File: BPS-LeaderDaughter.kicad_sch (KiCad schematic)
At the start: 0 parts

Commit message: Added strobe light + Som Connectors
Parts:
- added J1, J2: Conn_02x10_Odd_Even, symbol Connector_Generic:Conn_02x10_Odd_Even
- added J3: CAN_In, Connector_Molex:Molex_Micro-Fit_3.0_43045-0612_2x03_P3.00mm_Vertical, symbol Connector_Generic:Conn_02x03_Odd_Even
- added LOGO1: Dr. Hallock, UTSVT_Special:Hallock_Image_Tiny, symbol utsvt-misc:Logo_Placeholder
- added LOGO2: UTSVT Logo, UTSVT_Special:UTSVT_Logo_Symbol, symbol utsvt-misc:Logo_Placeholder
- added MH1, MH2: M.3, MountingHole:MountingHole_3mm, symbol Mechanical:MountingHole
Connections:
- new net 5V_Ext: J3.6 (Pin_6)
- new net CAN_H: J3.5 (Pin_5)
- new net CAN_L: J3.2 (Pin_2)
- new net Fault: J1.9 (Pin_9)
- new net GND1: J3.3 (Pin_3)
- new net GNDPWR: J3.1 (Pin_1)
- new net V_CAN_IN: J3.4 (Pin_4)
Other:
- added sheet Strobe Light (Strobe_Light.kicad_sch)
- note added: "Graphics/Logos"
- note added: "SOM Connectors"
- note added: "V1.0: 3 contactors + Fan controller circuit"
- note added: "Version History"

Commit message: added fan control heirarchical sheet
Other:
- added sheet Fan Control (Fan_Control.kicad_sch)
Changed lines of the file:
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@@
+    )
+  )
+  (sheet (at 30.48 64.77) (size 44.45 13.97) (fields_autoplaced)
+    (stroke (width 0.1524) (type solid))
+    (fill (color 0 0 0 0.0000))
+    (property "Sheetname" "Fan Control" (at 30.48 64.0584 0)
+      (effects (font (size 1.27 1.27)) (justify left bottom))
+    )
+    (property "Sheetfile" "Fan_Control.kicad_sch" (at 30.48 79.3246 0)
+      (effects (font (size 1.27 1.27)) (justify left top))
+    )
+    (instances
+      (project "BPS-LeaderDaughter"
+        (path "/2e9f4f51-d216-4952-a31c-e7104e0d4b1e" (page "3"))
+      )
     )
   )

Commit message: Standardized strobe liight
Parts:
- removed J1, J2: Conn_02x10_Odd_Even, symbol Connector_Generic:Conn_02x10_Odd_Even
- added J5, J6: DaughterConnector, 533072071, symbol utsvt-connectors:DaughterConnector
Connections:
- net Fault: now also J5.10

Commit message: Added Contactor Driver circuit
Parts:
- J5, J6: footprint 533072071 -> UTSVT_Connectors:533072071
Other:
- added sheet Array Contactor Driver (Contactor_Driver.kicad_sch)
- added sheet HV+ Contactor Driver (Contactor_Driver.kicad_sch)
- added sheet HV- Contactor Driver (Contactor_Driver.kicad_sch)
Changed lines of the file:
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@@
     (effects (font (size 1.27 1.27)) (justify left bottom))
   )
-  (symbol (lib_name "DaughterConnector_1") (lib_id "utsvt-connectors:DaughterConnector") (at 255.905 30.48 0) (unit 1)
+  (symbol (lib_id "utsvt-connectors:DaughterConnector") (at 255.905 30.48 0) (unit 1)
     (in_bom yes) (on_board yes) (dnp no) (fields_autoplaced)
     (property "Reference" "J6" (at 267.335 22.86 0)
@@
       (effects (font (size 1.27 1.27)))
     )
-    (property "Footprint" "533072071" (at 274.955 125.4 0)
+    (property "Footprint" "UTSVT_Connectors:533072071" (at 274.955 125.4 0)
       (effects (font (size 1.27 1.27)) (justify left top) hide)
     )
@@
       (effects (font (size 1.27 1.27)))
     )
-    (property "Footprint" "533072071" (at 245.745 125.4 0)
+    (property "Footprint" "UTSVT_Connectors:533072071" (at 245.745 125.4 0)
       (effects (font (size 1.27 1.27)) (justify left top) hide)
     )
@@
       )
     )
+  )
+  (sheet (at 30.48 114.3) (size 45.085 18.415) (fields_autoplaced)
+    (stroke (width 0.1524) (type solid))
+    (fill (color 0 0 0 0.0000))
+    (property "Sheetname" "HV- Contactor Driver" (at 30.48 113.5884 0)
+      (effects (font (size 1.27 1.27)) (justify left bottom))
+    )
+    (property "Sheetfile" "Contactor_Driver.kicad_sch" (at 30.48 133.2996 0)
+      (effects (font (size 1.27 1.27)) (justify left top))
+    )
+    (instances
+      (project "BPS-LeaderDaughter"
+        (path "/2e9f4f51-d216-4952-a31c-e7104e0d4b1e" (page "5"))
+      )
+    )
+  )
+  (sheet (at 30.48 86.995) (size 45.085 18.415) (fields_autoplaced)
+    (stroke (width 0.1524) (type solid))
+    (fill (color 0 0 0 0.0000))
+    (property "Sheetname" "HV+ Contactor Driver" (at 30.48 86.2834 0)
+      (effects (font (size 1.27 1.27)) (justify left bottom))
+    )
+    (property "Sheetfile" "Contactor_Driver.kicad_sch" (at 30.48 105.9946 0)
+      (effects (font (size 1.27 1.27)) (justify left top))
+    )
+    (instances
+      (project "BPS-LeaderDaughter"
+        (path "/2e9f4f51-d216-4952-a31c-e7104e0d4b1e" (page "4"))
+      )
+    )
+  )
+  (sheet (at 30.48 141.605) (size 45.085 18.415) (fields_autoplaced)
+    (stroke (width 0.1524) (type solid))
+    (fill (color 0 0 0 0.0000))
+    (property "Sheetname" "Array Contactor Driver" (at 30.48 140.8934 0)
+      (effects (font (size 1.27 1.27)) (justify left bottom))
+    )
+    (property "Sheetfile" "Contactor_Driver.kicad_sch" (at 30.48 160.6046 0)
+      (effects (font (size 1.27 1.27)) (justify left top))
+    )
+    (instances
+      (project "BPS-LeaderDaughter"
+        (path "/2e9f4f51-d216-4952-a31c-e7104e0d4b1e" (page "6"))
+      )
+    )

Commit message: Added more documentatino to the Contactor circuits
Connections:
- net Fault: now also J5.12; no longer J5.10
- net HV-_Sense: now reaches J5.14
- net HV+_Sense: now reaches J5.16
- net HV-_EN: now reaches J5.18
- net HV+_EN: now reaches J5.20
- net Array_EN: now reaches J5.8
- new net Array_Sense: J5.10
Other:
- sheet Array Contactor Driver ports: added Contactor_EN, Contactor_Sense; removed none
- sheet HV+ Contactor Driver ports: added Contactor_EN, Contactor_Sense; removed none
- sheet HV- Contactor Driver ports: added Contactor_EN, Contactor_Sense; removed none
Changed lines of the file:
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@@
 (kicad_sch (version 20230121) (generator eeschema)
   (paper "A4")
+  (wire (pts (xy 75.565 121.285) (xy 80.01 121.285))
+    (stroke (width 0) (type default))
+  )
+  (wire (pts (xy 215.265 35.56) (xy 226.695 35.56))
+    (stroke (width 0) (type default))
+  )
   (wire (pts (xy 227.33 65.405) (xy 245.11 65.405))
     (stroke (width 0) (type default))
@@
     (stroke (width 0) (type default))
   )
+  (wire (pts (xy 214.63 45.72) (xy 226.695 45.72))
+    (stroke (width 0) (type default))
+  )
   (wire (pts (xy 260.985 65.405) (xy 257.81 65.405))
     (stroke (width 0) (type default))
   )
+  (wire (pts (xy 218.44 30.48) (xy 226.695 30.48))
+    (stroke (width 0) (type default))
+  )
   (wire (pts (xy 233.68 70.485) (xy 245.11 70.485))
     (stroke (width 0) (type default))
   )
+  (wire (pts (xy 214.63 43.18) (xy 226.695 43.18))
+    (stroke (width 0) (type default))
+  )
+  (wire (pts (xy 218.44 33.02) (xy 226.695 33.02))
+    (stroke (width 0) (type default))
+  )
   (wire (pts (xy 227.33 66.04) (xy 227.33 65.405))
     (stroke (width 0) (type default))
   )
-  (wire (pts (xy 219.075 43.18) (xy 226.695 43.18))
+  (wire (pts (xy 75.565 127) (xy 80.01 127))
+    (stroke (width 0) (type default))
+  )
+  (wire (pts (xy 75.565 153.035) (xy 80.645 153.035))
+    (stroke (width 0) (type default))
+  )
+  (wire (pts (xy 219.71 40.64) (xy 226.695 40.64))
     (stroke (width 0) (type default))
   )
@@
     (stroke (width 0) (type default))
   )
+  (wire (pts (xy 75.565 92.075) (xy 80.01 92.075))
+    (stroke (width 0) (type default))
+  )
+  (wire (pts (xy 75.565 97.79) (xy 79.375 97.79))
+    (stroke (width 0) (type default))
+  )
   (wire (pts (xy 260.985 67.945) (xy 257.81 67.945))
+    (stroke (width 0) (type default))
+  )
+  (wire (pts (xy 75.565 148.59) (xy 80.645 148.59))
+    (stroke (width 0) (type default))
+  )
+  (wire (pts (xy 215.265 38.1) (xy 226.695 38.1))
     (stroke (width 0) (type default))
   )
@@
     (effects (font (size 1.27 1.27)) (justify left bottom))
   )
-  (label "Fault" (at 219.075 43.18 0) (fields_autoplaced)
+  (label "HV+_EN" (at 218.44 30.48 0) (fields_autoplaced)
+    (effects (font (size 1.27 1.27)) (justify left bottom))
+  )
+  (label "HV+_Sense" (at 80.01 92.075 0) (fields_autoplaced)
+    (effects (font (size 1.27 1.27)) (justify left bottom))
+  )
+  (label "Array_EN" (at 80.645 153.035 0) (fields_autoplaced)
+    (effects (font (size 1.27 1.27)) (justify left bottom))
+  )
+  (label "HV-_EN" (at 80.01 127 0) (fields_autoplaced)
+    (effects (font (size 1.27 1.27)) (justify left bottom))
+  )
+  (label "Fault" (at 219.71 40.64 0) (fields_autoplaced)
     (effects (font (size 1.27 1.27)) (justify left bottom))
   )
@@
     (effects (font (size 1.27 1.27)) (justify left bottom))
   )
+  (label "HV+_Sense" (at 215.265 35.56 0) (fields_autoplaced)
+    (effects (font (size 1.27 1.27)) (justify left bottom))
+  )
+  (label "HV+_EN" (at 79.375 97.79 0) (fields_autoplaced)
+    (effects (font (size 1.27 1.27)) (justify left bottom))
+  )
   (label "5V_Ext" (at 260.985 70.485 0) (fields_autoplaced)
     (effects (font (size 1.27 1.27)) (justify left bottom))
@@
     (effects (font (size 1.27 1.27)) (justify left bottom))
   )
+  (label "Array_EN" (at 214.63 45.72 0) (fields_autoplaced)
+    (effects (font (size 1.27 1.27)) (justify left bottom))
+  )
+  (label "HV-_EN" (at 218.44 33.02 0) (fields_autoplaced)
+    (effects (font (size 1.27 1.27)) (justify left bottom))
+  )
+  (label "Array_Sense" (at 80.645 148.59 0) (fields_autoplaced)
+    (effects (font (size 1.27 1.27)) (justify left bottom))
+  )
   (label "CAN_H" (at 233.68 70.485 0) (fields_autoplaced)
     (effects (font (size 1.27 1.27)) (justify left bottom))
   )
+  (label "Array_Sense" (at 214.63 43.18 0) (fields_autoplaced)
+    (effects (font (size 1.27 1.27)) (justify left bottom))
+  )
+  (label "HV-_Sense" (at 80.01 121.285 0) (fields_autoplaced)
+    (effects (font (size 1.27 1.27)) (justify left bottom))
+  )
   (label "Fault" (at 80.645 37.465 0) (fields_autoplaced)
+    (effects (font (size 1.27 1.27)) (justify left bottom))
+  )
+  (label "HV-_Sense" (at 215.265 38.1 0) (fields_autoplaced)
     (effects (font (size 1.27 1.27)) (justify left bottom))
   )
@@
       (effects (font (size 1.27 1.27)) (justify left top))
     )
+    (pin "Contactor_Sense" input (at 75.565 121.285 0)
+      (effects (font (size 1.27 1.27)) (justify right))
+    )
+    (pin "Contactor_EN" input (at 75.565 127 0)
+      (effects (font (size 1.27 1.27)) (justify right))
+    )
     (instances
       (project "BPS-LeaderDaughter"
@@
       (effects (font (size 1.27 1.27)) (justify left top))
     )
+    (pin "Contactor_Sense" input (at 75.565 92.075 0)
+      (effects (font (size 1.27 1.27)) (justify right))
+    )
+    (pin "Contactor_EN" input (at 75.565 97.79 0)
+      (effects (font (size 1.27 1.27)) (justify right))
+    )
     (instances
       (project "BPS-LeaderDaughter"
@@
       (effects (font (size 1.27 1.27)) (justify left top))
     )
-    (instances
+    (pin "Contactor_Sense" input (at 75.565 148.59 0)
+      (effects (font (size 1.27 1.27)) (justify right))
+    )
+    (pin "Contactor_EN" input (at 75.565 153.035 0)
+      (effects (font (size 1.27 1.27)) (justify right))
+    )
+    (instances

Commit message: Added more contactor footprints
Parts:
- removed J3: CAN_In, Connector_Molex:Molex_Micro-Fit_3.0_43045-0612_2x03_P3.00mm_Vertical, symbol Connector_Generic:Conn_02x03_Odd_Even
Changed lines of the file:
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@@
-    (stroke (width 0) (type default))
-  )
-  (wire (pts (xy 227.33 65.405) (xy 245.11 65.405))
     (stroke (width 0) (type default))
   )
@@
     (stroke (width 0) (type default))
   )
-  (wire (pts (xy 260.985 65.405) (xy 257.81 65.405))
-    (stroke (width 0) (type default))
-  )
   (wire (pts (xy 218.44 30.48) (xy 226.695 30.48))
     (stroke (width 0) (type default))
   )
-  (wire (pts (xy 233.68 70.485) (xy 245.11 70.485))
-    (stroke (width 0) (type default))
-  )
   (wire (pts (xy 214.63 43.18) (xy 226.695 43.18))
     (stroke (width 0) (type default))
@@
     (stroke (width 0) (type default))
   )
-  (wire (pts (xy 227.33 66.04) (xy 227.33 65.405))
-    (stroke (width 0) (type default))
-  )
   (wire (pts (xy 75.565 127) (xy 80.01 127))
     (stroke (width 0) (type default))
@@
     (stroke (width 0) (type default))
   )
-  (wire (pts (xy 257.81 70.485) (xy 260.985 70.485))
-    (stroke (width 0) (type default))
-  )
   (wire (pts (xy 75.565 92.075) (xy 80.01 92.075))
     (stroke (width 0) (type default))
@@
     (stroke (width 0) (type default))
   )
-  (wire (pts (xy 260.985 67.945) (xy 257.81 67.945))
-    (stroke (width 0) (type default))
-  )
   (wire (pts (xy 75.565 148.59) (xy 80.645 148.59))
     (stroke (width 0) (type default))
   )
   (wire (pts (xy 215.265 38.1) (xy 226.695 38.1))
-    (stroke (width 0) (type default))
-  )
-  (wire (pts (xy 232.41 71.12) (xy 232.41 67.945))
-    (stroke (width 0) (type default))
-  )
-  (wire (pts (xy 232.41 67.945) (xy 245.11 67.945))
     (stroke (width 0) (type default))
   )
@@
     (effects (font (size 1.27 1.27)) (justify left bottom))
   )
-  (label "V_CAN_IN" (at 260.985 67.945 0) (fields_autoplaced)
-    (effects (font (size 1.27 1.27)) (justify left bottom))
-  )
   (label "HV+_Sense" (at 215.265 35.56 0) (fields_autoplaced)
     (effects (font (size 1.27 1.27)) (justify left bottom))
@@
     (effects (font (size 1.27 1.27)) (justify left bottom))
   )
-  (label "5V_Ext" (at 260.985 70.485 0) (fields_autoplaced)
-    (effects (font (size 1.27 1.27)) (justify left bottom))
-  )
-  (label "CAN_L" (at 260.985 65.405 0) (fields_autoplaced)
-    (effects (font (size 1.27 1.27)) (justify left bottom))
-  )
   (label "Array_EN" (at 214.63 45.72 0) (fields_autoplaced)
     (effects (font (size 1.27 1.27)) (justify left bottom))
@@
   )
   (label "Array_Sense" (at 80.645 148.59 0) (fields_autoplaced)
-    (effects (font (size 1.27 1.27)) (justify left bottom))
-  )
-  (label "CAN_H" (at 233.68 70.485 0) (fields_autoplaced)
     (effects (font (size 1.27 1.27)) (justify left bottom))
   )
@@
     )
   )
-  (symbol (lib_id "Connector_Generic:Conn_02x03_Odd_Even") (at 250.19 67.945 0) (unit 1)
-    (in_bom yes) (on_board yes) (dnp no) (fields_autoplaced)
-    (property "Reference" "J3" (at 251.46 59.055 0)
-      (effects (font (size 1.27 1.27)))
-    )
-    (property "Value" "CAN_In" (at 251.46 61.595 0)
-      (effects (font (size 1.27 1.27)))
-    )
-    (property "Footprint" "Connector_Molex:Molex_Micro-Fit_3.0_43045-0612_2x03_P3.00mm_Vertical" (at 250.19 67.945 0)
-      (effects (font (size 1.27 1.27)) hide)
-    )
-    (property "Datasheet" "https://tools.molex.com/pdm_docs/sd/430450612_sd.pdf" (at 250.19 67.945 0)
-      (effects (font (size 1.27 1.27)) hide)
-    )
-    (property "P/N" "43045-0612" (at 250.19 67.945 0)
-      (effects (font (size 1.27 1.27)) hide)
-    )
-    (pin "1")
-    (pin "2")
-    (pin "3")
-    (pin "4")
-    (pin "5")
-    (pin "6")
-    (instances
-      (project "BPS-LeaderDaughter"
-        (path "/2e9f4f51-d216-4952-a31c-e7104e0d4b1e"
-          (reference "J3") (unit 1)
-        )
-      )
-      (project "BPS-PeripheralSOM"
-        (path "/d5ebd247-5a7c-47c2-8aee-beabaef72d6d/1d0c269d-60cf-499b-bfd2-5087981d6678"
-          (reference "J5") (unit 1)
-        )
-        (path "/d5ebd247-5a7c-47c2-8aee-beabaef72d6d"
-          (reference "J5") (unit 1)
-        )
-      )
-    )
-  )
   (symbol (lib_id "utsvt-misc:Logo_Placeholder") (at 236.855 146.685 0) (unit 1)
     (in_bom yes) (on_board yes) (dnp no)
@@
         )
       )
-    )
-  )
-  (symbol (lib_id "power:GND1") (at 232.41 71.12 0) (unit 1)
-    (in_bom yes) (on_board yes) (dnp no) (fields_autoplaced)
-    (property "Reference" "#PWR02" (at 232.41 77.47 0)
-      (effects (font (size 1.27 1.27)) hide)
-    )
-    (property "Value" "GND1" (at 232.41 75.565 0)
-      (effects (font (size 1.27 1.27)))
-    )
-    (property "Footprint" "" (at 232.41 71.12 0)
-      (effects (font (size 1.27 1.27)) hide)
-    )
-    (property "Datasheet" "" (at 232.41 71.12 0)
-      (effects (font (size 1.27 1.27)) hide)
-    )
-    (pin "1")
-    (instances
-      (project "BPS-LeaderDaughter"
-        (path "/2e9f4f51-d216-4952-a31c-e7104e0d4b1e"
-          (reference "#PWR02") (unit 1)
-        )
-      )
-      (project "BPS-PeripheralSOM"
-        (path "/d5ebd247-5a7c-47c2-8aee-beabaef72d6d/1d0c269d-60cf-499b-bfd2-5087981d6678"
-          (reference "#PWR013") (unit 1)
-        )
-        (path "/d5ebd247-5a7c-47c2-8aee-beabaef72d6d"
-          (reference "#PWR041") (unit 1)
-        )
-      )
-    )
-  )
-  (symbol (lib_id "power:GNDPWR") (at 227.33 66.04 0) (unit 1)
-    (in_bom yes) (on_board yes) (dnp no) (fields_autoplaced)
-    (property "Reference" "#PWR01" (at 227.33 71.12 0)
-      (effects (font (size 1.27 1.27)) hide)
-    )
-    (property "Value" "GNDPWR" (at 227.203 71.12 0)
-      (effects (font (size 1.27 1.27)))
-    )
-    (property "Footprint" "" (at 227.33 67.31 0)
-      (effects (font (size 1.27 1.27)) hide)
-    )
-    (property "Datasheet" "" (at 227.33 67.31 0)
-      (effects (font (size 1.27 1.27)) hide)
-    )
-    (pin "1")
-    (instances
-      (project "BPS-LeaderDaughter"
-        (path "/2e9f4f51-d216-4952-a31c-e7104e0d4b1e"
-          (reference "#PWR01") (unit 1)
-        )
-      )
-      (project "BPS-PeripheralSOM"
-        (path "/d5ebd247-5a7c-47c2-8aee-beabaef72d6d/1d0c269d-60cf-499b-bfd2-5087981d6678"
-          (reference "#PWR022") (unit 1)
-        )
-        (path "/d5ebd247-5a7c-47c2-8aee-beabaef72d6d"
-          (reference "#PWR038") (unit 1)
-        )
-      )

Commit message: Added fan sheet
Connections:
- net +12V: now reaches J5.19
- net SDA: now reaches J5.4
- net SCL: now reaches J5.6
- no-connect marks 0 -> 18
Other:
- sheet Fan Control ports: added SCL, SDA; removed none
Changed lines of the file:
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@@
 (kicad_sch (version 20230121) (generator eeschema)
   (paper "A4")
+  (no_connect (at 255.905 48.26))
+  (no_connect (at 255.905 43.18))
+  (no_connect (at 249.555 45.72))
+  (no_connect (at 249.555 48.26))
+  (no_connect (at 255.905 30.48))
+  (no_connect (at 255.905 33.02))
+  (no_connect (at 255.905 38.1))
+  (no_connect (at 249.555 50.8))
+  (no_connect (at 226.695 53.34))
+  (no_connect (at 249.555 38.1))
+  (no_connect (at 249.555 35.56))
+  (no_connect (at 255.905 35.56))
+  (no_connect (at 249.555 33.02))
+  (no_connect (at 255.905 40.64))
+  (no_connect (at 255.905 45.72))
+  (no_connect (at 249.555 40.64))
+  (no_connect (at 249.555 53.34))
+  (no_connect (at 249.555 43.18))
   (wire (pts (xy 75.565 121.285) (xy 80.01 121.285))
     (stroke (width 0) (type default))
@@
     (stroke (width 0) (type default))
   )
+  (wire (pts (xy 214.63 48.26) (xy 226.695 48.26))
+    (stroke (width 0) (type default))
+  )
   (wire (pts (xy 218.44 33.02) (xy 226.695 33.02))
     (stroke (width 0) (type default))
   )
+  (wire (pts (xy 214.63 50.8) (xy 226.695 50.8))
+    (stroke (width 0) (type default))
+  )
+  (wire (pts (xy 252.095 27.94) (xy 252.095 30.48))
+    (stroke (width 0) (type default))
+  )
   (wire (pts (xy 75.565 127) (xy 80.01 127))
     (stroke (width 0) (type default))
   )
   (wire (pts (xy 75.565 153.035) (xy 80.645 153.035))
+    (stroke (width 0) (type default))
+  )
+  (wire (pts (xy 252.095 30.48) (xy 249.555 30.48))
     (stroke (width 0) (type default))
   )
@@
     (effects (font (size 1.27 1.27)) (justify left bottom))
   )
+  (label "SCL" (at 214.63 48.26 0) (fields_autoplaced)
+    (effects (font (size 1.27 1.27)) (justify left bottom))
+  )
   (label "HV+_EN" (at 218.44 30.48 0) (fields_autoplaced)
     (effects (font (size 1.27 1.27)) (justify left bottom))
@@
   )
   (label "Array_Sense" (at 80.645 148.59 0) (fields_autoplaced)
+    (effects (font (size 1.27 1.27)) (justify left bottom))
+  )
+  (label "SDA" (at 214.63 50.8 0) (fields_autoplaced)
     (effects (font (size 1.27 1.27)) (justify left bottom))
   )
@@
     )
   )
+  (symbol (lib_id "power:+12V") (at 252.095 27.94 0) (unit 1)
+    (in_bom yes) (on_board yes) (dnp no) (fields_autoplaced)
+    (property "Reference" "#PWR068" (at 252.095 31.75 0)
+      (effects (font (size 1.27 1.27)) hide)
+    )
+    (property "Value" "+12V" (at 252.095 22.86 0)
+      (effects (font (size 1.27 1.27)))
+    )
+    (property "Footprint" "" (at 252.095 27.94 0)
+      (effects (font (size 1.27 1.27)) hide)
+    )
+    (property "Datasheet" "" (at 252.095 27.94 0)
+      (effects (font (size 1.27 1.27)) hide)
+    )
+    (pin "1")
+    (instances
+      (project "BPS-LeaderDaughter"
+        (path "/2e9f4f51-d216-4952-a31c-e7104e0d4b1e"
+          (reference "#PWR068") (unit 1)
+        )
+      )
+    )
+  )
   (symbol (lib_id "utsvt-connectors:DaughterConnector") (at 226.695 30.48 0) (unit 1)
     (in_bom yes) (on_board yes) (dnp no) (fields_autoplaced)
@@
       (effects (font (size 1.27 1.27)) (justify left top))
     )
-    (instances
+    (pin "SDA" input (at 74.93 69.85 0)
+      (effects (font (size 1.27 1.27)) (justify right))
+    )
+    (pin "SCL" input (at 74.93 73.66 0)
+      (effects (font (size 1.27 1.27)) (justify right))
+    )
+    (instances

Commit message: removed redundant contactor circuit
Connections:
- net +5V: now reaches J6.19
- net GND: now reaches J5.1
- net +3.3V: now reaches J5.17
- no-connect marks 18 -> 27
Other:
- moved on the sheet: J5
