File: BPS-LeaderDaughter.kicad_sch (KiCad schematic)
At the start: 6 parts, among them J5 DaughterConnector, J6 DaughterConnector

Commit message: Added even moreeeee Contactor p/n + added 4 more mounting holes
Parts:
- added MH3, MH4, MH5, MH6: M.3, MountingHole:MountingHole_3mm, symbol Mechanical:MountingHole
Changed lines of the file:
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@@
+    )
+  )
+  (symbol (lib_id "Mechanical:MountingHole") (at 277.495 146.685 0) (unit 1)
+    (in_bom yes) (on_board yes) (dnp no)
+    (property "Reference" "MH5" (at 280.035 145.5166 0)
+      (effects (font (size 1.27 1.27)) (justify left))
+    )
+    (property "Value" "M.3" (at 280.035 147.828 0)
+      (effects (font (size 1.27 1.27)) (justify left))
+    )
+    (property "Footprint" "MountingHole:MountingHole_3mm" (at 277.495 146.685 0)
+      (effects (font (size 1.27 1.27)) hide)
+    )
+    (property "Datasheet" "~" (at 277.495 146.685 0)
+      (effects (font (size 1.27 1.27)) hide)
+    )
+    (instances
+      (project "BPS-LeaderDaughter"
+        (path "/2e9f4f51-d216-4952-a31c-e7104e0d4b1e"
+          (reference "MH5") (unit 1)
+        )
+      )
+      (project "BPS-Leader"
+        (path "/c248b171-df31-4e8a-afb6-607fa2df334b"
+          (reference "MH1") (unit 1)
+        )
+      )
+      (project "BPS-PeripheralSOM"
+        (path "/d5ebd247-5a7c-47c2-8aee-beabaef72d6d"
+          (reference "MH1") (unit 1)
+        )
+      )
+    )
+  )
+  (symbol (lib_id "Mechanical:MountingHole") (at 267.335 154.94 0) (unit 1)
+    (in_bom yes) (on_board yes) (dnp no)
+    (property "Reference" "MH4" (at 269.875 153.7716 0)
+      (effects (font (size 1.27 1.27)) (justify left))
+    )
+    (property "Value" "M.3" (at 269.875 156.083 0)
+      (effects (font (size 1.27 1.27)) (justify left))
+    )
+    (property "Footprint" "MountingHole:MountingHole_3mm" (at 267.335 154.94 0)
+      (effects (font (size 1.27 1.27)) hide)
+    )
+    (property "Datasheet" "~" (at 267.335 154.94 0)
+      (effects (font (size 1.27 1.27)) hide)
+    )
+    (instances
+      (project "BPS-LeaderDaughter"
+        (path "/2e9f4f51-d216-4952-a31c-e7104e0d4b1e"
+          (reference "MH4") (unit 1)
+        )
+      )
+      (project "BPS-Leader"
+        (path "/c248b171-df31-4e8a-afb6-607fa2df334b"
+          (reference "MH2") (unit 1)
+        )
+      )
+      (project "BPS-PeripheralSOM"
+        (path "/d5ebd247-5a7c-47c2-8aee-beabaef72d6d"
+          (reference "MH2") (unit 1)
+        )
+      )
     )
   )
@@
         )
       )
+    )
+  )
+  (symbol (lib_id "Mechanical:MountingHole") (at 277.495 154.94 0) (unit 1)
+    (in_bom yes) (on_board yes) (dnp no)
+    (property "Reference" "MH6" (at 280.035 153.7716 0)
+      (effects (font (size 1.27 1.27)) (justify left))
+    )
+    (property "Value" "M.3" (at 280.035 156.083 0)
+      (effects (font (size 1.27 1.27)) (justify left))
+    )
+    (property "Footprint" "MountingHole:MountingHole_3mm" (at 277.495 154.94 0)
+      (effects (font (size 1.27 1.27)) hide)
+    )
+    (property "Datasheet" "~" (at 277.495 154.94 0)
+      (effects (font (size 1.27 1.27)) hide)
+    )
+    (instances
+      (project "BPS-LeaderDaughter"
+        (path "/2e9f4f51-d216-4952-a31c-e7104e0d4b1e"
+          (reference "MH6") (unit 1)
+        )
+      )
+      (project "BPS-Leader"
+        (path "/c248b171-df31-4e8a-afb6-607fa2df334b"
+          (reference "MH2") (unit 1)
+        )
+      )
+      (project "BPS-PeripheralSOM"
+        (path "/d5ebd247-5a7c-47c2-8aee-beabaef72d6d"
+          (reference "MH2") (unit 1)
+        )
+      )
+    )
+  )
+  (symbol (lib_id "Mechanical:MountingHole") (at 267.335 146.685 0) (unit 1)
+    (in_bom yes) (on_board yes) (dnp no)
+    (property "Reference" "MH3" (at 269.875 145.5166 0)
+      (effects (font (size 1.27 1.27)) (justify left))
+    )
+    (property "Value" "M.3" (at 269.875 147.828 0)
+      (effects (font (size 1.27 1.27)) (justify left))
+    )
+    (property "Footprint" "MountingHole:MountingHole_3mm" (at 267.335 146.685 0)
+      (effects (font (size 1.27 1.27)) hide)
+    )
+    (property "Datasheet" "~" (at 267.335 146.685 0)
+      (effects (font (size 1.27 1.27)) hide)
+    )
+    (instances
+      (project "BPS-LeaderDaughter"
+        (path "/2e9f4f51-d216-4952-a31c-e7104e0d4b1e"
+          (reference "MH3") (unit 1)
+        )
+      )
+      (project "BPS-Leader"
+        (path "/c248b171-df31-4e8a-afb6-607fa2df334b"
+          (reference "MH1") (unit 1)
+        )
+      )
+      (project "BPS-PeripheralSOM"
+        (path "/d5ebd247-5a7c-47c2-8aee-beabaef72d6d"
+          (reference "MH1") (unit 1)
+        )
+      )

Commit message: Added version history
Other:
- note added: "V1.0: - 3 Contactors + Fan controller circuit"
- note removed: "V1.0: 3 contactors + Fan controller circuit"
Changed lines of the file:
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@@
     (stroke (width 0) (type default))
   )
-  (wire (pts (xy 211.455 35.56) (xy 222.885 35.56))
+  (wire (pts (xy 210.82 35.56) (xy 222.885 35.56))
     (stroke (width 0) (type default))
   )
@@
     (stroke (width 0) (type default))
   )
-  (wire (pts (xy 214.63 30.48) (xy 222.885 30.48))
+  (wire (pts (xy 210.82 30.48) (xy 222.885 30.48))
     (stroke (width 0) (type default))
   )
@@
     (stroke (width 0) (type default))
   )
-  (wire (pts (xy 214.63 33.02) (xy 222.885 33.02))
+  (wire (pts (xy 210.82 33.02) (xy 222.885 33.02))
     (stroke (width 0) (type default))
   )
@@
     (stroke (width 0) (type default))
   )
-  (wire (pts (xy 215.9 40.64) (xy 222.885 40.64))
+  (wire (pts (xy 210.82 40.64) (xy 222.885 40.64))
     (stroke (width 0) (type default))
   )
@@
     (stroke (width 0) (type default))
   )
-  (wire (pts (xy 211.455 38.1) (xy 222.885 38.1))
+  (wire (pts (xy 210.82 38.1) (xy 222.885 38.1))
     (stroke (width 0) (type default))
   )
@@
   (wire (pts (xy 74.93 73.66) (xy 80.01 73.66))
     (stroke (width 0) (type default))
+  )
+  (rectangle (start 227.965 86.36) (end 280.67 113.665)
+    (stroke (width 0) (type default))
+    (fill (type none))
   )
   (text "SOM Connectors" (at 236.855 18.415 0)
@@
     (effects (font (size 2.54 2.54) (thickness 0.508) bold) (justify left bottom))
   )
-  (text "V1.0: 3 contactors + Fan controller circuit" (at 229.87 99.695 0)
+  (text "V1.0: \n- 3 Contactors + Fan controller circuit" (at 229.87 97.155 0)
     (effects (font (size 1.27 1.27)) (justify left bottom))
   )
@@
     (effects (font (size 1.27 1.27)) (justify left bottom))
   )
-  (label "HV+_EN" (at 214.63 30.48 0) (fields_autoplaced)
+  (label "HV+_EN" (at 210.82 30.48 0) (fields_autoplaced)
     (effects (font (size 1.27 1.27)) (justify left bottom))
   )
@@
     (effects (font (size 1.27 1.27)) (justify left bottom))
   )
-  (label "Fault" (at 215.9 40.64 0) (fields_autoplaced)
+  (label "Fault" (at 210.82 40.64 0) (fields_autoplaced)
     (effects (font (size 1.27 1.27)) (justify left bottom))
   )
-  (label "HV+_Sense" (at 211.455 35.56 0) (fields_autoplaced)
+  (label "HV+_Sense" (at 210.82 35.56 0) (fields_autoplaced)
     (effects (font (size 1.27 1.27)) (justify left bottom))
   )
@@
     (effects (font (size 1.27 1.27)) (justify left bottom))
   )
-  (label "HV-_EN" (at 214.63 33.02 0) (fields_autoplaced)
+  (label "HV-_EN" (at 210.82 33.02 0) (fields_autoplaced)
     (effects (font (size 1.27 1.27)) (justify left bottom))
   )
@@
     (effects (font (size 1.27 1.27)) (justify left bottom))
   )
-  (label "HV-_Sense" (at 211.455 38.1 0) (fields_autoplaced)
+  (label "HV-_Sense" (at 210.82 38.1 0) (fields_autoplaced)
     (effects (font (size 1.27 1.27)) (justify left bottom))
   )

Commit message: Combined fan and contactor stuff
Parts:
- renumbered J5 to J1, J6 to J2
Changed lines of the file:
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@@
   (symbol (lib_id "utsvt-connectors:DaughterConnector") (at 255.905 30.48 0) (unit 1)
     (in_bom yes) (on_board yes) (dnp no) (fields_autoplaced)
-    (property "Reference" "J6" (at 267.335 22.86 0)
+    (property "Reference" "J2" (at 267.335 22.86 0)
       (effects (font (size 1.27 1.27)))
     )
@@
       (project "BPS-LeaderDaughter"
         (path "/2e9f4f51-d216-4952-a31c-e7104e0d4b1e"
-          (reference "J6") (unit 1)
+          (reference "J2") (unit 1)
         )
       )
@@
   (symbol (lib_id "power:+3.3V") (at 252.73 31.115 0) (unit 1)
     (in_bom yes) (on_board yes) (dnp no) (fields_autoplaced)
-    (property "Reference" "#PWR071" (at 252.73 34.925 0)
+    (property "Reference" "#PWR03" (at 252.73 34.925 0)
       (effects (font (size 1.27 1.27)) hide)
     )
@@
       (project "BPS-LeaderDaughter"
         (path "/2e9f4f51-d216-4952-a31c-e7104e0d4b1e"
-          (reference "#PWR071") (unit 1)
+          (reference "#PWR03") (unit 1)
         )
       )
@@
   (symbol (lib_id "power:GND") (at 247.65 55.88 0) (unit 1)
     (in_bom yes) (on_board yes) (dnp no) (fields_autoplaced)
-    (property "Reference" "#PWR069" (at 247.65 62.23 0)
+    (property "Reference" "#PWR01" (at 247.65 62.23 0)
       (effects (font (size 1.27 1.27)) hide)
     )
@@
       (project "BPS-LeaderDaughter"
         (path "/2e9f4f51-d216-4952-a31c-e7104e0d4b1e"
-          (reference "#PWR069") (unit 1)
+          (reference "#PWR01") (unit 1)
         )
       )
@@
   (symbol (lib_id "power:+12V") (at 248.285 27.94 0) (unit 1)
     (in_bom yes) (on_board yes) (dnp no) (fields_autoplaced)
-    (property "Reference" "#PWR068" (at 248.285 31.75 0)
+    (property "Reference" "#PWR02" (at 248.285 31.75 0)
       (effects (font (size 1.27 1.27)) hide)
     )
@@
       (project "BPS-LeaderDaughter"
         (path "/2e9f4f51-d216-4952-a31c-e7104e0d4b1e"
-          (reference "#PWR068") (unit 1)
+          (reference "#PWR02") (unit 1)
         )
       )
@@
   (symbol (lib_id "utsvt-connectors:DaughterConnector") (at 222.885 30.48 0) (unit 1)
     (in_bom yes) (on_board yes) (dnp no) (fields_autoplaced)
-    (property "Reference" "J5" (at 234.315 22.86 0)
+    (property "Reference" "J1" (at 234.315 22.86 0)
       (effects (font (size 1.27 1.27)))
     )
@@
       (project "BPS-LeaderDaughter"
         (path "/2e9f4f51-d216-4952-a31c-e7104e0d4b1e"
-          (reference "J5") (unit 1)
+          (reference "J1") (unit 1)
         )
       )
@@
   (symbol (lib_id "power:+5V") (at 281.305 27.94 0) (unit 1)
     (in_bom yes) (on_board yes) (dnp no) (fields_autoplaced)
-    (property "Reference" "#PWR070" (at 281.305 31.75 0)
+    (property "Reference" "#PWR04" (at 281.305 31.75 0)
       (effects (font (size 1.27 1.27)) hide)
     )
@@
       (project "BPS-LeaderDaughter"
         (path "/2e9f4f51-d216-4952-a31c-e7104e0d4b1e"
-          (reference "#PWR070") (unit 1)
-        )
-      )
+          (reference "#PWR04") (unit 1)
+        )
+      )

Commit message: Started Ignition and nearly done with Contactor Circuit
Other:
- added sheet Ignition (Ignition.kicad_sch)
Changed lines of the file:
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@@
+    )
+  )
+  (sheet (at 30.48 167.005) (size 44.45 15.875) (fields_autoplaced)
+    (stroke (width 0.1524) (type solid))
+    (fill (color 0 0 0 0.0000))
+    (property "Sheetname" "Ignition" (at 30.48 166.2934 0)
+      (effects (font (size 1.27 1.27)) (justify left bottom))
+    )
+    (property "Sheetfile" "Ignition.kicad_sch" (at 30.48 183.4646 0)
+      (effects (font (size 1.27 1.27)) (justify left top))
+    )
+    (instances
+      (project "BPS-LeaderDaughter"
+        (path "/2e9f4f51-d216-4952-a31c-e7104e0d4b1e" (page "7"))
+      )
     )
   )

Commit message: Added new SOM connector layout
Connections:
- net +12V: now also J2.1, J2.2; no longer J1.19
- net +3.3V: now also J1.1, J1.2, J2.19, J2.20; no longer J1.17
- net +5V: now also J1.19, J1.20; no longer J2.19
- net Array_EN: now also J1.6; no longer J1.8
- net Array_Sense: now also J1.8; no longer J1.10
- net Fault: no longer J1.12
- net GND: now also J1.17, J1.18, J1.3, J1.4, J2.17, J2.18; no longer J1.1
- net HV+_EN: now also J1.16; no longer J1.20
- net HV+_Sense: now also J1.14; no longer J1.16
- net HV-_EN: now also J1.12; no longer J1.18
- net HV-_Sense: now also J1.10; no longer J1.14
- net SCL: now also J2.15; no longer J1.6
- net SDA: now also J2.13; no longer J1.4
- net GNDPWR: now reaches J2.3
- net GNDPWR: now also J2.4
- no-connect marks 27 -> 10
Other:
- moved on the sheet: J2

Commit message: Restructed main sheet
Connections:
- net Array_EN: now also J2.7; no longer J1.6
- net Array_Sense: now also J2.5; no longer J1.8
- net Fault: now also J1.6
- net HV+_EN: now also J2.16; no longer J1.16
- net HV+_Sense: now also J2.14; no longer J1.14
- net HV-_EN: now also J2.8; no longer J1.12
- net HV-_Sense: now also J2.6; no longer J1.10
- no-connect marks 10 -> 15
Other:
- moved on the sheet: J1, J2, MH1, MH2, MH3, MH4, MH5, MH6

Commit message: updated som connecters to match leadersom
Connections:
- net GNDPWR is gone; now on net GND: J2.3, J2.4
- net +12V: now also J1.1, J1.2; no longer J2.1, J2.2
- net +3.3V: now also J1.11, J1.9, J2.17, J2.18; no longer J1.1, J1.2
- net GND: now also J2.1, J2.2; no longer J2.17, J2.18
- net SCL: now also J1.15; no longer J2.15
- net SDA: now also J1.13; no longer J2.13
- net ~{SMBALERT}: now reaches J1.8
- no-connect marks 15 -> 12
Other:
- sheet Fan Control ports: added ~{SMBALERT}; removed none
- moved on the sheet: J1, J2
