File: BPS-LeaderDaughter.kicad_sch (KiCad schematic)
At the start: 10 parts, among them J1 DaughterConnector, J2 DaughterConnector

Commit message: Fixed LeaderSOM connections, strobe, ignition, and contactor layout
Connections:
- net Fault: now also J1.14; no longer J1.6
- net GND: now also J1.6
- no-connect marks 9 -> 8
Changed lines of the file:
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@@
   (junction (at 220.98 132.08) (diameter 0) (color 0 0 0 0)
+  )
+  (junction (at 253.365 96.52) (diameter 0) (color 0 0 0 0)
   )
   (junction (at 261.62 111.76) (diameter 0) (color 0 0 0 0)
@@
   (no_connect (at 229.87 93.98))
   (no_connect (at 229.87 121.92))
-  (no_connect (at 252.73 83.82))
   (no_connect (at 252.73 86.36))
   (no_connect (at 229.87 76.2))
@@
     (stroke (width 0) (type default))
   )
+  (wire (pts (xy 252.73 93.98) (xy 253.365 93.98))
+    (stroke (width 0) (type default))
+  )
   (wire (pts (xy 219.71 119.38) (xy 229.87 119.38))
     (stroke (width 0) (type default))
@@
     (stroke (width 0) (type default))
   )
+  (wire (pts (xy 253.365 96.52) (xy 252.73 96.52))
+    (stroke (width 0) (type default))
+  )
   (wire (pts (xy 252.73 134.62) (xy 261.62 134.62))
     (stroke (width 0) (type default))
@@
     (stroke (width 0) (type default))
   )
-  (wire (pts (xy 256.54 96.52) (xy 252.73 96.52))
+  (wire (pts (xy 256.54 96.52) (xy 253.365 96.52))
     (stroke (width 0) (type default))
   )
@@
     (stroke (width 0) (type default))
   )
-  (wire (pts (xy 260.35 93.98) (xy 252.73 93.98))
-    (stroke (width 0) (type default))
-  )
   (wire (pts (xy 229.87 132.08) (xy 220.98 132.08))
     (stroke (width 0) (type default))
   )
   (wire (pts (xy 74.93 97.79) (xy 78.74 97.79))
+    (stroke (width 0) (type default))
+  )
+  (wire (pts (xy 253.365 93.98) (xy 253.365 96.52))
+    (stroke (width 0) (type default))
+  )
+  (wire (pts (xy 252.73 83.82) (xy 262.89 83.82))
     (stroke (width 0) (type default))
   )
@@
     (effects (font (size 1.27 1.27)) (justify right bottom))
   )
-  (label "Fault" (at 260.35 93.98 180) (fields_autoplaced)
-    (effects (font (size 1.27 1.27)) (justify right bottom))
-  )
+  (label "Fault" (at 262.89 83.82 180) (fields_autoplaced)
+    (effects (font (size 1.27 1.27)) (justify right bottom))
+  )

Commit message: Traced Champers <3
Connections:
- net Array_EN: now also J1.12; no longer J2.7
- net Array_Sense: now also J1.10; no longer J2.5
- net Fault: now also J1.8; no longer J1.14
- net HV+_EN: now also J1.7; no longer J2.16
- net HV+_Sense: now also J1.5; no longer J2.14
- net HV-_EN: now also J2.16; no longer J2.8
- net HV-_Sense: now also J2.14; no longer J2.6
- net ~{SMBALERT}: now also J1.14; no longer J1.8
Changed lines of the file:
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@@
   (junction (at 228.6 86.36) (diameter 0) (color 0 0 0 0)
   )
-  (no_connect (at 229.87 91.44))
-  (no_connect (at 229.87 93.98))
+  (no_connect (at 252.73 127))
   (no_connect (at 229.87 121.92))
-  (no_connect (at 252.73 86.36))
+  (no_connect (at 229.87 129.54))
+  (no_connect (at 229.87 127))
   (no_connect (at 229.87 76.2))
-  (no_connect (at 252.73 88.9))
+  (no_connect (at 252.73 129.54))
   (no_connect (at 252.73 76.2))
   (no_connect (at 229.87 124.46))
@@
     (stroke (width 0) (type default))
   )
+  (wire (pts (xy 227.965 91.44) (xy 229.87 91.44))
+    (stroke (width 0) (type default))
+  )
   (wire (pts (xy 74.93 47.625) (xy 80.01 47.625))
     (stroke (width 0) (type default))
@@
     (stroke (width 0) (type default))
   )
-  (wire (pts (xy 267.335 119.38) (xy 252.73 119.38))
-    (stroke (width 0) (type default))
-  )
   (wire (pts (xy 228.6 86.36) (xy 229.87 86.36))
     (stroke (width 0) (type default))
@@
     (stroke (width 0) (type default))
   )
+  (wire (pts (xy 267.97 86.36) (xy 252.73 86.36))
+    (stroke (width 0) (type default))
+  )
   (wire (pts (xy 219.71 119.38) (xy 229.87 119.38))
     (stroke (width 0) (type default))
@@
     (stroke (width 0) (type default))
   )
-  (wire (pts (xy 229.87 127) (xy 222.25 127))
-    (stroke (width 0) (type default))
-  )
   (wire (pts (xy 252.73 114.3) (xy 261.62 114.3))
     (stroke (width 0) (type default))
@@
     (stroke (width 0) (type default))
   )
-  (wire (pts (xy 266.7 129.54) (xy 252.73 129.54))
+  (wire (pts (xy 252.73 88.9) (xy 268.605 88.9))
     (stroke (width 0) (type default))
   )
@@
     (stroke (width 0) (type default))
   )
-  (wire (pts (xy 266.7 127) (xy 252.73 127))
-    (stroke (width 0) (type default))
-  )
   (wire (pts (xy 73.66 152.4) (xy 78.105 152.4))
     (stroke (width 0) (type default))
@@
     (stroke (width 0) (type default))
   )
-  (wire (pts (xy 252.73 91.44) (xy 264.16 91.44))
+  (wire (pts (xy 252.73 83.82) (xy 263.525 83.82))
     (stroke (width 0) (type default))
   )
@@
     (stroke (width 0) (type default))
   )
-  (wire (pts (xy 267.335 116.84) (xy 252.73 116.84))
-    (stroke (width 0) (type default))
-  )
   (wire (pts (xy 252.73 123.19) (xy 252.73 124.46))
     (stroke (width 0) (type default))
   )
-  (wire (pts (xy 229.87 129.54) (xy 222.885 129.54))
-    (stroke (width 0) (type default))
-  )
   (wire (pts (xy 74.93 92.075) (xy 79.375 92.075))
     (stroke (width 0) (type default))
@@
     (stroke (width 0) (type default))
   )
-  (wire (pts (xy 252.73 83.82) (xy 262.89 83.82))
-    (stroke (width 0) (type default))
-  )
   (wire (pts (xy 255.905 123.19) (xy 252.73 123.19))
     (stroke (width 0) (type default))
@@
     (stroke (width 0) (type default))
   )
+  (wire (pts (xy 252.73 116.84) (xy 266.7 116.84))
+    (stroke (width 0) (type default))
+  )
   (wire (pts (xy 223.52 81.28) (xy 229.87 81.28))
     (stroke (width 0) (type default))
@@
     (stroke (width 0) (type default))
   )
+  (wire (pts (xy 227.965 93.98) (xy 229.87 93.98))
+    (stroke (width 0) (type default))
+  )
   (wire (pts (xy 261.62 114.3) (xy 261.62 111.76))
     (stroke (width 0) (type default))
@@
     (stroke (width 0) (type default))
   )
+  (wire (pts (xy 252.73 91.44) (xy 259.08 91.44))
+    (stroke (width 0) (type default))
+  )
   (wire (pts (xy 220.98 134.62) (xy 220.98 132.08))
     (stroke (width 0) (type default))
@@
   )
   (wire (pts (xy 74.93 51.435) (xy 80.01 51.435))
+    (stroke (width 0) (type default))
+  )
+  (wire (pts (xy 252.73 119.38) (xy 266.7 119.38))
     (stroke (width 0) (type default))
   )
@@
     (effects (font (size 1.27 1.27)) (justify left bottom))
   )
-  (label "HV+_EN" (at 267.335 116.84 180) (fields_autoplaced)
+  (label "HV+_EN" (at 227.965 91.44 180) (fields_autoplaced)
     (effects (font (size 1.27 1.27)) (justify right bottom))
   )
@@
     (effects (font (size 1.27 1.27)) (justify right bottom))
   )
-  (label "Fault" (at 262.89 83.82 180) (fields_autoplaced)
+  (label "Fault" (at 259.08 91.44 180) (fields_autoplaced)
     (effects (font (size 1.27 1.27)) (justify right bottom))
   )
@@
     (effects (font (size 1.27 1.27)) (justify left bottom))
   )
-  (label "HV+_Sense" (at 267.335 119.38 180) (fields_autoplaced)
+  (label "HV+_Sense" (at 227.965 93.98 180) (fields_autoplaced)
     (effects (font (size 1.27 1.27)) (justify right bottom))
   )
@@
     (effects (font (size 1.27 1.27)) (justify left bottom))
   )
-  (label "Array_EN" (at 222.25 127 180) (fields_autoplaced)
-    (effects (font (size 1.27 1.27)) (justify right bottom))
-  )
-  (label "HV-_EN" (at 266.7 127 180) (fields_autoplaced)
+  (label "Array_EN" (at 267.97 86.36 180) (fields_autoplaced)
+    (effects (font (size 1.27 1.27)) (justify right bottom))
+  )
+  (label "HV-_EN" (at 266.7 116.84 180) (fields_autoplaced)
     (effects (font (size 1.27 1.27)) (justify right bottom))
   )
@@
     (effects (font (size 1.27 1.27)) (justify left bottom))
   )
-  (label "Array_Sense" (at 222.885 129.54 180) (fields_autoplaced)
+  (label "Array_Sense" (at 268.605 88.9 180) (fields_autoplaced)
     (effects (font (size 1.27 1.27)) (justify right bottom))
   )
@@
     (effects (font (size 1.27 1.27)) (justify left bottom))
   )
-  (label "~{SMBALERT}" (at 264.16 91.44 180) (fields_autoplaced)
+  (label "~{SMBALERT}" (at 263.525 83.82 180) (fields_autoplaced)
     (effects (font (size 1.27 1.27)) (justify right bottom))
   )
@@
     (effects (font (size 1.27 1.27)) (justify left bottom))
   )
-  (label "HV-_Sense" (at 266.7 129.54 180) (fields_autoplaced)
-    (effects (font (size 1.27 1.27)) (justify right bottom))
-  )
+  (label "HV-_Sense" (at 266.7 119.38 180) (fields_autoplaced)
+    (effects (font (size 1.27 1.27)) (justify right bottom))
+  )

Commit message: magical unicorns
Parts:
- J1, J2: footprint UTSVT_Connectors:533072071 -> UTSVT_Connectors:Molex_53307-2071
Changed lines of the file:
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@@
       (effects (font (size 1.27 1.27)))
     )
-    (property "Footprint" "UTSVT_Connectors:533072071" (at 233.68 206.68 0)
+    (property "Footprint" "UTSVT_Connectors:Molex_53307-2071" (at 233.68 206.68 0)
       (effects (font (size 1.27 1.27)) (justify left top) hide)
     )
@@
       (effects (font (size 1.27 1.27)))
     )
-    (property "Footprint" "UTSVT_Connectors:533072071" (at 233.68 171.12 0)
-      (effects (font (size 1.27 1.27)) (justify left top) hide)
+    (property "Footprint" "UTSVT_Connectors:Molex_53307-2071" (at 233.68 171.12 0)
+      (effects (font (size 1.27 1.27)) (justify left top))
     )
     (property "Datasheet" "https://tools.molex.com/pdm_docs/sd/533072071_sd.pdf" (at 233.68 271.12 0)

Commit message: Cleaned up silkscreen
Other:
- note added: "To do: Schematic: Double check LeaderSOM Connector layout Fix part number and value for gate resistor on Strobe Check Orion datasheet again for fan connections for sanity check Sanity check for pullup math on fans PCB: Silkscreen"
- note removed: "To do: Schematic: Double check LeaderSOM Connector layout Fix part number and value for gate resistor on Strobe Check Orion datasheet again for fan connections for sanity check Sanity check for pullup math on fans PCB: Layout :cry: Fix spacing for LeaderSOM holes Silkscreen Silkscreen guide for 4 wire vs 3 wire fans Guide for driving fans with orion"
Changed lines of the file:
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@@
     (effects (font (size 2.54 2.54) (thickness 0.508) bold) (justify left bottom))
   )
-  (text "To do:\nSchematic:\n	Double check LeaderSOM Connector layout\n	Fix part number and value for gate resistor on Strobe\n	Check Orion datasheet again for fan connections for sanity check\n	Sanity check for pullup math on fans\nPCB:\n	Layout :cry:\n	Fix spacing for LeaderSOM holes\n	Silkscreen\n	Silkscreen guide for 4 wire vs 3 wire fans\n	Guide for driving fans with orion\n	\n"
-    (at 28.575 196.85 0)
+  (text "To do:\nSchematic:\n	Double check LeaderSOM Connector layout\n	Fix part number and value for gate resistor on Strobe\n	Check Orion datasheet again for fan connections for sanity check\n	Sanity check for pullup math on fans\nPCB:\n	Silkscreen\n"
+    (at 28.575 181.61 0)
     (effects (font (size 1.27 1.27)) (justify left bottom))
   )

Commit message: last sanity check + part numbers (ready for review)
Parts:
- J1, J2: Mouser Part Number 538-53307-2071 -> (none)
Other:
- note removed: "To do: Schematic: Double check LeaderSOM Connector layout Fix part number and value for gate resistor on Strobe Check Orion datasheet again for fan connections for sanity check Sanity check for pullup math on fans PCB: Silkscreen"
Changed lines of the file:
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@@
     (effects (font (size 2.54 2.54) (thickness 0.508) bold) (justify left bottom))
-  )
-  (text "To do:\nSchematic:\n	Double check LeaderSOM Connector layout\n	Fix part number and value for gate resistor on Strobe\n	Check Orion datasheet again for fan connections for sanity check\n	Sanity check for pullup math on fans\nPCB:\n	Silkscreen\n"
-    (at 28.575 181.61 0)
-    (effects (font (size 1.27 1.27)) (justify left bottom))
   )
   (text "V1.0: \n- 3 Contactors + Fan controller circuit" (at 219.075 43.18 0)
@@
       (effects (font (size 1.27 1.27)) (justify left top) hide)
     )
-    (property "Mouser Part Number" "538-53307-2071" (at 233.68 606.68 0)
+    (property "Mouser Part Number" "" (at 233.68 606.68 0)
       (effects (font (size 1.27 1.27)) (justify left top) hide)
     )
@@
       (effects (font (size 1.27 1.27)) (justify left top) hide)
     )
-    (property "Mouser Part Number" "538-53307-2071" (at 233.68 571.12 0)
-      (effects (font (size 1.27 1.27)) (justify left top) hide)
-    )
+    (property "Mouser Part Number" "" (at 233.68 571.12 0)
+      (effects (font (size 1.27 1.27)) (justify left top) hide)
+    )

Commit message: updated symbol and footprint libraries to use
Parts:
- J1, J2: footprint UTSVT_Connectors:Molex_53307-2071 -> UTSVT_Connectors:533072071; Mouser Part Number (none) -> 538-53307-2071
Changed lines of the file:
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@@
       (effects (font (size 1.27 1.27)))
     )
-    (property "Footprint" "UTSVT_Connectors:Molex_53307-2071" (at 233.68 206.68 0)
+    (property "Footprint" "UTSVT_Connectors:533072071" (at 233.68 206.68 0)
       (effects (font (size 1.27 1.27)) (justify left top) hide)
     )
@@
       (effects (font (size 1.27 1.27)) (justify left top) hide)
     )
-    (property "Mouser Part Number" "" (at 233.68 606.68 0)
+    (property "Mouser Part Number" "538-53307-2071" (at 233.68 606.68 0)
       (effects (font (size 1.27 1.27)) (justify left top) hide)
     )
@@
       (effects (font (size 1.27 1.27)))
     )
-    (property "Footprint" "UTSVT_Connectors:Molex_53307-2071" (at 233.68 171.12 0)
+    (property "Footprint" "UTSVT_Connectors:533072071" (at 233.68 171.12 0)
       (effects (font (size 1.27 1.27)) (justify left top))
     )
@@
       (effects (font (size 1.27 1.27)) (justify left top) hide)
     )
-    (property "Mouser Part Number" "" (at 233.68 571.12 0)
-      (effects (font (size 1.27 1.27)) (justify left top) hide)
-    )
+    (property "Mouser Part Number" "538-53307-2071" (at 233.68 571.12 0)
+      (effects (font (size 1.27 1.27)) (justify left top) hide)
+    )
