File: Contactor_Driver.kicad_sch (KiCad schematic)
At the start: 26 parts, among them J1 Conn_01x04, Q3 BUK9M23-80E, Q4 FDC2512, Q5 NTR4003NT1G, Q6 NMOS, U2 SI8261ABC-IS

Commit message: Added more documentatino to the Contactor circuits
Other:
- note added: "Clipping Voltage Logic to ensure that only 3.3V logic goes in to mcu"
- note added: "The upper mosfet is for voltage protection: If some high votlage spike comes in from the Contactor it won't send it through the rest of the circuit"
- note removed: "Should this by GND or GNDPWR?"
Changed lines of the file:
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@@
+    (effects (font (size 1.27 1.27)) (justify left bottom))
+  )
+  (text "Clipping Voltage Logic to \nensure that only 3.3V logic goes in to mcu"
+    (at 38.1 146.05 0)
     (effects (font (size 1.27 1.27)) (justify left bottom))
   )
@@
     (effects (font (size 1.27 1.27)) (justify left bottom))
   )
-  (text "Should this by GND or GNDPWR?" (at 61.595 130.175 0)
+  (text "The upper mosfet is for voltage protection:\nIf some high votlage spike comes in from the Contactor \nit won't send it through the rest of the circuit"
+    (at 228.6 24.13 0)
     (effects (font (size 1.27 1.27)) (justify left bottom))
   )

Commit message: Added part numbers and datasheet to isolator part
Parts:
- Q5: P/N (none) -> NTR4003NT1G
Changed lines of the file:
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@@
       (effects (font (size 1.27 1.27)) hide)
     )
-    (property "Datasheet" "~" (at 50.8 77.47 0)
+    (property "Datasheet" "https://www.mouser.com/datasheet/2/308/1/NTR4003N_D-2319203.pdf" (at 50.8 77.47 0)
       (effects (font (size 1.27 1.27)) hide)
     )
+    (property "P/N" "NTR4003NT1G" (at 50.8 77.47 0)
+      (effects (font (size 1.27 1.27)) hide)
+    )

Commit message: removed redundant contactor circuit
Parts:
- removed C8: 1u, Capacitor_SMD:C_0805_2012Metric, symbol Device:C
- removed D6: D, LED_SMD:LED_0805_2012Metric, symbol Device:D
- removed D9: V2F22HM3/H, UTSVT_Passive:V2F22HM, symbol Device:D
- removed Q6: NMOS, symbol Simulation_SPICE:NMOS
- removed R12: 100k, Resistor_SMD:R_0805_2012Metric, symbol Device:R
Other:
- note removed: "Lakshay's cool test circuit (ignore)"

Commit message: Added part numbers for Contactors and Strobe light
Parts:
- removed C4: 0.1u, Capacitor_SMD:C_0805_2012Metric, symbol Device:C
- removed C5: 10u, Capacitor_SMD:C_0805_2012Metric, symbol Device:C
- removed C6: C, Capacitor_SMD:C_0805_2012Metric, symbol Device:C
- removed D2: V2F22HM, UTSVT_Passive:V2F22HM, symbol Diode:C3D25170H
- removed D3: D, LED_SMD:LED_0805_2012Metric, symbol Device:D
- removed Q4: FDC2512, Package_TO_SOT_SMD:SuperSOT-6, symbol Transistor_FET:FDC2512
- removed R7, R9: R, Resistor_SMD:R_0805_2012Metric, symbol Device:R
- added C14, C4: 100nF, Capacitor_SMD:C_0805_2012Metric, symbol Device:C_Small
- added C5: 10uF, Capacitor_SMD:C_0805_2012Metric, symbol Device:C_Small
- added D2: V2F22HM3/H, UTSVT_Passive:V2F22HM, symbol Device:D
- added Q4: VND5N07-E, Package_TO_SOT_SMD:TO-252-2, symbol Device:Q_NMOS_GDS
- added R21: 1.5k, Resistor_SMD:R_0805_2012Metric, symbol Device:R
- added R22: 470, Resistor_SMD:R_0805_2012Metric, symbol Device:R
- C7: P/N (none) -> C0805C105K5PACTU
- D5: value D -> ContactorEn; Color (none) -> Green; P/N (none) -> APTD2012LCGCK
- D7: P/N (none) -> BAS70-04
- D8: value SZESD9B5.0ST5G -> SMAJ43CA
- R10, R8: value R -> 10k; Mouser Part Number (none) -> 71-CRCW080510K0FKEAC; P/N (none) -> CRCW080510K0FKEAC
- R11: value R -> 0; Mouser Part Number (none) -> 71-CRCW08050000Z0EAC; P/N (none) -> CRCW08050000Z0EAC
- R13: value R -> 100k
Connections:
- net +12V: now also R8.1, C4.1, C5.1, D2.1 (K)
- net +5V: now also R21.1, R22.2; no longer R8.1
- net CONTACTOR_V-: now also Q4.2 (D)
- net GNDPWR: now also C4.2, C5.2
- net at D4.2 (A), Q3.5 (D), R13.2: now also C14.2, D2.2 (A), Q4.3 (S)
- net at D4.1 (K), R13.1: now also R8.2, C14.1, Q4.1 (G)
- net at D5.2 (A): now also R21.2
- net at U2.2 (ANODE): now also R22.1; no longer R8.2
Other:
- note removed: "FIND BETTER PART"
- moved on the sheet: R13

Commit message: Added even moreeeee Contactor p/n + added 4 more mounting holes
Parts:
- D2, D4: P/N (none) -> V2F22HM
- D8: P/N (none) -> SMAJ43CA
- Q3: P/N (none) -> BUK9M23-80E
- R13: P/N (none) -> CRCW0805100KFKEAC
- U2: P/N (none) -> SI8261ABC-IS
Changed lines of the file:
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@@
       (effects (font (size 1.27 1.27)) (justify left) hide)
+    )
+    (property "P/N" "BUK9M23-80E" (at 210.82 78.105 0)
+      (effects (font (size 1.27 1.27)) hide)
     )
     (pin "1")
@@
       (effects (font (size 1.27 1.27)) hide)
     )
+    (property "P/N" "V2F22HM" (at 243.205 64.135 90)
+      (effects (font (size 1.27 1.27)) hide)
+    )
     (pin "1")
     (pin "2")
@@
       (effects (font (size 1.27 1.27)) hide)
     )
+    (property "P/N" "SMAJ43CA" (at 193.675 49.53 90)
+      (effects (font (size 1.27 1.27)) hide)
+    )
     (pin "1")
     (pin "2")
@@
       (effects (font (size 1.27 1.27)) hide)
     )
-    (property "Datasheet" "~" (at 182.88 67.31 0)
+    (property "Datasheet" "https://www.mouser.com/ProductDetail/Vishay-Dale/CRCW0805100KFKEAC?qs=sGAEpiMZZMvdGkrng054t0DrEhLhGh8gZRT9GjFuHWDV3jEqj5sSqw%3D%3D" (at 182.88 67.31 0)
+      (effects (font (size 1.27 1.27)) hide)
+    )
+    (property "P/N" "CRCW0805100KFKEAC" (at 182.88 67.31 0)
       (effects (font (size 1.27 1.27)) hide)
     )
@@
       (effects (font (size 1.27 1.27)) hide)
     )
+    (property "P/N" "V2F22HM" (at 176.53 67.31 90)
+      (effects (font (size 1.27 1.27)) hide)
+    )
     (pin "1")
     (pin "2")
@@
       (effects (font (size 1.27 1.27)) hide)
     )
+    (property "P/N" "SI8261ABC-IS" (at 82.55 57.785 0)
+      (effects (font (size 1.27 1.27)) hide)
+    )

Commit message: Combined fan and contactor stuff
Parts:
- removed Q4: VND5N07-E, Package_TO_SOT_SMD:TO-252-2, symbol Device:Q_NMOS_GDS
- added Q8: VND5N07-E, Package_TO_SOT_SMD:TO-252-2, symbol Device:Q_NMOS_GDS
- renumbered C14 to C6, D7 to D10, D5 to D11, D4 to D12, D8 to D13, D2 to D14, J1 to J9, Q5 to Q7, Q3 to Q9, R11 to R23, R10 to R24, R21 to R25, R22 to R26, R8 to R27, R13 to R28
Connections:
- net CONTACTOR_V-: now also Q8.2 (D)
- net at C6.2, D12.2 (A), D14.2 (A)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: now also Q8.3 (S)
- net at C6.1, D12.1 (K), R27.2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: now also Q8.1 (G)
