File: Contactor_Driver.kicad_sch (KiCad schematic)
At the start: 14 parts, among them J9 Conn_01x04, Q1 BUK9M3R3-40HX, U5 SI8261ABC-IS

Commit message: Finished Contactor Schematic (hopefully :( )
Parts:
- removed D28: SMAJ43CA, Diode_SMD:D_SOD-923, symbol Diode:SZESD9B5.0ST5G
Other:
- moved on the sheet: D25, R26
Changed lines of the file:
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@@
   (junction (at 93.98 55.88) (diameter 0) (color 0 0 0 0)
   )
-  (junction (at 170.18 54.61) (diameter 0) (color 0 0 0 0)
-  )
   (junction (at 66.04 99.06) (diameter 0) (color 0 0 0 0)
   )
@@
   (junction (at 186.69 72.39) (diameter 0) (color 0 0 0 0)
   )
-  (junction (at 170.18 38.1) (diameter 0) (color 0 0 0 0)
-  )
   (junction (at 186.69 44.45) (diameter 0) (color 0 0 0 0)
   )
-  (wire (pts (xy 170.18 54.61) (xy 186.69 54.61))
+  (wire (pts (xy 177.165 54.61) (xy 186.69 54.61))
     (stroke (width 0) (type default))
   )
@@
     (stroke (width 0) (type default))
   )
-  (wire (pts (xy 158.75 52.705) (xy 158.75 54.61))
+  (wire (pts (xy 177.165 52.705) (xy 177.165 54.61))
     (stroke (width 0) (type default))
   )
@@
     (stroke (width 0) (type default))
   )
-  (wire (pts (xy 170.18 50.8) (xy 170.18 54.61))
-    (stroke (width 0) (type default))
-  )
   (wire (pts (xy 186.69 31.75) (xy 186.69 38.1))
     (stroke (width 0) (type default))
@@
     (stroke (width 0) (type default))
   )
-  (wire (pts (xy 158.75 38.1) (xy 170.18 38.1))
-    (stroke (width 0) (type default))
-  )
-  (wire (pts (xy 158.75 45.72) (xy 158.75 47.625))
-    (stroke (width 0) (type default))
-  )
   (wire (pts (xy 57.15 99.06) (xy 66.04 99.06))
     (stroke (width 0) (type default))
@@
     (stroke (width 0) (type default))
   )
-  (wire (pts (xy 170.18 38.1) (xy 186.69 38.1))
+  (wire (pts (xy 177.165 38.1) (xy 186.69 38.1))
     (stroke (width 0) (type default))
   )
@@
     (stroke (width 0) (type default))
   )
-  (wire (pts (xy 170.18 38.1) (xy 170.18 43.18))
-    (stroke (width 0) (type default))
-  )
   (wire (pts (xy 109.855 53.34) (xy 103.505 53.34))
     (stroke (width 0) (type default))
@@
     (stroke (width 0) (type default))
   )
-  (wire (pts (xy 158.75 54.61) (xy 170.18 54.61))
-    (stroke (width 0) (type default))
-  )
   (wire (pts (xy 109.855 53.34) (xy 114.935 53.34))
     (stroke (width 0) (type default))
   )
   (wire (pts (xy 186.69 38.1) (xy 210.82 38.1))
+    (stroke (width 0) (type default))
+  )
+  (wire (pts (xy 177.165 45.72) (xy 177.165 47.625))
     (stroke (width 0) (type default))
   )
@@
     )
   )
-  (symbol (lib_id "Device:R") (at 158.75 41.91 0) (unit 1)
+  (symbol (lib_id "Device:R") (at 177.165 41.91 0) (unit 1)
     (in_bom yes) (on_board yes) (dnp no) (fields_autoplaced)
-    (property "Reference" "R26" (at 161.29 40.64 0)
-      (effects (font (size 1.27 1.27)) (justify left))
-    )
-    (property "Value" "10k" (at 161.29 43.18 0)
-      (effects (font (size 1.27 1.27)) (justify left))
-    )
-    (property "Footprint" "Resistor_SMD:R_0805_2012Metric" (at 156.972 41.91 90)
-      (effects (font (size 1.27 1.27)) hide)
-    )
-    (property "Datasheet" "~" (at 158.75 41.91 0)
+    (property "Reference" "R26" (at 179.705 40.64 0)
+      (effects (font (size 1.27 1.27)) (justify left))
+    )
+    (property "Value" "10k" (at 179.705 43.18 0)
+      (effects (font (size 1.27 1.27)) (justify left))
+    )
+    (property "Footprint" "Resistor_SMD:R_0805_2012Metric" (at 175.387 41.91 90)
+      (effects (font (size 1.27 1.27)) hide)
+    )
+    (property "Datasheet" "~" (at 177.165 41.91 0)
       (effects (font (size 1.27 1.27)) hide)
     )
@@
       (effects (font (size 1.27 1.27)) (justify left))
     )
-    (property "Value" "V2F22HM" (at 175.26 52.07 90)
+    (property "Value" "V2F22HM" (at 191.135 50.165 90)
       (effects (font (size 1.27 1.27)) (justify left))
     )
@@
     )
   )
-  (symbol (lib_id "Device:LED_Small") (at 158.75 50.165 90) (unit 1)
-    (in_bom yes) (on_board yes) (dnp no)
-    (property "Reference" "D25" (at 160.4772 48.9966 90)
+  (symbol (lib_id "Device:LED_Small") (at 177.165 50.165 90) (unit 1)
+    (in_bom yes) (on_board yes) (dnp no)
+    (property "Reference" "D25" (at 178.8922 48.9966 90)
       (effects (font (size 1.27 1.27)) (justify right))
     )
-    (property "Value" "Green" (at 160.4772 51.308 90)
+    (property "Value" "Green" (at 178.8922 51.308 90)
       (effects (font (size 1.27 1.27)) (justify right))
     )
-    (property "Footprint" "LED_SMD:LED_0805_2012Metric_Pad1.15x1.40mm_HandSolder" (at 158.75 50.165 90)
-      (effects (font (size 1.27 1.27)) hide)
-    )
-    (property "Datasheet" "" (at 158.75 50.165 90)
-      (effects (font (size 1.27 1.27)) hide)
-    )
-    (property "P/N" "LHR971-KN1" (at 158.75 50.165 0)
+    (property "Footprint" "LED_SMD:LED_0805_2012Metric_Pad1.15x1.40mm_HandSolder" (at 177.165 50.165 90)
+      (effects (font (size 1.27 1.27)) hide)
+    )
+    (property "Datasheet" "" (at 177.165 50.165 90)
+      (effects (font (size 1.27 1.27)) hide)
+    )
+    (property "P/N" "LHR971-KN1" (at 177.165 50.165 0)
       (effects (font (size 1.27 1.27)) hide)
     )
@@
         )
       )
-    )
-  )
-  (symbol (lib_id "Diode:SZESD9B5.0ST5G") (at 170.18 46.99 90) (unit 1)
-    (in_bom yes) (on_board yes) (dnp no)
-    (property "Reference" "D28" (at 173.355 45.72 90)
-      (effects (font (size 1.27 1.27)) (justify right))
-    )
-    (property "Value" "SMAJ43CA" (at 173.355 47.625 90)
-      (effects (font (size 1.27 1.27)) (justify right))
-    )
-    (property "Footprint" "Diode_SMD:D_SOD-923" (at 170.18 46.99 0)
-      (effects (font (size 1.27 1.27)) hide)
-    )
-    (property "Datasheet" "https://www.littelfuse.com/media?resourcetype=datasheets&itemid=13c2a823-03b8-4d1f-9ddc-9b44670aed9d&filename=littelfuse_tvs_diode_smaj_datasheet.pdf" (at 170.18 46.99 0)
-      (effects (font (size 1.27 1.27)) hide)
-    )
-    (property "P/N" "SMAJ43CA" (at 170.18 46.99 90)
-      (effects (font (size 1.27 1.27)) hide)
-    )
-    (pin "1")
-    (pin "2")
-    (instances
-      (project "BPS-LeaderDaughter"
-        (path "/2e9f4f51-d216-4952-a31c-e7104e0d4b1e/ae57cd3a-fadb-4313-835a-95d5b185a797"
-          (reference "D28") (unit 1)
-        )
-        (path "/2e9f4f51-d216-4952-a31c-e7104e0d4b1e/5e4c6ec4-73d4-4ed3-a75f-02eb4f9ac8b3"
-          (reference "D29") (unit 1)
-        )
-        (path "/2e9f4f51-d216-4952-a31c-e7104e0d4b1e/bb673292-4a5d-469b-b6b6-0dc7df3c162d"
-          (reference "D30") (unit 1)
-        )
-      )

Commit message: Started adding changes from review
Parts:
- removed Q1: BUK9M3R3-40HX, Package_TO_SOT_SMD:LFPAK33, symbol Transistor_FET:BUK9M23-80EX
- added Q?: BUK9M23-80E, Package_TO_SOT_SMD:LFPAK33, symbol Transistor_FET:BUK9M23-80EX
- R26: value 10k -> 5k
- R41: value R -> 50
Connections:
- net CONTACTOR_V-: now also Q?.5 (D)
- net GNDPWR: now also Q?.1 (S), Q?.2 (S), Q?.3 (S)
- net PWM_ISO: now also Q?.4 (G)
- net +5V renamed +3.3V
Other:
- note added: "Vf = 1.6 V If = 30 mA (3.3 - 1.6) / .030"
Changed lines of the file:
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@@
     (effects (font (size 2.54 2.54) (thickness 0.508) bold) (justify left bottom))
+  )
+  (text "Vf = 1.6 V\nIf = 30 mA\n(3.3 - 1.6) / .030" (at 42.545 45.085 0)
+    (effects (font (size 1.27 1.27)) (justify left bottom))
   )
   (text "The upper mosfet is for voltage protection:\nIf some high votlage spike comes in from the Contactor \nit won't send it through the rest of the circuit"
@@
     )
   )
+  (symbol (lib_id "Transistor_FET:BUK9M23-80EX") (at 184.15 61.595 0) (unit 1)
+    (in_bom yes) (on_board yes) (dnp no) (fields_autoplaced)
+    (property "Reference" "Q?" (at 190.5 60.325 0)
+      (effects (font (size 1.27 1.27)) (justify left))
+    )
+    (property "Value" "BUK9M23-80E" (at 190.5 62.865 0)
+      (effects (font (size 1.27 1.27)) (justify left))
+    )
+    (property "Footprint" "Package_TO_SOT_SMD:LFPAK33" (at 189.23 63.5 0)
+      (effects (font (size 1.27 1.27) italic) (justify left) hide)
+    )
+    (property "Datasheet" "https://assets.nexperia.com/documents/data-sheet/BUK9M23-80E.pdf" (at 184.15 61.595 90)
+      (effects (font (size 1.27 1.27)) (justify left) hide)
+    )
+    (property "P/N" "BUK9M23-80E" (at 184.15 61.595 0)
+      (effects (font (size 1.27 1.27)) hide)
+    )
+    (pin "1")
+    (pin "2")
+    (pin "3")
+    (pin "4")
+    (pin "5")
+    (instances
+      (project "BPS-LeaderDaughter"
+        (path "/2e9f4f51-d216-4952-a31c-e7104e0d4b1e/bf23a663-b938-440b-843e-ef7912c82d18"
+          (reference "Q?") (unit 1)
+        )
+        (path "/2e9f4f51-d216-4952-a31c-e7104e0d4b1e/bf23a663-b938-440b-843e-ef7912c82d18/cb70587e-88a7-4e34-a774-2566ee5ba031"
+          (reference "Q5") (unit 1)
+        )
+        (path "/2e9f4f51-d216-4952-a31c-e7104e0d4b1e/bf23a663-b938-440b-843e-ef7912c82d18/726bf2a6-1244-4795-8327-149588380c7e"
+          (reference "Q6") (unit 1)
+        )
+        (path "/2e9f4f51-d216-4952-a31c-e7104e0d4b1e/bf23a663-b938-440b-843e-ef7912c82d18/66fa18d5-534c-477b-b6ed-b26c28a08707"
+          (reference "Q7") (unit 1)
+        )
+        (path "/2e9f4f51-d216-4952-a31c-e7104e0d4b1e/bf23a663-b938-440b-843e-ef7912c82d18/3bf7416b-1505-491f-89b6-6e99a8c04638"
+          (reference "Q8") (unit 1)
+        )
+        (path "/2e9f4f51-d216-4952-a31c-e7104e0d4b1e/ae57cd3a-fadb-4313-835a-95d5b185a797"
+          (reference "Q1") (unit 1)
+        )
+        (path "/2e9f4f51-d216-4952-a31c-e7104e0d4b1e/5e4c6ec4-73d4-4ed3-a75f-02eb4f9ac8b3"
+          (reference "Q2") (unit 1)
+        )
+        (path "/2e9f4f51-d216-4952-a31c-e7104e0d4b1e/bb673292-4a5d-469b-b6b6-0dc7df3c162d"
+          (reference "Q4") (unit 1)
+        )
+      )
+    )
+  )
   (symbol (lib_id "Device:R") (at 177.165 41.91 0) (unit 1)
     (in_bom yes) (on_board yes) (dnp no) (fields_autoplaced)
-    (property "Reference" "R26" (at 179.705 40.64 0)
-      (effects (font (size 1.27 1.27)) (justify left))
-    )
-    (property "Value" "10k" (at 179.705 43.18 0)
+    (property "Reference" "R26" (at 179.07 40.64 0)
+      (effects (font (size 1.27 1.27)) (justify left))
+    )
+    (property "Value" "5k" (at 179.07 43.18 0)
       (effects (font (size 1.27 1.27)) (justify left))
     )
@@
     )
   )
-  (symbol (lib_id "Transistor_FET:BUK9M23-80EX") (at 184.15 61.595 0) (unit 1)
-    (in_bom yes) (on_board yes) (dnp no)
-    (property "Reference" "Q1" (at 189.23 62.865 0)
-      (effects (font (size 1.27 1.27)) (justify left))
-    )
-    (property "Value" "BUK9M3R3-40HX" (at 189.23 59.055 0)
-      (effects (font (size 1.27 1.27)) (justify left))
-    )
-    (property "Footprint" "Package_TO_SOT_SMD:LFPAK33" (at 189.23 63.5 0)
-      (effects (font (size 1.27 1.27) italic) (justify left) hide)
-    )
-    (property "Datasheet" "https://assets.nexperia.com/documents/data-sheet/BUK9M3R3-40H.pdf" (at 184.15 61.595 90)
-      (effects (font (size 1.27 1.27)) (justify left) hide)
-    )
-    (property "P/n" "BUK9M3R3-40HX" (at 184.15 61.595 0)
-      (effects (font (size 1.27 1.27)) hide)
-    )
-    (pin "1")
-    (pin "2")
-    (pin "3")
-    (pin "4")
-    (pin "5")
-    (instances
-      (project "BPS-LeaderDaughter"
-        (path "/2e9f4f51-d216-4952-a31c-e7104e0d4b1e/ae57cd3a-fadb-4313-835a-95d5b185a797"
-          (reference "Q1") (unit 1)
-        )
-        (path "/2e9f4f51-d216-4952-a31c-e7104e0d4b1e/5e4c6ec4-73d4-4ed3-a75f-02eb4f9ac8b3"
-          (reference "Q2") (unit 1)
-        )
-        (path "/2e9f4f51-d216-4952-a31c-e7104e0d4b1e/bb673292-4a5d-469b-b6b6-0dc7df3c162d"
-          (reference "Q10") (unit 1)
-        )
-      )
-      (project "BPS-Fan"
-        (path "/e60847d4-a954-40b9-b9c4-54b73957661c"
-          (reference "Q4") (unit 1)
-        )
-      )
-    )
-  )
   (symbol (lib_id "utsvt-chips:BAS70-04") (at 87.63 95.885 270) (unit 1)
     (in_bom yes) (on_board yes) (dnp no)
@@
     )
   )
-  (symbol (lib_id "power:+5V") (at 87.63 92.075 0) (unit 1)
-    (in_bom yes) (on_board yes) (dnp no)
-    (property "Reference" "#PWR029" (at 87.63 95.885 0)
-      (effects (font (size 1.27 1.27)) hide)
-    )
-    (property "Value" "+5V" (at 88.011 87.6808 0)
-      (effects (font (size 1.27 1.27)))
-    )
-    (property "Footprint" "" (at 87.63 92.075 0)
-      (effects (font (size 1.27 1.27)) hide)
-    )
-    (property "Datasheet" "" (at 87.63 92.075 0)
-      (effects (font (size 1.27 1.27)) hide)
-    )
-    (pin "1")
-    (instances
-      (project "BPS-LeaderDaughter"
-        (path "/2e9f4f51-d216-4952-a31c-e7104e0d4b1e/ae57cd3a-fadb-4313-835a-95d5b185a797"
-          (reference "#PWR029") (unit 1)
-        )
-        (path "/2e9f4f51-d216-4952-a31c-e7104e0d4b1e/5e4c6ec4-73d4-4ed3-a75f-02eb4f9ac8b3"
-          (reference "#PWR041") (unit 1)
-        )
-        (path "/2e9f4f51-d216-4952-a31c-e7104e0d4b1e/bb673292-4a5d-469b-b6b6-0dc7df3c162d"
-          (reference "#PWR053") (unit 1)
-        )
-      )
-      (project "BPS-Leader"
-        (path "/c248b171-df31-4e8a-afb6-607fa2df334b/00000000-0000-0000-0000-00005c38c674"
-          (reference "#PWR061") (unit 1)
-        )
-        (path "/c248b171-df31-4e8a-afb6-607fa2df334b/3faa4167-9e5e-4372-9a55-3c963a25ae73"
-          (reference "#PWR0114") (unit 1)
-        )
-        (path "/c248b171-df31-4e8a-afb6-607fa2df334b/bb594d23-7f65-4f42-8951-e176f5e7b2cb"
-          (reference "#PWR0114") (unit 1)
-        )
-      )
-    )
-  )
   (symbol (lib_id "power:GND") (at 66.04 109.855 0) (unit 1)
     (in_bom yes) (on_board yes) (dnp no)
@@
     )
   )
+  (symbol (lib_id "power:+3.3V") (at 87.63 92.075 0) (unit 1)
+    (in_bom yes) (on_board yes) (dnp no) (fields_autoplaced)
+    (property "Reference" "#PWR017" (at 87.63 95.885 0)
+      (effects (font (size 1.27 1.27)) hide)
+    )
+    (property "Value" "+3.3V" (at 87.63 87.63 0)
+      (effects (font (size 1.27 1.27)))
+    )
+    (property "Footprint" "" (at 87.63 92.075 0)
+      (effects (font (size 1.27 1.27)) hide)
+    )
+    (property "Datasheet" "" (at 87.63 92.075 0)
+      (effects (font (size 1.27 1.27)) hide)
+    )
+    (pin "1")
+    (instances
+      (project "BPS-LeaderDaughter"
+        (path "/2e9f4f51-d216-4952-a31c-e7104e0d4b1e/ae57cd3a-fadb-4313-835a-95d5b185a797"
+          (reference "#PWR017") (unit 1)
+        )
+        (path "/2e9f4f51-d216-4952-a31c-e7104e0d4b1e/5e4c6ec4-73d4-4ed3-a75f-02eb4f9ac8b3"
+          (reference "#PWR018") (unit 1)
+        )
+        (path "/2e9f4f51-d216-4952-a31c-e7104e0d4b1e/bb673292-4a5d-469b-b6b6-0dc7df3c162d"
+          (reference "#PWR019") (unit 1)
+        )
+      )
+    )
+  )
   (symbol (lib_id "Device:C") (at 210.82 45.085 0) (unit 1)
     (in_bom yes) (on_board yes) (dnp no) (fields_autoplaced)
@@
   (symbol (lib_id "Device:R") (at 62.23 53.34 90) (unit 1)
     (in_bom yes) (on_board yes) (dnp no) (fields_autoplaced)
-    (property "Reference" "R41" (at 62.23 47.625 90)
-      (effects (font (size 1.27 1.27)))
-    )
-    (property "Value" "R" (at 62.23 50.165 90)
-      (effects (font (size 1.27 1.27)))
-    )
+    (property "Reference" "R41" (at 62.23 46.99 90)
+      (effects (font (size 1.27 1.27)))
+    )
+    (property "Value" "50" (at 62.23 49.53 90)
+      (effects (font (size 1.27 1.27)))
+    )

Commit message: Fan layout updated
Parts:
- R41: footprint (none) -> Resistor_SMD:R_0805_2012Metric
- renumbered R26 to R7
Changed lines of the file:
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@@
   (symbol (lib_id "Device:R") (at 177.165 41.91 0) (unit 1)
     (in_bom yes) (on_board yes) (dnp no) (fields_autoplaced)
-    (property "Reference" "R26" (at 179.07 40.64 0)
+    (property "Reference" "R7" (at 179.07 40.64 0)
       (effects (font (size 1.27 1.27)) (justify left))
     )
@@
       (project "BPS-LeaderDaughter"
         (path "/2e9f4f51-d216-4952-a31c-e7104e0d4b1e/ae57cd3a-fadb-4313-835a-95d5b185a797"
-          (reference "R26") (unit 1)
-        )
-        (path "/2e9f4f51-d216-4952-a31c-e7104e0d4b1e/5e4c6ec4-73d4-4ed3-a75f-02eb4f9ac8b3"
-          (reference "R27") (unit 1)
-        )
-        (path "/2e9f4f51-d216-4952-a31c-e7104e0d4b1e/bb673292-4a5d-469b-b6b6-0dc7df3c162d"
-          (reference "R29") (unit 1)
+          (reference "R7") (unit 1)
+        )
+        (path "/2e9f4f51-d216-4952-a31c-e7104e0d4b1e/5e4c6ec4-73d4-4ed3-a75f-02eb4f9ac8b3"
+          (reference "R3") (unit 1)
+        )
+        (path "/2e9f4f51-d216-4952-a31c-e7104e0d4b1e/bb673292-4a5d-469b-b6b6-0dc7df3c162d"
+          (reference "R11") (unit 1)
         )
       )
@@
         )
         (path "/2e9f4f51-d216-4952-a31c-e7104e0d4b1e/5e4c6ec4-73d4-4ed3-a75f-02eb4f9ac8b3"
-          (reference "D16") (unit 1)
+          (reference "D14") (unit 1)
         )
         (path "/2e9f4f51-d216-4952-a31c-e7104e0d4b1e/bb673292-4a5d-469b-b6b6-0dc7df3c162d"
@@
   (symbol (lib_name "GNDPWR_4") (lib_id "power:GNDPWR") (at 210.82 50.8 0) (unit 1)
     (in_bom yes) (on_board yes) (dnp no) (fields_autoplaced)
-    (property "Reference" "#PWR012" (at 210.82 55.88 0)
+    (property "Reference" "#PWR0111" (at 210.82 55.88 0)
       (effects (font (size 1.27 1.27)) hide)
     )
@@
       (project "BPS-LeaderDaughter"
         (path "/2e9f4f51-d216-4952-a31c-e7104e0d4b1e/ae57cd3a-fadb-4313-835a-95d5b185a797"
-          (reference "#PWR012") (unit 1)
+          (reference "#PWR0111") (unit 1)
         )
         (path "/2e9f4f51-d216-4952-a31c-e7104e0d4b1e/5e4c6ec4-73d4-4ed3-a75f-02eb4f9ac8b3"
@@
   (symbol (lib_id "power:GND") (at 87.63 109.22 0) (unit 1)
     (in_bom yes) (on_board yes) (dnp no)
-    (property "Reference" "#PWR030" (at 87.63 115.57 0)
+    (property "Reference" "#PWR0107" (at 87.63 115.57 0)
       (effects (font (size 1.27 1.27)) hide)
     )
@@
       (project "BPS-LeaderDaughter"
         (path "/2e9f4f51-d216-4952-a31c-e7104e0d4b1e/ae57cd3a-fadb-4313-835a-95d5b185a797"
-          (reference "#PWR030") (unit 1)
+          (reference "#PWR0107") (unit 1)
         )
         (path "/2e9f4f51-d216-4952-a31c-e7104e0d4b1e/5e4c6ec4-73d4-4ed3-a75f-02eb4f9ac8b3"
@@
         )
         (path "/2e9f4f51-d216-4952-a31c-e7104e0d4b1e/5e4c6ec4-73d4-4ed3-a75f-02eb4f9ac8b3"
-          (reference "D15") (unit 2)
+          (reference "D13") (unit 2)
         )
         (path "/2e9f4f51-d216-4952-a31c-e7104e0d4b1e/bb673292-4a5d-469b-b6b6-0dc7df3c162d"
@@
         )
         (path "/2e9f4f51-d216-4952-a31c-e7104e0d4b1e/5e4c6ec4-73d4-4ed3-a75f-02eb4f9ac8b3"
-          (reference "D15") (unit 1)
+          (reference "D13") (unit 1)
         )
         (path "/2e9f4f51-d216-4952-a31c-e7104e0d4b1e/bb673292-4a5d-469b-b6b6-0dc7df3c162d"
@@
   (symbol (lib_name "GNDPWR_3") (lib_id "power:GNDPWR") (at 186.69 74.93 0) (unit 1)
     (in_bom yes) (on_board yes) (dnp no) (fields_autoplaced)
-    (property "Reference" "#PWR06" (at 186.69 80.01 0)
+    (property "Reference" "#PWR0110" (at 186.69 80.01 0)
       (effects (font (size 1.27 1.27)) hide)
     )
@@
       (project "BPS-LeaderDaughter"
         (path "/2e9f4f51-d216-4952-a31c-e7104e0d4b1e/ae57cd3a-fadb-4313-835a-95d5b185a797"
-          (reference "#PWR06") (unit 1)
-        )
-        (path "/2e9f4f51-d216-4952-a31c-e7104e0d4b1e/5e4c6ec4-73d4-4ed3-a75f-02eb4f9ac8b3"
-          (reference "#PWR07") (unit 1)
-        )
-        (path "/2e9f4f51-d216-4952-a31c-e7104e0d4b1e/bb673292-4a5d-469b-b6b6-0dc7df3c162d"
-          (reference "#PWR08") (unit 1)
+          (reference "#PWR0110") (unit 1)
+        )
+        (path "/2e9f4f51-d216-4952-a31c-e7104e0d4b1e/5e4c6ec4-73d4-4ed3-a75f-02eb4f9ac8b3"
+          (reference "#PWR0114") (unit 1)
+        )
+        (path "/2e9f4f51-d216-4952-a31c-e7104e0d4b1e/bb673292-4a5d-469b-b6b6-0dc7df3c162d"
+          (reference "#PWR0116") (unit 1)
         )
       )
@@
   (symbol (lib_id "power:+3.3V") (at 87.63 92.075 0) (unit 1)
     (in_bom yes) (on_board yes) (dnp no) (fields_autoplaced)
-    (property "Reference" "#PWR017" (at 87.63 95.885 0)
+    (property "Reference" "#PWR0109" (at 87.63 95.885 0)
       (effects (font (size 1.27 1.27)) hide)
     )
@@
       (project "BPS-LeaderDaughter"
         (path "/2e9f4f51-d216-4952-a31c-e7104e0d4b1e/ae57cd3a-fadb-4313-835a-95d5b185a797"
-          (reference "#PWR017") (unit 1)
-        )
-        (path "/2e9f4f51-d216-4952-a31c-e7104e0d4b1e/5e4c6ec4-73d4-4ed3-a75f-02eb4f9ac8b3"
-          (reference "#PWR018") (unit 1)
+          (reference "#PWR0109") (unit 1)
+        )
+        (path "/2e9f4f51-d216-4952-a31c-e7104e0d4b1e/5e4c6ec4-73d4-4ed3-a75f-02eb4f9ac8b3"
+          (reference "#PWR0113") (unit 1)
         )
         (path "/2e9f4f51-d216-4952-a31c-e7104e0d4b1e/bb673292-4a5d-469b-b6b6-0dc7df3c162d"
@@
   (symbol (lib_id "Device:R") (at 175.26 67.31 0) (unit 1)
     (in_bom yes) (on_board yes) (dnp no) (fields_autoplaced)
-    (property "Reference" "R5" (at 177.165 66.04 0)
-      (effects (font (size 1.27 1.27)) (justify left))
-    )
-    (property "Value" "100k" (at 177.165 68.58 0)
+    (property "Reference" "R5" (at 177.8 66.04 0)
+      (effects (font (size 1.27 1.27)) (justify left))
+    )
+    (property "Value" "100k" (at 177.8 68.58 0)
       (effects (font (size 1.27 1.27)) (justify left))
     )
@@
         )
         (path "/2e9f4f51-d216-4952-a31c-e7104e0d4b1e/bb673292-4a5d-469b-b6b6-0dc7df3c162d"
-          (reference "R25") (unit 1)
+          (reference "R9") (unit 1)
         )
       )
@@
   (symbol (lib_id "power:GND") (at 101.6 104.14 0) (unit 1)
     (in_bom yes) (on_board yes) (dnp no) (fields_autoplaced)
-    (property "Reference" "#PWR032" (at 101.6 110.49 0)
+    (property "Reference" "#PWR0108" (at 101.6 110.49 0)
       (effects (font (size 1.27 1.27)) hide)
     )
@@
       (project "BPS-LeaderDaughter"
         (path "/2e9f4f51-d216-4952-a31c-e7104e0d4b1e/ae57cd3a-fadb-4313-835a-95d5b185a797"
-          (reference "#PWR032") (unit 1)
+          (reference "#PWR0108") (unit 1)
         )
         (path "/2e9f4f51-d216-4952-a31c-e7104e0d4b1e/5e4c6ec4-73d4-4ed3-a75f-02eb4f9ac8b3"
@@
       (effects (font (size 1.27 1.27)))
     )
-    (property "Footprint" "" (at 62.23 55.118 90)
+    (property "Footprint" "Resistor_SMD:R_0805_2012Metric" (at 62.23 55.118 90)
       (effects (font (size 1.27 1.27)) hide)
     )
@@
   (symbol (lib_name "+12V_2") (lib_id "power:+12V") (at 186.69 31.75 0) (unit 1)
     (in_bom yes) (on_board yes) (dnp no) (fields_autoplaced)
-    (property "Reference" "#PWR09" (at 186.69 35.56 0)
+    (property "Reference" "#PWR0112" (at 186.69 35.56 0)
       (effects (font (size 1.27 1.27)) hide)
     )
@@
       (project "BPS-LeaderDaughter"
         (path "/2e9f4f51-d216-4952-a31c-e7104e0d4b1e/ae57cd3a-fadb-4313-835a-95d5b185a797"
-          (reference "#PWR09") (unit 1)
-        )
-        (path "/2e9f4f51-d216-4952-a31c-e7104e0d4b1e/5e4c6ec4-73d4-4ed3-a75f-02eb4f9ac8b3"
-          (reference "#PWR010") (unit 1)
-        )
-        (path "/2e9f4f51-d216-4952-a31c-e7104e0d4b1e/bb673292-4a5d-469b-b6b6-0dc7df3c162d"
-          (reference "#PWR011") (unit 1)
-        )
-      )
+          (reference "#PWR0112") (unit 1)
+        )
+        (path "/2e9f4f51-d216-4952-a31c-e7104e0d4b1e/5e4c6ec4-73d4-4ed3-a75f-02eb4f9ac8b3"
+          (reference "#PWR0115") (unit 1)
+        )
+        (path "/2e9f4f51-d216-4952-a31c-e7104e0d4b1e/bb673292-4a5d-469b-b6b6-0dc7df3c162d"
+          (reference "#PWR0128") (unit 1)
+        )
+      )
