File: Contactor_Driver.kicad_sch (KiCad schematic)
At the start: 13 parts, among them J9 Conn_01x04, U5 SI8261ABC-IS

Commit message: Fixed current limiting LEDs on the Optoisolator and FAN jumpers
Parts:
- C22: value 1uF -> 100nF
- R12: value R -> 1k
- R41: value 49.9 -> 80.6
- R7: value 5k -> 10k
Connections:
- net GNDPWR is gone; now on net GND: C16.2, C17.2, Q?.1 (S), Q?.2 (S), Q?.3 (S), R5.2, U5.5 (GND)
Other:
- note added: "Vf = 1.6 V If = 30 mA (3.3 - 1.6) / .030 = 56"
- note removed: "Clipping Voltage Logic to ensure that only 3.3V logic goes in to mcu"
- note removed: "The upper mosfet is for voltage protection: If some high votlage spike comes in from the Contactor it won't send it through the rest of the circuit"
- note removed: "Vf = 1.6 V If = 30 mA (3.3 - 1.6) / .030"
- moved on the sheet: C22, R12

Commit message: Made ignition connector 3 pin + fixed tach resistors
Parts:
- D2: footprint Diode_SMD:D_SOD-323F -> Diode_SMD:D_SOD-323; P/N 1N4148WS -> 1N4148WSQ-7-F
Connections:
- net GND: no longer C16.2, C17.2, Q?.1 (S), Q?.2 (S), Q?.3 (S), R5.2, U5.5 (GND)
- new net GND2: C16.2, C17.2, Q?.1 (S), Q?.2 (S), Q?.3 (S), R5.2, U5.5 (GND)

Commit message: why your schematic so broken >:(
Parts:
- R4: renamed from R41; value 80.6 -> 105
- renumbered C22 to C4, C16 to C5, C17 to C6, D10 to D2, D25 to D3, J9 to J5, R12 to R13, R5 to R6, U5 to U2
Other:
- note added: "Vf = 1.6 V If = 30 mA MAX, we drive at 20mA (3.3 - 1.6) / .020 = 85"
- note removed: "Vf = 1.6 V If = 30 mA (3.3 - 1.6) / .030 = 56"

Commit message: More layout progress, fix LeaderSOM holes, removed strobe isolator, fixed GND of contactor, weeeee
Connections:
- net GND2 is gone; now on net GND: C5.2, C6.2, Q?.1 (S), Q?.2 (S), Q?.3 (S), R6.2, U2.5 (GND)
Other:
- note added: "12V Contactor +/- should be planes"
- note removed: "ISOLATED"
Changed lines of the file:
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@@
-    (stroke (width 0) (type default))
-  )
-  (polyline (pts (xy 82.55 40.64) (xy 82.55 83.82))
     (stroke (width 0) (type default))
   )
@@
   (wire (pts (xy 177.165 45.72) (xy 177.165 47.625))
     (stroke (width 0) (type default))
-  )
-  (text "ISOLATED" (at 74.93 38.1 0)
-    (effects (font (size 2.54 2.54) (thickness 0.508) bold) (justify left bottom))
   )
   (text "Vf = 1.6 V\nIf = 30 mA MAX, we drive at 20mA\n(3.3 - 1.6) / .020 = 85\n"
@@
     (effects (font (size 1.27 1.27)) (justify left bottom))
   )
+  (text "12V\nContactor +/- should be planes" (at 163.195 86.36 0)
+    (effects (font (size 1.27 1.27)) (justify left bottom))
+  )
   (label "PWM_ISO" (at 96.52 55.88 0) (fields_autoplaced)
     (effects (font (size 1.27 1.27)) (justify left bottom))
@@
   (hierarchical_label "Contactor_EN" (shape input) (at 52.705 53.34 180) (fields_autoplaced)
     (effects (font (size 1.27 1.27)) (justify right))
-  )
-  (symbol (lib_id "power:GND2") (at 97.79 61.595 0) (unit 1)
-    (in_bom yes) (on_board yes) (dnp no) (fields_autoplaced)
-    (property "Reference" "#PWR030" (at 97.79 67.945 0)
-      (effects (font (size 1.27 1.27)) hide)
-    )
-    (property "Value" "GND2" (at 97.79 66.04 0)
-      (effects (font (size 1.27 1.27)))
-    )
-    (property "Footprint" "" (at 97.79 61.595 0)
-      (effects (font (size 1.27 1.27)) hide)
-    )
-    (property "Datasheet" "" (at 97.79 61.595 0)
-      (effects (font (size 1.27 1.27)) hide)
-    )
-    (pin "1")
-    (instances
-      (project "BPS-LeaderDaughter"
-        (path "/2e9f4f51-d216-4952-a31c-e7104e0d4b1e/ae57cd3a-fadb-4313-835a-95d5b185a797"
-          (reference "#PWR030") (unit 1)
-        )
-        (path "/2e9f4f51-d216-4952-a31c-e7104e0d4b1e/5e4c6ec4-73d4-4ed3-a75f-02eb4f9ac8b3"
-          (reference "#PWR040") (unit 1)
-        )
-        (path "/2e9f4f51-d216-4952-a31c-e7104e0d4b1e/bb673292-4a5d-469b-b6b6-0dc7df3c162d"
-          (reference "#PWR050") (unit 1)
-        )
-      )
-    )
-  )
-  (symbol (lib_id "power:GND2") (at 109.855 55.245 0) (unit 1)
-    (in_bom yes) (on_board yes) (dnp no) (fields_autoplaced)
-    (property "Reference" "#PWR033" (at 109.855 61.595 0)
-      (effects (font (size 1.27 1.27)) hide)
-    )
-    (property "Value" "GND2" (at 109.855 59.69 0)
-      (effects (font (size 1.27 1.27)))
-    )
-    (property "Footprint" "" (at 109.855 55.245 0)
-      (effects (font (size 1.27 1.27)) hide)
-    )
-    (property "Datasheet" "" (at 109.855 55.245 0)
-      (effects (font (size 1.27 1.27)) hide)
-    )
-    (pin "1")
-    (instances
-      (project "BPS-LeaderDaughter"
-        (path "/2e9f4f51-d216-4952-a31c-e7104e0d4b1e/ae57cd3a-fadb-4313-835a-95d5b185a797"
-          (reference "#PWR033") (unit 1)
-        )
-        (path "/2e9f4f51-d216-4952-a31c-e7104e0d4b1e/5e4c6ec4-73d4-4ed3-a75f-02eb4f9ac8b3"
-          (reference "#PWR043") (unit 1)
-        )
-        (path "/2e9f4f51-d216-4952-a31c-e7104e0d4b1e/bb673292-4a5d-469b-b6b6-0dc7df3c162d"
-          (reference "#PWR053") (unit 1)
-        )
-      )
-    )
   )
   (symbol (lib_id "Transistor_FET:BUK9M23-80EX") (at 184.15 61.595 0) (unit 1)
@@
     )
   )
+  (symbol (lib_id "power:GND") (at 186.69 74.93 0) (unit 1)
+    (in_bom yes) (on_board yes) (dnp no) (fields_autoplaced)
+    (property "Reference" "#PWR035" (at 186.69 81.28 0)
+      (effects (font (size 1.27 1.27)) hide)
+    )
+    (property "Value" "GND" (at 186.69 80.01 0)
+      (effects (font (size 1.27 1.27)))
+    )
+    (property "Footprint" "" (at 186.69 74.93 0)
+      (effects (font (size 1.27 1.27)) hide)
+    )
+    (property "Datasheet" "" (at 186.69 74.93 0)
+      (effects (font (size 1.27 1.27)) hide)
+    )
+    (pin "1")
+    (instances
+      (project "BPS-LeaderDaughter"
+        (path "/2e9f4f51-d216-4952-a31c-e7104e0d4b1e/ae57cd3a-fadb-4313-835a-95d5b185a797"
+          (reference "#PWR035") (unit 1)
+        )
+        (path "/2e9f4f51-d216-4952-a31c-e7104e0d4b1e/5e4c6ec4-73d4-4ed3-a75f-02eb4f9ac8b3"
+          (reference "#PWR045") (unit 1)
+        )
+        (path "/2e9f4f51-d216-4952-a31c-e7104e0d4b1e/bb673292-4a5d-469b-b6b6-0dc7df3c162d"
+          (reference "#PWR055") (unit 1)
+        )
+      )
+    )
+  )
   (symbol (lib_id "Device:LED_Small") (at 177.165 50.165 90) (unit 1)
     (in_bom yes) (on_board yes) (dnp no)
@@
     )
   )
+  (symbol (lib_id "power:GND") (at 109.855 55.245 0) (unit 1)
+    (in_bom yes) (on_board yes) (dnp no) (fields_autoplaced)
+    (property "Reference" "#PWR033" (at 109.855 61.595 0)
+      (effects (font (size 1.27 1.27)) hide)
+    )
+    (property "Value" "GND" (at 109.855 60.325 0)
+      (effects (font (size 1.27 1.27)))
+    )
+    (property "Footprint" "" (at 109.855 55.245 0)
+      (effects (font (size 1.27 1.27)) hide)
+    )
+    (property "Datasheet" "" (at 109.855 55.245 0)
+      (effects (font (size 1.27 1.27)) hide)
+    )
+    (pin "1")
+    (instances
+      (project "BPS-LeaderDaughter"
+        (path "/2e9f4f51-d216-4952-a31c-e7104e0d4b1e/ae57cd3a-fadb-4313-835a-95d5b185a797"
+          (reference "#PWR033") (unit 1)
+        )
+        (path "/2e9f4f51-d216-4952-a31c-e7104e0d4b1e/5e4c6ec4-73d4-4ed3-a75f-02eb4f9ac8b3"
+          (reference "#PWR043") (unit 1)
+        )
+        (path "/2e9f4f51-d216-4952-a31c-e7104e0d4b1e/bb673292-4a5d-469b-b6b6-0dc7df3c162d"
+          (reference "#PWR053") (unit 1)
+        )
+      )
+    )
+  )
+  (symbol (lib_id "power:GND") (at 97.79 61.595 0) (unit 1)
+    (in_bom yes) (on_board yes) (dnp no) (fields_autoplaced)
+    (property "Reference" "#PWR030" (at 97.79 67.945 0)
+      (effects (font (size 1.27 1.27)) hide)
+    )
+    (property "Value" "GND" (at 97.79 66.675 0)
+      (effects (font (size 1.27 1.27)))
+    )
+    (property "Footprint" "" (at 97.79 61.595 0)
+      (effects (font (size 1.27 1.27)) hide)
+    )
+    (property "Datasheet" "" (at 97.79 61.595 0)
+      (effects (font (size 1.27 1.27)) hide)
+    )
+    (pin "1")
+    (instances
+      (project "BPS-LeaderDaughter"
+        (path "/2e9f4f51-d216-4952-a31c-e7104e0d4b1e/ae57cd3a-fadb-4313-835a-95d5b185a797"
+          (reference "#PWR030") (unit 1)
+        )
+        (path "/2e9f4f51-d216-4952-a31c-e7104e0d4b1e/5e4c6ec4-73d4-4ed3-a75f-02eb4f9ac8b3"
+          (reference "#PWR040") (unit 1)
+        )
+        (path "/2e9f4f51-d216-4952-a31c-e7104e0d4b1e/bb673292-4a5d-469b-b6b6-0dc7df3c162d"
+          (reference "#PWR050") (unit 1)
+        )
+      )
+    )
+  )
   (symbol (lib_id "power:GND") (at 62.865 109.855 0) (unit 1)
     (in_bom yes) (on_board yes) (dnp no)
@@
         )
       )
-    )
-  )
-  (symbol (lib_id "power:GND2") (at 186.69 74.93 0) (unit 1)
-    (in_bom yes) (on_board yes) (dnp no) (fields_autoplaced)
-    (property "Reference" "#PWR035" (at 186.69 81.28 0)
-      (effects (font (size 1.27 1.27)) hide)
-    )
-    (property "Value" "GND2" (at 186.69 79.375 0)
-      (effects (font (size 1.27 1.27)))
-    )
-    (property "Footprint" "" (at 186.69 74.93 0)
-      (effects (font (size 1.27 1.27)) hide)
-    )
-    (property "Datasheet" "" (at 186.69 74.93 0)
-      (effects (font (size 1.27 1.27)) hide)
-    )
-    (pin "1")
-    (instances
-      (project "BPS-LeaderDaughter"
-        (path "/2e9f4f51-d216-4952-a31c-e7104e0d4b1e/ae57cd3a-fadb-4313-835a-95d5b185a797"
-          (reference "#PWR035") (unit 1)
-        )
-        (path "/2e9f4f51-d216-4952-a31c-e7104e0d4b1e/5e4c6ec4-73d4-4ed3-a75f-02eb4f9ac8b3"
-          (reference "#PWR045") (unit 1)
-        )
-        (path "/2e9f4f51-d216-4952-a31c-e7104e0d4b1e/bb673292-4a5d-469b-b6b6-0dc7df3c162d"
-          (reference "#PWR055") (unit 1)
-        )
-      )

Commit message: Fixed gate resistor on Strovbe
Other:
- note added: "12V GND Contactor +/- should be planes"
- note removed: "12V Contactor +/- should be planes"
Changed lines of the file:
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@@
     (effects (font (size 1.27 1.27)) (justify left bottom))
   )
-  (text "12V\nContactor +/- should be planes" (at 163.195 86.36 0)
+  (text "12V\nGND\nContactor +/- should be planes" (at 163.195 86.36 0)
     (effects (font (size 1.27 1.27)) (justify left bottom))
   )

Commit message: everythign on front
Parts:
- removed C5: 100nF, Capacitor_SMD:C_0805_2012Metric, symbol Device:C_Small
- removed C6: 10uF, Capacitor_SMD:C_0805_2012Metric, symbol Device:C_Small
- removed R4: 105, Resistor_SMD:R_0805_2012Metric, symbol Device:R
- removed U2: SI8261ABC-IS, Package_SO:SOIC-8_3.9x4.9mm_P1.27mm, symbol utsvt-bps:SI8261ABC-IS
- added R5: 1k, Resistor_SMD:R_0805_2012Metric, symbol Device:R
- renumbered C4 to C2, R13 to R12
Connections:
- net Contactor_EN: now also R5.1
- net PWM_ISO: no longer names the net of Q?.4 (G), R6.1
- net PWM_ISO: now also R5.2
Other:
- note removed: "Vf = 1.6 V If = 30 mA MAX, we drive at 20mA (3.3 - 1.6) / .020 = 85"
- moved on the sheet: D2, D3, Q?, R6, R7
