File: Fan_Control.kicad_sch (KiCad schematic)
At the start: 29 parts, among them IC1 ADT7470ARQZ-REEL7, J10 Fan 4, J3 Fan 1, J8 Fan 2, J9 Fan 3

Commit message: Fans - no connects and FULL_SPEED
Parts:
- removed J10: Fan 4, symbol Connector_Generic:Conn_01x04
- removed J3: Fan 1, symbol Connector_Generic:Conn_01x04
- removed J8: Fan 2, symbol Connector_Generic:Conn_01x04
- removed J9: Fan 3, symbol Connector_Generic:Conn_01x04
- added J1 (x4): Conn_01x04, UTSVT_Connectors:Molex_MicroFit3.0_1x4xP3.00mm_PolarizingPeg_Vertical, symbol Connector_Generic:Conn_01x04
Connections:
- net +12V: now also J1.1 (Pin_1), J1.1 (Pin_1), J1.1 (Pin_1), J1.1 (Pin_1)
- net GND: now also J1.4 (Pin_4), J1.4 (Pin_4), J1.4 (Pin_4), J1.4 (Pin_4)
- net PWM1: now also J1.3 (Pin_3)
- net PWM2: now also J1.3 (Pin_3)
- net PWM3: now also J1.3 (Pin_3)
- net PWM4: now also J1.3 (Pin_3)
- net TACH1_OUT: now also J1.2 (Pin_2)
- net TACH2_OUT: now also J1.2 (Pin_2)
- net TACH3_OUT: now also J1.2 (Pin_2)
- net TACH4_OUT: now also J1.2 (Pin_2)
- no-connect marks 0 -> 3

Commit message: PWM Fan Support for Orion
Parts:
- removed D27, D28: 1N4148, Diode_THT:D_DO-35_SOD27_P7.62mm_Horizontal, symbol Diode:1N4148
- added D24, D25: 1N4148WS, Diode_SMD:D_SOD-323F, symbol Diode:1N4148
- added J1: Conn_01x04, UTSVT_Connectors:Molex_MicroFit3.0_1x4xP3.00mm_PolarizingPeg_Vertical, symbol Connector_Generic:Conn_01x04
- added Q10, Q14, Q15, Q6: BUK9M23-80E, Package_TO_SOT_SMD:LFPAK33, symbol Transistor_FET:BUK9M23-80EX
- D26, D29: value 1N4148 -> 1N4148WS; footprint Diode_THT:D_DO-35_SOD27_P7.62mm_Horizontal -> Diode_SMD:D_SOD-323F; P/N 1N4148 -> 1N4148WS
Connections:
- net +12V: now also D24.1 (K), D25.1 (K), J1.1 (Pin_1)
- net GND: now also D24.2 (A), D25.2 (A), J1.4 (Pin_4), Q10.1 (S), Q10.2 (S), Q10.3 (S), Q14.1 (S), Q14.2 (S), Q14.3 (S), Q15.1 (S), Q15.2 (S), Q15.3 (S), Q6.1 (S), Q6.2 (S), Q6.3 (S)
- net PWM1 renamed ORION_PWM(24)
- net ORION_PWM(24): now also IC1.10 (PWM4), IC1.5 (PWM2), IC1.8 (PWM3), R28.2, R29.2, R30.2, J1.2 (Pin_2), Q10.4 (G), Q14.4 (G), Q15.4 (G), Q6.4 (G); no longer J1.3 (Pin_3)
- removed net PWM2: IC1.5 (PWM2), J1.3 (Pin_3), R30.2
- removed net PWM3: IC1.8 (PWM3), J1.3 (Pin_3), R29.2
- removed net PWM4: IC1.10 (PWM4), J1.3 (Pin_3), R28.2
- net TACH1 renamed ORION_TACH(9)
- net ORION_TACH(9): now also J1.3 (Pin_3)
- new net PWM1_IN: J1.3 (Pin_3), Q6.5 (D)
- new net PWM2_IN: J1.3 (Pin_3), Q10.5 (D)
- new net PWM3_IN: J1.3 (Pin_3), Q15.5 (D)
- new net PWM4_IN: J1.3 (Pin_3), Q14.5 (D)
Other:
- moved on the sheet: D29, R28, R29, R30, R31

Commit message: Combined fan and contactor stuff
Parts:
- removed D6, D9: 3.3V, Diode_SMD:D_SOD-523, symbol Device:D_Zener
- added D4, D5: 3.3V, Diode_SMD:D_SOD-523, symbol Device:D_Zener
- renumbered D17 to D2, D16 to D3, D26 to D6, D25 to D7, D24 to D8, D29 to D9, Q14 to Q3, Q15 to Q4, Q10 to Q5, R31 to R10, R32 to R11, R33 to R12, R34 to R13, R35 to R14, R36 to R15, R37 to R16, R38 to R17, R39 to R18, R40 to R19, R41 to R20, R42 to R21, R43 to R22, R28 to R7, R29 to R8, R30 to R9
Connections:
- net GND: now also D4.2 (A), D5.2 (A)
- net TACH3: now also D4.1 (K)
- net TACH4: now also D5.1 (K)

Commit message: Fans-Orion Pwms isolated
Parts:
- added JP1, JP2: Jumper_3_Open, symbol Jumper:Jumper_3_Open
Connections:
- removed net ORION_PWM(24): IC1.10 (PWM4), IC1.15 (PWM1), IC1.5 (PWM2), IC1.8 (PWM3), J1.2 (Pin_2), Q3.4 (G), Q4.4 (G), Q5.4 (G), Q6.4 (G), R10.2, R7.2, R8.2, R9.2
- new net: J1.2 (Pin_2), JP1.2 (C), JP2.2 (C)
- new net ORION_PWM1(24): IC1.15 (PWM1), JP1.3 (B), Q6.4 (G), R10.2
- new net ORION_PWM2(24): IC1.5 (PWM2), JP1.1 (A), Q5.4 (G), R9.2
- new net ORION_PWM3(24): IC1.8 (PWM3), JP2.3 (B), Q4.4 (G), R8.2
- new net ORION_PWM4(24): IC1.10 (PWM4), JP2.1 (A), Q3.4 (G), R7.2
Other:
- moved on the sheet: J1, Q3, Q4, Q5, Q6, R10, R7, R8, R9

Commit message: zener diode footprint -> 323
Parts:
- D2, D3, D4, D5: footprint Diode_SMD:D_SOD-523 -> Diode_SMD:D_SOD-323; P/N SZMM5Z3V3T1G -> SZMM3Z3V3T1G
- JP1, JP2: footprint (none) -> Connector_PinHeader_2.54mm:PinHeader_1x03_P2.54mm_Vertical
Changed lines of the file:
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@@
-    (stroke (width 0) (type default))
-  )
-  (wire (pts (xy 182.88 30.48) (xy 189.23 30.48))
     (stroke (width 0) (type default))
   )
@@
   )
   (label "PWM4_IN" (at 257.175 143.51 180) (fields_autoplaced)
-    (effects (font (size 1.27 1.27)) (justify right bottom))
-  )
-  (label "Ground(12)" (at 203.2 135.89 180) (fields_autoplaced)
     (effects (font (size 1.27 1.27)) (justify right bottom))
   )
@@
     (effects (font (size 1.27 1.27)) (justify right bottom))
   )
-  (label "ORION_12V(10)" (at 203.2 128.27 180) (fields_autoplaced)
-    (effects (font (size 1.27 1.27)) (justify right bottom))
-  )
   (label "ORION_PWM2(24)" (at 175.26 124.46 180) (fields_autoplaced)
     (effects (font (size 1.27 1.27)) (justify right bottom))
@@
   )
   (label "TACH3_OUT" (at 257.175 119.38 180) (fields_autoplaced)
-    (effects (font (size 1.27 1.27)) (justify right bottom))
-  )
-  (label "ORION_12V(10)" (at 182.88 30.48 180) (fields_autoplaced)
     (effects (font (size 1.27 1.27)) (justify right bottom))
   )
@@
     )
   )
-  (symbol (lib_id "Device:D_Zener") (at 143.51 83.82 270) (unit 1)
-    (in_bom yes) (on_board yes) (dnp no) (fields_autoplaced)
-    (property "Reference" "D5" (at 146.05 82.55 90)
-      (effects (font (size 1.27 1.27)) (justify left))
-    )
-    (property "Value" "3.3V" (at 146.05 85.09 90)
-      (effects (font (size 1.27 1.27)) (justify left))
-    )
-    (property "Footprint" "Diode_SMD:D_SOD-523" (at 143.51 83.82 0)
-      (effects (font (size 1.27 1.27)) hide)
-    )
-    (property "Datasheet" "https://www.mouser.com/datasheet/2/308/1/MM5Z2V4T1_D-2316295.pdf" (at 143.51 83.82 0)
-      (effects (font (size 1.27 1.27)) hide)
-    )
-    (property "P/N" "SZMM5Z3V3T1G" (at 143.51 83.82 90)
-      (effects (font (size 1.27 1.27)) hide)
-    )
-    (pin "1")
-    (pin "2")
-    (instances
-      (project "BPS-LeaderDaughter"
-        (path "/2e9f4f51-d216-4952-a31c-e7104e0d4b1e/bf23a663-b938-440b-843e-ef7912c82d18"
-          (reference "D5") (unit 1)
-        )
-      )
-    )
-  )
   (symbol (lib_id "Connector_Generic:Conn_01x04") (at 267.97 97.79 0) (unit 1)
     (in_bom yes) (on_board yes) (dnp no) (fields_autoplaced)
@@
       (effects (font (size 1.27 1.27)) (justify left))
     )
-    (property "Footprint" "" (at 180.34 118.11 0)
+    (property "Footprint" "Connector_PinHeader_2.54mm:PinHeader_1x03_P2.54mm_Vertical" (at 180.34 118.11 0)
       (effects (font (size 1.27 1.27)) hide)
     )
@@
       (effects (font (size 1.27 1.27)) (justify left))
     )
-    (property "Footprint" "Diode_SMD:D_SOD-523" (at 116.84 83.82 0)
-      (effects (font (size 1.27 1.27)) hide)
-    )
-    (property "Datasheet" "https://www.mouser.com/datasheet/2/308/1/MM5Z2V4T1_D-2316295.pdf" (at 116.84 83.82 0)
-      (effects (font (size 1.27 1.27)) hide)
-    )
-    (property "P/N" "SZMM5Z3V3T1G" (at 116.84 83.82 90)
+    (property "Footprint" "Diode_SMD:D_SOD-323" (at 116.84 83.82 0)
+      (effects (font (size 1.27 1.27)) hide)
+    )
+    (property "Datasheet" "https://www.mouser.com/datasheet/2/308/1/MM3Z2V4T1_D-2316321.pdf" (at 116.84 83.82 0)
+      (effects (font (size 1.27 1.27)) hide)
+    )
+    (property "P/N" "SZMM3Z3V3T1G" (at 116.84 83.82 90)
       (effects (font (size 1.27 1.27)) hide)
     )
@@
     )
   )
+  (symbol (lib_id "Device:D_Zener") (at 125.73 83.82 270) (unit 1)
+    (in_bom yes) (on_board yes) (dnp no) (fields_autoplaced)
+    (property "Reference" "D3" (at 128.27 82.55 90)
+      (effects (font (size 1.27 1.27)) (justify left))
+    )
+    (property "Value" "3.3V" (at 128.27 85.09 90)
+      (effects (font (size 1.27 1.27)) (justify left))
+    )
+    (property "Footprint" "Diode_SMD:D_SOD-323" (at 125.73 83.82 0)
+      (effects (font (size 1.27 1.27)) hide)
+    )
+    (property "Datasheet" "https://www.mouser.com/datasheet/2/308/1/MM3Z2V4T1_D-2316321.pdf" (at 125.73 83.82 0)
+      (effects (font (size 1.27 1.27)) hide)
+    )
+    (property "P/N" "SZMM3Z3V3T1G" (at 125.73 83.82 90)
+      (effects (font (size 1.27 1.27)) hide)
+    )
+    (pin "1")
+    (pin "2")
+    (instances
+      (project "BPS-LeaderDaughter"
+        (path "/2e9f4f51-d216-4952-a31c-e7104e0d4b1e/bf23a663-b938-440b-843e-ef7912c82d18"
+          (reference "D3") (unit 1)
+        )
+      )
+    )
+  )
   (symbol (lib_id "Device:R") (at 182.88 55.88 90) (unit 1)
     (in_bom yes) (on_board yes) (dnp no) (fields_autoplaced)
@@
     )
   )
-  (symbol (lib_id "Device:D_Zener") (at 125.73 83.82 270) (unit 1)
-    (in_bom yes) (on_board yes) (dnp no) (fields_autoplaced)
-    (property "Reference" "D3" (at 128.27 82.55 90)
-      (effects (font (size 1.27 1.27)) (justify left))
-    )
-    (property "Value" "3.3V" (at 128.27 85.09 90)
-      (effects (font (size 1.27 1.27)) (justify left))
-    )
-    (property "Footprint" "Diode_SMD:D_SOD-523" (at 125.73 83.82 0)
-      (effects (font (size 1.27 1.27)) hide)
-    )
-    (property "Datasheet" "https://www.mouser.com/datasheet/2/308/1/MM5Z2V4T1_D-2316295.pdf" (at 125.73 83.82 0)
-      (effects (font (size 1.27 1.27)) hide)
-    )
-    (property "P/N" "SZMM5Z3V3T1G" (at 125.73 83.82 90)
-      (effects (font (size 1.27 1.27)) hide)
-    )
-    (pin "1")
-    (pin "2")
-    (instances
-      (project "BPS-LeaderDaughter"
-        (path "/2e9f4f51-d216-4952-a31c-e7104e0d4b1e/bf23a663-b938-440b-843e-ef7912c82d18"
-          (reference "D3") (unit 1)
-        )
-      )
-    )
-  )
   (symbol (lib_id "Device:R") (at 170.18 83.82 0) (unit 1)
     (in_bom yes) (on_board yes) (dnp no) (fields_autoplaced)
@@
     )
   )
+  (symbol (lib_id "power:+12V") (at 203.2 128.27 0) (unit 1)
+    (in_bom yes) (on_board yes) (dnp no) (fields_autoplaced)
+    (property "Reference" "#PWR065" (at 203.2 132.08 0)
+      (effects (font (size 1.27 1.27)) hide)
+    )
+    (property "Value" "+12V" (at 203.2 123.19 0)
+      (effects (font (size 1.27 1.27)))
+    )
+    (property "Footprint" "" (at 203.2 128.27 0)
+      (effects (font (size 1.27 1.27)) hide)
+    )
+    (property "Datasheet" "" (at 203.2 128.27 0)
+      (effects (font (size 1.27 1.27)) hide)
+    )
+    (pin "1")
+    (instances
+      (project "BPS-LeaderDaughter"
+        (path "/2e9f4f51-d216-4952-a31c-e7104e0d4b1e/bf23a663-b938-440b-843e-ef7912c82d18"
+          (reference "#PWR065") (unit 1)
+        )
+      )
+    )
+  )
+  (symbol (lib_id "Device:D_Zener") (at 143.51 83.82 270) (unit 1)
+    (in_bom yes) (on_board yes) (dnp no) (fields_autoplaced)
+    (property "Reference" "D5" (at 146.05 82.55 90)
+      (effects (font (size 1.27 1.27)) (justify left))
+    )
+    (property "Value" "3.3V" (at 146.05 85.09 90)
+      (effects (font (size 1.27 1.27)) (justify left))
+    )
+    (property "Footprint" "Diode_SMD:D_SOD-323" (at 143.51 83.82 0)
+      (effects (font (size 1.27 1.27)) hide)
+    )
+    (property "Datasheet" "https://www.mouser.com/datasheet/2/308/1/MM3Z2V4T1_D-2316321.pdf" (at 143.51 83.82 0)
+      (effects (font (size 1.27 1.27)) hide)
+    )
+    (property "P/N" "SZMM3Z3V3T1G" (at 143.51 83.82 90)
+      (effects (font (size 1.27 1.27)) hide)
+    )
+    (pin "1")
+    (pin "2")
+    (instances
+      (project "BPS-LeaderDaughter"
+        (path "/2e9f4f51-d216-4952-a31c-e7104e0d4b1e/bf23a663-b938-440b-843e-ef7912c82d18"
+          (reference "D5") (unit 1)
+        )
+      )
+    )
+  )
   (symbol (lib_id "Device:R") (at 215.9 38.1 0) (unit 1)
     (in_bom yes) (on_board yes) (dnp no) (fields_autoplaced)
@@
     )
   )
+  (symbol (lib_id "Device:D_Zener") (at 134.62 83.82 270) (unit 1)
+    (in_bom yes) (on_board yes) (dnp no) (fields_autoplaced)
+    (property "Reference" "D4" (at 137.16 82.55 90)
+      (effects (font (size 1.27 1.27)) (justify left))
+    )
+    (property "Value" "3.3V" (at 137.16 85.09 90)
+      (effects (font (size 1.27 1.27)) (justify left))
+    )
+    (property "Footprint" "Diode_SMD:D_SOD-323" (at 134.62 83.82 0)
+      (effects (font (size 1.27 1.27)) hide)
+    )
+    (property "Datasheet" "https://www.mouser.com/datasheet/2/308/1/MM3Z2V4T1_D-2316321.pdf" (at 134.62 83.82 0)
+      (effects (font (size 1.27 1.27)) hide)
+    )
+    (property "P/N" "SZMM3Z3V3T1G" (at 134.62 83.82 90)
+      (effects (font (size 1.27 1.27)) hide)
+    )
+    (pin "1")
+    (pin "2")
+    (instances
+      (project "BPS-LeaderDaughter"
+        (path "/2e9f4f51-d216-4952-a31c-e7104e0d4b1e/bf23a663-b938-440b-843e-ef7912c82d18"
+          (reference "D4") (unit 1)
+        )
+      )
+    )
+  )
   (symbol (lib_id "power:+12V") (at 234.95 138.43 0) (unit 1)
     (in_bom yes) (on_board yes) (dnp no) (fields_autoplaced)
@@
       (effects (font (size 1.27 1.27)) (justify left))
     )
-    (property "Footprint" "" (at 180.34 143.51 0)
+    (property "Footprint" "Connector_PinHeader_2.54mm:PinHeader_1x03_P2.54mm_Vertical" (at 180.34 143.51 0)
       (effects (font (size 1.27 1.27)) hide)
     )
@@
         )
       )
-    )
-  )
-  (symbol (lib_id "Device:D_Zener") (at 134.62 83.82 270) (unit 1)
-    (in_bom yes) (on_board yes) (dnp no) (fields_autoplaced)
-    (property "Reference" "D4" (at 137.16 82.55 90)
-      (effects (font (size 1.27 1.27)) (justify left))
-    )
-    (property "Value" "3.3V" (at 137.16 85.09 90)
-      (effects (font (size 1.27 1.27)) (justify left))
-    )
-    (property "Footprint" "Diode_SMD:D_SOD-523" (at 134.62 83.82 0)
-      (effects (font (size 1.27 1.27)) hide)
-    )
-    (property "Datasheet" "https://www.mouser.com/datasheet/2/308/1/MM5Z2V4T1_D-2316295.pdf" (at 134.62 83.82 0)
-      (effects (font (size 1.27 1.27)) hide)
-    )
-    (property "P/N" "SZMM5Z3V3T1G" (at 134.62 83.82 90)
-      (effects (font (size 1.27 1.27)) hide)
-    )
-    (pin "1")
-    (pin "2")
-    (instances
-      (project "BPS-LeaderDaughter"
-        (path "/2e9f4f51-d216-4952-a31c-e7104e0d4b1e/bf23a663-b938-440b-843e-ef7912c82d18"
-          (reference "D4") (unit 1)
-        )
-      )
