File: Fan_Control.kicad_sch (KiCad schematic)
At the start: 12 parts, among them IC1 ADT7470ARQZ-REEL7, J1 Conn_01x04

Commit message: Fan layout on pcb. need to figure out IC
Parts:
- renumbered D6 to D2, D7 to D3, D8 to D4, D9 to D5, J1 to J?
Connections:
- net ORION_PWM1(24) is gone; now on net PWM1: JP1.3 (B)
- net ORION_PWM2(24) is gone; now on net PWM2: JP1.1 (A)
- net ORION_PWM3(24) is gone; now on net PWM3: JP2.3 (B)
- net ORION_PWM4(24) is gone; now on net PWM4: JP2.1 (A)
- net ORION_TACH(9) is gone; now on net TACH1: J?.3 (Pin_3)
- net +12V: now also J?.2 (Pin_2), J?.2 (Pin_2), J?.2 (Pin_2), J?.2 (Pin_2); no longer J?.1 (Pin_1), J?.1 (Pin_1), J?.1 (Pin_1), J?.1 (Pin_1)
- net GND: now also J?.1 (Pin_1), J?.1 (Pin_1), J?.1 (Pin_1), J?.1 (Pin_1); no longer J?.4 (Pin_4), J?.4 (Pin_4), J?.4 (Pin_4), J?.4 (Pin_4)
- net PWM1_OUT: now also J?.4 (Pin_4); no longer J?.3 (Pin_3)
- net PWM2_OUT: now also J?.4 (Pin_4); no longer J?.3 (Pin_3)
- net PWM3_OUT: now also J?.4 (Pin_4); no longer J?.3 (Pin_3)
- net PWM4_OUT: now also J?.4 (Pin_4); no longer J?.3 (Pin_3)
- net TACH1_IN: now also J?.3 (Pin_3); no longer J?.2 (Pin_2)
- net TACH2_IN: now also J?.3 (Pin_3); no longer J?.2 (Pin_2)
- net TACH3_IN: now also J?.3 (Pin_3); no longer J?.2 (Pin_2)
- net TACH4_IN: now also J?.3 (Pin_3); no longer J?.2 (Pin_2)
Other:
- sheet Fan_PWM1 ports: added none; removed ORION_PWM
- sheet Fan_PWM2 ports: added none; removed ORION_PWM
- sheet Fan_PWM3 ports: added none; removed ORION_PWM
- sheet Fan_PWM4 ports: added none; removed ORION_PWM
- moved on the sheet: D2, D3, D4, D5, J?

Commit message: Fan layout updated
Parts:
- added C1: 1uF, Capacitor_SMD:C_0805_2012Metric, symbol Device:C
Connections:
- net +3.3V: now also C1.1
- net GND: now also C1.2
- net ORION_PWM: now reaches J?.2 (Pin_2), JP1.2 (C), JP2.2 (C)
- net ~{SMBALERT}: now reaches IC1.14 (~{SMBALERT})
- no-connect marks 3 -> 2
Other:
- note added: "Bridge both jumpers when connecting ORION. All fans will recieve the same PWM control signal."
- moved on the sheet: D2, D3, D4, D5

Commit message: Fixed current limiting LEDs on the Optoisolator and FAN jumpers
Parts:
- removed JP1, JP2: Jumper_3_Open, Connector_PinHeader_2.54mm:PinHeader_1x03_P2.54mm_Vertical, symbol Jumper:Jumper_3_Open
- added JP1, JP2, JP3, JP4: Termination Resistors, Connector_PinHeader_2.54mm:PinHeader_1x02_P2.54mm_Vertical, symbol Jumper:Jumper_2_Open
Connections:
- net ORION_PWM: now also JP2.2 (B), JP3.1 (A)
- net PWM1: now also JP2.1 (A)
- net PWM2: now also JP3.2 (B), JP4.1 (A)
- net PWM3: now also JP1.1 (A), JP4.2 (B)
- net PWM4: now also JP1.2 (B)
Other:
- moved on the sheet: J?

Commit message: Made ignition connector 3 pin + fixed tach resistors
Parts:
- D2, D3, D4, D5: footprint Diode_SMD:D_SOD-323F -> Diode_SMD:D_SOD-323; P/N 1N4148WS -> 1N4148WSQ-7-F
Connections:
- net +3.3V: no longer IC1.3 (VCC)
- net GND: no longer C1.2
- new net: C1.2, IC1.3 (VCC)
Other:
- note added: "Max input for tach pins should be 5V, even if Vcc is 3.3V. As per page 22 of datasheet"
- note added: "Vih for Tach inputs at Vcc = 3.3V is 2.4V"
- moved on the sheet: C1

Commit message: revamp fans
Parts:
- removed D2, D3, D4, D5: 1N4148WS, Diode_SMD:D_SOD-323, symbol Diode:1N4148
- removed J? (x4): Conn_01x04, UTSVT_Connectors:Molex_MicroFit3.0_1x4xP3.00mm_PolarizingPeg_Vertical, symbol Connector_Generic:Conn_01x04
Other:
- removed sheet Fan_Tach1
- removed sheet Fan_Tach2
- removed sheet Fan_Tach3
- removed sheet Fan_Tach4
- sheet Fan_PWM1 ports: added TACH_OUT; removed PWM_OUT
- sheet Fan_PWM2 ports: added TACH_OUT; removed PWM_OUT
- sheet Fan_PWM3 ports: added TACH_OUT; removed PWM_OUT
- sheet Fan_PWM4 ports: added TACH_OUT; removed PWM_OUT

Commit message: why your schematic so broken >:(
Parts:
- renumbered JP2 to JP1, JP3 to JP2, JP4 to JP3, JP1 to JP4
Connections:
- net ORION_PWM: now also JP2.2 (B), JP3.2 (B), JP4.2 (B); no longer JP2.1 (A)
- net PWM2: now also JP2.1 (A); no longer JP2.2 (B), JP3.1 (A)
- net PWM3: now also JP3.1 (A); no longer JP3.2 (B), JP4.1 (A)
- net PWM4: now also JP4.1 (A); no longer JP4.2 (B)
Other:
- note added: "Bridge all jumpers when connecting ORION. All fans will recieve the same PWM control signal."
- note removed: "Bridge both jumpers when connecting ORION. All fans will recieve the same PWM control signal."
- moved on the sheet: C1, IC1, J?, JP1, JP2, JP3, JP4
