File: Fan_Control.kicad_sch (KiCad schematic)
At the start: 7 parts, among them IC1 ADT7470ARQZ-REEL7

Commit message: everythign on front
Connections:
- net +3.3V: now also IC1.3 (VCC)
- net GND: now also C1.2
Other:
- moved on the sheet: C1
Changed lines of the file:
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@@
   (junction (at 80.01 153.67) (diameter 0) (color 0 0 0 0)
+  )
+  (junction (at 20.32 111.125) (diameter 0) (color 0 0 0 0)
   )
   (junction (at 69.215 153.67) (diameter 0) (color 0 0 0 0)
@@
     (stroke (width 0) (type default))
   )
+  (wire (pts (xy 20.32 121.92) (xy 20.32 118.745))
+    (stroke (width 0) (type default))
+  )
   (wire (pts (xy 80.01 138.43) (xy 80.01 153.67))
     (stroke (width 0) (type default))
@@
     (stroke (width 0) (type default))
   )
-  (wire (pts (xy 20.32 101.6) (xy 20.32 102.235))
-    (stroke (width 0) (type default))
-  )
   (wire (pts (xy 25.4 63.5) (xy 29.21 63.5))
     (stroke (width 0) (type default))
@@
     (stroke (width 0) (type default))
   )
-  (wire (pts (xy 20.32 109.855) (xy 20.32 111.125))
+  (wire (pts (xy 20.32 107.315) (xy 20.32 111.125))
     (stroke (width 0) (type default))
   )
@@
     )
   )
-  (symbol (lib_id "power:+3.3V") (at 20.32 101.6 0) (unit 1)
-    (in_bom yes) (on_board yes) (dnp no)
-    (property "Reference" "#PWR021" (at 20.32 105.41 0)
-      (effects (font (size 1.27 1.27)) hide)
-    )
-    (property "Value" "+3.3V" (at 17.78 96.52 0)
+  (symbol (lib_id "power:+3.3V") (at 20.32 107.315 0) (unit 1)
+    (in_bom yes) (on_board yes) (dnp no)
+    (property "Reference" "#PWR017" (at 20.32 111.125 0)
+      (effects (font (size 1.27 1.27)) hide)
+    )
+    (property "Value" "+3.3V" (at 17.78 102.235 0)
       (effects (font (size 1.27 1.27)) (justify left))
     )
-    (property "Footprint" "" (at 20.32 101.6 0)
-      (effects (font (size 1.27 1.27)) hide)
-    )
-    (property "Datasheet" "" (at 20.32 101.6 0)
-      (effects (font (size 1.27 1.27)) hide)
-    )
-    (pin "1")
-    (instances
-      (project "BPS-LeaderDaughter"
-        (path "/2e9f4f51-d216-4952-a31c-e7104e0d4b1e/bf23a663-b938-440b-843e-ef7912c82d18"
-          (reference "#PWR021") (unit 1)
+    (property "Footprint" "" (at 20.32 107.315 0)
+      (effects (font (size 1.27 1.27)) hide)
+    )
+    (property "Datasheet" "" (at 20.32 107.315 0)
+      (effects (font (size 1.27 1.27)) hide)
+    )
+    (pin "1")
+    (instances
+      (project "BPS-LeaderDaughter"
+        (path "/2e9f4f51-d216-4952-a31c-e7104e0d4b1e/bf23a663-b938-440b-843e-ef7912c82d18"
+          (reference "#PWR017") (unit 1)
         )
       )
@@
         )
         (path "/2e9f4f51-d216-4952-a31c-e7104e0d4b1e/bf23a663-b938-440b-843e-ef7912c82d18"
-          (reference "#PWR022") (unit 1)
+          (reference "#PWR019") (unit 1)
         )
       )
@@
   (symbol (lib_id "power:+3.3V") (at 97.79 113.665 270) (mirror x) (unit 1)
     (in_bom yes) (on_board yes) (dnp no) (fields_autoplaced)
-    (property "Reference" "#PWR025" (at 93.98 113.665 0)
+    (property "Reference" "#PWR022" (at 93.98 113.665 0)
       (effects (font (size 1.27 1.27)) hide)
     )
@@
       (project "BPS-LeaderDaughter"
         (path "/2e9f4f51-d216-4952-a31c-e7104e0d4b1e/bf23a663-b938-440b-843e-ef7912c82d18"
-          (reference "#PWR025") (unit 1)
-        )
-      )
-    )
-  )
-  (symbol (lib_id "Device:C") (at 20.32 106.045 0) (unit 1)
+          (reference "#PWR022") (unit 1)
+        )
+      )
+    )
+  )
+  (symbol (lib_id "Device:C") (at 20.32 114.935 0) (unit 1)
     (in_bom yes) (on_board yes) (dnp no) (fields_autoplaced)
-    (property "Reference" "C1" (at 24.13 104.775 0)
+    (property "Reference" "C1" (at 24.13 113.665 0)
       (effects (font (size 1.27 1.27)) (justify left))
     )
-    (property "Value" "1uF" (at 24.13 107.315 0)
+    (property "Value" "1uF" (at 24.13 116.205 0)
       (effects (font (size 1.27 1.27)) (justify left))
     )
-    (property "Footprint" "Capacitor_SMD:C_0805_2012Metric" (at 21.2852 109.855 0)
-      (effects (font (size 1.27 1.27)) hide)
-    )
-    (property "Datasheet" "~" (at 20.32 106.045 0)
+    (property "Footprint" "Capacitor_SMD:C_0805_2012Metric" (at 21.2852 118.745 0)
+      (effects (font (size 1.27 1.27)) hide)
+    )
+    (property "Datasheet" "~" (at 20.32 114.935 0)
       (effects (font (size 1.27 1.27)) hide)
     )
@@
         )
         (path "/2e9f4f51-d216-4952-a31c-e7104e0d4b1e/bf23a663-b938-440b-843e-ef7912c82d18"
-          (reference "C3") (unit 1)
+          (reference "C1") (unit 1)
         )
       )
@@
         )
         (path "/2e9f4f51-d216-4952-a31c-e7104e0d4b1e/bf23a663-b938-440b-843e-ef7912c82d18"
-          (reference "#PWR024") (unit 1)
+          (reference "#PWR021") (unit 1)
         )
       )
@@
     )
   )
+  (symbol (lib_id "power:GND") (at 20.32 121.92 0) (unit 1)
+    (in_bom yes) (on_board yes) (dnp no)
+    (property "Reference" "#PWR?" (at 20.32 128.27 0)
+      (effects (font (size 1.27 1.27)) hide)
+    )
+    (property "Value" "GND" (at 20.447 126.3142 0)
+      (effects (font (size 1.27 1.27)))
+    )
+    (property "Footprint" "" (at 20.32 121.92 0)
+      (effects (font (size 1.27 1.27)) hide)
+    )
+    (property "Datasheet" "" (at 20.32 121.92 0)
+      (effects (font (size 1.27 1.27)) hide)
+    )
+    (pin "1")
+    (instances
+      (project "BPS-LeaderDaughter"
+        (path "/2e9f4f51-d216-4952-a31c-e7104e0d4b1e"
+          (reference "#PWR?") (unit 1)
+        )
+        (path "/2e9f4f51-d216-4952-a31c-e7104e0d4b1e/55cfe956-9550-49f5-88d2-e32c6d523ac3"
+          (reference "#PWR?") (unit 1)
+        )
+        (path "/2e9f4f51-d216-4952-a31c-e7104e0d4b1e/bf23a663-b938-440b-843e-ef7912c82d18"
+          (reference "#PWR018") (unit 1)
+        )
+      )
+      (project "BPS-Leader"
+        (path "/c248b171-df31-4e8a-afb6-607fa2df334b/00000000-0000-0000-0000-00005d923d59"
+          (reference "#PWR?") (unit 1)
+        )
+      )
+    )
+  )
   (symbol (lib_id "Jumper:Jumper_2_Open") (at 69.215 161.925 90) (unit 1)
     (in_bom yes) (on_board yes) (dnp no)
@@
   (symbol (lib_id "power:+12V") (at 92.71 135.89 0) (unit 1)
     (in_bom yes) (on_board yes) (dnp no) (fields_autoplaced)
-    (property "Reference" "#PWR023" (at 92.71 139.7 0)
+    (property "Reference" "#PWR020" (at 92.71 139.7 0)
       (effects (font (size 1.27 1.27)) hide)
     )
@@
       (project "BPS-LeaderDaughter"
         (path "/2e9f4f51-d216-4952-a31c-e7104e0d4b1e/bf23a663-b938-440b-843e-ef7912c82d18"
-          (reference "#PWR023") (unit 1)
-        )
-      )
+          (reference "#PWR020") (unit 1)
+        )
+      )

Commit message: Used standard footprint cuz Champers sucks (╯°□°)╯︵ ┻━┻
Parts:
- IC1: footprint UTSVT_ICs:ADT7470ARQZ-REEL7 -> Package_SO:QSOP-16_3.9x4.9mm_P0.635mm
Changed lines of the file:
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@@
       (effects (font (size 1.27 1.27)))
     )
-    (property "Footprint" "UTSVT_ICs:ADT7470ARQZ-REEL7" (at 87.63 200.965 0)
+    (property "Footprint" "Package_SO:QSOP-16_3.9x4.9mm_P0.635mm" (at 87.63 200.965 0)
       (effects (font (size 1.27 1.27)) (justify left top) hide)
     )

Commit message: magical unicorns
Parts:
- IC1: symbol utsvt-chips:ADT7470ARQZ-REEL7 -> utsvt-chips:ADT7470ARQZ
Changed lines of the file:
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@@
     )
   )
-  (symbol (lib_id "utsvt-chips:ADT7470ARQZ-REEL7") (at 40.64 106.045 0) (unit 1)
+  (symbol (lib_id "utsvt-chips:ADT7470ARQZ") (at 40.64 106.045 0) (unit 1)
     (in_bom yes) (on_board yes) (dnp no) (fields_autoplaced)
-    (property "Reference" "IC1" (at 66.04 98.425 0)
+    (property "Reference" "IC1" (at 66.04 99.06 0)
       (effects (font (size 1.27 1.27)))
     )
-    (property "Value" "ADT7470ARQZ-REEL7" (at 66.04 100.965 0)
+    (property "Value" "ADT7470ARQZ-REEL7" (at 66.04 101.6 0)
       (effects (font (size 1.27 1.27)))
     )

Commit message: last sanity check + part numbers (ready for review)
Parts:
- C1: P/N (none) -> C0805C105K5PACTU
- IC1: Mouser Part Number 584-ADT7470ARQZ-R7 -> (none)
Other:
- note added: "GND connects to Orion Pin 12 (Ground)"
- note added: "Orion 12V connects to Orion Pin 10 (Fan Enable/ Multi Purpose Output 3)"
- note added: "Orion Tach connects to Orion Pin 9 (Multi Purpose Inptu 3)"
- note added: "Orion_PWM connects to Orion Pin 24 (Fan PWM/ Multi Purpose Output 4)"
Changed lines of the file:
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@@
     (stroke (width 0) (type default))
+  )
+  (text "Orion 12V connects to Orion Pin 10 (Fan Enable/ Multi Purpose Output 3)"
+    (at 117.475 135.89 0)
+    (effects (font (size 1.27 1.27)) (justify left bottom))
+  )
+  (text "Orion_PWM connects to Orion Pin 24 (Fan PWM/ Multi Purpose Output 4)"
+    (at 117.475 138.43 0)
+    (effects (font (size 1.27 1.27)) (justify left bottom))
   )
   (text "Max input for tach pins should be 5V, even if Vcc is 3.3V.\nAs per page 22 of datasheet"
@@
   )
   (text "Vih for Tach inputs at Vcc = 3.3V is 2.4V" (at 105.41 118.745 0)
+    (effects (font (size 1.27 1.27)) (justify left bottom))
+  )
+  (text "GND connects to Orion Pin 12 (Ground)" (at 117.475 146.05 0)
+    (effects (font (size 1.27 1.27)) (justify left bottom))
+  )
+  (text "Orion Tach connects to Orion Pin 9 (Multi Purpose Inptu 3)"
+    (at 117.475 143.51 0)
     (effects (font (size 1.27 1.27)) (justify left bottom))
   )
@@
       (effects (font (size 1.27 1.27)) hide)
     )
+    (property "P/N" "C0805C105K5PACTU" (at 20.32 114.935 0)
+      (effects (font (size 1.27 1.27)) hide)
+    )
     (pin "1")
     (pin "2")
@@
       (effects (font (size 1.27 1.27)) (justify left top) hide)
     )
-    (property "Mouser Part Number" "584-ADT7470ARQZ-R7" (at 87.63 600.965 0)
+    (property "Mouser Part Number" "" (at 87.63 600.965 0)
       (effects (font (size 1.27 1.27)) (justify left top) hide)
     )

Commit message: updated symbol and footprint libraries to use
Parts:
- IC1: Mouser Part Number (none) -> 584-ADT7470ARQZ-R7
Changed lines of the file:
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@@
       (effects (font (size 1.27 1.27)) (justify left top) hide)
     )
-    (property "Mouser Part Number" "" (at 87.63 600.965 0)
+    (property "Mouser Part Number" "584-ADT7470ARQZ-R7" (at 87.63 600.965 0)
       (effects (font (size 1.27 1.27)) (justify left top) hide)
     )

Commit message: bom + gerbers
Parts:
- J?: P/N 0436500428 -> 436500244
Changed lines of the file:
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@@
       (effects (font (size 1.27 1.27)) hide)
     )
-    (property "P/N" "0436500428" (at 104.14 138.43 0)
+    (property "P/N" "436500244" (at 104.14 138.43 0)
       (effects (font (size 1.27 1.27)) hide)
     )
