File: BPS-LeaderDaughter.kicad_pcb (KiCad board)
At the start: 2 copper layers, 50 x 124 mm, 104 parts, among them IC1 ADT7470ARQZ-REEL7, J1 DaughterConnector, J10 Conn_01x04, J11 Conn_01x04, J12 ErrorLightConn, J2 DaughterConnector, J3 Conn_01x04, J4 Conn_01x04, J5 Conn_01x04, J6 Conn_01x04, J7 Conn_01x04, J8 Conn_01x04, J9 Conn_01x04, Q1 BUK9M23-80E, Q2 BUK9M23-80E, Q3 BUK9M23-80E, Q4 BUK9M23-80E, Q5 BUK9M23-80E, Q6 BUK9M23-80E, Q7 BUK9M23-80E, Q8 BUK9M23-80E, U2 SI8261ABC-IS, U5 SI8261ABC-IS, U6 SI8261ABC-IS, U7 SI8261ABC-IS

Commit message: Workday changes
Parts:
- moved D15 0.50 mm to (135.0, 85.8)
- moved D2 0.50 mm to (130.0, 89.3)
- moved D6 0.50 mm to (130.0, 85.3)
- moved J5 0.50 mm to (137.5, 94.1)
- moved Q5 0.50 mm to (133.0, 84.8)
- moved R13 0.50 mm to (135.0, 83.8)
- moved R14 0.50 mm to (135.0, 87.8)
- moved R15 0.50 mm to (135.0, 89.7)
- moved R16 0.50 mm to (135.0, 81.8)
- moved R17 0.50 mm to (130.0, 87.3)
Changed lines of the file:
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@@
   )
   (footprint "Package_TO_SOT_SMD:LFPAK33" (layer "F.Cu")
-    (at 132.475 84.8275 -90)
+    (at 132.975 84.8275 -90)
     (descr "LFPAK33 SOT-1210 https://assets.nexperia.com/documents/outline-drawing/SOT1210.pdf")
     (tags "LFPAK33 SOT-1210")
@@
   )
   (footprint "UTSVT_Connectors:Molex_MicroFit3.0_1x4xP3.00mm_PolarizingPeg_Vertical" (layer "F.Cu")
-    (at 137 94.1 180)
+    (at 137.5 94.1 180)
     (property "P/N" "0436500428")
     (property "Sheetfile" "Fan_Control.kicad_sch")
@@
   )
   (footprint "Diode_SMD:D_SOD-323F" (layer "B.Cu")
-    (at 129.4775 89.2925 180)
+    (at 129.9775 89.2925 180)
     (descr "SOD-323F http://www.nxp.com/documents/outline_drawing/SOD323F.pdf")
     (tags "SOD-323F")
@@
   )
   (footprint "Resistor_SMD:R_0805_2012Metric" (layer "B.Cu")
-    (at 134.475 89.6575 180)
+    (at 134.975 89.6575 180)
     (descr "Resistor SMD 0805 (2012 Metric), square (rectangular) end terminal, IPC_7351 nominal, (Body size source: IPC-SM-782 page 72, https://www.pcb-3d.com/wordpress/wp-content/uploads/ipc-sm-782a_amendment_1_and_2.pdf), generated with kicad-footprint-generator")
     (tags "resistor")
@@
   )
   (footprint "Diode_SMD:D_SOD-323" (layer "B.Cu")
-    (at 134.475 85.7575 180)
+    (at 134.975 85.7575 180)
     (descr "SOD-323")
     (tags "SOD-323")
@@
   )
   (footprint "Resistor_SMD:R_0805_2012Metric" (layer "B.Cu")
-    (at 134.475 81.7575 180)
+    (at 134.975 81.7575 180)
     (descr "Resistor SMD 0805 (2012 Metric), square (rectangular) end terminal, IPC_7351 nominal, (Body size source: IPC-SM-782 page 72, https://www.pcb-3d.com/wordpress/wp-content/uploads/ipc-sm-782a_amendment_1_and_2.pdf), generated with kicad-footprint-generator")
     (tags "resistor")
@@
   )
   (footprint "Resistor_SMD:R_0805_2012Metric" (layer "B.Cu")
-    (at 134.475 87.7575 180)
+    (at 134.975 87.7575 180)
     (descr "Resistor SMD 0805 (2012 Metric), square (rectangular) end terminal, IPC_7351 nominal, (Body size source: IPC-SM-782 page 72, https://www.pcb-3d.com/wordpress/wp-content/uploads/ipc-sm-782a_amendment_1_and_2.pdf), generated with kicad-footprint-generator")
     (tags "resistor")
@@
   )
   (footprint "Resistor_SMD:R_0805_2012Metric" (layer "B.Cu")
-    (at 134.475 83.7575 180)
+    (at 134.975 83.7575 180)
     (descr "Resistor SMD 0805 (2012 Metric), square (rectangular) end terminal, IPC_7351 nominal, (Body size source: IPC-SM-782 page 72, https://www.pcb-3d.com/wordpress/wp-content/uploads/ipc-sm-782a_amendment_1_and_2.pdf), generated with kicad-footprint-generator")
     (tags "resistor")
@@
   )
   (footprint "Diode_SMD:D_SOD-323F" (layer "B.Cu")
-    (at 129.4775 85.2925 180)
+    (at 129.9775 85.2925 180)
     (descr "SOD-323F http://www.nxp.com/documents/outline_drawing/SOD323F.pdf")
     (tags "SOD-323F")
@@
   )
   (footprint "Resistor_SMD:R_0805_2012Metric" (layer "B.Cu")
-    (at 129.5 87.2925 180)
+    (at 130 87.2925 180)
     (descr "Resistor SMD 0805 (2012 Metric), square (rectangular) end terminal, IPC_7351 nominal, (Body size source: IPC-SM-782 page 72, https://www.pcb-3d.com/wordpress/wp-content/uploads/ipc-sm-782a_amendment_1_and_2.pdf), generated with kicad-footprint-generator")
     (tags "resistor")
@@
     (effects (font (size 1 1) (thickness 0.15)) (justify left bottom))
   )
-  (gr_text "2" (at 133.5 97.6 -90) (layer "F.SilkS")
+  (gr_text "2" (at 134 97.6 -90) (layer "F.SilkS")
     (effects (font (size 1 1) (thickness 0.15)) (justify left bottom))
   )
@@
     (effects (font (size 1 1) (thickness 0.15)) (justify bottom))
   )
-  (gr_text "3" (at 130.5 97.6 -90) (layer "F.SilkS")
+  (gr_text "3" (at 131 97.6 -90) (layer "F.SilkS")
     (effects (font (size 1 1) (thickness 0.15)) (justify left bottom))
   )
-  (gr_text "4" (at 127.75 97.6 -90) (layer "F.SilkS")
+  (gr_text "4" (at 128.25 97.6 -90) (layer "F.SilkS")
     (effects (font (size 1 1) (thickness 0.15)) (justify left bottom))
   )
@@
     (effects (font (size 1 1) (thickness 0.15)) (justify bottom))
   )
-  (gr_text "FAN 1" (at 139.75 97.85 -90) (layer "F.SilkS")
+  (gr_text "FAN 1" (at 140.25 97.85 -90) (layer "F.SilkS")
     (effects (font (size 1 1) (thickness 0.15)) (justify left bottom))
   )
@@
     (effects (font (size 1 1) (thickness 0.15)) (justify bottom))
   )
-  (gr_text "1" (at 136.5 97.6 -90) (layer "F.SilkS")
+  (gr_text "1" (at 137 97.6 -90) (layer "F.SilkS")
     (effects (font (size 1 1) (thickness 0.15)) (justify left bottom))
   )
