File: BPS-LeaderDaughter.kicad_pcb (KiCad board)
At the start: 2 copper layers, 50 x 124 mm, 104 parts, among them IC1 ADT7470ARQZ-REEL7, J1 DaughterConnector, J10 Conn_01x04, J11 Conn_01x04, J12 ErrorLightConn, J2 DaughterConnector, J3 Conn_01x04, J4 Conn_01x04, J5 Conn_01x04, J6 Conn_01x04, J7 Conn_01x04, J8 Conn_01x04, J9 Conn_01x04, Q1 BUK9M23-80E, Q2 BUK9M23-80E, Q3 BUK9M23-80E, Q4 BUK9M23-80E, Q5 BUK9M23-80E, Q6 BUK9M23-80E, Q7 BUK9M23-80E, Q8 BUK9M23-80E, U2 SI8261ABC-IS, U5 SI8261ABC-IS, U6 SI8261ABC-IS, U7 SI8261ABC-IS

Commit message: Made ignition connector 3 pin + fixed tach resistors
Parts:
- removed D21: 1N4148WS, Diode_SMD:D_SOD-323F
- removed J3: Conn_01x04, UTSVT_Connectors:Molex_MicroFit3.0_1x4xP3.00mm_PolarizingPeg_Vertical
- added D12: 1N4148WS, Diode_SMD:D_SOD-323, F.Cu at (7.96, 0.97)
- added J13: Conn_01x03, Connector_Molex:Molex_Micro-Fit_3.0_43650-0315_1x03_P3.00mm_Vertical, F.Cu at (177.0, 150.0)
- added JP3: Termination Resistors, Connector_PinHeader_2.54mm:PinHeader_1x02_P2.54mm_Vertical, F.Cu at (169.2, 130.6)
- added JP4: Termination Resistors, Connector_PinHeader_2.54mm:PinHeader_1x02_P2.54mm_Vertical, F.Cu at (173.9, 130.6)
- added R33: 100k, Resistor_SMD:R_0805_2012Metric, F.Cu at (170.7, 139.0)
- added R34: 35, Resistor_SMD:R_0805_2012Metric, F.Cu at (191.1, 143.1)
- added R35: 35, Resistor_SMD:R_0805_2012Metric, F.Cu at (191.1, 146.0)
- added R36: 100k, Resistor_SMD:R_0805_2012Metric, F.Cu at (170.7, 141.9)
- added U1: EL3H7, Package_SO:SOP-4_4.4x2.6mm_P1.27mm, F.Cu at (159.8, 142.2)
- added U4: EL3H7, Package_SO:SOP-4_4.4x2.6mm_P1.27mm, F.Cu at (159.8, 146.4)
- C22, C23, C24: value 1uF -> 100nF
- D1: value LED -> Green; footprint LED_SMD:LED_0805_2012Metric -> LED_SMD:LED_0805_2012Metric_Pad1.15x1.40mm_HandSolder; moved to F.Cu
- D11, D14, D6, D7, D8, D9: footprint Diode_SMD:D_SOD-323F -> Diode_SMD:D_SOD-323
- D2, D3, D4, D5: footprint Diode_SMD:D_SOD-323F -> Diode_SMD:D_SOD-323; moved to F.Cu
- JP1, JP2: value Jumper_3_Open -> Termination Resistors; footprint Connector_PinHeader_2.54mm:PinHeader_1x03_P2.54mm_Vertical -> Connector_PinHeader_2.54mm:PinHeader_1x02_P2.54mm_Vertical
- R1: value 1k -> 10k; moved to F.Cu
- R10, R12, R8: value R -> 1k
- R11, R3, R7: value 5k -> 10k
- R15, R26, R29, R32: value 100k -> 10k
- R2: value 1k -> 80.6
- R41, R42, R43: value 49.9 -> 80.6
- moved D11 197.9 mm to (7.96, 5.92)
- moved D14 196.0 mm to (7.96, 10.9), turned to 0 degrees
- moved D2 155.8 mm to (1.67, 0.97), turned to 0 degrees
- moved D3 145.2 mm to (1.67, 3.92), turned to 0 degrees
- moved D4 126.8 mm to (1.67, 6.88), turned to 0 degrees
- moved D5 115.8 mm to (1.67, 9.82), turned to 0 degrees
- moved R1 86.3 mm to (177.1, 142.0), turned to 0 degrees
- moved D1 86.2 mm to (177.3, 139.0), turned to 0 degrees
- moved JP2 74.3 mm to (164.6, 130.6)
- moved JP1 58.9 mm to (159.9, 130.6)
Connections:
- C16 pad 2: GNDPWR -> GND2
- C17 pad 2: GNDPWR -> GND2
- C18 pad 2: GNDPWR -> GND2
- C19 pad 2: GNDPWR -> GND2
- C20 pad 2: GNDPWR -> GND2
- C21 pad 2: GNDPWR -> GND2
- C8 pad 2: GNDPWR -> GND2
- C9 pad 2: GNDPWR -> GND2
- D1 pad 1: GNDPWR -> Net-(D1-K)
- D14 pad 2: /HV- Contactor Driver/CONTACTOR_V- -> /Array Contactor Driver/CONTACTOR_V-
- J12 pad 2: Net-(J12-Pin_2) -> Net-(D1-K)
- J2 pad 10: unconnected-(J2-Pad10) -> GND
- J2 pad 12: unconnected-(J2-Pad12) -> GND
- J2 pad 13: unconnected-(J2-Pad13) -> /Motor_IG
- J2 pad 15: unconnected-(J2-Pad15) -> /Arr_IG
- JP1 pad 1: /Fan Control/PWM2 -> /Fan Control/PWM3
- JP1 pad 2: /Fan Control/ORION_PWM -> /Fan Control/PWM4
- JP2 pad 1: /Fan Control/PWM4 -> /Fan Control/PWM1
- Q1 pad 1: GNDPWR -> GND2
- Q1 pad 2: GNDPWR -> GND2
- Q1 pad 3: GNDPWR -> GND2
- Q2 pad 1: GNDPWR -> GND2
- Q2 pad 2: GNDPWR -> GND2
- Q2 pad 3: GNDPWR -> GND2
- Q3 pad 1: GNDPWR -> GND2
- Q3 pad 2: GNDPWR -> GND2
- Q3 pad 3: GNDPWR -> GND2
- Q3 pad 5: Net-(J12-Pin_2) -> Net-(D1-K)
- Q4 pad 1: GNDPWR -> GND2
- Q4 pad 2: GNDPWR -> GND2
- Q4 pad 3: GNDPWR -> GND2
- R1 pad 1: Net-(Q3-G) -> +12V
- R4 pad 2: GNDPWR -> GND2
- R5 pad 2: GNDPWR -> GND2
- R6 pad 2: GNDPWR -> GND2
- R9 pad 2: GNDPWR -> GND2
- U2 pad 5: GNDPWR -> GND2
- U5 pad 5: GNDPWR -> GND2
- U6 pad 5: GNDPWR -> GND2
- U7 pad 5: GNDPWR -> GND2

Commit message: Fixed optoisolator resistor values
Parts:
- R13, R24, R27, R30: value 4.7k -> 10k
- R14, R25, R28, R31: value 10k -> 20k
- moved JP4 77.4 mm to (110.0, 87.0), turned to 180 degrees
- moved JP2 76.5 mm to (111.0, 76.0), turned to 90 degrees
- moved JP3 74.6 mm to (118.5, 76.0), turned to 90 degrees
- moved J1 68.8 mm to (41.4, 115.2)
- moved J2 68.8 mm to (53.4, 115.2)
- moved MH5 68.8 mm to (66.9, 141.1)
- moved MH6 68.8 mm to (26.4, 141.1)
- moved JP1 57.3 mm to (126.0, 84.5)
- moved R2 14.0 mm to (105.0, 107.9), turned to -90 degrees
- moved U2 9.75 mm to (102.0, 108.0), turned to 180 degrees
- moved J13 9.00 mm to (168.0, 150.0)
- moved C9 8.37 mm to (101.0, 108.0), turned to 90 degrees
- moved C8 5.65 mm to (99.0, 108.0), turned to 90 degrees
- moved R4 3.62 mm to (93.0, 108.1), turned to 90 degrees
- moved Q3 1.98 mm to (95.6, 108.0), turned to 180 degrees
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Connections:
- C4 pad 2: GND -> Net-(IC1-VCC)
- IC1 pad 3: +3.3V -> Net-(IC1-VCC)

Commit message: why your schematic so broken >:(
Parts:
- removed C16, C18, C20, C22, C23, C24: 100nF, Capacitor_SMD:C_0805_2012Metric
- removed C17, C19, C21: 10uF, Capacitor_SMD:C_0805_2012Metric
- removed D20: BAS70-04, Package_TO_SOT_SMD:SOT-23
- removed D25, D26, D27: Green, LED_SMD:LED_0805_2012Metric_Pad1.15x1.40mm_HandSolder
- removed J13: Conn_01x03, Connector_Molex:Molex_Micro-Fit_3.0_43650-0315_1x03_P3.00mm_Vertical
- removed R41, R42, R43: 80.6, Resistor_SMD:R_0805_2012Metric
- removed U7: SI8261ABC-IS, Package_SO:SOIC-8_3.9x4.9mm_P1.27mm
- added C1: 100nF, Capacitor_SMD:C_0805_2012Metric, F.Cu at (164.0, 110.7)
- added C10: 100nF, Capacitor_SMD:C_0805_2012Metric, F.Cu at (418.7, -15.3)
- added C11: 100nF, Capacitor_SMD:C_0805_2012Metric, F.Cu at (418.7, -12.3)
- added C12: 10uF, Capacitor_SMD:C_0805_2012Metric, F.Cu at (418.7, -9.30)
- added C2: 10uF, Capacitor_SMD:C_0805_2012Metric, F.Cu at (164.0, 113.0)
- added C3: 1uF, Capacitor_SMD:C_0805_2012Metric, F.Cu at (121.4, 87.6)
- added C5: 100nF, Capacitor_SMD:C_0805_2012Metric, F.Cu at (400.6, 380.6)
- added C6: 10uF, Capacitor_SMD:C_0805_2012Metric, F.Cu at (400.6, 383.6)
- added C7: 100nF, Capacitor_SMD:C_0805_2012Metric, F.Cu at (491.0, 193.7)
- added J3: ErrorLightConn, UTSVT_Connectors:Molex_MicroFit3.0_1x2xP3.00mm_PolarizingPeg_Vertical, F.Cu at (169.9, 106.2)
- added JP5: Termination Resistors, Connector_PinHeader_2.54mm:PinHeader_1x02_P2.54mm_Vertical, F.Cu at (93.7, 70.1)
- added JP6: Termination Resistors, Connector_PinHeader_2.54mm:PinHeader_1x02_P2.54mm_Vertical, F.Cu at (124.2, 70.1)
- added JP7: Termination Resistors, Connector_PinHeader_2.54mm:PinHeader_1x02_P2.54mm_Vertical, F.Cu at (57.3, 476.2)
- added JP8: Termination Resistors, Connector_PinHeader_2.54mm:PinHeader_1x02_P2.54mm_Vertical, F.Cu at (-167.2, 199.5)
- added R37: 10k, Resistor_SMD:R_0805_2012Metric, F.Cu at (-265.8, 74.3)
- added R38: 20k, Resistor_SMD:R_0805_2012Metric, F.Cu at (-265.9, 77.6)
- added R39: 10k, Resistor_SMD:R_0805_2012Metric, F.Cu at (-265.9, 81.1)
- added U3: SI8261ABC-IS, Package_SO:SOIC-8_3.9x4.9mm_P1.27mm, F.Cu at (493.0, 189.0)
- C4: value 1uF -> 100nF
- D10, D13: value BAS70-04 -> 1N4148WS; footprint Package_TO_SOT_SMD:SOT-23 -> Diode_SMD:D_SOD-323
- D12, D14: value 1N4148WS -> 3.3V
- D15, D17: value 3.3V -> 1N4148WS; moved to F.Cu
- D16, D18, R20, R21, R24, R27, R28, R29, R32: moved to F.Cu
- D2, D5, D8: value 1N4148WS -> BAS70-04; footprint Diode_SMD:D_SOD-323 -> Package_TO_SOT_SMD:SOT-23
- D3, D6: value 1N4148WS -> Green; footprint Diode_SMD:D_SOD-323 -> LED_SMD:LED_0805_2012Metric_Pad1.15x1.40mm_HandSolder
- D9: value 1N4148WS -> Green; footprint Diode_SMD:D_SOD-323 -> LED_SMD:LED_0805_2012Metric_Pad1.15x1.40mm_HandSolder; moved to F.Cu
- J12: value ErrorLightConn -> Conn_01x04; footprint UTSVT_Connectors:Molex_MicroFit3.0_1x2xP3.00mm_PolarizingPeg_Vertical -> UTSVT_Connectors:Molex_MicroFit3.0_1x4xP3.00mm_PolarizingPeg_Vertical
- J8: value Conn_01x04 -> Conn_01x03; footprint UTSVT_Connectors:Molex_MicroFit3.0_1x4xP3.00mm_PolarizingPeg_Vertical -> Connector_Molex:Molex_Micro-Fit_3.0_43650-0315_1x03_P3.00mm_Vertical
- R1: value 10k -> 80.6
- R10: value 1k -> 100k
- R12, R8: value 1k -> 105
- R13: value 10k -> 1k
- R14: value 20k -> 100k
- R17, R19: value 100k -> 604
- R2: value 80.6 -> 10k; moved to F.Cu
- R22: value 100k -> 10k; moved to F.Cu
- R23: value 100k -> 20k; moved to F.Cu
- R25, R31: value 20k -> 100k; moved to F.Cu
- R26, R30: value 10k -> 100k; moved to F.Cu
- R3: value 10k -> 100k
- R33: value 100k -> 20k
- R34: value 35 -> 10k
- R35: value 35 -> 100k
- R4: value 100k -> 105
- R5, R9: value 100k -> 1k
- U1, U4: value EL3H7 -> SI8261ABC-IS; footprint Package_SO:SOP-4_4.4x2.6mm_P1.27mm -> Package_SO:SOIC-8_3.9x4.9mm_P1.27mm
- U5, U6: value SI8261ABC-IS -> EL3H7; footprint Package_SO:SOIC-8_3.9x4.9mm_P1.27mm -> Package_SO:SOP-4_4.4x2.6mm_P1.27mm
- moved D2 500.7 mm to (396.3, 309.1)
- moved D3 500.7 mm to (396.3, 312.0)
- moved D4 500.3 mm to (402.1, 306.8), turned to 180 degrees
- moved D5 482.1 mm to (469.5, 126.1)
- moved R8 435.6 mm to (545.9, 190.1), turned to 180 degrees
- moved R35 409.5 mm to (-217.7, 169.6), turned to -90 degrees
- moved D6 409.3 mm to (536.4, 124.5)
- moved D16 399.5 mm to (79.6, 463.7)
- moved D10 399.0 mm to (462.3, -23.5)
- moved R30 396.8 mm to (75.2, 460.8)
- moved R32 396.7 mm to (75.2, 466.7)
- moved R31 395.8 mm to (75.2, 463.7)
- moved R7 395.5 mm to (464.6, 359.9)
- moved J12 392.9 mm to (-294.4, 106.9)
- moved R36 388.7 mm to (-217.7, 156.8), turned to 90 degrees
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Connections:
- C4 pad 1: +3.3V -> /HV+_Sense
- C4 pad 2: Net-(IC1-VCC) -> GND
- D10 pad 1: GND -> +12V
- D10 pad 2: +3.3V -> /Array Contactor Driver/CONTACTOR_V-
- D11 pad 2: /HV+ Contactor Driver/CONTACTOR_V- -> GND
- D12 pad 1: +12V -> /Fan Control/TACH1
- D12 pad 2: /HV- Contactor Driver/CONTACTOR_V- -> GND
- D13 pad 1: GND -> +12V
- D13 pad 2: +3.3V -> GND
- D14 pad 1: +12V -> /Fan Control/TACH2
- D14 pad 2: /Array Contactor Driver/CONTACTOR_V- -> GND
- D15 pad 1: /Fan Control/TACH1 -> +12V
- D16 pad 1: /Fan Control/TACH2 -> /Fan Control/TACH3
- D17 pad 1: /Fan Control/TACH3 -> +12V
- D2 pad 1: +12V -> GND
- D2 pad 2: GND -> +3.3V
- D3 pad 1: +12V -> /HV+ Contactor Driver/CONTACTOR_V-
- D3 pad 2: GND -> Net-(D3-A)
- D4 pad 2: GND -> /HV+ Contactor Driver/CONTACTOR_V-
- D5 pad 1: +12V -> GND
- D5 pad 2: GND -> +3.3V
- D6 pad 1: +12V -> /HV- Contactor Driver/CONTACTOR_V-
- D6 pad 2: /Fan Control/PWM1_OUT -> Net-(D6-A)
- D7 pad 2: /Fan Control/PWM2_OUT -> /HV- Contactor Driver/CONTACTOR_V-
- D8 pad 1: +12V -> GND
- D8 pad 2: /Fan Control/PWM3_OUT -> +3.3V
- D9 pad 1: +12V -> /Array Contactor Driver/CONTACTOR_V-
- D9 pad 2: /Fan Control/PWM4_OUT -> Net-(D9-A)
- J10 pad 1: +12V -> Net-(J10-Pin_1)
- J10 pad 2: /HV- Contactor Driver/CONTACTOR_V- -> +12V
- J10 pad 3: GND -> /Fan Control/Fan_PWM2/TACH_IN
- J10 pad 4: Net-(J10-Pin_4) -> /Fan Control/PWM2
- J11 pad 1: +12V -> Net-(J11-Pin_1)
- J11 pad 2: /Array Contactor Driver/CONTACTOR_V- -> +12V
- J11 pad 3: GND -> /Fan Control/Fan_PWM3/TACH_IN
- J11 pad 4: Net-(J11-Pin_4) -> /Fan Control/PWM3
- J12 pad 1: +12V -> Net-(J12-Pin_1)
- J12 pad 2: Net-(D1-K) -> +12V
- J5 pad 1: GND -> +12V
- J5 pad 2: +12V -> /HV+ Contactor Driver/CONTACTOR_V-
- J5 pad 3: /Fan Control/TACH1_IN -> GND
- J5 pad 4: /Fan Control/PWM1_OUT -> Net-(J5-Pin_4)
- J6 pad 1: GND -> +12V
- J6 pad 2: +12V -> /HV- Contactor Driver/CONTACTOR_V-
- J6 pad 3: /Fan Control/TACH2_IN -> GND
- J6 pad 4: /Fan Control/PWM2_OUT -> Net-(J6-Pin_4)
- J7 pad 1: GND -> +12V
- J7 pad 2: +12V -> /Array Contactor Driver/CONTACTOR_V-
- J7 pad 3: /Fan Control/TACH3_IN -> GND
- J7 pad 4: /Fan Control/PWM3_OUT -> Net-(J7-Pin_4)
- J8 pad 1: GND -> Net-(J8-Pin_1)
- J8 pad 2: +12V -> Net-(J8-Pin_2)
- J8 pad 3: /Fan Control/TACH4_IN -> GND
- J9 pad 1: +12V -> Net-(J9-Pin_1)
- J9 pad 2: /HV+ Contactor Driver/CONTACTOR_V- -> +12V
- J9 pad 3: GND -> /Fan Control/Fan_PWM1/TACH_IN
- J9 pad 4: Net-(J9-Pin_4) -> /Fan Control/PWM1
- JP1 pad 1: /Fan Control/PWM3 -> /Fan Control/PWM1
- JP1 pad 2: /Fan Control/PWM4 -> /Fan Control/ORION_PWM
- JP2 pad 1: /Fan Control/PWM1 -> /Fan Control/PWM2
- JP3 pad 1: /Fan Control/ORION_PWM -> /Fan Control/PWM3
- JP3 pad 2: /Fan Control/PWM2 -> /Fan Control/ORION_PWM
- JP4 pad 1: /Fan Control/PWM2 -> /Fan Control/PWM4
- JP4 pad 2: /Fan Control/PWM3 -> /Fan Control/ORION_PWM
- Q1 pad 4: /HV+ Contactor Driver/PWM_ISO -> Net-(Q1-G)
- Q1 pad 5: /HV+ Contactor Driver/CONTACTOR_V- -> Net-(D1-K)
- Q2 pad 4: /HV- Contactor Driver/PWM_ISO -> /HV+ Contactor Driver/PWM_ISO
- Q2 pad 5: /HV- Contactor Driver/CONTACTOR_V- -> /HV+ Contactor Driver/CONTACTOR_V-
- Q3 pad 4: Net-(Q3-G) -> /HV- Contactor Driver/PWM_ISO
- Q3 pad 5: Net-(D1-K) -> /HV- Contactor Driver/CONTACTOR_V-
- Q5 pad 4: /Fan Control/PWM1 -> Net-(JP5-B)
- Q5 pad 5: /Fan Control/PWM1_OUT -> Net-(J9-Pin_1)
- Q6 pad 4: /Fan Control/PWM2 -> Net-(JP6-B)
- Q6 pad 5: /Fan Control/PWM2_OUT -> Net-(J10-Pin_1)
- Q7 pad 4: /Fan Control/PWM3 -> Net-(JP7-B)
- Q7 pad 5: /Fan Control/PWM3_OUT -> Net-(J11-Pin_1)
- Q8 pad 4: /Fan Control/PWM4 -> Net-(JP8-B)
- Q8 pad 5: /Fan Control/PWM4_OUT -> Net-(J12-Pin_1)
- R1 pad 1: +12V -> /Fault
- R1 pad 2: Net-(D1-A) -> Net-(U1-ANODE)
- R10 pad 1: /HV-_Sense -> /HV- Contactor Driver/PWM_ISO
- R10 pad 2: Net-(J10-Pin_4) -> GND2
- R11 pad 2: Net-(D27-A) -> Net-(D6-A)
- R12 pad 1: /Array_Sense -> /Array_EN
- R12 pad 2: Net-(J11-Pin_4) -> Net-(U4-ANODE)
- R13 pad 1: /Fan Control/TACH1 -> /Array_Sense
- R13 pad 2: GND -> Net-(J7-Pin_4)
- R14 pad 1: /Fan Control/TACH1 -> /Array Contactor Driver/PWM_ISO
- R14 pad 2: /Fan Control/TACH1_IN -> GND2
- R15 pad 2: /Fan Control/TACH1_IN -> Net-(D9-A)
- R16 pad 1: +3.3V -> GND
- R16 pad 2: /Fan Control/PWM1 -> /Motor_IG
- R17 pad 1: +12V -> Net-(R17-Pad1)
- R17 pad 2: /Fan Control/PWM1_OUT -> Net-(J8-Pin_1)
- R18 pad 1: +3.3V -> GND
- R18 pad 2: /Fan Control/PWM2 -> /Arr_IG
- R19 pad 1: +12V -> Net-(R19-Pad1)
- R19 pad 2: /Fan Control/PWM2_OUT -> Net-(J8-Pin_2)
- R2 pad 1: /Fault -> +12V
- R2 pad 2: Net-(U2-ANODE) -> Net-(D1-A)
- R20 pad 2: /Fan Control/PWM3 -> /Fan Control/PWM1
- R21 pad 1: +12V -> +3.3V
- R21 pad 2: /Fan Control/PWM3_OUT -> Net-(JP5-B)
- R22 pad 1: +3.3V -> +12V
- R22 pad 2: /Fan Control/PWM4 -> /Fan Control/Fan_PWM1/TACH_IN
- R23 pad 1: +12V -> /Fan Control/Fan_PWM1/TACH_IN
- R23 pad 2: /Fan Control/PWM4_OUT -> /Fan Control/TACH1
- R24 pad 1: /Fan Control/TACH2 -> /Fan Control/TACH1
- R25 pad 1: /Fan Control/TACH2 -> +3.3V
- R25 pad 2: /Fan Control/TACH2_IN -> /Fan Control/PWM2
- R26 pad 1: +12V -> +3.3V
- R26 pad 2: /Fan Control/TACH2_IN -> Net-(JP6-B)
- R27 pad 1: /Fan Control/TACH3 -> +12V
- R27 pad 2: GND -> /Fan Control/Fan_PWM2/TACH_IN
- R28 pad 1: /Fan Control/TACH3 -> /Fan Control/Fan_PWM2/TACH_IN
- R28 pad 2: /Fan Control/TACH3_IN -> /Fan Control/TACH2
- R29 pad 1: +12V -> /Fan Control/TACH2
- R29 pad 2: /Fan Control/TACH3_IN -> GND
- R3 pad 1: +12V -> Net-(Q1-G)
- R3 pad 2: Net-(D26-A) -> GND2
- R30 pad 1: /Fan Control/TACH4 -> +3.3V
- R30 pad 2: GND -> /Fan Control/PWM3
- R31 pad 1: /Fan Control/TACH4 -> +3.3V
- R31 pad 2: /Fan Control/TACH4_IN -> Net-(JP7-B)
- R32 pad 2: /Fan Control/TACH4_IN -> /Fan Control/Fan_PWM3/TACH_IN
- R33 pad 1: /Arr_IG -> /Fan Control/Fan_PWM3/TACH_IN
- R33 pad 2: +3.3V -> /Fan Control/TACH3
- R34 pad 1: Net-(R34-Pad1) -> /Fan Control/TACH3
- R34 pad 2: Net-(J13-Pin_2) -> GND
- R35 pad 1: Net-(R35-Pad1) -> +3.3V
- R35 pad 2: Net-(J13-Pin_1) -> /Fan Control/PWM4
- R36 pad 1: /Motor_IG -> +3.3V
- R36 pad 2: +3.3V -> Net-(JP8-B)
- R4 pad 1: Net-(Q3-G) -> /HV+_EN
- R4 pad 2: GND2 -> Net-(U2-ANODE)
- R5 pad 1: /HV+ Contactor Driver/PWM_ISO -> /HV+_Sense
- R5 pad 2: GND2 -> Net-(J5-Pin_4)
- R6 pad 1: /HV- Contactor Driver/PWM_ISO -> /HV+ Contactor Driver/PWM_ISO
- R7 pad 2: Net-(D25-A) -> Net-(D3-A)
- R8 pad 1: /HV+_Sense -> /HV-_EN
- R8 pad 2: Net-(J9-Pin_4) -> Net-(U3-ANODE)
- R9 pad 1: /Array Contactor Driver/PWM_ISO -> /HV-_Sense
- R9 pad 2: GND2 -> Net-(J6-Pin_4)
- U1 pad 1: Net-(R35-Pad1) -> unconnected-(U1-NC-Pad1)
- U1 pad 2: GND -> Net-(U1-ANODE)
- U1 pad 4: /Motor_IG -> unconnected-(U1-NC-Pad4)
- U2 pad 6: Net-(Q3-G) -> /HV+ Contactor Driver/PWM_ISO
- U2 pad 7: Net-(Q3-G) -> /HV+ Contactor Driver/PWM_ISO
- U4 pad 1: Net-(R34-Pad1) -> unconnected-(U4-NC-Pad1)
- U4 pad 2: GND -> Net-(U4-ANODE)
- U4 pad 4: /Arr_IG -> unconnected-(U4-NC-Pad4)
- U5 pad 1: unconnected-(U5-NC-Pad1) -> Net-(R17-Pad1)
- U5 pad 2: Net-(U5-ANODE) -> GND
- U5 pad 3: GND -> /Motor_IG
- U5 pad 4: unconnected-(U5-NC-Pad4) -> +3.3V
- U6 pad 1: unconnected-(U6-NC-Pad1) -> Net-(R19-Pad1)
- U6 pad 2: Net-(U6-ANODE) -> GND
- U6 pad 3: GND -> /Arr_IG
- U6 pad 4: unconnected-(U6-NC-Pad4) -> +3.3V
Routing:
- net +12V: track 0.00 -> 37.5 mm
- net /Fan Control/ORION_PWM: track 0.00 -> 25.6 mm
- net Net-(Q1-G): track 0.00 -> 15.8 mm
- net Net-(JP5-B): track 0.00 -> 12.9 mm
- net /Fan Control/PWM1: track 0.00 -> 12.2 mm
- net /Fan Control/Fan_PWM1/TACH_IN: track 0.00 -> 10.8 mm
- net Net-(D1-K): track 0.00 -> 10.0 mm
- net Net-(J9-Pin_1): track 0.00 -> 6.69 mm
- net Net-(J10-Pin_1): track 0.00 -> 6.69 mm
- net /Fan Control/TACH1: track 0.00 -> 5.14 mm
- net Net-(U1-ANODE): track 0.00 -> 2.99 mm
Other:
- board text added: "Grid size is .01in"

Commit message: More layout progress, fix LeaderSOM holes, removed strobe isolator, fixed GND of contactor, weeeee
Parts:
- removed C1: 100nF, Capacitor_SMD:C_0805_2012Metric
- removed C2: 10uF, Capacitor_SMD:C_0805_2012Metric
- removed U1: SI8261ABC-IS, Package_SO:SOIC-8_3.9x4.9mm_P1.27mm
- C10, C11, C12, C3, C5, C6, C7, D10, D12, D14, D16, D18, D4, R10, R20, R21, R25, R26, R3, R30, R31, R35, R36: moved to B.Cu
- D6, D8, R15, R4: moved to F.Cu
- R1: value 80.6 -> 105; moved to B.Cu
- moved J12 430.7 mm to (135.6, 81.6)
- moved R14 425.9 mm to (112.1, 171.9), turned to 90 degrees
- moved R7 421.8 mm to (97.4, 152.1), turned to 90 degrees
- moved R13 421.7 mm to (120.1, 171.9), turned to -90 degrees
- moved R15 420.4 mm to (114.0, 167.0), turned to 90 degrees
- moved J11 411.7 mm to (105.0, 82.0)
- moved D6 411.5 mm to (125.9, 153.1), turned to 90 degrees
- moved R8 408.1 mm to (139.5, 153.4), turned to -90 degrees
- moved D10 402.8 mm to (110.1, 172.0), turned to 90 degrees
- moved J7 395.7 mm to (112.5, 176.9), turned to 0 degrees
- moved R37 393.7 mm to (127.6, 89.0), turned to -90 degrees
- moved R38 391.6 mm to (125.6, 89.0), turned to -90 degrees
- moved Q8 391.1 mm to (133.0, 89.0), turned to 0 degrees
- moved JP7 391.0 mm to (107.1, 88.5)
- moved R39 389.5 mm to (123.6, 89.0), turned to -90 degrees
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Connections:
- C11 pad 2: GND2 -> GND
- C12 pad 2: GND2 -> GND
- C5 pad 2: GND2 -> GND
- C6 pad 2: GND2 -> GND
- C8 pad 2: GND2 -> GND
- C9 pad 2: GND2 -> GND
- Q1 pad 1: GND2 -> GND
- Q1 pad 2: GND2 -> GND
- Q1 pad 3: GND2 -> GND
- Q2 pad 1: GND2 -> GND
- Q2 pad 2: GND2 -> GND
- Q2 pad 3: GND2 -> GND
- Q3 pad 1: GND2 -> GND
- Q3 pad 2: GND2 -> GND
- Q3 pad 3: GND2 -> GND
- Q4 pad 1: GND2 -> GND
- Q4 pad 2: GND2 -> GND
- Q4 pad 3: GND2 -> GND
- R1 pad 2: Net-(U1-ANODE) -> Net-(Q1-G)
- R10 pad 2: GND2 -> GND
- R14 pad 2: GND2 -> GND
- R3 pad 2: GND2 -> GND
- R6 pad 2: GND2 -> GND
- U2 pad 5: GND2 -> GND
- U3 pad 5: GND2 -> GND
- U4 pad 5: GND2 -> GND
Routing:
- net +12V: track 37.5 -> 0.00 mm
- net /Fan Control/ORION_PWM: track 25.6 -> 0.00 mm
- net Net-(Q1-G): track 15.8 -> 0.00 mm
- net Net-(JP5-B): track 12.9 -> 0.00 mm
- net /Fan Control/PWM1: track 12.2 -> 0.00 mm
- net /Fan Control/Fan_PWM1/TACH_IN: track 10.8 -> 0.00 mm
- net Net-(D1-K): track 10.0 -> 0.00 mm
- net Net-(J9-Pin_1): track 6.69 -> 0.00 mm
- net Net-(J10-Pin_1): track 6.69 -> 0.00 mm
- net /Fan Control/TACH1: track 5.14 -> 0.00 mm
- net Net-(U1-ANODE): track 2.99 -> 0.00 mm
- net Net-(J6-Pin_4): vias 0 -> 2
- net Net-(J5-Pin_4): vias 0 -> 2
- net /HV- Contactor Driver/PWM_ISO: vias 0 -> 2
- net /HV+ Contactor Driver/PWM_ISO: vias 0 -> 2
Other:
- board text removed: "FAN 1"

Commit message: Made connectors all on one side
Parts:
- moved J7 88.3 mm to (120.5, 89.0), turned to 180 degrees
- moved D10 77.0 mm to (121.6, 95.9), turned to -90 degrees
- moved D8 76.7 mm to (110.6, 95.9), turned to 0 degrees
- moved R13 76.5 mm to (111.6, 95.9), turned to 90 degrees
- moved R14 76.4 mm to (119.6, 95.9), turned to -90 degrees
- moved Q4 76.2 mm to (118.0, 95.9), turned to 180 degrees
- moved C10 76.2 mm to (113.6, 95.9), turned to 90 degrees
- moved D9 65.8 mm to (121.6, 101.9), turned to -90 degrees
- moved R15 65.3 mm to (119.6, 101.9), turned to -90 degrees
- moved J2 63.3 mm to (109.0, 166.9), turned to 0 degrees
- moved J1 62.9 mm to (121.0, 166.9), turned to 0 degrees
- moved C12 61.2 mm to (111.5, 101.0), turned to -90 degrees
- moved C11 61.0 mm to (113.5, 101.0), turned to -90 degrees
- moved R12 61.0 mm to (108.0, 101.6), turned to 90 degrees
- moved U4 60.3 mm to (113.0, 101.3), turned to 0 degrees
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Routing:
- net Net-(J7-Pin_4): vias 0 -> 2
- net /Array Contactor Driver/PWM_ISO: vias 0 -> 2
Other:
- board size 50 x 124 mm -> 50 x 131 mm

Commit message: everythign on front
Parts:
- removed C10, C11, C5, C7, C8: 100nF, Capacitor_SMD:C_0805_2012Metric
- removed C12, C6, C9: 10uF, Capacitor_SMD:C_0805_2012Metric
- removed U3, U4: SI8261ABC-IS, Package_SO:SOIC-8_3.9x4.9mm_P1.27mm
- removed U5, U6: EL3H7, Package_SO:SOP-4_4.4x2.6mm_P1.27mm
- added C1: 1uF, Capacitor_SMD:C_0805_2012Metric, F.Cu at (115.6, 84.1)
- added C2: 100nF, Capacitor_SMD:C_0805_2012Metric, F.Cu at (122.9, 96.8)
- added U1: EL3H7, Package_SO:SOP-4_4.4x2.6mm_P1.27mm, F.Cu at (123.6, 167.5)
- C3: value 1uF -> 100nF; moved to F.Cu
- C4, D10, D12, D14, D16, D18, D4, R13, R14, R16, R17, R18, R19, R20, R21, R25, R26, R3, R30, R31, R35, R36, R5, R6: moved to F.Cu
- R1: value 105 -> 1k; moved to F.Cu
- R12, R4, R8: value 105 -> 1k
- U2: value SI8261ABC-IS -> EL3H7; footprint Package_SO:SOIC-8_3.9x4.9mm_P1.27mm -> Package_SO:SOP-4_4.4x2.6mm_P1.27mm
- moved J3 92.0 mm to (103.3, 176.9), turned to 0 degrees
- moved J6 89.7 mm to (45.9, 126.5), turned to -90 degrees
- moved J8 89.3 mm to (123.5, 176.9), turned to 0 degrees
- moved R19 85.5 mm to (129.2, 172.8), turned to 0 degrees
- moved D7 83.6 mm to (51.8, 125.5), turned to 0 degrees
- moved R2 83.5 mm to (101.8, 170.8), turned to 90 degrees
- moved D1 83.3 mm to (99.7, 170.8), turned to 90 degrees
- moved R10 81.9 mm to (51.9, 127.5), turned to 0 degrees
- moved R17 81.8 mm to (123.6, 172.8)
- moved Q3 80.7 mm to (51.8, 129.0), turned to -90 degrees
- moved Q1 79.4 mm to (108.8, 171.4), turned to -90 degrees
- moved R3 79.1 mm to (105.8, 170.8)
- moved R1 78.9 mm to (103.8, 170.8)
- moved C3 77.9 mm to (58.3, 132.0), turned to 0 degrees
- moved D6 76.9 mm to (57.8, 125.5), turned to 0 degrees
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Connections:
- C3 pad 1: +3.3V -> /HV-_Sense
- C3 pad 2: Net-(IC1-VCC) -> GND
- C4 pad 1: /HV+_Sense -> /Array_Sense
- IC1 pad 3: Net-(IC1-VCC) -> +3.3V
- Q2 pad 4: /HV+ Contactor Driver/PWM_ISO -> Net-(Q2-G)
- Q3 pad 4: /HV- Contactor Driver/PWM_ISO -> Net-(Q3-G)
- Q4 pad 4: /Array Contactor Driver/PWM_ISO -> Net-(Q4-G)
- R10 pad 1: /HV- Contactor Driver/PWM_ISO -> Net-(Q3-G)
- R12 pad 1: /Array_EN -> /Array_Sense
- R12 pad 2: Net-(U4-ANODE) -> Net-(J7-Pin_4)
- R13 pad 1: /Array_Sense -> /Array_EN
- R13 pad 2: Net-(J7-Pin_4) -> Net-(Q4-G)
- R14 pad 1: /Array Contactor Driver/PWM_ISO -> Net-(Q4-G)
- R4 pad 1: /HV+_EN -> /HV+_Sense
- R4 pad 2: Net-(U2-ANODE) -> Net-(J5-Pin_4)
- R5 pad 1: /HV+_Sense -> /HV+_EN
- R5 pad 2: Net-(J5-Pin_4) -> Net-(Q2-G)
- R6 pad 1: /HV+ Contactor Driver/PWM_ISO -> Net-(Q2-G)
- R8 pad 1: /HV-_EN -> /HV-_Sense
- R8 pad 2: Net-(U3-ANODE) -> Net-(J6-Pin_4)
- R9 pad 1: /HV-_Sense -> /HV-_EN
- R9 pad 2: Net-(J6-Pin_4) -> Net-(Q3-G)
- U2 pad 1: unconnected-(U2-NC-Pad1) -> Net-(R19-Pad1)
- U2 pad 2: Net-(U2-ANODE) -> GND
- U2 pad 3: GND -> /Arr_IG
- U2 pad 4: unconnected-(U2-NC-Pad4) -> +3.3V
Routing:
- net +12V: track 0.00 -> 23.5 mm
- net Net-(D1-K): track 0.00 -> 17.7 mm
- net /Array Contactor Driver/CONTACTOR_V-: track 0.00 -> 15.0 mm
- net Net-(JP7-B): track 0.00 -> 12.9 mm
- net Net-(J7-Pin_4): track 0.00 -> 10.3 mm, vias 2 -> 0
- net /Fan Control/TACH3: track 0.00 -> 9.74 mm
- net /Fan Control/PWM3: track 0.00 -> 8.57 mm
- net /Fan Control/Fan_PWM3/TACH_IN: track 0.00 -> 7.41 mm
- net Net-(Q4-G): track 0.00 -> 5.72 mm
- net Net-(Q1-G): track 0.00 -> 4.86 mm
- net Net-(J11-Pin_1): track 0.00 -> 4.66 mm
- net Net-(D1-A): track 0.00 -> 2.08 mm
- net /Array_Sense: track 0.00 -> 1.95 mm
- net Net-(D9-A): track 0.00 -> 1.72 mm
- net Net-(Q3-G): vias 0 -> 1
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Other:
- board text added: "Array Contactor"
- board text added: "Error Light"
- board text added: "FAN 1"
- board text added: "HV+ Contactor"
- board text added: "Orion"

Commit message: Layout and arrange other Contactor circuit
Parts:
- D7, R10, R9: moved to F.Cu
- moved J6 77.9 mm to (120.6, 104.5), turned to 180 degrees
- moved R9 71.7 mm to (118.5, 109.1), turned to 90 degrees
- moved D7 70.7 mm to (120.6, 109.1), turned to 90 degrees
- moved R11 70.6 mm to (123.5, 101.3), turned to 180 degrees
- moved J8 69.7 mm to (136.7, 108.5), turned to 180 degrees
- moved J3 68.5 mm to (99.1, 108.5), turned to 180 degrees
- moved R10 67.2 mm to (116.5, 109.1), turned to -90 degrees
- moved D6 66.5 mm to (119.8, 101.3)
- moved Q3 64.5 mm to (113.3, 109.6), turned to 90 degrees
- moved R8 63.7 mm to (108.9, 101.3)
- moved D5 63.2 mm to (109.2, 109.8)
- moved C3 62.4 mm to (112.7, 101.3)
- moved R17 61.6 mm to (136.6, 112.6), turned to 180 degrees
- moved R19 60.2 mm to (131.0, 112.6), turned to 180 degrees
- moved Q1 59.3 mm to (93.6, 114.0), turned to 90 degrees
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Routing:
- net /HV- Contactor Driver/CONTACTOR_V-: track 0.00 -> 15.0 mm
- net Net-(J7-Pin_4): track 10.3 -> 0.00 mm
- net /Array Contactor Driver/CONTACTOR_V-: track 15.0 -> 6.58 mm
- net Net-(Q3-G): track 0.00 -> 5.72 mm, vias 1 -> 0
- net Net-(Q4-G): track 5.72 -> 0.00 mm
- net /Array_Sense: track 1.95 -> 0.00 mm
- net Net-(D6-A): track 0.00 -> 1.72 mm
- net Net-(J6-Pin_4): vias 2 -> 0
- net /HV-_Sense: vias 1 -> 0
