File: BPS-LeaderDaughter.kicad_pcb (KiCad board)
At the start: 2 copper layers, 50 x 130 mm, 94 parts, among them IC1 ADT7470ARQZ-REEL7, J1 DaughterConnector, J10 Conn_01x04, J11 Conn_01x04, J12 Conn_01x04, J2 DaughterConnector, J3 ErrorLightConn, J4 Conn_01x04, J5 Conn_01x04, J6 Conn_01x04, J7 Conn_01x04, J8 Conn_01x03, J9 Conn_01x04, Q1 BUK9M23-80E, Q2 BUK9M23-80E, Q3 BUK9M23-80E, Q4 BUK9M23-80E, Q5 BUK9M23-80E, Q6 BUK9M23-80E, Q7 BUK9M23-80E, Q8 BUK9M23-80E, U1 EL3H7, U2 EL3H7

Commit message: let's ignore the 18 remaining DRC issues
Parts:
- J1, J2: footprint UTSVT_Connectors:533072071 -> UTSVT_Connectors:Molex_53307-2071
- moved J1 0.27 mm to (146.2, 91.8)
- moved J2 0.27 mm to (158.2, 91.8)
- moved MH5 0.27 mm to (171.7, 117.7), turned to 0 degrees
- moved MH6 0.27 mm to (131.2, 117.7), turned to 0 degrees
- moved J3 0.06 mm to (136.4, 82.5)
- turned MH1 to 180 degrees
- turned MH2 to 180 degrees
Routing:
- net +3.3V: track 145.1 -> 111.5 mm
- net GND: track 43.3 -> 31.6 mm, vias 5 -> 6
- net /SDA: track 49.0 -> 43.0 mm
- net /~{SMBALERT}: track 46.7 -> 41.4 mm
- net /SCL: track 45.1 -> 40.7 mm
- net /Fan Control/PWM4: track 25.9 -> 29.0 mm
- net /Fault: vias 2 -> 1
- added copper zone on F.Cu, net +3.3V
Other:
- board text added: "HV- Contactor"
- board text added: "Ignition"
- board text added: "Strobe Light"

Commit message: Cleaned up silkscreen
Parts:
- added J1: DaughterConnector, UTSVT_Connectors:Molex_53307-2071, F.Cu at (146.2, 91.8)
- moved LOGO2 111.7 mm to (152.1, 126.0)
- moved LOGO1 104.0 mm to (151.9, 104.5)
- moved MH1 0.83 mm to (173.6, 29.1)
- moved MH2 0.76 mm to (130.6, 29.1)
- moved MH4 0.72 mm to (173.6, 152.1)
- moved MH3 0.64 mm to (130.6, 152.1)
Routing:
- net GND: track 31.6 -> 31.9 mm, vias 6 -> 7
Other:
- outline, holes or cut-outs redrawn
- board text added: "Arr"
- board text added: "BPS-LeaderDaughter V1.0 Fall 2023"
- board text added: "Bridge to use Orion for fans"
- board text added: "Cont-"
- board text added: "Lakshay and Jamey were here"
- board text added: "Motor"
- board text added: "Sense"
- board text added: "Short for 4 wire fan"
- board text added: "Tach"
- board text added: "locked"
- board text removed: "1"
- board text removed: "12V(OR 10)"
- board text removed: "2"
- board text removed: "3"
- board text removed: "3 WIRE"
- board text removed: "4"
- board text removed: "4 WIRE"
- board text removed: "BRIDGE"
- board text removed: "GND(OR 12)"
- board text removed: "ORION PWM"
- board text removed: "PWM(OR 24)"
- board text removed: "TACH"
- board text removed: "TACH(OR 9)"
- board text removed: "USB"

Commit message: LAKSHAY CHOSE THE WRONG DIODE >:(
Parts:
- removed the J1 at (146.2, 91.8)
- D10, D11, D13, D15, D17, D4, D7: value 1N4148WS -> 1N4448W; footprint Diode_SMD:D_SOD-323 -> Diode_SMD:D_SOD-123; moved to F.Cu
- R17, R19: value 604 -> 600
- moved D13 78.0 mm to (99.5, 78.2), turned to 0 degrees
- moved D17 74.6 mm to (99.5, 83.6), turned to 0 degrees
- moved D7 72.4 mm to (99.5, 67.5), turned to 0 degrees
- moved D10 60.4 mm to (99.5, 72.9), turned to 0 degrees
- moved D11 47.3 mm to (107.3, 78.2), turned to 0 degrees
- moved D4 36.5 mm to (107.3, 67.5), turned to 0 degrees
- moved D15 34.3 mm to (107.3, 72.9), turned to 0 degrees
Other:
- board text added: "Lakshay and Jamey were here Champers snuck in too"
- board text removed: "Lakshay and Jamey were here"

Commit message: I̶̤̒'̶̝͊m̴͂ͅ ̵͓͆n̷̙͘ǫ̷̛t̴͖̿ ̶̝͝l̴͍̐ó̷̪s̶̲̀i̶͎̊n̴̛͙ǵ̸̢ ̴̱̋m̴̢̈́y̴̺͒ ̶̋͜m̵̟̔i̷̹͝n̴̞̅ḏ̷͠.̴̠̌ ̶̲̕Ÿ̴̱́o̶̰̐ù̸̡ ̸̣̌a̷̭͘r̷̨̔e̴͈̅ ̵͕͊≯̤͊:̶̯̅)̵̟̕
Parts:
- D10, D11, D13, D15, D17, D4, D7: moved to B.Cu
- moved D13 78.0 mm to (170.9, 47.0), turned to -90 degrees
- moved D17 74.6 mm to (170.9, 62.0), turned to -90 degrees
- moved D7 71.8 mm to (170.6, 77.8), turned to -135 degrees
- moved D10 60.3 mm to (159.7, 77.5), turned to -90 degrees
- moved D11 46.9 mm to (137.4, 42.3), turned to -90 degrees
- moved D4 37.0 mm to (144.4, 67.1), turned to -45 degrees
- moved D15 33.9 mm to (137.4, 57.2), turned to -90 degrees
- moved D12 0.52 mm to (131.1, 47.6)
- moved R23 0.52 mm to (133.1, 46.1)
- moved R32 0.52 mm to (135.1, 59.0)
- moved D16 0.52 mm to (131.1, 62.6)
- moved R22 0.52 mm to (135.1, 44.0)
- moved R33 0.52 mm to (133.1, 61.0)
- moved R24 0.52 mm to (129.0, 49.1)
- moved R34 0.52 mm to (129.0, 64.1)
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Routing:
- net /HV+_Sense: track 29.4 -> 34.0 mm
- net /Fan Control/TACH4: track 14.8 -> 16.8 mm
- net +12V: track 52.7 -> 54.7 mm
- net /Array Contactor Driver/CONTACTOR_V-: track 10.9 -> 11.9 mm
- net /HV- Contactor Driver/CONTACTOR_V-: track 10.9 -> 11.9 mm
- net /HV+ Contactor Driver/CONTACTOR_V-: track 10.9 -> 11.9 mm
- net +3.3V: track 111.5 -> 112.5 mm
- net /Fan Control/TACH3: track 34.1 -> 34.7 mm
- net /Fan Control/TACH1: track 44.4 -> 44.9 mm

Commit message: clearance WOOHOOO
Routing:
- net +3.3V: track 112.5 -> 116.8 mm
Changed lines of the file:
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@@
   (segment (start 153.0298 52.6542) (end 152.4 53.284) (width 0.25) (layer "F.Cu") (net 15))
   (segment (start 134.112 77.978) (end 144.739 77.978) (width 1) (layer "F.Cu") (net 15))
+  (segment (start 160.95 89.62) (end 160.95 93.92) (width 0.25) (layer "F.Cu") (net 15))
   (segment (start 157.988 56.388) (end 152.842 56.388) (width 1) (layer "F.Cu") (net 15))
   (segment (start 152.4 53.284) (end 152.842 53.726) (width 0.25) (layer "F.Cu") (net 15))
@@
   (zone (net 1) (net_name "+12V") (layer "F.Cu") (hatch edge 0.5)
     (priority 2)
-    (connect_pads (clearance 0.5))
+    (connect_pads thru_hole_only (clearance 0.5))
     (min_thickness 0.25) (filled_areas_thickness no)
     (fill yes (thermal_gap 0.5) (thermal_bridge_width 0.5))
@@
   (zone (net 3) (net_name "GND") (layer "B.Cu") (hatch edge 0.5)
     (priority 2)
-    (connect_pads (clearance 0.5))
+    (connect_pads thru_hole_only (clearance 0.5))
     (min_thickness 0.25) (filled_areas_thickness no)
     (fill yes (thermal_gap 0.5) (thermal_bridge_width 0.5))

Commit message: fix ignition
Connections:
- J8 pad 3: GND -> GND1
Routing:
- net GND1: track 6.52 -> 12.6 mm
Changed lines of the file:
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@@
       (net 53 "Net-(J8-Pin_2)") (pinfunction "Pin_2") (pintype "passive"))
     (pad "3" thru_hole oval (at 6 0 180) (size 1.5 2.02) (drill 1.02) (layers "*.Cu" "*.Mask")
-      (net 3 "GND") (pinfunction "Pin_3") (pintype "passive"))
+      (net 63 "GND1") (pinfunction "Pin_3") (pintype "passive"))
     (model "${KICAD6_3DMODEL_DIR}/Connector_Molex.3dshapes/Molex_Micro-Fit_3.0_43650-0315_1x03_P3.00mm_Vertical.wrl"
       (offset (xyz 0 0 0))
@@
     (effects (font (size 1 1) (thickness 0.15)) (justify left bottom))
   )
-  (gr_text "Short for \n4 wire fan" (at 156.21 44.958) (layer "F.SilkS")
+  (gr_text "Short for \n4 wire fan" (at 156.21 44.704) (layer "F.SilkS")
     (effects (font (size 1 1) (thickness 0.15)) (justify left bottom))
   )
@@
   (segment (start 166.10425 88.7605) (end 166.10425 86.7645) (width 0.25) (layer "B.Cu") (net 51))
   (segment (start 166.10425 86.7645) (end 165.82675 86.487) (width 0.25) (layer "B.Cu") (net 51))
-  (segment (start 170.65275 86.487) (end 170.65275 84.0495) (width 1) (layer "B.Cu") (net 52))
-  (segment (start 170.65275 84.0495) (end 172.15225 82.55) (width 1) (layer "B.Cu") (net 52))
-  (segment (start 167.65175 84.0505) (end 169.15225 82.55) (width 1) (layer "B.Cu") (net 53))
-  (segment (start 167.65175 86.487) (end 167.65175 84.0505) (width 1) (layer "B.Cu") (net 53))
+  (segment (start 172.15225 82.55) (end 172.15225 84.9875) (width 0.25) (layer "B.Cu") (net 52))
+  (segment (start 172.15225 84.9875) (end 170.65275 86.487) (width 0.25) (layer "B.Cu") (net 52))
+  (segment (start 169.15225 84.9865) (end 167.65175 86.487) (width 0.25) (layer "B.Cu") (net 53))
+  (segment (start 169.15225 82.55) (end 169.15225 84.9865) (width 0.25) (layer "B.Cu") (net 53))
   (segment (start 174.851281 45.366719) (end 174.851281 43.263463) (width 2) (layer "B.Cu") (net 54))
   (segment (start 174.126 47.870818) (end 174.126 46.092) (width 2) (layer "B.Cu") (net 54))
@@
   (segment (start 174.126 61.078) (end 174.851281 60.352719) (width 2) (layer "B.Cu") (net 56))
   (segment (start 174.851281 58.249463) (end 172.22689 55.625072) (width 2) (layer "B.Cu") (net 56))
-  (segment (start 172.20025 89.505082) (end 172.20025 88.7605) (width 1) (layer "B.Cu") (net 63))
-  (segment (start 171.432332 90.273) (end 172.20025 89.505082) (width 1) (layer "B.Cu") (net 63))
-  (segment (start 168.88675 90.273) (end 171.432332 90.273) (width 1) (layer "B.Cu") (net 63))
-  (segment (start 167.37425 88.7605) (end 168.88675 90.273) (width 1) (layer "B.Cu") (net 63))
+  (segment (start 167.37425 88.7605) (end 168.51175 89.898) (width 0.25) (layer "B.Cu") (net 63))
+  (segment (start 166.15225 82.55) (end 166.66425 83.062) (width 0.25) (layer "B.Cu") (net 63))
+  (segment (start 166.66425 87.67025) (end 167.37425 88.38025) (width 0.25) (layer "B.Cu") (net 63))
+  (segment (start 167.37425 88.38025) (end 167.37425 88.7605) (width 0.25) (layer "B.Cu") (net 63))
+  (segment (start 171.281158 89.898) (end 172.20025 88.978908) (width 0.25) (layer "B.Cu") (net 63))
+  (segment (start 166.66425 83.062) (end 166.66425 87.67025) (width 0.25) (layer "B.Cu") (net 63))
+  (segment (start 172.20025 88.978908) (end 172.20025 88.7605) (width 0.25) (layer "B.Cu") (net 63))
+  (segment (start 168.51175 89.898) (end 171.281158 89.898) (width 0.25) (layer "B.Cu") (net 63))
   (zone (net 15) (net_name "+3.3V") (layer "F.Cu") (hatch edge 0.5)
     (connect_pads (clearance 0.5))
@@
     (members
       08d72c95-7431-4f9d-a9a0-300bdd637d84
-      1dec5c28-2197-461d-a009-2770957e8ab4
-      31906bf2-3bb6-4815-a195-1cac88bc277c
       3a20bc03-fb63-4e1b-8c9d-53d70b80404e
       3e679f9b-2ad5-4507-81b8-b2acdc014c94
-      3ed813bf-92eb-4064-972d-369c654e3fca
       4249f035-cf5a-4919-8ec5-e40993e8eb12
       4f1e0587-57cb-4540-ac2f-816e51325a02
-      586a0d2a-d866-496a-a06f-503d43d8bdaa
       5bb532c5-35ec-46a5-a8f5-ad8f72477daf
       67459f1c-2816-4b14-96d6-d75e28554baf
-      73341c24-b374-48c1-8e74-39f687a00c91
+      6b849cf5-3e28-4375-9e33-35e0567a38a7
       7398a944-a892-4efd-ac09-75dab8717db2
-      88ad8560-f5c3-408b-8299-13783c2cad38
-      926ece64-d53a-4fb1-88eb-373f407035ae
       927464bb-42d6-4745-9785-2936f5985c27
       9be2a224-f9f8-4c88-8e8d-35d614630824
-      b1a94acc-44f5-4685-8733-b11e5bc62d5e
       bc7ecdfc-b7c5-4bd4-b454-a410898fab4a
       cb6411a1-5c92-43ca-8027-6a64e5561a56
+      d859fcb5-4079-433a-81f5-378352fdca06
       dbb4f5ea-0255-4092-990a-3cb9f686f362
-      e2e17b12-760d-4f70-89f9-8ced827c288e
-      fdb77cd3-22d2-478d-b621-787d317e1a99
     )
   )

Commit message: Island vacationgit add . !
Routing:
- net +12V: track 54.7 -> 82.6 mm
- net /Fan Control/ORION_PWM: track 26.6 -> 24.0 mm
- net /Fan Control/PWM1: track 51.2 -> 50.5 mm
- net /Fan Control/TACH1: track 44.9 -> 45.6 mm
- net GND: track 31.9 -> 31.8 mm, vias 7 -> 9
- added copper zone on F.Cu, net GND
