File: Strobe_Light.kicad_sch (KiCad schematic)
At the start: 15 parts, among them J4 ErrorLightConn, Q1 NTR4003NT1G, Q2 VND5N07-E, U1 SI8261ABC-IS

Commit message: Standardized strobe liight
Parts:
- C2: P/N (none) -> 0805YC106KAT2A
- J4: P/N (none) -> 43650-0227
- Q1: P/N (none) -> NTR4003NT1G
- Q2: P/N (none) -> VND5N07-E
- R1, R5: P/N (none) -> CRCW08050000Z0EAC
- R2, R6: P/N (none) -> CRCW080510K0FKEAC
- TP1: Mouser Part Number (none) -> 534-5005; P/N (none) -> 5005
- U1: Mouser Part Number (none) -> 634-SI8261AAC-C-ISR; P/N (none) -> SI8261AAC-C-ISR
Changed lines of the file:
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@@
       (effects (font (size 1.27 1.27)) hide)
     )
-    (property "Datasheet" "~" (at 200.025 80.01 0)
+    (property "Datasheet" "https://www.mouser.com/datasheet/2/276/0436500227_PCB_HEADERS-168471.pdf" (at 200.025 80.01 0)
+      (effects (font (size 1.27 1.27)) hide)
+    )
+    (property "P/N" "43650-0227" (at 200.025 80.01 0)
       (effects (font (size 1.27 1.27)) hide)
     )
@@
   (symbol (lib_id "Device:R") (at 97.155 104.14 270) (unit 1)
     (in_bom yes) (on_board yes) (dnp no)
-    (property "Reference" "R1" (at 97.155 101.6 90)
-      (effects (font (size 1.27 1.27)))
-    )
-    (property "Value" "0" (at 97.155 104.14 90)
+    (property "Reference" "R1" (at 97.155 97.79 90)
+      (effects (font (size 1.27 1.27)))
+    )
+    (property "Value" "0" (at 97.155 100.33 90)
       (effects (font (size 1.27 1.27)))
     )
@@
       (effects (font (size 1.27 1.27)) hide)
     )
-    (property "Datasheet" "~" (at 97.155 104.14 0)
+    (property "Datasheet" "https://www.vishay.com/docs/28773/crcwce3.pdf" (at 97.155 104.14 0)
+      (effects (font (size 1.27 1.27)) hide)
+    )
+    (property "P/N" "CRCW08050000Z0EAC" (at 97.155 104.14 90)
       (effects (font (size 1.27 1.27)) hide)
     )
@@
       (effects (font (size 1.27 1.27)) hide)
     )
-    (property "Datasheet" "~" (at 116.205 82.55 0)
+    (property "Datasheet" "https://www.mouser.com/datasheet/2/216/APTD2012LSURCK-1101937.pdf" (at 116.205 82.55 0)
       (effects (font (size 1.27 1.27)) hide)
     )
@@
       (effects (font (size 1.27 1.27)) hide)
     )
-    (property "Datasheet" "~" (at 189.865 93.98 0)
+    (property "Datasheet" "https://www.mouser.com/datasheet/2/389/vnd5n07_e-1852681.pdf" (at 189.865 93.98 0)
+      (effects (font (size 1.27 1.27)) hide)
+    )
+    (property "P/N" "VND5N07-E" (at 189.865 93.98 0)
       (effects (font (size 1.27 1.27)) hide)
     )
@@
       (effects (font (size 1.27 1.27)))
     )
-    (property "Value" "470" (at 126.365 86.36 90)
+    (property "Value" "470" (at 130.81 86.995 0)
       (effects (font (size 1.27 1.27)))
     )
@@
       (effects (font (size 1.27 1.27)) hide)
     )
-    (property "Datasheet" "~" (at 113.665 104.14 0)
+    (property "Datasheet" "https://www.mouser.com/datasheet/2/308/1/NTR4003N_D-2319203.pdf" (at 113.665 104.14 0)
+      (effects (font (size 1.27 1.27)) hide)
+    )
+    (property "P/N" "NTR4003NT1G" (at 113.665 104.14 0)
       (effects (font (size 1.27 1.27)) hide)
     )
@@
       (effects (font (size 1.27 1.27)) hide)
     )
-    (property "Datasheet" "~" (at 175.895 93.98 0)
+    (property "Datasheet" "https://www.vishay.com/docs/28773/crcwce3.pdf" (at 175.895 93.98 0)
+      (effects (font (size 1.27 1.27)) hide)
+    )
+    (property "P/N" "CRCW08050000Z0EAC" (at 175.895 93.98 0)
       (effects (font (size 1.27 1.27)) hide)
     )
@@
       (effects (font (size 1.27 1.27)) (justify left))
     )
-    (property "Value" "10k" (at 104.775 111.76 90)
+    (property "Value" "10k" (at 106.68 111.125 0)
       (effects (font (size 1.27 1.27)) (justify left))
     )
@@
       (effects (font (size 1.27 1.27)) hide)
     )
-    (property "Datasheet" "~" (at 104.775 109.22 0)
+    (property "Datasheet" "https://www.vishay.com/docs/28773/crcwce3.pdf" (at 104.775 109.22 0)
+      (effects (font (size 1.27 1.27)) hide)
+    )
+    (property "P/N" "CRCW080510K0FKEAC" (at 104.775 109.22 0)
       (effects (font (size 1.27 1.27)) hide)
     )
@@
       (effects (font (size 1.27 1.27)) hide)
     )
-    (property "Datasheet" "~" (at 182.245 68.58 0)
+    (property "Datasheet" "https://www.mouser.com/datasheet/2/40/AVX_X7RDielectric_777024-1853642.pdf" (at 182.245 68.58 0)
+      (effects (font (size 1.27 1.27)) hide)
+    )
+    (property "P/N" "0805YC106KAT2A" (at 182.245 68.58 0)
       (effects (font (size 1.27 1.27)) hide)
     )
@@
       (effects (font (size 1.27 1.27)) hide)
     )
-    (property "Datasheet" "https://www.silabs.com/documents/public/data-sheets/Si826x.pdf" (at 146.685 86.36 0)
+    (property "Datasheet" "https://www.mouser.com/datasheet/2/472/Si826x-2507538.pdf" (at 146.685 86.36 0)
+      (effects (font (size 1.27 1.27)) hide)
+    )
+    (property "P/N" "SI8261AAC-C-ISR" (at 146.685 86.36 0)
+      (effects (font (size 1.27 1.27)) hide)
+    )
+    (property "Mouser Part Number" "634-SI8261AAC-C-ISR" (at 146.685 86.36 0)
       (effects (font (size 1.27 1.27)) hide)
     )
@@
       (effects (font (size 1.27 1.27)) hide)
     )
-    (property "Datasheet" "~" (at 172.085 90.17 0)
+    (property "Datasheet" "https://www.mouser.com/datasheet/2/215/5005_5009-741322.pdf" (at 172.085 90.17 0)
+      (effects (font (size 1.27 1.27)) hide)
+    )
+    (property "Mouser Part Number" "534-5005" (at 167.005 90.17 0)
+      (effects (font (size 1.27 1.27)) hide)
+    )
+    (property "P/N" "5005" (at 167.005 90.17 0)
       (effects (font (size 1.27 1.27)) hide)
     )
@@
       (effects (font (size 1.27 1.27)) (justify left))
     )
-    (property "Value" "10k" (at 182.245 102.87 90)
+    (property "Value" "10k" (at 183.515 102.235 0)
       (effects (font (size 1.27 1.27)) (justify left))
     )
@@
       (effects (font (size 1.27 1.27)) hide)
     )
-    (property "Datasheet" "~" (at 182.245 100.33 0)
+    (property "Datasheet" "https://www.vishay.com/docs/28773/crcwce3.pdf" (at 182.245 100.33 0)
+      (effects (font (size 1.27 1.27)) hide)
+    )
+    (property "P/N" "CRCW080510K0FKEAC" (at 182.245 100.33 0)
       (effects (font (size 1.27 1.27)) hide)
     )
@@
       (effects (font (size 1.27 1.27)) (justify left))
     )
-    (property "Value" "1.6k" (at 116.205 93.98 90)
-      (effects (font (size 1.27 1.27)) (justify left))
-    )
+    (property "Value" "1.6k" (at 118.11 92.075 0)
+      (effects (font (size 1.27 1.27)) (justify left))
+    )

Commit message: Added part numbers for Contactors and Strobe light
Parts:
- removed C1: 0.1u, Capacitor_SMD:C_0805_2012Metric, symbol Device:C
- removed C3: 1u, Capacitor_SMD:C_0805_2012Metric, symbol Device:C
- removed R3: 1.6k, Resistor_SMD:R_0805_2012Metric, symbol Device:R
- removed R4: 470, Resistor_SMD:R_0805_2012Metric, symbol Device:R
- added C4: 100nF, Capacitor_SMD:C_0805_2012Metric, symbol Device:C_Small
- added C7: 1u, Capacitor_SMD:C_0805_2012Metric, symbol Device:C
- added R21: 1.5k, Resistor_SMD:R_0805_2012Metric, symbol Device:R
- added R22: 470, Resistor_SMD:R_0805_2012Metric, symbol Device:R
Connections:
- net +12V: now also C4.1, C7.1
- net +5V: now also R22.2
- net GNDPWR: now also C4.2, C7.2
- net at D1.1 (K): now also R21.1
- net at U1.2 (ANODE): now also R22.1
- net at Q1.3 (D), U1.3 (CATHODE): now also R21.2

Commit message: Finished comments for Strobe Light and started resolving them for Contactor
Parts:
- removed C2: 10u, Capacitor_SMD:C_0805_2012Metric, symbol Device:C
- removed C4: 100nF, Capacitor_SMD:C_0805_2012Metric, symbol Device:C_Small
- removed D1: Fault, LED_SMD:LED_0805_2012Metric, symbol Device:D
- removed Q1: NTR4003NT1G, Package_TO_SOT_SMD:SOT-23, symbol Device:Q_NMOS_GSD
- removed R2, R6: 10k, Resistor_SMD:R_0805_2012Metric, symbol Device:R
- removed R21: 1.5k, Resistor_SMD:R_0805_2012Metric, symbol Device:R
- removed R22: 470, Resistor_SMD:R_0805_2012Metric, symbol Device:R
- removed R5: 0, Resistor_SMD:R_0805_2012Metric, symbol Device:R
- removed TP1: StrobeLightGate_TP, TestPoint:TestPoint_Keystone_5005-5009_Compact, symbol Connector:TestPoint
- added C16: 100nF, Capacitor_SMD:C_0805_2012Metric, symbol Device:C_Small
- added C17: 10uF, Capacitor_SMD:C_0805_2012Metric, symbol Device:C_Small
- added D1: LED, LED_SMD:LED_0805_2012Metric, symbol Device:LED
- added R23: R, symbol Device:R
- added R28: 100k, Resistor_SMD:R_0805_2012Metric, symbol Device:R
- R1: value 0 -> 1k; Mouser Part Number (none) -> 71-CRCW08051K00FKEAC; P/N CRCW08050000Z0EAC -> CRCW08051K00FKEAC
Connections:
- net +12V: now also C16.1, C17.1; no longer J4.1 (Pin_1)
- net FAULT: now also R23.1; no longer R1.2
- net GND: now also U1.3 (CATHODE)
- net GNDPWR: now also C16.2, C17.2, D1.1 (K), R28.2; no longer C7.2
- net at R1.1: now also Q2.1 (G), U1.6 (VO), U1.7 (VO), R28.1
- net at U1.2 (ANODE): now also R23.2
- new net: C7.2, J4.1 (Pin_1)
- new net: D1.2 (A), R1.2
Other:
- note removed: "Extra transistor interface present because the Si8261 Isolator requires 6mA to turn but we wanted an LED indicator on the board to tell us the Contactor is on. The max current output of an STM32 pin is 8mA and adding a LED in parallel will exceed the max."
- note removed: "Local (Leader Board) GND (Internal)"
- note removed: "Please check footprint and symbol matches! 1: G 2: D 3: S"
- note removed: "Power GND (External)"

Commit message: added no connects to Ignition switch and removed redundant Strobe coupling cap
Parts:
- removed C7: 1u, Capacitor_SMD:C_0805_2012Metric, symbol Device:C
- R23: value R -> 1k
Connections:
- net +12V: now also J4.1 (Pin_1)
Changed lines of the file:
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@@
-    (stroke (width 0) (type default))
-  )
-  (wire (pts (xy 196.85 78.105) (xy 196.85 80.645))
     (stroke (width 0) (type default))
   )
@@
     (stroke (width 0) (type default))
   )
-  (wire (pts (xy 196.85 88.265) (xy 196.85 88.9))
+  (wire (pts (xy 196.85 78.105) (xy 196.85 88.9))
     (stroke (width 0) (type default))
   )
@@
         (path "/c248b171-df31-4e8a-afb6-607fa2df334b/00000000-0000-0000-0000-00005d923d59"
           (reference "Q4") (unit 1)
-        )
-      )
-    )
-  )
-  (symbol (lib_id "Device:C") (at 196.85 84.455 0) (unit 1)
-    (in_bom yes) (on_board yes) (dnp no)
-    (property "Reference" "C7" (at 201.295 83.185 0)
-      (effects (font (size 1.27 1.27)))
-    )
-    (property "Value" "1u" (at 201.295 85.725 0)
-      (effects (font (size 1.27 1.27)))
-    )
-    (property "Footprint" "Capacitor_SMD:C_0805_2012Metric" (at 197.8152 88.265 0)
-      (effects (font (size 1.27 1.27)) hide)
-    )
-    (property "Datasheet" "https://www.mouser.com/datasheet/2/447/KEM_C1006_X5R_SMD-3316465.pdf" (at 196.85 84.455 0)
-      (effects (font (size 1.27 1.27)) hide)
-    )
-    (property "P/N" "C0805C105K5PACTU" (at 196.85 84.455 0)
-      (effects (font (size 1.27 1.27)) hide)
-    )
-    (pin "1")
-    (pin "2")
-    (instances
-      (project "BPS-LeaderDaughter"
-        (path "/2e9f4f51-d216-4952-a31c-e7104e0d4b1e/ae57cd3a-fadb-4313-835a-95d5b185a797"
-          (reference "C7") (unit 1)
-        )
-        (path "/2e9f4f51-d216-4952-a31c-e7104e0d4b1e/5e4c6ec4-73d4-4ed3-a75f-02eb4f9ac8b3"
-          (reference "C12") (unit 1)
-        )
-        (path "/2e9f4f51-d216-4952-a31c-e7104e0d4b1e/bb673292-4a5d-469b-b6b6-0dc7df3c162d"
-          (reference "C17") (unit 1)
-        )
-        (path "/2e9f4f51-d216-4952-a31c-e7104e0d4b1e/55cfe956-9550-49f5-88d2-e32c6d523ac3"
-          (reference "C4") (unit 1)
-        )
-      )
-      (project "BPS-Leader"
-        (path "/c248b171-df31-4e8a-afb6-607fa2df334b/00000000-0000-0000-0000-00005c38c674"
-          (reference "C22") (unit 1)
-        )
-        (path "/c248b171-df31-4e8a-afb6-607fa2df334b/3faa4167-9e5e-4372-9a55-3c963a25ae73"
-          (reference "C46") (unit 1)
-        )
-        (path "/c248b171-df31-4e8a-afb6-607fa2df334b/bb594d23-7f65-4f42-8951-e176f5e7b2cb"
-          (reference "C46") (unit 1)
         )
       )
@@
   (symbol (lib_id "Device:R") (at 123.825 95.885 90) (unit 1)
     (in_bom yes) (on_board yes) (dnp no) (fields_autoplaced)
-    (property "Reference" "R23" (at 123.825 89.535 90)
-      (effects (font (size 1.27 1.27)))
-    )
-    (property "Value" "R" (at 123.825 92.075 90)
-      (effects (font (size 1.27 1.27)))
-    )
+    (property "Reference" "R23" (at 123.825 90.17 90)
+      (effects (font (size 1.27 1.27)))
+    )
+    (property "Value" "1k" (at 123.825 92.71 90)
+      (effects (font (size 1.27 1.27)))
+    )

Commit message: Started adding changes from review
Parts:
- removed Q2: VND5N07-E, Package_TO_SOT_SMD:TO-252-2, symbol Device:Q_NMOS_GDS
- added Q?: BUK9M23-80E, Package_TO_SOT_SMD:LFPAK33, symbol Transistor_FET:BUK9M23-80EX
Connections:
- net GNDPWR: now also Q?.1 (S), Q?.2 (S), Q?.3 (S)
- net at R1.1, R28.1, U1.6 (VO)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: now also Q?.4 (G)
- net at J4.2 (Pin_2): now also Q?.5 (D)
Changed lines of the file:
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@@
-    )
-  )
-  (symbol (lib_id "Device:Q_NMOS_GDS") (at 196.215 98.425 0) (unit 1)
-    (in_bom yes) (on_board yes) (dnp no)
-    (property "Reference" "Q2" (at 201.422 97.2566 0)
-      (effects (font (size 1.27 1.27)) (justify left))
-    )
-    (property "Value" "VND5N07-E" (at 201.422 99.568 0)
-      (effects (font (size 1.27 1.27)) (justify left))
-    )
-    (property "Footprint" "Package_TO_SOT_SMD:TO-252-2" (at 201.295 95.885 0)
-      (effects (font (size 1.27 1.27)) hide)
-    )
-    (property "Datasheet" "https://www.mouser.com/datasheet/2/389/vnd5n07_e-1852681.pdf" (at 196.215 98.425 0)
-      (effects (font (size 1.27 1.27)) hide)
-    )
-    (property "P/N" "VND5N07-E" (at 196.215 98.425 0)
-      (effects (font (size 1.27 1.27)) hide)
-    )
-    (pin "1")
-    (pin "2")
-    (pin "3")
-    (instances
-      (project "BPS-LeaderDaughter"
-        (path "/2e9f4f51-d216-4952-a31c-e7104e0d4b1e"
-          (reference "Q2") (unit 1)
-        )
-        (path "/2e9f4f51-d216-4952-a31c-e7104e0d4b1e/55cfe956-9550-49f5-88d2-e32c6d523ac3"
-          (reference "Q7") (unit 1)
-        )
-      )
-      (project "BPS-Leader"
-        (path "/c248b171-df31-4e8a-afb6-607fa2df334b/00000000-0000-0000-0000-00005d923d59"
-          (reference "Q4") (unit 1)
-        )
-      )
     )
   )
@@
         )
       )
+    )
+  )
+  (symbol (lib_id "Transistor_FET:BUK9M23-80EX") (at 196.215 98.425 0) (unit 1)
+    (in_bom yes) (on_board yes) (dnp no) (fields_autoplaced)
+    (property "Reference" "Q?" (at 202.565 97.155 0)
+      (effects (font (size 1.27 1.27)) (justify left))
+    )
+    (property "Value" "BUK9M23-80E" (at 202.565 99.695 0)
+      (effects (font (size 1.27 1.27)) (justify left))
+    )
+    (property "Footprint" "Package_TO_SOT_SMD:LFPAK33" (at 201.295 100.33 0)
+      (effects (font (size 1.27 1.27) italic) (justify left) hide)
+    )
+    (property "Datasheet" "https://assets.nexperia.com/documents/data-sheet/BUK9M23-80E.pdf" (at 196.215 98.425 90)
+      (effects (font (size 1.27 1.27)) (justify left) hide)
+    )
+    (property "P/N" "BUK9M23-80E" (at 196.215 98.425 0)
+      (effects (font (size 1.27 1.27)) hide)
+    )
+    (pin "1")
+    (pin "2")
+    (pin "3")
+    (pin "4")
+    (pin "5")
+    (instances
+      (project "BPS-LeaderDaughter"
+        (path "/2e9f4f51-d216-4952-a31c-e7104e0d4b1e/bf23a663-b938-440b-843e-ef7912c82d18"
+          (reference "Q?") (unit 1)
+        )
+        (path "/2e9f4f51-d216-4952-a31c-e7104e0d4b1e/bf23a663-b938-440b-843e-ef7912c82d18/cb70587e-88a7-4e34-a774-2566ee5ba031"
+          (reference "Q5") (unit 1)
+        )
+        (path "/2e9f4f51-d216-4952-a31c-e7104e0d4b1e/bf23a663-b938-440b-843e-ef7912c82d18/726bf2a6-1244-4795-8327-149588380c7e"
+          (reference "Q6") (unit 1)
+        )
+        (path "/2e9f4f51-d216-4952-a31c-e7104e0d4b1e/bf23a663-b938-440b-843e-ef7912c82d18/66fa18d5-534c-477b-b6ed-b26c28a08707"
+          (reference "Q7") (unit 1)
+        )
+        (path "/2e9f4f51-d216-4952-a31c-e7104e0d4b1e/bf23a663-b938-440b-843e-ef7912c82d18/3bf7416b-1505-491f-89b6-6e99a8c04638"
+          (reference "Q8") (unit 1)
+        )
+        (path "/2e9f4f51-d216-4952-a31c-e7104e0d4b1e/55cfe956-9550-49f5-88d2-e32c6d523ac3"
+          (reference "Q3") (unit 1)
+        )
+      )

Commit message: Fan layout updated
Parts:
- R2: renamed from R23; footprint (none) -> Resistor_SMD:R_0805_2012Metric
Changed lines of the file:
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@@
         )
         (path "/2e9f4f51-d216-4952-a31c-e7104e0d4b1e/55cfe956-9550-49f5-88d2-e32c6d523ac3"
-          (reference "#PWR05") (unit 1)
+          (reference "#PWR0101") (unit 1)
         )
       )
@@
         )
         (path "/2e9f4f51-d216-4952-a31c-e7104e0d4b1e/55cfe956-9550-49f5-88d2-e32c6d523ac3"
-          (reference "R24") (unit 1)
+          (reference "R4") (unit 1)
         )
       )
@@
   (symbol (lib_id "Device:R") (at 123.825 95.885 90) (unit 1)
     (in_bom yes) (on_board yes) (dnp no) (fields_autoplaced)
-    (property "Reference" "R23" (at 123.825 90.17 90)
+    (property "Reference" "R2" (at 123.825 90.17 90)
       (effects (font (size 1.27 1.27)))
     )
@@
       (effects (font (size 1.27 1.27)))
     )
-    (property "Footprint" "" (at 123.825 97.663 90)
+    (property "Footprint" "Resistor_SMD:R_0805_2012Metric" (at 123.825 97.663 90)
       (effects (font (size 1.27 1.27)) hide)
     )
@@
       (project "BPS-LeaderDaughter"
         (path "/2e9f4f51-d216-4952-a31c-e7104e0d4b1e/55cfe956-9550-49f5-88d2-e32c6d523ac3"
-          (reference "R23") (unit 1)
-        )
-      )
+          (reference "R2") (unit 1)
+        )
+      )

Commit message: Fixed current limiting LEDs on the Optoisolator and FAN jumpers
Parts:
- removed D1: LED, LED_SMD:LED_0805_2012Metric, symbol Device:LED
- removed R1: 1k, Resistor_SMD:R_0805_2012Metric, symbol Device:R
- added D25: Green, LED_SMD:LED_0805_2012Metric_Pad1.15x1.40mm_HandSolder, symbol Device:LED_Small
- added R7: 10k, Resistor_SMD:R_0805_2012Metric, symbol Device:R
- R2: value 1k -> 80.6
Connections:
- net GNDPWR is gone; now on net GND: C16.2, C17.2, Q?.1 (S), Q?.2 (S), Q?.3 (S), R28.2, U1.5 (GND)
- net +12V: now also R7.1
- net at J4.2 (Pin_2), Q?.5 (D): now also D25.1 (K)
- new net: D25.2 (A), R7.2
Other:
- moved on the sheet: J4, Q?
