File: Strobe_Light.kicad_sch (KiCad schematic)
At the start: 6 parts, among them J4 ErrorLightConn

Commit message: Fixed LeaderSOM connections, strobe, ignition, and contactor layout
Connections:
- net Strobe_-: now reaches D25.1 (K), J4.2 (Pin_2), Q?.5 (D)
Changed lines of the file:
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@@
   (junction (at 104.775 82.55) (diameter 0) (color 0 0 0 0)
+  )
+  (junction (at 113.665 76.835) (diameter 0) (color 0 0 0 0)
   )
   (junction (at 111.76 59.69) (diameter 0) (color 0 0 0 0)
@@
   )
   (wire (pts (xy 103.505 67.31) (xy 103.505 69.215))
+    (stroke (width 0) (type default))
+  )
+  (wire (pts (xy 113.665 76.835) (xy 116.84 76.835))
     (stroke (width 0) (type default))
   )
@@
     (stroke (width 0) (type default))
   )
-  (wire (pts (xy 113.665 75.565) (xy 113.665 77.47))
+  (wire (pts (xy 113.665 75.565) (xy 113.665 76.835))
     (stroke (width 0) (type default))
   )
@@
   )
   (wire (pts (xy 109.855 93.345) (xy 113.665 93.345))
+    (stroke (width 0) (type default))
+  )
+  (wire (pts (xy 113.665 76.835) (xy 113.665 77.47))
     (stroke (width 0) (type default))
   )
@@
     (effects (font (size 2.54 2.54) (thickness 0.508) bold) (justify left bottom))
   )
+  (label "Strobe_-" (at 116.84 76.835 0) (fields_autoplaced)
+    (effects (font (size 1.27 1.27)) (justify left bottom))
+  )
   (hierarchical_label "FAULT" (shape input) (at 90.17 82.55 180) (fields_autoplaced)

Commit message: last sanity check + part numbers (ready for review)
Parts:
- R4: P/N (none) -> CRCW08051K00FKEAC; P/n RCC080549R9FKEA -> (none)
- R7: P/N (none) -> RT0603FRE0710KL
Changed lines of the file:
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@@
       (effects (font (size 1.27 1.27)) hide)
     )
-    (property "P/n" "RCC080549R9FKEA " (at 96.52 82.55 90)
+    (property "P/n" "" (at 96.52 82.55 90)
+      (effects (font (size 1.27 1.27)) hide)
+    )
+    (property "P/N" "CRCW08051K00FKEAC" (at 96.52 82.55 0)
       (effects (font (size 1.27 1.27)) hide)
     )
@@
       (effects (font (size 1.27 1.27)) hide)
     )
+    (property "P/N" "RT0603FRE0710KL " (at 103.505 63.5 0)
+      (effects (font (size 1.27 1.27)) hide)
+    )

Commit message: BOM complete
Parts:
- J4: P/N 43650-0227 -> 43650-0215
- R7: P/N RT0603FRE0710KL -> CRCW080510K0FKEAC
Changed lines of the file:
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@@
       (effects (font (size 1.27 1.27)) hide)
     )
-    (property "P/N" "43650-0227" (at 119.38 69.85 0)
+    (property "P/N" "43650-0215" (at 119.38 69.85 0)
       (effects (font (size 1.27 1.27)) hide)
     )
@@
       (effects (font (size 1.27 1.27)) hide)
     )
-    (property "P/N" "RT0603FRE0710KL " (at 103.505 63.5 0)
+    (property "P/N" "CRCW080510K0FKEAC" (at 103.505 63.5 0)
       (effects (font (size 1.27 1.27)) hide)
     )

Commit message: bom + gerbers
Parts:
- D25: P/N LHR971-KN1 -> APTD2012LCGCK
Changed lines of the file:
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@@
       (effects (font (size 1.27 1.27)) hide)
     )
-    (property "P/N" "LHR971-KN1" (at 103.505 71.755 0)
+    (property "P/N" "APTD2012LCGCK" (at 103.505 71.755 0)
       (effects (font (size 1.27 1.27)) hide)
     )
