File: Fan_Tach.kicad_sch (KiCad schematic)
At the start: 4 parts

Commit message: Fan layout on pcb. need to figure out IC
Parts:
- renumbered D25 to D?, R47 to R?, R46 to R?, R45 to R?

Commit message: Made ignition connector 3 pin + fixed tach resistors
Parts:
- R?: value 100k -> 10k
Other:
- note added: "2 V < VPULL-UP × R13/(RPULL-UP + R14 + R13) < 5 V"
Changed lines of the file:
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@@
     (stroke (width 0) (type default))
+  )
+  (text "2 V < VPULL-UP × R13/(RPULL-UP + R14 + R13) < 5 V" (at 113.665 112.395 0)
+    (effects (font (size 1.27 1.27)) (justify left bottom))
   )
   (hierarchical_label "TACH" (shape input) (at 123.19 80.01 180) (fields_autoplaced)
@@
       (effects (font (size 1.27 1.27)) (justify left))
     )
-    (property "Value" "100k" (at 160.02 73.66 0)
+    (property "Value" "10k" (at 160.02 73.66 0)
       (effects (font (size 1.27 1.27)) (justify left))
     )
@@
       (effects (font (size 1.27 1.27)) hide)
     )
-    (property "Datasheet" "https://www.mouser.com/ProductDetail/603-RT0603FRE0710KL" (at 157.48 72.39 0)
+    (property "Datasheet" "~" (at 157.48 72.39 0)
       (effects (font (size 1.27 1.27)) hide)
     )
@@
       (effects (font (size 1.27 1.27)) hide)
     )
-    (property "Datasheet" "https://www.mouser.com/ProductDetail/603-RT0603FRE0710KL" (at 148.59 80.01 0)
+    (property "Datasheet" "~" (at 148.59 80.01 0)
       (effects (font (size 1.27 1.27)) hide)
     )
@@
       (effects (font (size 1.27 1.27)) hide)
     )
-    (property "Datasheet" "https://www.mouser.com/datasheet/2/308/1/MM3Z2V4T1_D-2316321.pdf" (at 129.54 87.63 0)
+    (property "Datasheet" "~" (at 129.54 87.63 0)
       (effects (font (size 1.27 1.27)) hide)
     )
@@
       (effects (font (size 1.27 1.27)) hide)
     )
-    (property "Datasheet" "https://www.mouser.com/ProductDetail/603-RT0603FRE074K7L" (at 139.7 87.63 0)
+    (property "Datasheet" "~" (at 139.7 87.63 0)
       (effects (font (size 1.27 1.27)) hide)
     )

Commit message: forgor to save Fan tach
Parts:
- R?: value 10k -> 20k
- R?: value 4.7k -> 10k
Changed lines of the file:
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@@
       (effects (font (size 1.27 1.27)))
     )
-    (property "Value" "10k" (at 148.59 76.2 90)
+    (property "Value" "20k" (at 148.59 76.2 90)
       (effects (font (size 1.27 1.27)))
     )
@@
       (effects (font (size 1.27 1.27)) (justify left))
     )
-    (property "Value" "4.7k" (at 142.24 88.9 0)
+    (property "Value" "10k" (at 142.24 88.9 0)
       (effects (font (size 1.27 1.27)) (justify left))
     )
