File: Fan_PWM.kicad_sch (KiCad schematic)
At the start: 3 parts, among them Q6 BUK9M23-80E

Commit message: Fan layout on pcb. need to figure out IC
Parts:
- renumbered Q6 to Q?, R41 to R?, R10 to R?
Connections:
- net ORION_PWM renamed PWM_IN

Commit message: Fan layout updated
Parts:
- added D2: 1N4148WS, Diode_SMD:D_SOD-323F, symbol Diode:1N4148
Connections:
- net +12V: now also D2.1 (K)
- net PWM_OUT: now also D2.2 (A)
Changed lines of the file:
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@@
   (junction (at 104.14 54.61) (diameter 0) (color 0 0 0 0)
   )
+  (junction (at 125.73 54.61) (diameter 0) (color 0 0 0 0)
+  )
+  (junction (at 115.57 39.37) (diameter 0) (color 0 0 0 0)
+  )
+  (wire (pts (xy 125.73 54.61) (xy 133.35 54.61))
+    (stroke (width 0) (type default))
+  )
   (wire (pts (xy 86.36 59.69) (xy 86.36 49.53))
     (stroke (width 0) (type default))
@@
     (stroke (width 0) (type default))
   )
+  (wire (pts (xy 125.73 49.53) (xy 125.73 54.61))
+    (stroke (width 0) (type default))
+  )
+  (wire (pts (xy 125.73 41.91) (xy 125.73 39.37))
+    (stroke (width 0) (type default))
+  )
+  (wire (pts (xy 115.57 39.37) (xy 104.14 39.37))
+    (stroke (width 0) (type default))
+  )
   (wire (pts (xy 93.98 54.61) (xy 104.14 54.61))
     (stroke (width 0) (type default))
@@
     (stroke (width 0) (type default))
   )
-  (wire (pts (xy 104.14 41.91) (xy 104.14 36.83))
+  (wire (pts (xy 104.14 41.91) (xy 104.14 39.37))
+    (stroke (width 0) (type default))
+  )
+  (wire (pts (xy 125.73 39.37) (xy 115.57 39.37))
     (stroke (width 0) (type default))
   )
@@
     (stroke (width 0) (type default))
   )
-  (wire (pts (xy 104.14 54.61) (xy 111.76 54.61))
-    (stroke (width 0) (type default))
-  )
-  (hierarchical_label "PWM_OUT" (shape input) (at 111.76 54.61 0) (fields_autoplaced)
+  (wire (pts (xy 115.57 39.37) (xy 115.57 36.83))
+    (stroke (width 0) (type default))
+  )
+  (wire (pts (xy 104.14 54.61) (xy 125.73 54.61))
+    (stroke (width 0) (type default))
+  )
+  (hierarchical_label "PWM_OUT" (shape input) (at 133.35 54.61 0) (fields_autoplaced)
     (effects (font (size 1.27 1.27)) (justify left))
   )
@@
     )
   )
-  (symbol (lib_id "power:+12V") (at 104.14 36.83 0) (unit 1)
-    (in_bom yes) (on_board yes) (dnp no) (fields_autoplaced)
-    (property "Reference" "#PWR?" (at 104.14 40.64 0)
-      (effects (font (size 1.27 1.27)) hide)
-    )
-    (property "Value" "+12V" (at 104.14 31.75 0)
+  (symbol (lib_id "power:+12V") (at 115.57 36.83 0) (unit 1)
+    (in_bom yes) (on_board yes) (dnp no) (fields_autoplaced)
+    (property "Reference" "#PWR?" (at 115.57 40.64 0)
+      (effects (font (size 1.27 1.27)) hide)
+    )
+    (property "Value" "+12V" (at 115.57 31.75 0)
       (effects (font (size 1.27 1.27)))
     )
-    (property "Footprint" "" (at 104.14 36.83 0)
-      (effects (font (size 1.27 1.27)) hide)
-    )
-    (property "Datasheet" "" (at 104.14 36.83 0)
+    (property "Footprint" "" (at 115.57 36.83 0)
+      (effects (font (size 1.27 1.27)) hide)
+    )
+    (property "Datasheet" "" (at 115.57 36.83 0)
       (effects (font (size 1.27 1.27)) hide)
     )
@@
         )
         (path "/2e9f4f51-d216-4952-a31c-e7104e0d4b1e/bf23a663-b938-440b-843e-ef7912c82d18/726bf2a6-1244-4795-8327-149588380c7e"
-          (reference "#PWR077") (unit 1)
-        )
-        (path "/2e9f4f51-d216-4952-a31c-e7104e0d4b1e/bf23a663-b938-440b-843e-ef7912c82d18/66fa18d5-534c-477b-b6ed-b26c28a08707"
-          (reference "#PWR080") (unit 1)
-        )
-        (path "/2e9f4f51-d216-4952-a31c-e7104e0d4b1e/bf23a663-b938-440b-843e-ef7912c82d18/3bf7416b-1505-491f-89b6-6e99a8c04638"
-          (reference "#PWR083") (unit 1)
+          (reference "#PWR0121") (unit 1)
+        )
+        (path "/2e9f4f51-d216-4952-a31c-e7104e0d4b1e/bf23a663-b938-440b-843e-ef7912c82d18/66fa18d5-534c-477b-b6ed-b26c28a08707"
+          (reference "#PWR0124") (unit 1)
+        )
+        (path "/2e9f4f51-d216-4952-a31c-e7104e0d4b1e/bf23a663-b938-440b-843e-ef7912c82d18/3bf7416b-1505-491f-89b6-6e99a8c04638"
+          (reference "#PWR0127") (unit 1)
+        )
+      )
+    )
+  )
+  (symbol (lib_id "Diode:1N4148") (at 125.73 45.72 270) (unit 1)
+    (in_bom yes) (on_board yes) (dnp no)
+    (property "Reference" "D2" (at 128.27 44.45 90)
+      (effects (font (size 1.27 1.27)) (justify left))
+    )
+    (property "Value" "1N4148WS" (at 128.27 46.99 90)
+      (effects (font (size 1.27 1.27)) (justify left))
+    )
+    (property "Footprint" "Diode_SMD:D_SOD-323F" (at 125.73 45.72 0)
+      (effects (font (size 1.27 1.27)) hide)
+    )
+    (property "Datasheet" "https://assets.nexperia.com/documents/data-sheet/1N4148_1N4448.pdf" (at 125.73 45.72 0)
+      (effects (font (size 1.27 1.27)) hide)
+    )
+    (property "Sim.Device" "D" (at 125.73 45.72 0)
+      (effects (font (size 1.27 1.27)) hide)
+    )
+    (property "Sim.Pins" "1=K 2=A" (at 125.73 45.72 0)
+      (effects (font (size 1.27 1.27)) hide)
+    )
+    (property "P/N" "1N4148WS" (at 125.73 45.72 90)
+      (effects (font (size 1.27 1.27)) hide)
+    )
+    (pin "1")
+    (pin "2")
+    (instances
+      (project "BPS-LeaderDaughter"
+        (path "/2e9f4f51-d216-4952-a31c-e7104e0d4b1e/bf23a663-b938-440b-843e-ef7912c82d18"
+          (reference "D2") (unit 1)
+        )
+        (path "/2e9f4f51-d216-4952-a31c-e7104e0d4b1e/bf23a663-b938-440b-843e-ef7912c82d18/cb70587e-88a7-4e34-a774-2566ee5ba031"
+          (reference "D6") (unit 1)
+        )
+        (path "/2e9f4f51-d216-4952-a31c-e7104e0d4b1e/bf23a663-b938-440b-843e-ef7912c82d18/726bf2a6-1244-4795-8327-149588380c7e"
+          (reference "D7") (unit 1)
+        )
+        (path "/2e9f4f51-d216-4952-a31c-e7104e0d4b1e/bf23a663-b938-440b-843e-ef7912c82d18/66fa18d5-534c-477b-b6ed-b26c28a08707"
+          (reference "D8") (unit 1)
+        )
+        (path "/2e9f4f51-d216-4952-a31c-e7104e0d4b1e/bf23a663-b938-440b-843e-ef7912c82d18/3bf7416b-1505-491f-89b6-6e99a8c04638"
+          (reference "D9") (unit 1)
         )
       )
@@
         )
         (path "/2e9f4f51-d216-4952-a31c-e7104e0d4b1e/bf23a663-b938-440b-843e-ef7912c82d18/726bf2a6-1244-4795-8327-149588380c7e"
-          (reference "#PWR076") (unit 1)
-        )
-        (path "/2e9f4f51-d216-4952-a31c-e7104e0d4b1e/bf23a663-b938-440b-843e-ef7912c82d18/66fa18d5-534c-477b-b6ed-b26c28a08707"
-          (reference "#PWR079") (unit 1)
-        )
-        (path "/2e9f4f51-d216-4952-a31c-e7104e0d4b1e/bf23a663-b938-440b-843e-ef7912c82d18/3bf7416b-1505-491f-89b6-6e99a8c04638"
-          (reference "#PWR082") (unit 1)
+          (reference "#PWR0119") (unit 1)
+        )
+        (path "/2e9f4f51-d216-4952-a31c-e7104e0d4b1e/bf23a663-b938-440b-843e-ef7912c82d18/66fa18d5-534c-477b-b6ed-b26c28a08707"
+          (reference "#PWR0122") (unit 1)
+        )
+        (path "/2e9f4f51-d216-4952-a31c-e7104e0d4b1e/bf23a663-b938-440b-843e-ef7912c82d18/3bf7416b-1505-491f-89b6-6e99a8c04638"
+          (reference "#PWR0125") (unit 1)
         )
       )
@@
         )
         (path "/2e9f4f51-d216-4952-a31c-e7104e0d4b1e/bf23a663-b938-440b-843e-ef7912c82d18/726bf2a6-1244-4795-8327-149588380c7e"
-          (reference "#PWR075") (unit 1)
-        )
-        (path "/2e9f4f51-d216-4952-a31c-e7104e0d4b1e/bf23a663-b938-440b-843e-ef7912c82d18/66fa18d5-534c-477b-b6ed-b26c28a08707"
-          (reference "#PWR078") (unit 1)
-        )
-        (path "/2e9f4f51-d216-4952-a31c-e7104e0d4b1e/bf23a663-b938-440b-843e-ef7912c82d18/3bf7416b-1505-491f-89b6-6e99a8c04638"
-          (reference "#PWR081") (unit 1)
-        )
-      )
+          (reference "#PWR0120") (unit 1)
+        )
+        (path "/2e9f4f51-d216-4952-a31c-e7104e0d4b1e/bf23a663-b938-440b-843e-ef7912c82d18/66fa18d5-534c-477b-b6ed-b26c28a08707"
+          (reference "#PWR0123") (unit 1)
+        )
+        (path "/2e9f4f51-d216-4952-a31c-e7104e0d4b1e/bf23a663-b938-440b-843e-ef7912c82d18/3bf7416b-1505-491f-89b6-6e99a8c04638"
+          (reference "#PWR0126") (unit 1)
+        )
+      )

Commit message: Made ignition connector 3 pin + fixed tach resistors
Parts:
- D2: footprint Diode_SMD:D_SOD-323F -> Diode_SMD:D_SOD-323; P/N 1N4148WS -> 1N4148WSQ-7-F
Changed lines of the file:
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@@
     (stroke (width 0) (type default))
   )
-  (wire (pts (xy 93.98 64.77) (xy 93.98 69.85))
+  (wire (pts (xy 93.98 64.77) (xy 93.98 71.12))
     (stroke (width 0) (type default))
   )
@@
       (effects (font (size 1.27 1.27)) hide)
     )
-    (property "Datasheet" "https://www.mouser.com/ProductDetail/603-RT0603FRE0710KL" (at 104.14 45.72 0)
+    (property "Datasheet" "~" (at 104.14 45.72 0)
       (effects (font (size 1.27 1.27)) hide)
     )
@@
       (effects (font (size 1.27 1.27)) hide)
     )
-    (property "Datasheet" "https://www.mouser.com/ProductDetail/603-RT0603FRE0710KL" (at 86.36 45.72 0)
+    (property "Datasheet" "~" (at 86.36 45.72 0)
       (effects (font (size 1.27 1.27)) hide)
     )
@@
       (effects (font (size 1.27 1.27)) (justify left))
     )
-    (property "Footprint" "Diode_SMD:D_SOD-323F" (at 125.73 45.72 0)
+    (property "Footprint" "Diode_SMD:D_SOD-323" (at 125.73 45.72 0)
       (effects (font (size 1.27 1.27)) hide)
     )
@@
       (effects (font (size 1.27 1.27)) hide)
     )
-    (property "P/N" "1N4148WS" (at 125.73 45.72 90)
+    (property "P/N" "1N4148WSQ-7-F" (at 125.73 45.72 90)
       (effects (font (size 1.27 1.27)) hide)
     )
@@
     )
   )
-  (symbol (lib_id "power:GND") (at 93.98 69.85 0) (unit 1)
+  (symbol (lib_id "power:GND") (at 93.98 71.12 0) (unit 1)
     (in_bom yes) (on_board yes) (dnp no)
-    (property "Reference" "#PWR?" (at 93.98 76.2 0)
-      (effects (font (size 1.27 1.27)) hide)
-    )
-    (property "Value" "GND" (at 94.107 74.2442 0)
+    (property "Reference" "#PWR?" (at 93.98 77.47 0)
+      (effects (font (size 1.27 1.27)) hide)
+    )
+    (property "Value" "GND" (at 94.107 75.5142 0)
       (effects (font (size 1.27 1.27)))
     )
-    (property "Footprint" "" (at 93.98 69.85 0)
-      (effects (font (size 1.27 1.27)) hide)
-    )
-    (property "Datasheet" "" (at 93.98 69.85 0)
-      (effects (font (size 1.27 1.27)) hide)
-    )
+    (property "Footprint" "" (at 93.98 71.12 0)
+      (effects (font (size 1.27 1.27)) hide)
+    )
+    (property "Datasheet" "" (at 93.98 71.12 0)
+      (effects (font (size 1.27 1.27)) hide)
+    )

Commit message: revamp fans
Parts:
- removed R?: 100k, Resistor_SMD:R_0805_2012Metric, symbol Device:R
- added D?: 3.3V, Diode_SMD:D_SOD-323, symbol Device:D_Zener
- added J?: Conn_01x04, UTSVT_Connectors:Molex_MicroFit3.0_1x4xP3.00mm_PolarizingPeg_Vertical, symbol Connector_Generic:Conn_01x04
- added JP2: Termination Resistors, Connector_PinHeader_2.54mm:PinHeader_1x02_P2.54mm_Vertical, symbol Jumper:Jumper_2_Open
- added R? (x2): 10k, Resistor_SMD:R_0805_2012Metric, symbol Device:R
- added R?: 100k, Resistor_SMD:R_0805_2012Metric, symbol Device:R
- added R?: 20k, Resistor_SMD:R_0805_2012Metric, symbol Device:R
Connections:
- net +12V: now also D2.2 (A), J?.2 (Pin_2), R?.1; no longer D2.1 (K)
- net +3.3V: now also R?.1
- net GND: now also D2.1 (K), D?.2 (A), R?.2
- net PWM_IN: now also J?.4 (Pin_4), JP2.1 (A), R?.2; no longer Q?.4 (G), R?.2
- net PWM_OUT: no longer names the net of Q?.5 (D)
- net PWM_OUT: now also J?.1 (Pin_1); no longer D2.2 (A)
- new net: JP2.2 (B), Q?.4 (G), R?.2
- new net TACH_IN: J?.3 (Pin_3), R?.1, R?.2
- new net TACH_OUT: D?.1 (K), R?.1, R?.2
Other:
- note added: "2 V < VPULL-UP × R13/(RPULL-UP + R14 + R13) < 5 V"
- note added: "PWM"
- note added: "SHORT THIS FOR 4 PIN FANS"
- note added: "TACH"
- moved on the sheet: Q?, R?

Commit message: why your schematic so broken >:(
Connections:
- net +12V: now also D2.1 (K); no longer D2.2 (A)
- net GND: now also D2.2 (A); no longer D2.1 (K)
Other:
- moved on the sheet: D2

Commit message: More laying out, fixed board constraints, added labs to important fan nets
Connections:
- net Fan_-: now reaches J?.1 (Pin_1), Q?.5 (D)
Changed lines of the file:
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@@
   (junction (at 123.19 61.595) (diameter 0) (color 0 0 0 0)
   )
+  (junction (at 62.23 69.85) (diameter 0) (color 0 0 0 0)
+  )
   (junction (at 34.925 76.2) (diameter 0) (color 0 0 0 0)
   )
@@
     (stroke (width 0) (type default))
   )
+  (wire (pts (xy 62.23 69.85) (xy 64.135 69.85))
+    (stroke (width 0) (type default))
+  )
   (wire (pts (xy 34.925 76.2) (xy 40.005 76.2))
     (stroke (width 0) (type default))
@@
     (stroke (width 0) (type default))
   )
-  (wire (pts (xy 62.23 71.12) (xy 62.23 55.88))
+  (wire (pts (xy 62.23 71.12) (xy 62.23 69.85))
     (stroke (width 0) (type default))
   )
@@
   )
   (wire (pts (xy 155.575 61.595) (xy 155.575 65.405))
+    (stroke (width 0) (type default))
+  )
+  (wire (pts (xy 62.23 69.85) (xy 62.23 55.88))
     (stroke (width 0) (type default))
   )
@@
   )
   (text "2 V < VPULL-UP × R13/(RPULL-UP + R14 + R13) < 5 V" (at 113.665 88.9 0)
+    (effects (font (size 1.27 1.27)) (justify left bottom))
+  )
+  (label "Fan_-" (at 64.135 69.85 0) (fields_autoplaced)
     (effects (font (size 1.27 1.27)) (justify left bottom))
   )
@@
   )
   (symbol (lib_id "Device:R") (at 34.925 68.58 0) (unit 1)
-    (in_bom yes) (on_board yes) (dnp no) (fields_autoplaced)
+    (in_bom yes) (on_board yes) (dnp no)
     (property "Reference" "R?" (at 37.465 67.31 0)
       (effects (font (size 1.27 1.27)) (justify left))

Commit message: last sanity check + part numbers (ready for review)
Other:
- note added: "2 V < VPULL-UP × (RtachPULL-DOWN)/(RPULL-UP + Rtach + RtachPULL-DOWN) < 5 V"
- note added: "Equation from page 22 of datasheet"
- note added: "RPULL-UP"
- note added: "RtachPULL-DOWN"
- note removed: "2 V < VPULL-UP × R13/(RPULL-UP + R14 + R13) < 5 V"
Changed lines of the file:
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@@
     (fill (type none))
   )
-  (rectangle (start 106.045 38.735) (end 177.8 91.44)
+  (rectangle (start 106.045 38.735) (end 196.215 91.44)
     (stroke (width 0) (type default))
     (fill (type none))
@@
     (effects (font (size 1.27 1.27)) (justify left bottom))
   )
+  (text "RPULL-UP" (at 125.095 50.165 0)
+    (effects (font (size 1.27 1.27)) (justify left bottom))
+  )
+  (text "Equation from page 22 of datasheet" (at 106.68 90.17 0)
+    (effects (font (size 1.27 1.27)) (justify left bottom))
+  )
   (text "PWM" (at 20.32 36.83 0)
     (effects (font (size 2.54 2.54) (thickness 0.508) bold) (justify left bottom))
   )
-  (text "2 V < VPULL-UP × R13/(RPULL-UP + R14 + R13) < 5 V" (at 113.665 88.9 0)
+  (text " RtachPULL-DOWN" (at 157.48 66.04 0)
     (effects (font (size 1.27 1.27)) (justify left bottom))
   )
+  (text "2 V < VPULL-UP × (RtachPULL-DOWN)/(RPULL-UP + Rtach + RtachPULL-DOWN) < 5 V"
+    (at 106.68 87.63 0)
+    (effects (font (size 1.27 1.27)) (justify left bottom))
+  )
