File: Fan_PWM.kicad_sch (KiCad schematic)
At the start: 10 parts

Commit message: LAKSHAY CHOSE THE WRONG DIODE >:(
Parts:
- removed D2: 1N4148WS, Diode_SMD:D_SOD-323, symbol Diode:1N4148
- added D4: 1N4448W, Diode_SMD:D_SOD-123, symbol Diode:1N4448W
Connections:
- net +12V: now also D4.1 (K)
- net GND: now also D4.2 (A)
Changed lines of the file:
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@@
+    )
+  )
+  (symbol (lib_id "Diode:1N4448W") (at 87.63 58.42 270) (unit 1)
+    (in_bom yes) (on_board yes) (dnp no) (fields_autoplaced)
+    (property "Reference" "D4" (at 90.17 57.15 90)
+      (effects (font (size 1.27 1.27)) (justify left))
+    )
+    (property "Value" "1N4448W" (at 90.17 59.69 90)
+      (effects (font (size 1.27 1.27)) (justify left))
+    )
+    (property "Footprint" "Diode_SMD:D_SOD-123" (at 83.185 58.42 0)
+      (effects (font (size 1.27 1.27)) hide)
+    )
+    (property "Datasheet" "https://www.vishay.com/docs/85722/1n4448w.pdf" (at 87.63 58.42 0)
+      (effects (font (size 1.27 1.27)) hide)
+    )
+    (property "Sim.Device" "D" (at 87.63 58.42 0)
+      (effects (font (size 1.27 1.27)) hide)
+    )
+    (property "Sim.Pins" "1=K 2=A" (at 87.63 58.42 0)
+      (effects (font (size 1.27 1.27)) hide)
+    )
+    (pin "2")
+    (pin "1")
+    (instances
+      (project "BPS-LeaderDaughter"
+        (path "/2e9f4f51-d216-4952-a31c-e7104e0d4b1e/ae57cd3a-fadb-4313-835a-95d5b185a797"
+          (reference "D4") (unit 1)
+        )
+        (path "/2e9f4f51-d216-4952-a31c-e7104e0d4b1e/5e4c6ec4-73d4-4ed3-a75f-02eb4f9ac8b3"
+          (reference "D7") (unit 1)
+        )
+        (path "/2e9f4f51-d216-4952-a31c-e7104e0d4b1e/bb673292-4a5d-469b-b6b6-0dc7df3c162d"
+          (reference "D10") (unit 1)
+        )
+        (path "/2e9f4f51-d216-4952-a31c-e7104e0d4b1e/bf23a663-b938-440b-843e-ef7912c82d18/cb70587e-88a7-4e34-a774-2566ee5ba031"
+          (reference "D11") (unit 1)
+        )
+        (path "/2e9f4f51-d216-4952-a31c-e7104e0d4b1e/bf23a663-b938-440b-843e-ef7912c82d18/6987911b-7d09-4745-9ed2-ae46961723fc"
+          (reference "D13") (unit 1)
+        )
+        (path "/2e9f4f51-d216-4952-a31c-e7104e0d4b1e/bf23a663-b938-440b-843e-ef7912c82d18/5bfa400a-1062-4778-999e-70160150bf07"
+          (reference "D15") (unit 1)
+        )
+        (path "/2e9f4f51-d216-4952-a31c-e7104e0d4b1e/bf23a663-b938-440b-843e-ef7912c82d18/9e6063ac-d7b1-4ab6-8b9c-50a1e9762dc9"
+          (reference "D17") (unit 1)
+        )
+      )
     )
   )
@@
         )
       )
-    )
-  )
-  (symbol (lib_id "Diode:1N4148") (at 87.63 58.42 270) (unit 1)
-    (in_bom yes) (on_board yes) (dnp no)
-    (property "Reference" "D2" (at 74.93 57.15 90)
-      (effects (font (size 1.27 1.27)) (justify left))
-    )
-    (property "Value" "1N4148WS" (at 74.93 59.69 90)
-      (effects (font (size 1.27 1.27)) (justify left))
-    )
-    (property "Footprint" "Diode_SMD:D_SOD-323" (at 87.63 58.42 0)
-      (effects (font (size 1.27 1.27)) hide)
-    )
-    (property "Datasheet" "https://assets.nexperia.com/documents/data-sheet/1N4148_1N4448.pdf" (at 87.63 58.42 0)
-      (effects (font (size 1.27 1.27)) hide)
-    )
-    (property "Sim.Device" "D" (at 87.63 58.42 0)
-      (effects (font (size 1.27 1.27)) hide)
-    )
-    (property "Sim.Pins" "1=K 2=A" (at 87.63 58.42 0)
-      (effects (font (size 1.27 1.27)) hide)
-    )
-    (property "P/N" "1N4148WSQ-7-F" (at 87.63 58.42 90)
-      (effects (font (size 1.27 1.27)) hide)
-    )
-    (pin "1")
-    (pin "2")
-    (instances
-      (project "BPS-LeaderDaughter"
-        (path "/2e9f4f51-d216-4952-a31c-e7104e0d4b1e/bf23a663-b938-440b-843e-ef7912c82d18"
-          (reference "D2") (unit 1)
-        )
-        (path "/2e9f4f51-d216-4952-a31c-e7104e0d4b1e/bf23a663-b938-440b-843e-ef7912c82d18/cb70587e-88a7-4e34-a774-2566ee5ba031"
-          (reference "D11") (unit 1)
-        )
-        (path "/2e9f4f51-d216-4952-a31c-e7104e0d4b1e/bf23a663-b938-440b-843e-ef7912c82d18/6987911b-7d09-4745-9ed2-ae46961723fc"
-          (reference "D13") (unit 1)
-        )
-        (path "/2e9f4f51-d216-4952-a31c-e7104e0d4b1e/bf23a663-b938-440b-843e-ef7912c82d18/5bfa400a-1062-4778-999e-70160150bf07"
-          (reference "D15") (unit 1)
-        )
-        (path "/2e9f4f51-d216-4952-a31c-e7104e0d4b1e/bf23a663-b938-440b-843e-ef7912c82d18/9e6063ac-d7b1-4ab6-8b9c-50a1e9762dc9"
-          (reference "D17") (unit 1)
-        )
-      )

Commit message: Started BOM
Parts:
- D4: P/N (none) -> 1N4448W
Changed lines of the file:
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@@
+      (effects (font (size 1.27 1.27)) hide)
+    )
+    (property "P/N" "1N4448W" (at 87.63 58.42 0)
       (effects (font (size 1.27 1.27)) hide)
     )

Commit message: BOM complete
Parts:
- D?: P/N SZMM3Z3V3T1G -> BZT52B3V3
- J?: P/N 0436500428 -> 436500244
- R?: P/N RT0603FRE074K7L -> CRCW080510K0FKEAC
- R?: P/N RT0603FRE0710KL -> CRCW080510K0FKEAC
- R? (x2): P/N RT0603FRE0710KL -> CRCW0805100KFKEAC
- R?: P/N RT0603FRE0710KL -> CRCW080522K1FKEA
Changed lines of the file:
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@@
       (effects (font (size 1.27 1.27)) hide)
     )
-    (property "P/N" "RT0603FRE074K7L " (at 155.575 69.215 0)
+    (property "P/N" "CRCW080510K0FKEAC" (at 155.575 69.215 0)
       (effects (font (size 1.27 1.27)) hide)
     )
@@
       (effects (font (size 1.27 1.27)) hide)
     )
-    (property "P/N" "RT0603FRE0710KL " (at 123.19 53.975 90)
+    (property "P/N" "CRCW080510K0FKEAC" (at 123.19 53.975 90)
       (effects (font (size 1.27 1.27)) hide)
     )
@@
       (effects (font (size 1.27 1.27)) hide)
     )
-    (property "P/N" "RT0603FRE0710KL " (at 52.705 68.58 90)
+    (property "P/N" "CRCW0805100KFKEAC" (at 52.705 68.58 90)
       (effects (font (size 1.27 1.27)) hide)
     )
@@
       (effects (font (size 1.27 1.27)) hide)
     )
-    (property "P/N" "0436500428" (at 48.895 53.34 0)
+    (property "P/N" "436500244" (at 48.895 53.34 0)
       (effects (font (size 1.27 1.27)) hide)
     )
@@
       (effects (font (size 1.27 1.27)) hide)
     )
-    (property "P/N" "SZMM3Z3V3T1G" (at 145.415 69.215 90)
+    (property "P/N" "BZT52B3V3" (at 145.415 69.215 90)
       (effects (font (size 1.27 1.27)) hide)
     )
@@
       (effects (font (size 1.27 1.27)) hide)
     )
-    (property "Datasheet" "https://www.vishay.com/docs/85722/1n4448w.pdf" (at 87.63 58.42 0)
+    (property "Datasheet" "https://www.mouser.com/datasheet/2/849/1n4148w-3324072.pdf" (at 87.63 58.42 0)
       (effects (font (size 1.27 1.27)) hide)
     )
@@
       (effects (font (size 1.27 1.27)) hide)
     )
-    (property "P/N" "RT0603FRE0710KL " (at 34.925 68.58 90)
+    (property "P/N" "CRCW0805100KFKEAC" (at 34.925 68.58 90)
       (effects (font (size 1.27 1.27)) hide)
     )
@@
       (effects (font (size 1.27 1.27)) hide)
     )
-    (property "P/N" "RT0603FRE0710KL " (at 136.525 61.595 90)
-      (effects (font (size 1.27 1.27)) hide)
-    )
+    (property "P/N" "CRCW080522K1FKEA" (at 136.525 61.595 90)
+      (effects (font (size 1.27 1.27)) hide)
+    )

Commit message: yipee
Parts:
- gave numbers to parts that had none: 8
- renumbered D4 to D11, JP2 to JP5
