File: Ignition.kicad_sch (KiCad schematic)
At the start: 1 part, among them SW1 SW_Rotary2x6

Commit message: added no connects to Ignition switch and removed redundant Strobe coupling cap
Connections:
- no-connect marks 0 -> 14
Changed lines of the file:
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@@
 (kicad_sch (version 20230121) (generator eeschema)
   (paper "A4")
+  (no_connect (at 128.27 85.725))
+  (no_connect (at 128.27 70.485))
+  (no_connect (at 128.27 75.565))
+  (no_connect (at 128.27 93.345))
+  (no_connect (at 128.27 67.945))
+  (no_connect (at 128.27 98.425))
+  (no_connect (at 128.27 80.645))
+  (no_connect (at 151.13 90.805))
+  (no_connect (at 128.27 88.265))
+  (no_connect (at 128.27 73.025))
+  (no_connect (at 128.27 90.805))
+  (no_connect (at 151.13 73.025))
+  (no_connect (at 128.27 95.885))
+  (no_connect (at 128.27 78.105))
   (rectangle (start 88.265 109.855) (end 90.805 109.855)
     (stroke (width 0) (type default))

Commit message: Started new skinny layout
Parts:
- removed SW1: SW_Rotary2x6, Connector_Molex:Molex_Micro-Fit_3.0_43045-1412_2x07_P3.00mm_Vertical, symbol Switch:SW_Rotary2x6
- added J?: Conn_01x04, UTSVT_Connectors:Molex_MicroFit3.0_1x4xP3.00mm_PolarizingPeg_Vertical, symbol Connector_Generic:Conn_01x04
Connections:
- new net +12V: J?.1 (Pin_1)
- new net ARR_ON: J?.2 (Pin_2)
- new net GND: J?.4 (Pin_4)
- new net MOTOR_ON: J?.3 (Pin_3)
- no-connect marks 14 -> 0
Changed lines of the file:
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@@
 (kicad_sch (version 20230121) (generator eeschema)
   (paper "A4")
-  (no_connect (at 128.27 85.725))
-  (no_connect (at 128.27 70.485))
-  (no_connect (at 128.27 75.565))
-  (no_connect (at 128.27 93.345))
-  (no_connect (at 128.27 67.945))
-  (no_connect (at 128.27 98.425))
-  (no_connect (at 128.27 80.645))
-  (no_connect (at 151.13 90.805))
-  (no_connect (at 128.27 88.265))
-  (no_connect (at 128.27 73.025))
-  (no_connect (at 128.27 90.805))
-  (no_connect (at 151.13 73.025))
-  (no_connect (at 128.27 95.885))
-  (no_connect (at 128.27 78.105))
+  (junction (at 255.27 40.64) (diameter 0) (color 0 0 0 0)
+  )
+  (wire (pts (xy 121.285 112.395) (xy 125.095 112.395))
+    (stroke (width 0) (type default))
+  )
+  (wire (pts (xy 254 40.64) (xy 255.27 40.64))
+    (stroke (width 0) (type default))
+  )
+  (wire (pts (xy 254 43.18) (xy 255.27 43.18))
+    (stroke (width 0) (type default))
+  )
+  (wire (pts (xy 122.555 117.475) (xy 125.095 117.475))
+    (stroke (width 0) (type default))
+  )
+  (wire (pts (xy 121.285 114.935) (xy 125.095 114.935))
+    (stroke (width 0) (type default))
+  )
+  (wire (pts (xy 122.555 120.015) (xy 122.555 117.475))
+    (stroke (width 0) (type default))
+  )
+  (wire (pts (xy 255.27 43.18) (xy 255.27 40.64))
+    (stroke (width 0) (type default))
+  )
+  (wire (pts (xy 255.27 40.64) (xy 255.27 38.1))
+    (stroke (width 0) (type default))
+  )
+  (wire (pts (xy 122.555 109.855) (xy 125.095 109.855))
+    (stroke (width 0) (type default))
+  )
+  (wire (pts (xy 122.555 106.68) (xy 122.555 109.855))
+    (stroke (width 0) (type default))
+  )
   (rectangle (start 88.265 109.855) (end 90.805 109.855)
     (stroke (width 0) (type default))
@@
     (effects (font (size 1.27 1.27)) (justify left bottom))
   )
-  (symbol (lib_id "Switch:SW_Rotary2x6") (at 140.97 83.185 180) (unit 1)
-    (in_bom yes) (on_board yes) (dnp no)
-    (property "Reference" "SW1" (at 139.7 62.23 0)
-      (effects (font (size 1.27 1.27)))
-    )
-    (property "Value" "SW_Rotary2x6" (at 139.7 64.5414 0)
-      (effects (font (size 1.27 1.27)))
-    )
-    (property "Footprint" "Connector_Molex:Molex_Micro-Fit_3.0_43045-1412_2x07_P3.00mm_Vertical" (at 143.51 98.425 0)
-      (effects (font (size 1.27 1.27)) hide)
-    )
-    (property "Datasheet" "https://www.molex.com/molex/search/partSearch?query=430451412&pQuery=" (at 143.51 98.425 0)
-      (effects (font (size 1.27 1.27)) hide)
-    )
-    (property "P/N" "430451412" (at 140.97 83.185 0)
+  (hierarchical_label "MOTOR_ON" (shape input) (at 121.285 114.935 180) (fields_autoplaced)
+    (effects (font (size 1.27 1.27)) (justify right))
+  )
+  (hierarchical_label "ARR_ON" (shape input) (at 121.285 112.395 180) (fields_autoplaced)
+    (effects (font (size 1.27 1.27)) (justify right))
+  )
+  (symbol (lib_id "Connector_Generic:Conn_01x04") (at 130.175 112.395 0) (unit 1)
+    (in_bom yes) (on_board yes) (dnp no) (fields_autoplaced)
+    (property "Reference" "J?" (at 132.715 112.395 0)
+      (effects (font (size 1.27 1.27)) (justify left))
+    )
+    (property "Value" "Conn_01x04" (at 132.715 114.935 0)
+      (effects (font (size 1.27 1.27)) (justify left))
+    )
+    (property "Footprint" "UTSVT_Connectors:Molex_MicroFit3.0_1x4xP3.00mm_PolarizingPeg_Vertical" (at 130.175 112.395 0)
+      (effects (font (size 1.27 1.27)) hide)
+    )
+    (property "Datasheet" "https://www.mouser.com/datasheet/2/276/3/0436500428_PCB_HEADERS-2866587.pdf" (at 130.175 112.395 0)
+      (effects (font (size 1.27 1.27)) hide)
+    )
+    (property "P/N" "0436500428" (at 130.175 112.395 0)
       (effects (font (size 1.27 1.27)) hide)
     )
     (pin "1")
-    (pin "10")
-    (pin "11")
-    (pin "12")
-    (pin "13")
-    (pin "14")
     (pin "2")
     (pin "3")
     (pin "4")
-    (pin "5")
-    (pin "6")
-    (pin "7")
-    (pin "8")
-    (pin "9")
+    (instances
+      (project "BPS-LeaderDaughter"
+        (path "/2e9f4f51-d216-4952-a31c-e7104e0d4b1e/ae57cd3a-fadb-4313-835a-95d5b185a797"
+          (reference "J?") (unit 1)
+        )
+        (path "/2e9f4f51-d216-4952-a31c-e7104e0d4b1e/5e4c6ec4-73d4-4ed3-a75f-02eb4f9ac8b3"
+          (reference "J?") (unit 1)
+        )
+        (path "/2e9f4f51-d216-4952-a31c-e7104e0d4b1e/bb673292-4a5d-469b-b6b6-0dc7df3c162d"
+          (reference "J?") (unit 1)
+        )
+        (path "/2e9f4f51-d216-4952-a31c-e7104e0d4b1e/bf23a663-b938-440b-843e-ef7912c82d18"
+          (reference "J5") (unit 1)
+        )
+        (path "/2e9f4f51-d216-4952-a31c-e7104e0d4b1e/115507eb-1e24-4553-a6e1-1fcd332a9a2b"
+          (reference "J3") (unit 1)
+        )
+      )
+    )
+  )
+  (symbol (lib_id "power:GND") (at 122.555 120.015 0) (unit 1)
+    (in_bom yes) (on_board yes) (dnp no) (fields_autoplaced)
+    (property "Reference" "#PWR04" (at 122.555 126.365 0)
+      (effects (font (size 1.27 1.27)) hide)
+    )
+    (property "Value" "GND" (at 122.555 124.46 0)
+      (effects (font (size 1.27 1.27)))
+    )
+    (property "Footprint" "" (at 122.555 120.015 0)
+      (effects (font (size 1.27 1.27)) hide)
+    )
+    (property "Datasheet" "" (at 122.555 120.015 0)
+      (effects (font (size 1.27 1.27)) hide)
+    )
+    (pin "1")
     (instances
       (project "BPS-LeaderDaughter"
         (path "/2e9f4f51-d216-4952-a31c-e7104e0d4b1e/115507eb-1e24-4553-a6e1-1fcd332a9a2b"
-          (reference "SW1") (unit 1)
+          (reference "#PWR04") (unit 1)
         )
       )
-      (project "Dashboard"
-        (path "/66218487-e316-4467-9eba-79d4626ab24e/00000000-0000-0000-0000-00005f6b59ce"
-          (reference "SW8") (unit 1)
+    )
+  )
+  (symbol (lib_id "power:+12V") (at 122.555 106.68 0) (unit 1)
+    (in_bom yes) (on_board yes) (dnp no) (fields_autoplaced)
+    (property "Reference" "#PWR03" (at 122.555 110.49 0)
+      (effects (font (size 1.27 1.27)) hide)
+    )
+    (property "Value" "+12V" (at 122.555 101.6 0)
+      (effects (font (size 1.27 1.27)))
+    )
+    (property "Footprint" "" (at 122.555 106.68 0)
+      (effects (font (size 1.27 1.27)) hide)
+    )
+    (property "Datasheet" "" (at 122.555 106.68 0)
+      (effects (font (size 1.27 1.27)) hide)
+    )
+    (pin "1")
+    (instances
+      (project "BPS-LeaderDaughter"
+        (path "/2e9f4f51-d216-4952-a31c-e7104e0d4b1e/115507eb-1e24-4553-a6e1-1fcd332a9a2b"
+          (reference "#PWR03") (unit 1)
         )
       )

Commit message: Made ignition connector 3 pin + fixed tach resistors
Parts:
- removed J?: Conn_01x04, UTSVT_Connectors:Molex_MicroFit3.0_1x4xP3.00mm_PolarizingPeg_Vertical, symbol Connector_Generic:Conn_01x04
- added J13: Conn_01x03, Connector_Molex:Molex_Micro-Fit_3.0_43650-0315_1x03_P3.00mm_Vertical, symbol Connector_Generic:Conn_01x03
- added R17 (x2): 100k, Resistor_SMD:R_0805_2012Metric, symbol Device:R_Small
- added R34, R35: 35, Resistor_SMD:R_0805_2012Metric, symbol Device:R
- added U1, U4: EL3H7, Package_SO:SOP-4_4.4x2.6mm_P1.27mm, symbol Isolator:EL817
Connections:
- net ARR_ON: now also R17.1, U4.4
- net GND: now also J13.3 (Pin_3), U1.2, U1.3, U4.2, U4.3
- net MOTOR_ON: now also R17.1, U1.4
- new net: R34.1, U4.1
- new net: J13.2 (Pin_2), R34.2
- new net: R35.1, U1.1
- new net: J13.1 (Pin_1), R35.2
- new net +3.3V: R17.2, R17.2
Other:
- note added: "Assumes 2 pole 6 way Ignition Switch The input signals are 12V"

Commit message: Fixed optoisolator resistor values
Parts:
- R34, R35: value 35 -> 100
Changed lines of the file:
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@@
   )
   (symbol (lib_id "Device:R") (at 118.745 78.74 90) (unit 1)
-    (in_bom yes) (on_board yes) (dnp no) (fields_autoplaced)
+    (in_bom yes) (on_board yes) (dnp no)
     (property "Reference" "R34" (at 118.745 81.28 90)
       (effects (font (size 1.27 1.27)))
     )
-    (property "Value" "35" (at 118.745 83.82 90)
+    (property "Value" "100" (at 118.745 83.82 90)
       (effects (font (size 1.27 1.27)))
     )
@@
   )
   (symbol (lib_id "Device:R") (at 74.93 76.2 90) (unit 1)
-    (in_bom yes) (on_board yes) (dnp no) (fields_autoplaced)
+    (in_bom yes) (on_board yes) (dnp no)
     (property "Reference" "R35" (at 74.93 79.375 90)
       (effects (font (size 1.27 1.27)))
     )
-    (property "Value" "35" (at 74.93 81.915 90)
+    (property "Value" "100" (at 74.93 81.915 90)
       (effects (font (size 1.27 1.27)))
     )

Commit message: why your schematic so broken >:(
Parts:
- R17: renamed from R35; value 100 -> 604
- R19: renamed from R34; value 100 -> 604
- renumbered J13 to J8, U1 to U5, U4 to U6
Connections:
- net +3.3V: now also U5.4, U6.4; no longer R17.2, R17.2
- net ARR_ON: now also R17.2, U6.3; no longer R17.1, U6.4
- net GND: now also R17.1, R17.1; no longer U5.3, U6.3
- net MOTOR_ON: now also R17.2, U5.3; no longer R17.1, U5.4
Other:
- moved on the sheet: R17

Commit message: everythign on front
Parts:
- renumbered U5 to U1, U6 to U2
Changed lines of the file:
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@@
   (symbol (lib_id "power:GND") (at 143.51 81.915 0) (unit 1)
     (in_bom yes) (on_board yes) (dnp no) (fields_autoplaced)
-    (property "Reference" "#PWR062" (at 143.51 88.265 0)
+    (property "Reference" "#PWR047" (at 143.51 88.265 0)
       (effects (font (size 1.27 1.27)) hide)
     )
@@
       (project "BPS-LeaderDaughter"
         (path "/2e9f4f51-d216-4952-a31c-e7104e0d4b1e/115507eb-1e24-4553-a6e1-1fcd332a9a2b"
-          (reference "#PWR062") (unit 1)
+          (reference "#PWR047") (unit 1)
         )
       )
@@
   (symbol (lib_id "Isolator:EL817") (at 102.87 87.63 270) (unit 1)
     (in_bom yes) (on_board yes) (dnp no) (fields_autoplaced)
-    (property "Reference" "U6" (at 107.95 86.36 90)
+    (property "Reference" "U2" (at 107.95 86.36 90)
       (effects (font (size 1.27 1.27)) (justify left))
     )
@@
       (project "BPS-LeaderDaughter"
         (path "/2e9f4f51-d216-4952-a31c-e7104e0d4b1e/115507eb-1e24-4553-a6e1-1fcd332a9a2b"
-          (reference "U6") (unit 1)
+          (reference "U2") (unit 1)
         )
       )
@@
   (symbol (lib_id "power:+3.3V") (at 118.11 93.98 0) (unit 1)
     (in_bom yes) (on_board yes) (dnp no) (fields_autoplaced)
-    (property "Reference" "#PWR061" (at 118.11 97.79 0)
+    (property "Reference" "#PWR046" (at 118.11 97.79 0)
       (effects (font (size 1.27 1.27)) hide)
     )
@@
       (project "BPS-LeaderDaughter"
         (path "/2e9f4f51-d216-4952-a31c-e7104e0d4b1e/115507eb-1e24-4553-a6e1-1fcd332a9a2b"
-          (reference "#PWR061") (unit 1)
+          (reference "#PWR046") (unit 1)
         )
       )
@@
   (symbol (lib_id "Isolator:EL817") (at 59.055 88.265 270) (unit 1)
     (in_bom yes) (on_board yes) (dnp no) (fields_autoplaced)
-    (property "Reference" "U5" (at 64.135 86.995 90)
+    (property "Reference" "U1" (at 64.135 86.995 90)
       (effects (font (size 1.27 1.27)) (justify left))
     )
@@
       (project "BPS-LeaderDaughter"
         (path "/2e9f4f51-d216-4952-a31c-e7104e0d4b1e/115507eb-1e24-4553-a6e1-1fcd332a9a2b"
-          (reference "U5") (unit 1)
+          (reference "U1") (unit 1)
         )
       )
@@
   (symbol (lib_id "power:GND") (at 56.515 107.315 0) (unit 1)
     (in_bom yes) (on_board yes) (dnp no) (fields_autoplaced)
-    (property "Reference" "#PWR057" (at 56.515 113.665 0)
+    (property "Reference" "#PWR042" (at 56.515 113.665 0)
       (effects (font (size 1.27 1.27)) hide)
     )
@@
       (project "BPS-LeaderDaughter"
         (path "/2e9f4f51-d216-4952-a31c-e7104e0d4b1e/115507eb-1e24-4553-a6e1-1fcd332a9a2b"
-          (reference "#PWR057") (unit 1)
+          (reference "#PWR042") (unit 1)
         )
       )
@@
   (symbol (lib_id "power:GND") (at 100.33 106.68 0) (unit 1)
     (in_bom yes) (on_board yes) (dnp no) (fields_autoplaced)
-    (property "Reference" "#PWR060" (at 100.33 113.03 0)
+    (property "Reference" "#PWR045" (at 100.33 113.03 0)
       (effects (font (size 1.27 1.27)) hide)
     )
@@
       (project "BPS-LeaderDaughter"
         (path "/2e9f4f51-d216-4952-a31c-e7104e0d4b1e/115507eb-1e24-4553-a6e1-1fcd332a9a2b"
-          (reference "#PWR060") (unit 1)
+          (reference "#PWR045") (unit 1)
         )
       )
@@
   (symbol (lib_id "power:+3.3V") (at 74.295 94.615 0) (unit 1)
     (in_bom yes) (on_board yes) (dnp no) (fields_autoplaced)
-    (property "Reference" "#PWR058" (at 74.295 98.425 0)
+    (property "Reference" "#PWR043" (at 74.295 98.425 0)
       (effects (font (size 1.27 1.27)) hide)
     )
@@
       (project "BPS-LeaderDaughter"
         (path "/2e9f4f51-d216-4952-a31c-e7104e0d4b1e/115507eb-1e24-4553-a6e1-1fcd332a9a2b"
-          (reference "#PWR058") (unit 1)
+          (reference "#PWR043") (unit 1)
         )
       )
@@
   (symbol (lib_id "power:GND") (at 91.44 82.55 0) (unit 1)
     (in_bom yes) (on_board yes) (dnp no) (fields_autoplaced)
-    (property "Reference" "#PWR059" (at 91.44 88.9 0)
+    (property "Reference" "#PWR044" (at 91.44 88.9 0)
       (effects (font (size 1.27 1.27)) hide)
     )
@@
       (project "BPS-LeaderDaughter"
         (path "/2e9f4f51-d216-4952-a31c-e7104e0d4b1e/115507eb-1e24-4553-a6e1-1fcd332a9a2b"
-          (reference "#PWR059") (unit 1)
+          (reference "#PWR044") (unit 1)
         )
       )
@@
   (symbol (lib_id "power:GND") (at 47.625 83.185 0) (unit 1)
     (in_bom yes) (on_board yes) (dnp no) (fields_autoplaced)
-    (property "Reference" "#PWR056" (at 47.625 89.535 0)
+    (property "Reference" "#PWR041" (at 47.625 89.535 0)
       (effects (font (size 1.27 1.27)) hide)
     )
@@
       (project "BPS-LeaderDaughter"
         (path "/2e9f4f51-d216-4952-a31c-e7104e0d4b1e/115507eb-1e24-4553-a6e1-1fcd332a9a2b"
-          (reference "#PWR056") (unit 1)
-        )
-      )
+          (reference "#PWR041") (unit 1)
+        )
+      )

Commit message: Traced Champers <3
Connections:
- net GND: no longer U1.2, U2.2
- new net GND1: U1.2, U2.2
Changed lines of the file:
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@@
+    )
+  )
+  (symbol (lib_id "power:GND1") (at 91.44 82.55 0) (unit 1)
+    (in_bom yes) (on_board yes) (dnp no) (fields_autoplaced)
+    (property "Reference" "#PWR03" (at 91.44 88.9 0)
+      (effects (font (size 1.27 1.27)) hide)
+    )
+    (property "Value" "GND1" (at 91.44 87.63 0)
+      (effects (font (size 1.27 1.27)))
+    )
+    (property "Footprint" "" (at 91.44 82.55 0)
+      (effects (font (size 1.27 1.27)) hide)
+    )
+    (property "Datasheet" "" (at 91.44 82.55 0)
+      (effects (font (size 1.27 1.27)) hide)
+    )
+    (pin "1")
+    (instances
+      (project "BPS-LeaderDaughter"
+        (path "/2e9f4f51-d216-4952-a31c-e7104e0d4b1e/115507eb-1e24-4553-a6e1-1fcd332a9a2b"
+          (reference "#PWR03") (unit 1)
+        )
+      )
     )
   )
@@
     )
   )
-  (symbol (lib_id "power:GND") (at 91.44 82.55 0) (unit 1)
+  (symbol (lib_id "power:GND1") (at 47.625 83.185 0) (unit 1)
     (in_bom yes) (on_board yes) (dnp no) (fields_autoplaced)
-    (property "Reference" "#PWR044" (at 91.44 88.9 0)
+    (property "Reference" "#PWR012" (at 47.625 89.535 0)
       (effects (font (size 1.27 1.27)) hide)
     )
-    (property "Value" "GND" (at 91.44 87.63 0)
+    (property "Value" "GND1" (at 47.625 88.265 0)
       (effects (font (size 1.27 1.27)))
     )
-    (property "Footprint" "" (at 91.44 82.55 0)
+    (property "Footprint" "" (at 47.625 83.185 0)
       (effects (font (size 1.27 1.27)) hide)
     )
-    (property "Datasheet" "" (at 91.44 82.55 0)
+    (property "Datasheet" "" (at 47.625 83.185 0)
       (effects (font (size 1.27 1.27)) hide)
     )
@@
       (project "BPS-LeaderDaughter"
         (path "/2e9f4f51-d216-4952-a31c-e7104e0d4b1e/115507eb-1e24-4553-a6e1-1fcd332a9a2b"
-          (reference "#PWR044") (unit 1)
+          (reference "#PWR012") (unit 1)
         )
       )
@@
         )
       )
-    )
-  )
-  (symbol (lib_id "power:GND") (at 47.625 83.185 0) (unit 1)
-    (in_bom yes) (on_board yes) (dnp no) (fields_autoplaced)
-    (property "Reference" "#PWR041" (at 47.625 89.535 0)
-      (effects (font (size 1.27 1.27)) hide)
-    )
-    (property "Value" "GND" (at 47.625 88.265 0)
-      (effects (font (size 1.27 1.27)))
-    )
-    (property "Footprint" "" (at 47.625 83.185 0)
-      (effects (font (size 1.27 1.27)) hide)
-    )
-    (property "Datasheet" "" (at 47.625 83.185 0)
-      (effects (font (size 1.27 1.27)) hide)
-    )
-    (pin "1")
-    (instances
-      (project "BPS-LeaderDaughter"
-        (path "/2e9f4f51-d216-4952-a31c-e7104e0d4b1e/115507eb-1e24-4553-a6e1-1fcd332a9a2b"
-          (reference "#PWR041") (unit 1)
-        )
-      )

Commit message: last sanity check + part numbers (ready for review)
Parts:
- J8: P/N (none) -> 436500315; P/n 436500315 -> (none)
- R17: P/N (none) -> CRCW0805100KFKEAC
- R17, R19: value 604 -> 600; P/N (none) -> CRCW0805600RFKEAHP
- U1, U2: P/N (none) -> EL3H7(D)(TA)-VG; PN EL3H7(D)(TA)-VG -> (none)
Changed lines of the file:
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@@
+      (effects (font (size 1.27 1.27)) hide)
+    )
+    (property "P/N" "CRCW0805100KFKEAC" (at 56.515 102.87 0)
       (effects (font (size 1.27 1.27)) hide)
     )
@@
       (effects (font (size 1.27 1.27)) hide)
     )
-    (property "PN" "EL3H7(D)(TA)-VG" (at 102.87 87.63 0)
+    (property "PN" "" (at 102.87 87.63 0)
+      (effects (font (size 1.27 1.27)) hide)
+    )
+    (property "P/N" "EL3H7(D)(TA)-VG" (at 102.87 87.63 0)
       (effects (font (size 1.27 1.27)) hide)
     )
@@
       (effects (font (size 1.27 1.27)))
     )
-    (property "Value" "604" (at 118.745 83.82 90)
+    (property "Value" "600" (at 118.745 83.82 90)
       (effects (font (size 1.27 1.27)))
     )
@@
     )
     (property "Datasheet" "~" (at 118.745 78.74 0)
+      (effects (font (size 1.27 1.27)) hide)
+    )
+    (property "P/N" "CRCW0805600RFKEAHP" (at 118.745 78.74 0)
       (effects (font (size 1.27 1.27)) hide)
     )
@@
       (effects (font (size 1.27 1.27)) hide)
     )
-    (property "PN" "EL3H7(D)(TA)-VG" (at 59.055 88.265 0)
+    (property "PN" "" (at 59.055 88.265 0)
+      (effects (font (size 1.27 1.27)) hide)
+    )
+    (property "P/N" "EL3H7(D)(TA)-VG" (at 59.055 88.265 0)
       (effects (font (size 1.27 1.27)) hide)
     )
@@
       (effects (font (size 1.27 1.27)))
     )
-    (property "Value" "604" (at 74.93 81.915 90)
+    (property "Value" "600" (at 74.93 81.915 90)
       (effects (font (size 1.27 1.27)))
     )
@@
       (effects (font (size 1.27 1.27)) hide)
     )
+    (property "P/N" "CRCW0805600RFKEAHP" (at 74.93 76.2 0)
+      (effects (font (size 1.27 1.27)) hide)
+    )
     (pin "1")
     (pin "2")
@@
       (effects (font (size 1.27 1.27)) hide)
     )
-    (property "P/n" "436500315" (at 151.13 78.74 0)
+    (property "P/n" "" (at 151.13 78.74 0)
+      (effects (font (size 1.27 1.27)) hide)
+    )
+    (property "P/N" "436500315" (at 151.13 78.74 0)
       (effects (font (size 1.27 1.27)) hide)
     )
@@
       (effects (font (size 1.27 1.27)) hide)
     )
+    (property "P/N" "CRCW0805100KFKEAC" (at 100.33 102.235 0)
+      (effects (font (size 1.27 1.27)) hide)
+    )
