File: Ignition.kicad_sch (KiCad schematic)
At the start: 7 parts, among them J8 Conn_01x03, U1 EL3H7, U2 EL3H7

Commit message: fix ignition
Connections:
- net GND: no longer J8.3 (Pin_3)
- net GND1: now also J8.3 (Pin_3)
Changed lines of the file:
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@@
     (effects (font (size 1.27 1.27)) (justify left))
-  )
-  (symbol (lib_id "power:GND") (at 143.51 81.915 0) (unit 1)
-    (in_bom yes) (on_board yes) (dnp no) (fields_autoplaced)
-    (property "Reference" "#PWR047" (at 143.51 88.265 0)
-      (effects (font (size 1.27 1.27)) hide)
-    )
-    (property "Value" "GND" (at 143.51 86.995 0)
-      (effects (font (size 1.27 1.27)))
-    )
-    (property "Footprint" "" (at 143.51 81.915 0)
-      (effects (font (size 1.27 1.27)) hide)
-    )
-    (property "Datasheet" "" (at 143.51 81.915 0)
-      (effects (font (size 1.27 1.27)) hide)
-    )
-    (pin "1")
-    (instances
-      (project "BPS-LeaderDaughter"
-        (path "/2e9f4f51-d216-4952-a31c-e7104e0d4b1e/115507eb-1e24-4553-a6e1-1fcd332a9a2b"
-          (reference "#PWR047") (unit 1)
-        )
-      )
-    )
   )
   (symbol (lib_id "Device:R_Small") (at 56.515 102.87 180) (unit 1)
@@
         )
       )
+    )
+  )
+  (symbol (lib_id "power:GND1") (at 143.51 81.915 0) (unit 1)
+    (in_bom yes) (on_board yes) (dnp no) (fields_autoplaced)
+    (property "Reference" "#PWR023" (at 143.51 88.265 0)
+      (effects (font (size 1.27 1.27)) hide)
+    )
+    (property "Value" "GND1" (at 143.51 86.995 0)
+      (effects (font (size 1.27 1.27)))
+    )
+    (property "Footprint" "" (at 143.51 81.915 0)
+      (effects (font (size 1.27 1.27)) hide)
+    )
+    (property "Datasheet" "" (at 143.51 81.915 0)
+      (effects (font (size 1.27 1.27)) hide)
+    )
+    (pin "1")
+    (instances
+      (project "BPS-LeaderDaughter"
+        (path "/2e9f4f51-d216-4952-a31c-e7104e0d4b1e/115507eb-1e24-4553-a6e1-1fcd332a9a2b"
+          (reference "#PWR023") (unit 1)
+        )
+      )
