File: BPS-Leader.kicad_sch (KiCad schematic)
At the start: 8 parts, among them IC1 ADT7470ARQZ, J1 HV+ Connector, J2 HV- Connector, J3 Array Connector, J4 Fan1, J5 Fan2, J6 Fan3, J7 Fan4

Commit message: Preliminary Schematic Finished
Parts:
- removed IC1: ADT7470ARQZ, Package_SO:QSOP-16_3.9x4.9mm_P0.635mm, symbol utsvt-chips:ADT7470ARQZ
- added J8: lSOMconn, Connector_Molex:Molex_Micro-Fit_3.0_43650-0415_1x04_P3.00mm_Vertical, symbol Connector_Generic:Conn_01x04
- added J9: Strobe_Conn, Connector_Molex:Molex_Micro-Fit_3.0_43650-0215_1x02_P3.00mm_Vertical, symbol Connector_Generic:Conn_01x02
- added U1: EMC2305-1-AP-TR, footprints:QFN16_4x4MC_MCH-M, symbol 2024-11-02_21-04-42:EMC2305-1-AP-TR
- added U2: PeripheralSOM, UTSVT_Special:PeripheralSOM, symbol utsvt-misc:PeripheralSOM
- J1: renamed from J4; footprint (none) -> Connector_Molex:Molex_Micro-Fit_3.0_43650-0315_1x03_P3.00mm_Vertical
- J2: renamed from J5; footprint (none) -> Connector_Molex:Molex_Micro-Fit_3.0_43650-0315_1x03_P3.00mm_Vertical
- J3: renamed from J6; footprint (none) -> Connector_Molex:Molex_Micro-Fit_3.0_43650-0315_1x03_P3.00mm_Vertical
- J4: renamed from J7; footprint (none) -> Connector_Molex:Molex_Micro-Fit_3.0_43650-0315_1x03_P3.00mm_Vertical
- renumbered J1 to J5, J2 to J6, J3 to J7
Connections:
- net -SNSGND is gone; now on net GND: J6.4 (Pin_4)
- net aSNSGND is gone; now on net GND: J7.4 (Pin_4)
- net Array SENSE: now also U2.3 (SPI2_MISO)
- net CS: now also U2.19 (SPI1_NSS)
- net Fan1_EN: now also U1.5 (PWM1)
- net Fan2_EN: now also U1.7 (PWM2)
- net Fan3_EN: now also U1.9 (PWM3)
- net Fan4_EN: now also U1.13 (PWM4)
- net HV+ SENSE: now also U2.20 (PA1(ADC))
- net HV- SENSE: now also U2.18 (PA2(ADC))
- net SCLK: now also U2.13 (SPI1_SCK)
- net SDI: now also U2.17 (SPI1_MOSI)
- net SDO: now also U2.15 (SPI1_MISO)
- net Tach1: now also U1.6 (TACH1)
- net Tach2: now also U1.8 (TACH2)
- net Tach3: now also U1.10 (TACH3)
- net Tach4: now also U1.14 (TACH4)
- net +SNSGND renamed GND
- net GND: now also J8.1 (Pin_1), U1.HTAB (EPAD), U2.11 (GND), U2.4 (GND)
- new net +12V: J8.4 (Pin_4), U2.22 (+12V_In)
- new net +3.3V: U1.3 (VDD), U2.2 (+3.3V), U2.9 (+3.3V)
- new net ADDRSEL_FAN: U1.4 (ADDR_SEL), U2.7 (SPI2_NSS)
- new net AVDD: U2.10 (VDDA(3.3V))
- new net CAN_H: J8.2 (Pin_2), U2.23 (CAN_H)
- new net CAN_L: J8.3 (Pin_3), U2.21 (CAN_L)
- new net FanError: U1.12 (*ALERT), U2.5 (SPI2_SCK)
- new net GNDA: U2.12 (GNDA)
- new net SCL: U1.2 (SMCLK), U2.14 (I2C1_SCL)
- new net SDA: U1.1 (SMDATA), U2.16 (I2C1_SDA)
- new net Strobe Light/High: J9.1 (Pin_1)
- new net Strobe Light/Low: J9.2 (Pin_2)
- no-connect marks 0 -> 7
Other:
- added sheet Strobe Light (strobe.kicad_sch)
- sheet ADC1 ports: added AVDD; removed none

Commit message: Added pull-up resistors to the fan control chip
Parts:
- removed U1: EMC2305-1-AP-TR, footprints:QFN16_4x4MC_MCH-M, symbol 2024-11-02_21-04-42:EMC2305-1-AP-TR
Connections:
- net Strobe_EN: now reaches U2.1 (SPI2_MOSI)
- net Tach1 renamed F1TACH
- net Tach2 renamed F2TACH
- net Tach3 renamed F3TACH
- net Tach4 renamed F4TACH
- no-connect marks 7 -> 3
Other:
- added sheet Fan Control (fancntrlr.kicad_sch)
- sheet Strobe Light ports: added EN; removed none
- note added: "FAN CONTROL"
- moved on the sheet: J9

Commit message: Preliminary Schematic
Parts:
- added J1: E-STOP, Connector_Molex:Molex_Micro-Fit_3.0_43650-0215_1x02_P3.00mm_Vertical, symbol Connector_Generic:Conn_01x02
- added J12: ADC SPI, Connector_PinHeader_2.54mm:PinHeader_2x04_P2.54mm_Vertical, symbol Connector_Generic:Conn_02x04_Odd_Even
- added J13: Fan I2C, Connector_PinHeader_2.54mm:PinHeader_2x04_P2.54mm_Vertical, symbol Connector_Generic:Conn_02x04_Odd_Even
- added J9: Fan5, Connector_Molex:Molex_Micro-Fit_3.0_43650-0315_1x03_P3.00mm_Vertical, symbol Connector_Generic:Conn_01x03
- added JP1: E-Stop Bypass, Connector_PinHeader_2.54mm:PinHeader_1x02_P2.54mm_Vertical, symbol Jumper:Jumper_2_Small_Open
- renumbered J9 to J10, J8 to J11, J1 to J2, J2 to J3, J3 to J4, J4 to J5, J5 to J6, J6 to J8, U2 to U1
Connections:
- net ADDRSEL_FAN: now also J13.5 (Pin_5), J13.6 (Pin_6)
- net CS: now also J12.1 (Pin_1), J12.2 (Pin_2)
- net FanError: now also J13.7 (Pin_7), J13.8 (Pin_8)
- net HV-_EN: now also J1.1 (Pin_1), JP1.2 (B)
- net SCL: now also J13.3 (Pin_3), J13.4 (Pin_4)
- net SCLK: now also J12.5 (Pin_5), J12.6 (Pin_6)
- net SDA: now also J13.1 (Pin_1), J13.2 (Pin_2)
- net SDI: now also J12.3 (Pin_3), J12.4 (Pin_4)
- net SDO: now also J12.7 (Pin_7), J12.8 (Pin_8)
- new net F5TACH: J9.3 (Pin_3)
- new net Fan5/High: J9.1 (Pin_1)
- new net Fan5/Low: J9.2 (Pin_2)
- new net HV- Contactor/EN: J1.2 (Pin_2), JP1.1 (A)
Other:
- added sheet Fan5 (currentsense.kicad_sch)
- sheet ADC1 ports: added Fan5; removed none
- sheet Fan Control ports: added PWM5, TACH5; removed none
- note added: "Logic Analyzer"
- note added: "Strobe Light"
- moved on the sheet: J10, J8
