File: BPS-Leader.kicad_sch (KiCad schematic)
At the start: 21 parts, among them J10 Fan2, J11 Fan3, J12 Fan4, J13 HV+ Connector, J14 HV- Connector, J15 Array Connector, J17 Fan5, J18 Strobe_Conn, J19 ADC SPI, J2 CarPowerConnector, J20 Fan I2C, J21 Segment1 Connector, J22 Segment2 Connector, J3 CANconn, J4 Fan I2C, J5 CANconn2, J6 I-CanConn, J8 E-STOP, J9 Fan1

Commit message: everything should be finished now; tracks cleaned up, silkscreen issues fixed, new shunt/feedback/protection resistors chosen, BOM made, some other stuff i forgot probably
Parts:
- J1: P/N (none) -> 533072471
- J10, J11, J12, J17, J9: P/N (none) -> 436500315
- J13, J14, J15, J21, J22, J6: P/N (none) -> 436500244
- J18, J2, J3, J5, J8: P/N (none) -> 436500215
Changed lines of the file:
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@@
 			)
 		)
+		(property "P/N" "533072471"
+			(at 234.95 55.88 0)
+			(effects
+				(font
+					(size 1.27 1.27)
+				)
+				(hide yes)
+			)
+		)
 		(pin "7"
 		)
@@
 			)
 		)
-		(property "Datasheet" ""
+		(property "Datasheet" "https://www.molex.com/molex/search/partSearch?query=436500215&pQuery="
 			(at 198.12 69.85 0)
 			(effects
@@
 			)
 		)
+		(property "P/N" "436500215"
+			(at 198.12 69.85 0)
+			(effects
+				(font
+					(size 1.27 1.27)
+				)
+				(hide yes)
+			)
+		)
 		(pin "1"
 		)
@@
 			)
 		)
-		(property "Datasheet" "~"
+		(property "Datasheet" "https://www.mouser.com/ProductDetail/Molex/43650-0244?qs=XoD1gVtqLQuEe6RJ38AzJQ%3D%3D"
 			(at 158.75 129.54 0)
 			(effects
@@
 			)
 		)
+		(property "P/N" "436500244"
+			(at 158.75 129.54 0)
+			(effects
+				(font
+					(size 1.27 1.27)
+				)
+				(hide yes)
+			)
+		)
 		(pin "1"
 		)
@@
 			)
 		)
-		(property "Datasheet" "~"
+		(property "Datasheet" "https://www.mouser.com/ProductDetail/Molex/43650-0244?qs=XoD1gVtqLQuEe6RJ38AzJQ%3D%3D"
 			(at 67.31 81.28 0)
 			(effects
@@
 			)
 		)
+		(property "P/N" "436500244"
+			(at 67.31 81.28 0)
+			(effects
+				(font
+					(size 1.27 1.27)
+				)
+				(hide yes)
+			)
+		)
 		(pin "1"
 		)
@@
 			)
 		)
-		(property "Datasheet" "~"
+		(property "Datasheet" "https://www.molex.com/molex/search/partSearch?query=436500315&pQuery="
 			(at 55.88 123.19 0)
 			(effects
@@
 			)
 		)
+		(property "P/N" "436500315"
+			(at 55.88 123.19 0)
+			(effects
+				(font
+					(size 1.27 1.27)
+				)
+				(hide yes)
+			)
+		)
 		(pin "3"
 		)
@@
 			)
 		)
+		(property "P/N" ""
+			(at 48.26 83.82 0)
+			(effects
+				(font
+					(size 1.27 1.27)
+				)
+				(hide yes)
+			)
+		)
 		(pin "2"
 		)
@@
 			)
 		)
-		(property "Datasheet" "~"
+		(property "Datasheet" "https://www.molex.com/molex/search/partSearch?query=436500215&pQuery="
 			(at 109.22 64.77 0)
 			(effects
@@
 			)
 		)
+		(property "P/N" "436500215"
+			(at 109.22 64.77 0)
+			(effects
+				(font
+					(size 1.27 1.27)
+				)
+				(hide yes)
+			)
+		)
 		(pin "2"
 		)
@@
 			)
 		)
-		(property "Datasheet" "~"
+		(property "Datasheet" "https://www.mouser.com/ProductDetail/Molex/43650-0244?qs=XoD1gVtqLQuEe6RJ38AzJQ%3D%3D"
 			(at 67.31 62.23 0)
 			(effects
@@
 			)
 		)
+		(property "P/N" "436500244"
+			(at 67.31 62.23 0)
+			(effects
+				(font
+					(size 1.27 1.27)
+				)
+				(hide yes)
+			)
+		)
 		(pin "1"
 		)
@@
 			)
 		)
-		(property "Datasheet" "~"
+		(property "Datasheet" "https://www.molex.com/molex/search/partSearch?query=436500215&pQuery="
 			(at 203.2 85.09 0)
 			(effects
@@
 			)
 		)
+		(property "P/N" "436500215"
+			(at 203.2 85.09 0)
+			(effects
+				(font
+					(size 1.27 1.27)
+				)
+				(hide yes)
+			)
+		)
 		(pin "2"
 		)
@@
 			)
 		)
+		(property "P/N" ""
+			(at 146.05 59.69 0)
+			(effects
+				(font
+					(size 1.27 1.27)
+				)
+				(hide yes)
+			)
+		)
 		(pin "5"
 		)
@@
 			)
 		)
-		(property "Datasheet" "~"
+		(property "Datasheet" "https://www.mouser.com/ProductDetail/Molex/43650-0244?qs=XoD1gVtqLQuEe6RJ38AzJQ%3D%3D"
 			(at 67.31 100.33 0)
 			(effects
@@
 			)
 		)
+		(property "P/N" "436500244"
+			(at 67.31 100.33 0)
+			(effects
+				(font
+					(size 1.27 1.27)
+				)
+				(hide yes)
+			)
+		)
 		(pin "1"
 		)
@@
 			)
 		)
-		(property "Datasheet" "~"
+		(property "Datasheet" "https://www.molex.com/molex/search/partSearch?query=436500315&pQuery="
 			(at 106.68 123.19 0)
 			(effects
@@
 			)
 		)
+		(property "P/N" "436500315"
+			(at 106.68 123.19 0)
+			(effects
+				(font
+					(size 1.27 1.27)
+				)
+				(hide yes)
+			)
+		)
 		(pin "3"
 		)
@@
 			)
 		)
-		(property "Datasheet" "~"
+		(property "Datasheet" "https://www.mouser.com/ProductDetail/Molex/43650-0244?qs=XoD1gVtqLQuEe6RJ38AzJQ%3D%3D"
 			(at 203.2 49.53 0)
 			(effects
@@
 			)
 		)
+		(property "P/N" "436500244"
+			(at 203.2 49.53 0)
+			(effects
+				(font
+					(size 1.27 1.27)
+				)
+				(hide yes)
+			)
+		)
 		(pin "3"
 		)
@@
 			)
 		)
+		(property "P/N" ""
+			(at 146.05 43.18 0)
+			(effects
+				(font
+					(size 1.27 1.27)
+				)
+				(hide yes)
+			)
+		)
 		(pin "5"
 		)
@@
 			)
 		)
-		(property "Datasheet" "~"
+		(property "Datasheet" "https://www.mouser.com/ProductDetail/Molex/43650-0244?qs=XoD1gVtqLQuEe6RJ38AzJQ%3D%3D"
 			(at 158.75 147.32 0)
 			(effects
@@
 			)
 		)
+		(property "P/N" "436500244"
+			(at 158.75 147.32 0)
+			(effects
+				(font
+					(size 1.27 1.27)
+				)
+				(hide yes)
+			)
+		)
 		(pin "1"
 		)
@@
 			)
 		)
+		(property "P/N" ""
+			(at 146.05 26.67 0)
+			(effects
+				(font
+					(size 1.27 1.27)
+				)
+				(hide yes)
+			)
+		)
 		(pin "5"
 		)
@@
 			)
 		)
-		(property "Datasheet" "~"
+		(property "Datasheet" "https://www.molex.com/molex/search/partSearch?query=436500315&pQuery="
 			(at 55.88 142.24 0)
 			(effects
@@
 			)
 		)
+		(property "P/N" "436500315"
+			(at 55.88 142.24 0)
+			(effects
+				(font
+					(size 1.27 1.27)
+				)
+				(hide yes)
+			)
+		)
 		(pin "3"
 		)
@@
 			)
 		)
-		(property "Datasheet" "~"
+		(property "Datasheet" "https://www.molex.com/molex/search/partSearch?query=436500215&pQuery="
 			(at 203.2 92.71 0)
 			(effects
@@
 			)
 		)
+		(property "P/N" "436500215"
+			(at 203.2 92.71 0)
+			(effects
+				(font
+					(size 1.27 1.27)
+				)
+				(hide yes)
+			)
+		)
 		(pin "2"
 		)
@@
 			)
 		)
-		(property "Datasheet" "~"
+		(property "Datasheet" "https://www.molex.com/molex/search/partSearch?query=436500315&pQuery="
 			(at 55.88 180.34 0)
 			(effects
@@
 			)
 		)
+		(property "P/N" "436500315"
+			(at 55.88 180.34 0)
+			(effects
+				(font
+					(size 1.27 1.27)
+				)
+				(hide yes)
+			)
+		)
 		(pin "3"
 		)
@@
 			)
 		)
+		(property "P/N" "533072471"
+			(at 234.95 22.86 0)
+			(effects
+				(font
+					(size 1.27 1.27)
+				)
+				(hide yes)
+			)
+		)
 		(pin "7"
 		)
@@
 			)
 		)
-		(property "Datasheet" "~"
+		(property "Datasheet" "https://www.molex.com/molex/search/partSearch?query=436500215&pQuery="
 			(at 50.8 92.71 0)
 			(effects
@@
 			)
 		)
+		(property "P/N" "436500215"
+			(at 50.8 92.71 0)
+			(effects
+				(font
+					(size 1.27 1.27)
+				)
+				(hide yes)
+			)
+		)
 		(pin "2"
 		)
@@
 			)
 		)
-		(property "Datasheet" "~"
+		(property "Datasheet" "https://www.molex.com/molex/search/partSearch?query=436500315&pQuery="
 			(at 55.88 161.29 0)
 			(effects
@@
 			(at 55.88 161.29 0)
 			(effects
+				(font
+					(size 1.27 1.27)
+				)
+				(hide yes)
+			)
+		)
+		(property "P/N" "436500315"
+			(at 55.88 161.29 0)
+			(effects
