File: BPS-Leader.kicad_pcb (KiCad board)
At the start: 2 copper layers, 126 parts, among them J1 Fan1, J2 Fan2, J3 Fan3, J4 Fan4, J5 HV+ Connector, J6 HV- Connector, J7 Array Connector, J8 lSOMconn, J9 Strobe_Conn, Q1 IRLML0030, Q2 IRLML0030, Q3 IRLML0030, Q4 IRLML0030, Q5 IRLML0030, Q6 IRLML0030, Q7 IRLML0030, Q8 IRLML0030, U1 EMC2305-1-AP-TR, U10 INA180B1, U2 PeripheralSOM, U3 TLA2518IRTER, U4 INA180B1, U5 INA180B1, U6 INA180B1, U7 INA180B1, U8 INA180B1, U9 INA180B1

Commit message: Added pull-up resistors to the fan control chip
Parts:
- added R67: 100k, Resistor_SMD:R_0805_2012Metric, F.Cu at (94.5, 107.7)
- added R68: 100k, Resistor_SMD:R_0805_2012Metric, F.Cu at (94.5, 110.6)
- added R69: 100k, Resistor_SMD:R_0805_2012Metric, F.Cu at (94.5, 113.6)
- added R70: 100k, Resistor_SMD:R_0805_2012Metric, F.Cu at (94.5, 116.5)
- added R71: 100k, Resistor_SMD:R_0805_2012Metric, F.Cu at (98.9, 107.7)
- added R72: 100k, Resistor_SMD:R_0805_2012Metric, F.Cu at (98.9, 110.6)
- added R73: 100k, Resistor_SMD:R_0805_2012Metric, F.Cu at (98.9, 113.6)
- added R74: 100k, Resistor_SMD:R_0805_2012Metric, F.Cu at (98.9, 116.5)
- added R75: 100k, Resistor_SMD:R_0805_2012Metric, F.Cu at (103.3, 107.7)
- added R76: 100k, Resistor_SMD:R_0805_2012Metric, F.Cu at (103.3, 110.6)
- added R77: 100k, Resistor_SMD:R_0805_2012Metric, F.Cu at (103.3, 113.6)
- added R78: 100k, Resistor_SMD:R_0805_2012Metric, F.Cu at (103.3, 116.5)
- U1: footprint footprints:QFN16_4x4MC_MCH-M -> footprints:QFN16_4x4MC_MCH
- moved C4 81.0 mm to (94.5, 82.8)
- moved C5 81.0 mm to (94.5, 85.8)
- moved D1 81.0 mm to (107.8, 74.0)
- moved D2 81.0 mm to (107.8, 77.0)
- moved Q1 81.0 mm to (104.3, 83.7)
- moved R1 81.0 mm to (94.5, 74.0)
- moved R2 81.0 mm to (94.5, 76.9)
- moved R3 81.0 mm to (94.5, 79.9)
- moved R4 81.0 mm to (98.9, 74.0)
- moved R5 81.0 mm to (98.9, 76.9)
- moved R6 81.0 mm to (98.9, 79.9)
- moved R7 81.0 mm to (103.3, 74.0)
- moved R8 81.0 mm to (103.3, 76.9)
- moved R9 81.0 mm to (103.3, 79.9)
- moved U4 81.0 mm to (99.3, 83.7)
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Connections:
- net /Tach1 renamed /F1TACH
- net /Tach2 renamed /F2TACH
- net /Tach3 renamed /F3TACH
- net /Tach4 renamed /F4TACH
- R64 pad 1: /Strobe Light/EN -> /Strobe_EN
- R66 pad 1: /Strobe Light/EN -> /Strobe_EN
- U2 pad 1: unconnected-(U2-SPI2_MOSI-Pad1) -> /Strobe_EN

Commit message: adjusted shunt, added bypass caps to fan, high net removed, opamp output test pins added
Parts:
- removed R16, R18, R25, R27, R34, R36, R43, R45, R52, R54, R7, R9: R, Resistor_SMD:R_0805_2012Metric
- removed R64: 100k, Resistor_SMD:R_0805_2012Metric
- removed R66: 1k, Resistor_SMD:R_0805_2012Metric
- added C18: 1.1uF, Capacitor_SMD:C_0805_2012Metric, F.Cu at (127.0, 34.1)
- added C19: 2.2uF, Capacitor_SMD:C_0805_2012Metric, F.Cu at (127.0, 37.1)
- added C20: 0.16uF, Capacitor_SMD:C_0805_2012Metric, F.Cu at (89.2, 112.5)
- added C21: 0.16uF, Capacitor_SMD:C_0805_2012Metric, F.Cu at (127.0, 85.4)
- added C22: 0.16uF, Capacitor_SMD:C_0805_2012Metric, F.Cu at (105.7, 112.5)
- added C23: 0.16uF, Capacitor_SMD:C_0805_2012Metric, F.Cu at (127.0, 62.7)
- added C24: 0.16uF, Capacitor_SMD:C_0805_2012Metric, F.Cu at (56.3, 112.5)
- added C25: 0.16uF, Capacitor_SMD:C_0805_2012Metric, F.Cu at (72.8, 112.5)
- added C26: 0.16uF, Capacitor_SMD:C_0805_2012Metric, F.Cu at (127.0, 108.0)
- added C27: 0.16uF, Capacitor_SMD:C_0805_2012Metric, F.Cu at (127.0, 40.1)
- added C28: 1uF, Capacitor_SMD:C_0805_2012Metric, F.Cu at (139.0, 108.3)
- added C29: 1uF, Capacitor_SMD:C_0805_2012Metric, F.Cu at (139.0, 111.3)
- added D17: Green, Diode_SMD:D_0805_2012Metric, F.Cu at (122.5, 34.1)
- added D18: 1N448W, Diode_SMD:D_0805_2012Metric, F.Cu at (122.5, 37.1)
- added D19: 1N448W, Diode_SMD:D_0805_2012Metric, F.Cu at (84.8, 112.5)
- added D20: 1N448W, Diode_SMD:D_0805_2012Metric, F.Cu at (122.5, 85.4)
- added D21: 1N448W, Diode_SMD:D_0805_2012Metric, F.Cu at (101.3, 112.5)
- added D22: 1N448W, Diode_SMD:D_0805_2012Metric, F.Cu at (122.5, 62.8)
- added D23: 1N448W, Diode_SMD:D_0805_2012Metric, F.Cu at (51.9, 112.5)
- added D24: 1N448W, Diode_SMD:D_0805_2012Metric, F.Cu at (68.4, 112.5)
- added D25: 1N448W, Diode_SMD:D_0805_2012Metric, F.Cu at (122.5, 108.1)
- added D26: 1N448W, Diode_SMD:D_0805_2012Metric, F.Cu at (122.5, 40.1)
- added D27: 1N448W, Diode_SMD:D_0805_2012Metric, F.Cu at (84.8, 115.6)
- added D28: 1N448W, Diode_SMD:D_0805_2012Metric, F.Cu at (122.5, 88.5)
- added D29: 1N448W, Diode_SMD:D_0805_2012Metric, F.Cu at (101.3, 115.6)
- added D30: 1N448W, Diode_SMD:D_0805_2012Metric, F.Cu at (122.5, 65.8)
- added D31: 1N448W, Diode_SMD:D_0805_2012Metric, F.Cu at (51.9, 115.6)
- added D32: 1N448W, Diode_SMD:D_0805_2012Metric, F.Cu at (68.4, 115.6)
- added D33: 1N448W, Diode_SMD:D_0805_2012Metric, F.Cu at (122.5, 111.1)
- added D34: 1N448W, Diode_SMD:D_0805_2012Metric, F.Cu at (122.5, 43.2)
- added J10: Strobe_Conn, Connector_Molex:Molex_Micro-Fit_3.0_43650-0215_1x02_P3.00mm_Vertical, F.Cu at (106.5, 43.9)
- added J11: ADC SPI, Connector_PinHeader_2.54mm:PinHeader_2x04_P2.54mm_Vertical, F.Cu at (47.6, 86.0)
- added J12: Fan I2C, Connector_PinHeader_2.54mm:PinHeader_2x04_P2.54mm_Vertical, F.Cu at (54.8, 86.0)
- added J13: lSOMconn, Connector_Molex:Molex_Micro-Fit_3.0_43650-0415_1x04_P3.00mm_Vertical, F.Cu at (91.9, 98.6)
- added J14: Fan5_test, Connector_PinHeader_2.54mm:PinHeader_1x01_P2.54mm_Vertical, F.Cu at (62.0, 86.0)
- added J15: Fan1_test, Connector_PinHeader_2.54mm:PinHeader_1x01_P2.54mm_Vertical, F.Cu at (62.0, 90.7)
- added J16: Fan2_test, Connector_PinHeader_2.54mm:PinHeader_1x01_P2.54mm_Vertical, F.Cu at (66.6, 86.0)
- added J17: Fan3_test, Connector_PinHeader_2.54mm:PinHeader_1x01_P2.54mm_Vertical, F.Cu at (66.6, 90.7)
- added J18: Fan4_test, Connector_PinHeader_2.54mm:PinHeader_1x01_P2.54mm_Vertical, F.Cu at (71.3, 86.0)
- added J19: Array_test, Connector_PinHeader_2.54mm:PinHeader_1x01_P2.54mm_Vertical, F.Cu at (71.3, 90.7)
- added J20: HV-_test, Connector_PinHeader_2.54mm:PinHeader_1x01_P2.54mm_Vertical, F.Cu at (75.9, 86.0)
- added J21: HV+_test, Connector_PinHeader_2.54mm:PinHeader_1x01_P2.54mm_Vertical, F.Cu at (75.9, 90.7)
- added JP1: E-Stop Bypass, Connector_PinHeader_2.54mm:PinHeader_1x02_P2.54mm_Vertical, F.Cu at (80.6, 86.0)
- added Q9: IRLML0030, Package_TO_SOT_SMD:SOT-23, F.Cu at (127.9, 47.1)
- added R79: 5, Resistor_SMD:R_0805_2012Metric, F.Cu at (118.1, 45.8)
- added R80: 5, Resistor_SMD:R_0805_2012Metric, F.Cu at (118.1, 48.8)
- added R82: 0.9, Resistor_SMD:R_0805_2012Metric, F.Cu at (118.1, 51.7)
- added U11: INA180A2, Package_TO_SOT_SMD:SOT-23-5, F.Cu at (122.9, 47.1)
- J1: value Fan1 -> E-STOP; footprint Connector_Molex:Molex_Micro-Fit_3.0_43650-0315_1x03_P3.00mm_Vertical -> Connector_Molex:Molex_Micro-Fit_3.0_43650-0215_1x02_P3.00mm_Vertical
- J2: value Fan2 -> Fan1
- J3: value Fan3 -> Fan2
- J4: value Fan4 -> Fan3
- J5: value HV+ Connector -> Fan4; footprint Connector_Molex:Molex_Micro-Fit_3.0_43650-0415_1x04_P3.00mm_Vertical -> Connector_Molex:Molex_Micro-Fit_3.0_43650-0315_1x03_P3.00mm_Vertical
- J6: value HV- Connector -> HV+ Connector
- J8: value lSOMconn -> HV- Connector
- J9: value Strobe_Conn -> Fan5; footprint Connector_Molex:Molex_Micro-Fit_3.0_43650-0215_1x02_P3.00mm_Vertical -> Connector_Molex:Molex_Micro-Fit_3.0_43650-0315_1x03_P3.00mm_Vertical
- R13, R22, R31, R4, R40, R49, R61: value R -> 3m
- R14, R15, R23, R24, R32, R33, R41, R42, R5, R50, R51, R6, R62, R63: value R -> 5
- R17, R26, R35, R44, R53, R8: value R -> 0.9
- R58: value R -> 100k
- R59: value R -> 10k
- R60: value R -> 1k
- R65: value 10k -> 0.9
- R72: value 100k -> 33k
- R74: value 100k -> 15k
- R76: value 100k -> 10k
- R77: value 100k -> 1k
- R78: value 100k -> 3m
- U1: value EMC2305-1-AP-TR -> PeripheralSOM; footprint footprints:QFN16_4x4MC_MCH -> UTSVT_Special:PeripheralSOM
- U10: value INA180B1 -> EMC2305-1-AP-TR; footprint Package_TO_SOT_SMD:SOT-23-5 -> footprints:QFN16_4x4MC_MCH
- U2: value PeripheralSOM -> TLA2518IRTER; footprint UTSVT_Special:PeripheralSOM -> footprints:WQFN16_RTE_TEX
- U3: value TLA2518IRTER -> INA180A2; footprint footprints:WQFN16_RTE_TEX -> Package_TO_SOT_SMD:SOT-23-5
- U4, U5, U6, U7, U8, U9: value INA180B1 -> INA180A2
- moved C10 110.3 mm to (127.0, 56.7)
- moved C11 110.3 mm to (127.0, 59.7)
- moved R28 98.1 mm to (118.1, 56.7)
- moved R29 98.1 mm to (118.1, 59.6)
- moved R30 98.1 mm to (118.1, 62.6)
- moved Q4 96.5 mm to (127.9, 69.8)
- moved U2 91.9 mm to (139.5, 80.6)
- moved D7 90.6 mm to (122.5, 56.7)
- moved D8 90.6 mm to (122.5, 59.8)
- moved R31 90.1 mm to (118.1, 65.5)
- moved R32 90.1 mm to (118.1, 68.5)
- moved R33 90.1 mm to (118.1, 71.4)
- moved R35 83.7 mm to (118.1, 74.4)
- moved U1 75.7 mm to (64.6, 54.9)
- moved R75 75.1 mm to (118.1, 34.0)
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Connections:
- C1 pad 1: /AVDD -> +3.3V
- C1 pad 2: GNDA -> GND
- C2 pad 2: Net-(U3-DECAP) -> Net-(U2-DECAP)
- D1 pad 1: /HV+ contactor/Low -> /Fan5/Low
- D10 pad 2: /Fan2/Low -> /Fan1/Low
- D11 pad 1: /Fan3/Low -> /Fan2/Low
- D12 pad 2: /Fan3/Low -> /Fan2/Low
- D13 pad 1: /Fan4/Low -> /Strobe Light/Low
- D14 pad 2: /Fan4/Low -> /Strobe Light/Low
- D15 pad 1: /Strobe Light/Low -> /Fan3/Low
- D16 pad 2: /Strobe Light/Low -> /Fan3/Low
- D2 pad 2: /HV+ contactor/Low -> /Fan5/Low
- D3 pad 1: /HV- Contactor/Low -> /HV+ contactor/Low
- D4 pad 2: /HV- Contactor/Low -> /HV+ contactor/Low
- D5 pad 1: /Array Contactor/Low -> /HV- Contactor/Low
- D6 pad 2: /Array Contactor/Low -> /HV- Contactor/Low
- D7 pad 1: /Fan1/Low -> /Array Contactor/Low
- D8 pad 2: /Fan1/Low -> /Array Contactor/Low
- D9 pad 1: /Fan2/Low -> /Fan1/Low
- J1 pad 1: /Fan1/High -> /HV-_EN
- J1 pad 2: /Fan1/Low -> /HV- Contactor/EN
- J2 pad 1: /Fan2/High -> +12V
- J2 pad 2: /Fan2/Low -> /Fan1/Low
- J2 pad 3: /F2TACH -> /F1TACH
- J3 pad 1: /Fan3/High -> +12V
- J3 pad 2: /Fan3/Low -> /Fan2/Low
- J3 pad 3: /F3TACH -> /F2TACH
- J4 pad 1: /Fan4/High -> +12V
- J4 pad 2: /Fan4/Low -> /Fan3/Low
- J4 pad 3: /F4TACH -> /F3TACH
- J5 pad 1: /HV+ contactor/High -> +12V
- J5 pad 2: /HV+ contactor/Low -> /Fan4/Low
- J5 pad 3: /HV+ SENSE -> /F4TACH
- J6 pad 1: /HV- Contactor/High -> +12V
- J6 pad 2: /HV- Contactor/Low -> /HV+ contactor/Low
- J6 pad 3: /HV- SENSE -> /HV+ SENSE
- J7 pad 1: /Array Contactor/High -> +12V
- J8 pad 1: GND -> +12V
- J8 pad 2: /CAN_H -> /HV- Contactor/Low
- J8 pad 3: /CAN_L -> /HV- SENSE
- J8 pad 4: +12V -> GND
- J9 pad 2: /Strobe Light/Low -> /Fan5/Low
- Q1 pad 3: /HV+ contactor/Low -> /Fan5/Low
- Q2 pad 3: /HV- Contactor/Low -> /HV+ contactor/Low
- Q3 pad 3: /Array Contactor/Low -> /HV- Contactor/Low
- Q4 pad 3: /Fan1/Low -> /Array Contactor/Low
- Q5 pad 3: /Fan2/Low -> /Fan1/Low
- Q6 pad 3: /Fan3/Low -> /Fan2/Low
- Q7 pad 3: /Fan4/Low -> /Strobe Light/Low
- Q8 pad 3: /Strobe Light/Low -> /Fan3/Low
- R1 pad 1: /HV+_EN -> /Fan5_EN
- R10 pad 1: /HV-_EN -> /HV+_EN
- R12 pad 1: /HV-_EN -> /HV+_EN
- R13 pad 2: /HV- Contactor/High -> Net-(R13-Pad2)
- R14 pad 2: Net-(U5-+) -> Net-(U4-+)
- R15 pad 1: /HV- Contactor/High -> Net-(R13-Pad2)
- R15 pad 2: Net-(U5--) -> Net-(U4--)
- R17 pad 1: Net-(U5--) -> Net-(U4--)
- R17 pad 2: Net-(R17-Pad2) -> /HV+_Current
- R19 pad 1: /Array_EN -> /HV- Contactor/EN
- R21 pad 1: /Array_EN -> /HV- Contactor/EN
- R22 pad 2: /Array Contactor/High -> Net-(R22-Pad2)
- R23 pad 2: Net-(U6-+) -> Net-(U5-+)
- R24 pad 1: /Array Contactor/High -> Net-(R22-Pad2)
- R24 pad 2: Net-(U6--) -> Net-(U5--)
- R26 pad 1: Net-(U6--) -> Net-(U5--)
- R26 pad 2: Net-(R26-Pad2) -> /HV-_Current
- R28 pad 1: /Fan1_EN -> /Array_EN
- R3 pad 1: /HV+_EN -> /Fan5_EN
- R30 pad 1: /Fan1_EN -> /Array_EN
- R31 pad 2: /Fan1/High -> Net-(R31-Pad2)
- R32 pad 2: Net-(U7-+) -> Net-(U6-+)
- R33 pad 1: /Fan1/High -> Net-(R31-Pad2)
- R33 pad 2: Net-(U7--) -> Net-(U6--)
- R35 pad 1: Net-(U7--) -> Net-(U6--)
- R35 pad 2: Net-(R35-Pad2) -> /Array_Current
- R37 pad 1: /Fan2_EN -> /Fan1_EN
- R39 pad 1: /Fan2_EN -> /Fan1_EN
- R4 pad 2: /HV+ contactor/High -> Net-(R4-Pad2)
- R40 pad 2: /Fan2/High -> Net-(R40-Pad2)
- R41 pad 2: Net-(U8-+) -> Net-(U7-+)
- R42 pad 1: /Fan2/High -> Net-(R40-Pad2)
- R42 pad 2: Net-(U8--) -> Net-(U7--)
- R44 pad 1: Net-(U8--) -> Net-(U7--)
- R44 pad 2: Net-(R44-Pad2) -> /FAN1_Current
- R46 pad 1: /Fan3_EN -> /Fan2_EN
- R48 pad 1: /Fan3_EN -> /Fan2_EN
- R49 pad 2: /Fan3/High -> Net-(R49-Pad2)
- R5 pad 2: Net-(U4-+) -> Net-(U3-+)
- R50 pad 2: Net-(U9-+) -> Net-(U8-+)
- R51 pad 1: /Fan3/High -> Net-(R49-Pad2)
- R51 pad 2: Net-(U9--) -> Net-(U8--)
- R53 pad 1: Net-(U9--) -> Net-(U8--)
- R53 pad 2: Net-(R53-Pad2) -> /FAN2_Current
- R55 pad 1: /Fan4_EN -> /Strobe_EN
- R57 pad 1: /Fan4_EN -> /Strobe_EN
- R58 pad 1: +12V -> /Fan3_EN
- R58 pad 2: /Fan4/High -> GND
- R59 pad 2: Net-(U10-+) -> Net-(D15-A)
- R6 pad 1: /HV+ contactor/High -> Net-(R4-Pad2)
- R6 pad 2: Net-(U4--) -> Net-(U3--)
- R60 pad 1: /Fan4/High -> /Fan3_EN
- R60 pad 2: Net-(U10--) -> Net-(Q8-G)
- R61 pad 1: Net-(U10-+) -> +12V
- R61 pad 2: GND -> Net-(R61-Pad2)
- R62 pad 1: Net-(U10--) -> +12V
- R62 pad 2: Net-(R62-Pad2) -> Net-(U9-+)
- R63 pad 1: Net-(R62-Pad2) -> Net-(R61-Pad2)
- R63 pad 2: /FAN4_Current -> Net-(U9--)
- R65 pad 1: +12V -> Net-(U9--)
- R65 pad 2: Net-(D15-A) -> /FAN3_Current
- R67 pad 2: /ADDRSEL_FAN -> /F1TACH
- R68 pad 2: /Fan1_EN -> /F2TACH
- R69 pad 2: /Fan2_EN -> /F3TACH
- R70 pad 2: /F1TACH -> /F4TACH
- R71 pad 2: /Fan3_EN -> /F5TACH
- R72 pad 2: /Fan4_EN -> /ADDRSEL_FAN
- R73 pad 2: /F2TACH -> /FanError
- R74 pad 2: /F3TACH -> Net-(U10-CLK)
- R75 pad 1: +3.3V -> /Fan4_EN
- R75 pad 2: /F4TACH -> GND
- R76 pad 1: +3.3V -> +12V
- R76 pad 2: /SDA -> Net-(D17-A)
- R77 pad 1: +3.3V -> /Fan4_EN
- R77 pad 2: /SCL -> Net-(Q9-G)
- R78 pad 1: +3.3V -> +12V
- R78 pad 2: /FanError -> Net-(R78-Pad2)
- R8 pad 1: Net-(U4--) -> Net-(U3--)
- R8 pad 2: Net-(R8-Pad2) -> /FAN5_Current
- U1 pad 1: /SDA -> /Strobe_EN
- U1 pad 10: /F3TACH -> unconnected-(U1-VDDA(3.3V)-Pad10)
- U1 pad 11: unconnected-(U1-CLK-Pad11) -> GND
- U1 pad 12: /FanError -> GNDA
- U1 pad 13: /Fan4_EN -> /SCLK
- U1 pad 14: /F4TACH -> /SCL
- U1 pad 15: unconnected-(U1-PWM5-Pad15) -> /SDO
- U1 pad 16: unconnected-(U1-TACH5-Pad16) -> /SDA
- U1 pad 2: /SCL -> +3.3V
- U1 pad 3: +3.3V -> /Array SENSE
- U1 pad 4: /ADDRSEL_FAN -> GND
- U1 pad 5: /Fan1_EN -> /FanError
- U1 pad 6: /F1TACH -> unconnected-(U1-I2C2_SDA-Pad6)
- U1 pad 7: /Fan2_EN -> /ADDRSEL_FAN
- U1 pad 8: /F2TACH -> unconnected-(U1-I2C2_SCL-Pad8)
- U1 pad 9: /Fan3_EN -> +3.3V
- U10 pad 1: Net-(U10-+) -> /SDA
- U10 pad 2: GND -> /SCL
- U10 pad 3: Net-(U10--) -> +3.3V
- U10 pad 4: Net-(R62-Pad2) -> /ADDRSEL_FAN
- U10 pad 5: +3.3V -> /Fan1_EN
- U2 pad 1: /Strobe_EN -> /Array_Current
- U2 pad 10: /AVDD -> +3.3V
- U2 pad 11: GND -> /CS
- U2 pad 12: GNDA -> /SDO
- U2 pad 14: /SCL -> /SDI
- U2 pad 15: /SDO -> /HV+_Current
- U2 pad 16: /SDA -> /HV-_Current
- U2 pad 17: /SDI -> GND
- U2 pad 2: +3.3V -> /FAN1_Current
- U2 pad 3: /Array SENSE -> /FAN2_Current
- U2 pad 4: GND -> /FAN3_Current
- U2 pad 5: /FanError -> /FAN4_Current
- U2 pad 6: unconnected-(U2-I2C2_SDA-Pad6) -> /FAN5_Current
- U2 pad 7: /ADDRSEL_FAN -> +3.3V
- U2 pad 8: unconnected-(U2-I2C2_SCL-Pad8) -> Net-(U2-DECAP)
- U2 pad 9: +3.3V -> GND
- U3 pad 1: /Array_Current -> /FAN5_Current
- U3 pad 2: /FAN1_Current -> GND
- U3 pad 3: /FAN2_Current -> Net-(U3-+)
- U3 pad 4: /FAN3_Current -> Net-(U3--)
- U3 pad 5: /FAN4_Current -> +3.3V
- U4 pad 1: Net-(U4-+) -> /HV+_Current
- U4 pad 3: Net-(U4--) -> Net-(U4-+)
- U4 pad 4: Net-(R8-Pad2) -> Net-(U4--)
- U5 pad 1: Net-(U5-+) -> /HV-_Current
- U5 pad 3: Net-(U5--) -> Net-(U5-+)
- U5 pad 4: Net-(R17-Pad2) -> Net-(U5--)
- U6 pad 1: Net-(U6-+) -> /Array_Current
- U6 pad 3: Net-(U6--) -> Net-(U6-+)
- U6 pad 4: Net-(R26-Pad2) -> Net-(U6--)
- U7 pad 1: Net-(U7-+) -> /FAN1_Current
- U7 pad 3: Net-(U7--) -> Net-(U7-+)
- U7 pad 4: Net-(R35-Pad2) -> Net-(U7--)
- U8 pad 1: Net-(U8-+) -> /FAN2_Current
- U8 pad 3: Net-(U8--) -> Net-(U8-+)
- U8 pad 4: Net-(R44-Pad2) -> Net-(U8--)
- U9 pad 1: Net-(U9-+) -> /FAN3_Current
- U9 pad 3: Net-(U9--) -> Net-(U9-+)
- U9 pad 4: Net-(R53-Pad2) -> Net-(U9--)

Commit message: preliminary schematic completed
Parts:
- moved U1 158.1 mm to (222.7, 53.3), turned to -90 degrees
- renumbered C8 to C10, C22 to C11, C9 to C12, C10 to C13, C23 to C14, C11 to C15, C12 to C16, C24 to C17, C13 to C18, C14 to C19, C25 to C20, C15 to C21, C16 to C22, C26 to C23, C17 to C24, C28 to C25, C29 to C26, C18 to C27, C27 to C28, C19 to C29, C20 to C5, C5 to C6, C6 to C7, C21 to C8, C7 to C9, D6 to D10, D29 to D11, D21 to D12, D7 to D13, D8 to D14, D30 to D15, D22 to D16, D9 to D17, D10 to D18, D31 to D19, D23 to D20, D11 to D21, D12 to D22, D32 to D23, D13 to D25, D14 to D26, D15 to D27, D16 to D28, D33 to D29, D27 to D3, D25 to D30, D17 to D31, D18 to D32, D34 to D33, D26 to D34, D19 to D4, D3 to D5, D4 to D6, D28 to D7, D20 to D8, D5 to D9, J20 to J1, J3 to J10, J4 to J11, J5 to J12, J6 to J13, J8 to J14, J7 to J15, J14 to J16, J9 to J17, J10 to J18, J11 to J19, J21 to J2, J12 to J20, J13 to J21, J19 to J3, J15 to J4, J16 to J5, J17 to J6, J18 to J7, J1 to J8, J2 to J9, R12 to R10, R13 to R11, R14 to R12, R15 to R13, R17 to R14, R19 to R15, R20 to R16, R21 to R17, R22 to R18, R23 to R19, R24 to R20, R26 to R21, R28 to R22, R29 to R23, R30 to R24, R31 to R25, R32 to R26, R33 to R27, R35 to R28, R37 to R29, R38 to R30, R39 to R31, R40 to R32, R41 to R33, R42 to R34, R44 to R35, R46 to R36, R47 to R37, R48 to R38, R49 to R39, R50 to R40, R51 to R41, R53 to R42, R55 to R43, R56 to R44, R57 to R45, R58 to R46, R59 to R47, R60 to R48, R61 to R49, R62 to R50, R63 to R51, R65 to R52, R67 to R53, R68 to R54, R69 to R55, R70 to R56, R71 to R57, R72 to R58, R73 to R59, R74 to R60, R75 to R61, R76 to R62, R77 to R63, R78 to R64, R79 to R65, R80 to R66, R82 to R67, R8 to R7, R10 to R8, R11 to R9

Commit message: Very rough layout of the board - maybe too long?
Parts:
- removed D26: 1N448W, Diode_SMD:D_0805_2012Metric
- removed J1: HV-_test, Connector_PinHeader_2.54mm:PinHeader_1x01_P2.54mm_Vertical
- removed J16: Fan5_test, Connector_PinHeader_2.54mm:PinHeader_1x01_P2.54mm_Vertical
- removed J2: HV+_test, Connector_PinHeader_2.54mm:PinHeader_1x01_P2.54mm_Vertical
- removed J3: Array_test, Connector_PinHeader_2.54mm:PinHeader_1x01_P2.54mm_Vertical
- removed J5: Fan2_test, Connector_PinHeader_2.54mm:PinHeader_1x01_P2.54mm_Vertical
- removed J6: Fan3_test, Connector_PinHeader_2.54mm:PinHeader_1x01_P2.54mm_Vertical
- removed J7: Fan4_test, Connector_PinHeader_2.54mm:PinHeader_1x01_P2.54mm_Vertical
- added J22: Segment2 Connector, Connector_Molex:Molex_Micro-Fit_3.0_43650-0415_1x04_P3.00mm_Vertical, F.Cu at (176.4, 158.8)
- added J23: lSOMconn, Connector_Molex:Molex_Micro-Fit_3.0_43650-0415_1x04_P3.00mm_Vertical, F.Cu at (133.8, 41.8)
- added Q10: IRLML0030, Package_TO_SOT_SMD:SOT-23, F.Cu at (142.3, 102.2)
- added Q11: IRLML0030, Package_TO_SOT_SMD:SOT-23, F.Cu at (142.1, 81.6)
- added R68: 3m, Resistor_SMD:R_0805_2012Metric, F.Cu at (143.2, 78.0)
- added R69: 5, Resistor_SMD:R_0805_2012Metric, F.Cu at (145.9, 77.0)
- added R70: 5, Resistor_SMD:R_0805_2012Metric, F.Cu at (145.9, 79.1)
- added R71: 0.9, Resistor_SMD:R_0805_2012Metric, F.Cu at (150.5, 81.4)
- J21: value lSOMconn -> Segment1 Connector
- J4: value Fan1_test -> Fan I2C; footprint Connector_PinHeader_2.54mm:PinHeader_1x01_P2.54mm_Vertical -> Connector_PinHeader_2.54mm:PinHeader_2x04_P2.54mm_Vertical
- R10, R63: value 1k -> 100k
- R11, R49: value 3m -> 1k
- R12, R19, R26, R33, R40, R50, R65: value 5 -> 100k
- R13, R20, R27, R34, R41, R51, R66: value 5 -> 10k
- R14, R21, R28, R35, R42, R52, R67: value 0.9 -> 1k
- R15, R22, R29, R36, R43, R53: value 100k -> 3m
- R16, R23, R30, R37, R44: value 10k -> 5
- R17, R24, R31, R38, R45: value 1k -> 5
- R18, R25, R32, R39: value 3m -> 0.9
- R46, R56: value 100k -> 0.9
- R47: value 10k -> 100k
- R48: value 1k -> 10k
- R54, R55: value 100k -> 5
- R58: value 33k -> 100k
- R60: value 15k -> 100k
- R62: value 10k -> 33k
- R64: value 3m -> 15k
- R9: value 10k -> 1k
- moved R29 129.1 mm to (176.1, 116.2), turned to 90 degrees
- moved R30 126.1 mm to (173.3, 117.2), turned to 180 degrees
- moved R31 125.9 mm to (173.3, 115.1), turned to 180 degrees
- moved J19 124.6 mm to (170.3, 107.3), turned to 180 degrees
- moved Q5 122.3 mm to (177.1, 143.6)
- moved R32 121.3 mm to (168.8, 112.9), turned to 180 degrees
- moved J8 120.9 mm to (133.9, 153.8), turned to -90 degrees
- moved J4 116.8 mm to (177.5, 107.3), turned to 180 degrees
- moved J20 110.7 mm to (163.4, 107.3), turned to 180 degrees
- moved J14 110.5 mm to (185.4, 149.6), turned to 90 degrees
- moved J13 108.8 mm to (185.4, 130.6), turned to 90 degrees
- moved R22 107.5 mm to (176.1, 147.1), turned to 90 degrees
- moved R23 104.3 mm to (173.3, 148.2), turned to 180 degrees
- moved D20 104.0 mm to (155.1, 125.3)
- moved D19 103.9 mm to (155.1, 127.3)
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Connections:
- J21 pad 1: GND -> +12V
- J21 pad 2: /CAN_H -> /Battery segments/Low1
- J21 pad 3: /CAN_L -> /Seg1Sense
- J21 pad 4: +12V -> GND
- Q2 pad 3: /HV+ contactor/Low -> /Battery segments/Low1
- Q3 pad 3: /HV- Contactor/Low -> /Battery segments/Low2
- Q4 pad 3: /Array Contactor/Low -> /HV+ contactor/Low
- Q5 pad 3: /Fan1/Low -> /HV- Contactor/Low
- Q6 pad 3: /Fan2/Low -> /Array Contactor/Low
- Q7 pad 3: /Strobe Light/Low -> /Fan1/Low
- Q8 pad 3: /Fan3/Low -> /Fan2/Low
- Q9 pad 3: /Fan4/Low -> /Strobe Light/Low
- R10 pad 1: /HV+_EN -> /SegEN
- R10 pad 2: Net-(Q2-G) -> GND
- R11 pad 1: +12V -> /SegEN
- R11 pad 2: Net-(R11-Pad2) -> Net-(Q3-G)
- R12 pad 1: +12V -> /HV+_EN
- R12 pad 2: Net-(U4-+) -> GND
- R13 pad 1: Net-(R11-Pad2) -> +12V
- R13 pad 2: Net-(U4--) -> Net-(D5-A)
- R14 pad 1: Net-(U4--) -> /HV+_EN
- R14 pad 2: /HV+_Current -> Net-(Q4-G)
- R15 pad 1: /HV- Contactor/EN -> +12V
- R15 pad 2: GND -> Net-(R15-Pad2)
- R16 pad 2: Net-(D9-A) -> Net-(U4-+)
- R17 pad 1: /HV- Contactor/EN -> Net-(R15-Pad2)
- R17 pad 2: Net-(Q3-G) -> Net-(U4--)
- R18 pad 1: +12V -> Net-(U4--)
- R18 pad 2: Net-(R18-Pad2) -> /HV+_Current
- R19 pad 1: +12V -> /HV- Contactor/EN
- R19 pad 2: Net-(U5-+) -> GND
- R20 pad 1: Net-(R18-Pad2) -> +12V
- R20 pad 2: Net-(U5--) -> Net-(D9-A)
- R21 pad 1: Net-(U5--) -> /HV- Contactor/EN
- R21 pad 2: /HV-_Current -> Net-(Q5-G)
- R22 pad 1: /Array_EN -> +12V
- R22 pad 2: GND -> Net-(R22-Pad2)
- R23 pad 2: Net-(D13-A) -> Net-(U5-+)
- R24 pad 1: /Array_EN -> Net-(R22-Pad2)
- R24 pad 2: Net-(Q4-G) -> Net-(U5--)
- R25 pad 1: +12V -> Net-(U5--)
- R25 pad 2: Net-(R25-Pad2) -> /HV-_Current
- R26 pad 1: +12V -> /Array_EN
- R26 pad 2: Net-(U6-+) -> GND
- R27 pad 1: Net-(R25-Pad2) -> +12V
- R27 pad 2: Net-(U6--) -> Net-(D13-A)
- R28 pad 1: Net-(U6--) -> /Array_EN
- R28 pad 2: /Array_Current -> Net-(Q6-G)
- R29 pad 1: /Fan1_EN -> +12V
- R29 pad 2: GND -> Net-(R29-Pad2)
- R30 pad 2: Net-(D17-A) -> Net-(U6-+)
- R31 pad 1: /Fan1_EN -> Net-(R29-Pad2)
- R31 pad 2: Net-(Q5-G) -> Net-(U6--)
- R32 pad 1: +12V -> Net-(U6--)
- R32 pad 2: Net-(R32-Pad2) -> /Array_Current
- R33 pad 1: +12V -> /Fan1_EN
- R33 pad 2: Net-(U7-+) -> GND
- R34 pad 1: Net-(R32-Pad2) -> +12V
- R34 pad 2: Net-(U7--) -> Net-(D17-A)
- R35 pad 1: Net-(U7--) -> /Fan1_EN
- R35 pad 2: /FAN1_Current -> Net-(Q7-G)
- R36 pad 1: /Fan2_EN -> +12V
- R36 pad 2: GND -> Net-(R36-Pad2)
- R37 pad 2: Net-(D21-A) -> Net-(U7-+)
- R38 pad 1: /Fan2_EN -> Net-(R36-Pad2)
- R38 pad 2: Net-(Q6-G) -> Net-(U7--)
- R39 pad 1: +12V -> Net-(U7--)
- R39 pad 2: Net-(R39-Pad2) -> /FAN1_Current
- R40 pad 1: +12V -> /Fan2_EN
- R40 pad 2: Net-(U8-+) -> GND
- R41 pad 1: Net-(R39-Pad2) -> +12V
- R41 pad 2: Net-(U8--) -> Net-(D21-A)
- R42 pad 1: Net-(U8--) -> /Fan2_EN
- R42 pad 2: /FAN2_Current -> Net-(Q8-G)
- R43 pad 1: /Strobe_EN -> +12V
- R43 pad 2: GND -> Net-(R43-Pad2)
- R44 pad 2: Net-(D25-A) -> Net-(U8-+)
- R45 pad 1: /Strobe_EN -> Net-(R43-Pad2)
- R45 pad 2: Net-(Q7-G) -> Net-(U8--)
- R46 pad 1: /Fan3_EN -> Net-(U8--)
- R46 pad 2: GND -> /FAN2_Current
- R47 pad 1: +12V -> /Strobe_EN
- R47 pad 2: Net-(D27-A) -> GND
- R48 pad 1: /Fan3_EN -> +12V
- R48 pad 2: Net-(Q8-G) -> Net-(D25-A)
- R49 pad 1: +12V -> /Strobe_EN
- R49 pad 2: Net-(R49-Pad2) -> Net-(Q9-G)
- R50 pad 1: +12V -> /Fan3_EN
- R50 pad 2: Net-(U9-+) -> GND
- R51 pad 1: Net-(R49-Pad2) -> +12V
- R51 pad 2: Net-(U9--) -> Net-(D27-A)
- R52 pad 1: Net-(U9--) -> /Fan3_EN
- R52 pad 2: /FAN3_Current -> Net-(Q10-G)
- R53 pad 1: +3.3V -> +12V
- R53 pad 2: /F1TACH -> Net-(R53-Pad2)
- R54 pad 1: +3.3V -> +12V
- R54 pad 2: /F2TACH -> Net-(U9-+)
- R55 pad 1: +3.3V -> Net-(R53-Pad2)
- R55 pad 2: /F3TACH -> Net-(U9--)
- R56 pad 1: +3.3V -> Net-(U9--)
- R56 pad 2: /F4TACH -> /FAN3_Current
- R57 pad 2: /F5TACH -> /F1TACH
- R58 pad 2: /ADDRSEL_FAN -> /F2TACH
- R59 pad 2: /FanError -> /F3TACH
- R60 pad 2: Net-(U10-CLK) -> /F4TACH
- R61 pad 1: /Fan4_EN -> +3.3V
- R61 pad 2: GND -> /F5TACH
- R62 pad 1: +12V -> +3.3V
- R62 pad 2: Net-(D31-A) -> /ADDRSEL_FAN
- R63 pad 1: /Fan4_EN -> +3.3V
- R63 pad 2: Net-(Q9-G) -> /FanError
- R64 pad 1: +12V -> +3.3V
- R64 pad 2: Net-(R64-Pad2) -> Net-(U10-CLK)
- R65 pad 1: +12V -> /Fan4_EN
- R65 pad 2: Net-(U11-+) -> GND
- R66 pad 1: Net-(R64-Pad2) -> +12V
- R66 pad 2: Net-(U11--) -> Net-(D31-A)
- R67 pad 1: Net-(U11--) -> /Fan4_EN
- R67 pad 2: /FAN4_Current -> Net-(Q11-G)
- R8 pad 1: /HV+_EN -> /SegEN
- R9 pad 1: +12V -> /SegEN
- R9 pad 2: Net-(D5-A) -> Net-(Q2-G)
Routing:
- net GND: track 0.00 -> 103.7 mm, vias 0 -> 31
- net +12V: track 0.00 -> 85.2 mm
- net +3.3V: track 0.00 -> 68.3 mm
- net /HV+_Current: track 0.00 -> 17.1 mm
- net /FAN5_Current: track 0.00 -> 16.9 mm
- net /FAN3_Current: track 0.00 -> 16.7 mm
- net /HV-_Current: track 0.00 -> 15.9 mm
- net /FAN4_Current: track 0.00 -> 15.7 mm
- net /FAN1_Current: track 0.00 -> 15.5 mm
- net /FAN2_Current: track 0.00 -> 15.4 mm
- net /Array_Current: track 0.00 -> 15.0 mm
- net /HV+ contactor/Low: track 0.00 -> 12.1 mm
- net /HV- Contactor/Low: track 0.00 -> 12.0 mm
- net /Fan2/Low: track 0.00 -> 11.7 mm
- net /Fan5/Low: track 0.00 -> 11.6 mm
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
Commit message: Made a bit shorter
Parts:
- moved J22 44.8 mm to (135.3, 140.9)
- moved R10 30.1 mm to (149.6, 139.6), turned to -90 degrees
- moved JP1 29.6 mm to (168.8, 150.5)
- moved R11 29.1 mm to (151.6, 139.6), turned to -90 degrees
- moved R49 28.7 mm to (165.1, 136.8), turned to 180 degrees
- moved R47 27.5 mm to (165.1, 134.7), turned to 180 degrees
- moved J8 26.5 mm to (160.0, 149.6), turned to 0 degrees
- moved J18 26.1 mm to (160.0, 140.8), turned to 0 degrees
- moved Q3 24.6 mm to (150.7, 143.3), turned to -90 degrees
- moved J21 24.0 mm to (135.3, 149.5)
- moved Q9 23.6 mm to (161.6, 135.7), turned to -90 degrees
- moved R8 20.6 mm to (149.7, 147.1), turned to -90 degrees
- moved R48 20.3 mm to (158.1, 136.8), turned to 180 degrees
- moved R9 19.2 mm to (151.7, 147.1), turned to -90 degrees
- moved D25 18.6 mm to (158.1, 134.7), turned to 180 degrees
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Routing:
- net /Battery segments/Low2: track 0.00 -> 13.8 mm
- net /Battery segments/Low1: track 0.00 -> 13.4 mm
- net GND: track 103.7 -> 110.9 mm
- net /HV- Contactor/Low: track 12.0 -> 5.15 mm
- net +12V: track 85.2 -> 79.3 mm
- net +3.3V: track 68.3 -> 64.4 mm

Commit message: slightly better layout
Parts:
- moved U2 67.4 mm to (155.5, 144.6)
- moved C1 67.4 mm to (159.6, 145.8)
- moved C2 67.4 mm to (158.3, 148.6)
- moved C3 67.4 mm to (156.3, 148.6)
- moved J18 37.4 mm to (123.8, 150.2), turned to -90 degrees
- moved R49 36.4 mm to (131.8, 151.6), turned to -90 degrees
- moved Q9 36.3 mm to (128.9, 151.6), turned to 180 degrees
- moved R47 35.5 mm to (133.8, 151.6), turned to -90 degrees
- moved R48 32.3 mm to (127.8, 148.0), turned to 90 degrees
- moved D25 31.2 mm to (129.8, 148.0), turned to 90 degrees
- moved J22 30.6 mm to (159.0, 160.2)
- moved J4 30.4 mm to (154.1, 126.6), turned to 0 degrees
- moved JP1 30.4 mm to (138.8, 155.2), turned to -90 degrees
- moved J8 29.8 mm to (131.2, 157.2), turned to -90 degrees
- moved R20 23.7 mm to (165.8, 155.6), turned to 0 degrees
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Routing:
- net GND: track 110.9 -> 95.5 mm
- net /Battery segments/Low2: track 13.8 -> 0.00 mm
- net /Battery segments/Low1: track 13.4 -> 0.00 mm
- net /HV- Contactor/EN: track 2.03 -> 11.7 mm
- net /HV+ contactor/Low: track 12.1 -> 5.41 mm
- net +12V: track 79.3 -> 73.4 mm
- net /HV-_EN: track 0.00 -> 5.87 mm
- net /HV-_Current: track 15.9 -> 12.0 mm
- net /Array_Current: track 15.0 -> 11.2 mm
- net /HV+_Current: track 17.1 -> 13.3 mm
- net Net-(Q9-G): track 2.71 -> 0.40 mm
- net /Strobe_EN: track 2.03 -> 0.00 mm
- net Net-(D25-A): track 1.98 -> 0.00 mm
- net /Array Contactor/Low: track 6.16 -> 5.15 mm

Commit message: i beveled the edges; ics still need to be put in good spots and traces made
Parts:
- added H1: MountingHole, MountingHole:MountingHole_3mm, F.Cu at (176.2, 160.8)
- added H1: MountingHole, MountingHole:MountingHole_3mm, F.Cu at (123.2, 160.8)
- added H1: MountingHole, MountingHole:MountingHole_3mm, F.Cu at (123.2, 43.2)
- moved U1 97.1 mm to (250.4, 31.6)
- moved Q9 1.96 mm to (128.9, 149.6)
- moved R47 1.96 mm to (133.8, 149.6)
- moved R48 1.96 mm to (127.8, 146.1)
- moved R49 1.96 mm to (131.8, 149.6)
- moved D25 1.96 mm to (129.8, 146.0)
- moved J8 1.40 mm to (131.2, 155.8)
- moved JP1 1.40 mm to (138.8, 153.8)
Routing:
- net /HV- Contactor/EN: track 11.7 -> 2.20 mm
- net /Fan3/Low: track 5.60 -> 12.0 mm
- net /HV-_EN: track 5.87 -> 0.00 mm
- net +12V: track 73.4 -> 78.8 mm
- net /FAN4_Current: track 15.7 -> 11.5 mm
- net /FAN3_Current: track 16.7 -> 13.6 mm
Other:
- board outline added: 59.4 x 124 mm

Commit message: most traces completed - need leaderSOM to finish. need to correct silkscreen issues.
Parts:
- moved J20 72.8 mm to (130.3, 43.7), turned to 0 degrees
- moved J19 68.5 mm to (130.4, 59.6), turned to 0 degrees
- moved C16 64.0 mm to (145.3, 75.5)
- moved C18 64.0 mm to (143.3, 75.5)
- moved D1 64.0 mm to (129.1, 139.0)
- moved D3 64.0 mm to (145.1, 136.7)
- moved Q1 64.0 mm to (132.2, 139.0)
- moved R38 64.0 mm to (135.9, 72.5)
- moved R39 64.0 mm to (140.5, 74.8)
- moved U7 64.0 mm to (141.5, 71.7)
- moved C5 64.0 mm to (138.8, 135.5)
- moved D17 64.0 mm to (129.1, 75.0)
- moved D19 64.0 mm to (145.1, 72.7)
- moved D2 64.0 mm to (131.2, 135.4)
- moved D4 64.0 mm to (145.1, 134.7)
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Connections:
- J23 pad 1: GND -> +12V
- J23 pad 2: /CAN_H -> /CAN_L
- J23 pad 3: /CAN_L -> /CAN_H
- J23 pad 4: +12V -> GND
- J4 pad 1: /FAN1_Current -> /FAN4_Current
- J4 pad 3: /FAN2_Current -> /FAN3_Current
- J4 pad 4: /HV+_Current -> /Array_Current
- J4 pad 5: /FAN3_Current -> /FAN2_Current
- J4 pad 6: /HV-_EN -> /HV-_Current
- J4 pad 7: /FAN4_Current -> /FAN1_Current
- J4 pad 8: /Array_Current -> /HV+_Current
Routing:
- net +3.3V: track 64.4 -> 251.8 mm, vias 0 -> 16
- net /F5TACH: track 1.85 -> 105.7 mm, vias 0 -> 1
- net /Fan5_EN: track 6.72 -> 105.7 mm
- net /F4TACH: track 1.86 -> 87.5 mm, vias 0 -> 1
- net /Seg1Sense: track 0.00 -> 84.2 mm, vias 0 -> 3
- net /HV+ SENSE: track 0.00 -> 81.8 mm, vias 0 -> 3
- net /Fan4_EN: track 4.96 -> 85.0 mm, vias 0 -> 2
- net /Seg2Sense: track 0.00 -> 78.9 mm, vias 0 -> 2
- net /FAN5_Current: track 16.9 -> 91.0 mm, vias 0 -> 2
- net /HV+_Current: track 13.3 -> 83.2 mm, vias 0 -> 1
- net /SegEN: track 4.00 -> 70.8 mm, vias 0 -> 2
- net /F3TACH: track 2.39 -> 68.8 mm, vias 0 -> 1
- net /FAN4_Current: track 11.5 -> 74.5 mm, vias 0 -> 2
- net /HV- SENSE: track 0.00 -> 62.8 mm, vias 0 -> 3
- net /Fan3_EN: track 4.33 -> 60.4 mm, vias 0 -> 2
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- added copper zone on F.Cu, net +12V
- added copper zone on F.Cu, net /SegEN
- added copper zone on B.Cu, net GND
