File: BPS-Leader.kicad_pcb (KiCad board)
At the start: 2 copper layers, 59.4 x 124 mm, 175 parts, among them J10 Fan2, J11 Fan3, J12 Fan4, J13 HV+ Connector, J14 HV- Connector, J15 Array Connector, J17 Fan5, J18 Strobe_Conn, J19 ADC SPI, J20 Fan I2C, J21 Segment1 Connector, J22 Segment2 Connector, J23 lSOMconn, J4 Fan I2C, J8 E-STOP, J9 Fan1, Q1 IRLML0030, Q10 IRLML0030, Q11 IRLML0030, Q2 IRLML0030, Q3 IRLML0030, Q4 IRLML0030, Q5 IRLML0030, Q6 IRLML0030, Q7 IRLML0030, Q8 IRLML0030, Q9 IRLML0030, U1 PeripheralSOM, U10 EMC2305-1-AP-TR, U11 INA180A2, U2 TLA2518IRTER, U3 INA180A2, U4 INA180A2, U5 INA180A2, U6 INA180A2, U7 INA180A2, U8 INA180A2, U9 INA180A2

Commit message: need to find a spot for the 3 new connectors and also flip the old connectors and also finish traces to leadersom
Parts:
- removed J23: lSOMconn, Connector_Molex:Molex_Micro-Fit_3.0_43650-0415_1x04_P3.00mm_Vertical
- removed U1: PeripheralSOM, UTSVT_Special:PeripheralSOM
- added J1: ~, UTSVT_Special:LeaderSOM, F.Cu at (180.5, 68.9)
- added J2: CarPowerConnector, Connector_Molex:Molex_Micro-Fit_3.0_43650-0215_1x02_P3.00mm_Vertical, F.Cu at (89.4, 68.8)
- added J3: CANconn, Connector_Molex:Molex_Micro-Fit_3.0_43650-0215_1x02_P3.00mm_Vertical, F.Cu at (111.2, 55.4)
- added J5: CANconn2, Connector_Molex:Molex_Micro-Fit_3.0_43650-0215_1x02_P3.00mm_Vertical, F.Cu at (108.8, 83.2)
- added J6: I-CanConn, Connector_Molex:Molex_Micro-Fit_3.0_43650-0415_1x04_P3.00mm_Vertical, F.Cu at (123.0, 60.8)
- moved R61 17.9 mm to (162.2, 81.9), turned to 90 degrees
- moved R60 17.6 mm to (160.1, 83.7), turned to 90 degrees
- moved R59 17.0 mm to (153.0, 87.2)
- moved R63 17.0 mm to (157.0, 87.2)
- moved R64 17.0 mm to (155.0, 87.2)
- moved C25 16.8 mm to (156.0, 77.0), turned to -90 degrees
- moved C26 16.8 mm to (158.0, 77.0), turned to -90 degrees
- moved R62 16.8 mm to (154.0, 77.0)
- moved U10 16.8 mm to (155.7, 82.1)
- moved R57 15.9 mm to (150.9, 80.5), turned to -90 degrees
- moved R58 15.8 mm to (148.9, 82.4), turned to -90 degrees
- moved C1 12.6 mm to (161.9, 96.1)
- moved C2 12.6 mm to (163.9, 96.1)
- moved C3 12.6 mm to (165.9, 96.1)
- moved U2 12.6 mm to (162.8, 91.8)
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Routing:
- net /Array SENSE: track 46.7 -> 80.6 mm
- net /CAN_L: track 42.0 -> 9.49 mm, vias 0 -> 1
- net /CAN_H: track 42.2 -> 12.6 mm, vias 0 -> 1
- net /HV- SENSE: track 62.8 -> 89.7 mm
- net /HV+ SENSE: track 81.8 -> 106.7 mm
- net +3.3V: track 251.8 -> 227.6 mm, vias 16 -> 14
- net /SegEN: track 70.8 -> 93.4 mm, vias 2 -> 0
- net /Fan5_EN: track 105.7 -> 83.4 mm, vias 0 -> 2
- net /FAN5_Current: track 91.0 -> 70.2 mm, vias 2 -> 3
- net /Fan4_EN: track 85.0 -> 64.5 mm, vias 2 -> 4
- net /Fan3_EN: track 60.4 -> 42.6 mm
- net /Fan2_EN: track 45.0 -> 27.3 mm
- net /Seg1Sense: track 84.2 -> 100.1 mm, vias 3 -> 1
- net /FAN4_Current: track 74.5 -> 59.6 mm, vias 2 -> 3
- net /FAN3_Current: track 64.0 -> 49.1 mm, vias 2 -> 3
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- added copper zone on F.Cu, net +3.3V
- added copper zone on F.Cu, net GND
- removed copper zone on F.Cu, net +12V
- removed copper zone on F.Cu, net /SegEN
Other:
- board size 59.4 x 124 mm -> 59.5 x 124 mm

Commit message: Traces completed, no drc electrical errors. need to clean up silkscreen.
Parts:
- moved J19 75.2 mm to (157.5, 131.9)
- moved J20 75.2 mm to (157.5, 120.6)
- moved J2 39.6 mm to (128.5, 62.3), turned to 0 degrees
- moved J5 37.7 mm to (128.4, 51.0), turned to 0 degrees
- moved J3 21.2 mm to (128.4, 43.0), turned to 0 degrees
- moved J21 9.04 mm to (149.2, 161.0), turned to 180 degrees
- moved J14 9.04 mm to (176.4, 124.8), turned to -90 degrees
- moved J13 9.04 mm to (176.4, 143.8), turned to -90 degrees
- moved J15 9.04 mm to (176.4, 105.8), turned to -90 degrees
- moved J22 9.02 mm to (168.0, 160.8), turned to 180 degrees
- moved D25 8.22 mm to (125.8, 153.2), turned to -90 degrees
- moved R48 7.11 mm to (127.8, 153.2)
- moved J10 6.92 mm to (120.4, 92.2), turned to 90 degrees
- moved J11 6.90 mm to (120.4, 108.2), turned to 90 degrees
- moved J12 6.90 mm to (120.4, 124.2), turned to 90 degrees
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Connections:
- J10 pad 1: +12V -> /F2TACH
- J10 pad 3: /F2TACH -> +12V
- J11 pad 1: +12V -> /F3TACH
- J11 pad 3: /F3TACH -> +12V
- J12 pad 1: +12V -> /F4TACH
- J12 pad 3: /F4TACH -> +12V
- J13 pad 1: +12V -> GND
- J13 pad 2: /HV+ contactor/Low -> /HV+ SENSE
- J13 pad 3: /HV+ SENSE -> /HV+ contactor/Low
- J13 pad 4: GND -> +12V
- J14 pad 1: +12V -> GND
- J14 pad 2: /HV- Contactor/Low -> /HV- SENSE
- J14 pad 3: /HV- SENSE -> /HV- Contactor/Low
- J14 pad 4: GND -> +12V
- J15 pad 1: +12V -> GND
- J15 pad 2: /Array Contactor/Low -> /Array SENSE
- J15 pad 3: /Array SENSE -> /Array Contactor/Low
- J15 pad 4: GND -> +12V
- J17 pad 1: +12V -> /F5TACH
- J17 pad 3: /F5TACH -> +12V
- J21 pad 2: /Battery segments/Low1 -> /Seg1Sense
- J21 pad 3: /Seg1Sense -> /Battery segments/Low1
- J22 pad 2: /Battery segments/Low2 -> /Seg2Sense
- J22 pad 3: /Seg2Sense -> /Battery segments/Low2
- J3 pad 1: /CAN_H -> /CAN_L
- J3 pad 2: /CAN_L -> /CAN_H
- J5 pad 1: /CAN_H -> /CAN_L
- J5 pad 2: /CAN_L -> /CAN_H
- J9 pad 1: +12V -> /F1TACH
- J9 pad 3: /F1TACH -> +12V
- JP1 pad 1: /HV- Contactor/EN -> /HV-_EN
- JP1 pad 2: /HV-_EN -> /HV- Contactor/EN
Routing:
- net /Strobe_EN: track 2.00 -> 98.1 mm, vias 0 -> 2
- net +3.3V: track 227.6 -> 313.9 mm, vias 14 -> 19
- net /CS: track 3.14 -> 80.9 mm, vias 1 -> 3
- net /SDI: track 4.33 -> 79.9 mm, vias 1 -> 3
- net /ADDRSEL_FAN: track 2.55 -> 75.5 mm, vias 0 -> 5
- net /I-CAN_H: track 0.00 -> 72.6 mm, vias 0 -> 1
- net /SCLK: track 3.67 -> 75.1 mm, vias 1 -> 3
- net /I-CAN_L: track 0.00 -> 70.6 mm, vias 0 -> 1
- net /FanError: track 2.34 -> 72.2 mm, vias 0 -> 3
- net /SDO: track 3.20 -> 70.9 mm, vias 1 -> 3
- net /SDA: track 18.2 -> 80.9 mm, vias 0 -> 2
- net /SCL: track 18.9 -> 74.8 mm, vias 2 -> 3
- net /CAN_L: track 9.49 -> 59.7 mm
- net /CAN_H: track 12.6 -> 56.3 mm
- net +12V: track 82.4 -> 118.7 mm, vias 0 -> 3
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- added copper zone on F.Cu, net +12V
Other:
- board size 59.5 x 124 mm -> 62.4 x 124 mm

Commit message: enable signals added for contactors.....
Connections:
- J1 pad 11: /Seg1Sense -> /HV+_EN
- J1 pad 17: /Seg2Sense -> /HV-_EN
- J1 pad 42: /FanError -> /Array_EN
Routing:
- net /HV-_EN: track 8.23 -> 116.1 mm, vias 0 -> 1
- net /Seg1Sense: track 97.7 -> 0.36 mm, vias 1 -> 0
- net /Seg2Sense: track 92.5 -> 0.00 mm
- net /HV+_EN: track 2.03 -> 93.4 mm, vias 0 -> 2
- net /Array_EN: track 2.03 -> 54.8 mm, vias 0 -> 2
- net /FanError: track 72.2 -> 50.9 mm, vias 3 -> 2
- net +3.3V: track 313.9 -> 330.1 mm, vias 19 -> 20
- net /F5TACH: track 102.0 -> 100.0 mm
- net /Fan4_EN: track 67.6 -> 66.6 mm
- net /HV+ SENSE: track 106.8 -> 106.2 mm
- removed copper zone on F.Cu, net +3.3V

Commit message: tracks cleaned up, yep.
Routing:
- net /FanError: track 50.9 -> 38.4 mm
Changed lines of the file:
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@@
 	)
 	(segment
-		(start 158.1 78)
-		(end 158.2 78.1)
-		(width 0.4)
-		(layer "F.Cu")
-		(net 1)
-	)
-	(segment
 		(start 169.392 113.6385)
 		(end 169.8775 114.124)
@@
 	)
 	(segment
-		(start 158.1 77.973999)
-		(end 158.1 78)
-		(width 0.4)
-		(layer "F.Cu")
-		(net 1)
-	)
-	(segment
 		(start 169.665 147.496)
 		(end 169.665 147.2265)
@@
 	)
 	(segment
-		(start 154.55 152.2)
-		(end 137.9 152.2)
+		(start 135.6 152.2)
+		(end 134 153.8)
 		(width 0.2)
 		(layer "B.Cu")
@@
 	)
 	(segment
-		(start 134 153.8)
-		(end 136.3 153.8)
-		(width 0.2)
-		(layer "B.Cu")
-		(net 48)
-	)
-	(segment
-		(start 137.9 152.2)
-		(end 136.3 153.8)
+		(start 154.55 152.2)
+		(end 135.6 152.2)
 		(width 0.2)
 		(layer "B.Cu")
@@
 	(segment
 		(start 149.644213 97.609899)
-		(end 150.034315 98)
+		(end 150.2 98.165685)
 		(width 0.2)
 		(layer "F.Cu")
@@
 	)
 	(segment
-		(start 150.034315 98)
-		(end 150.2 98.165685)
-		(width 0.2)
-		(layer "F.Cu")
-		(net 57)
-	)
-	(segment
 		(start 149.644213 97.609898)
 		(end 149.644213 97.609899)
@@
 	(segment
 		(start 167.313731 89.383327)
-		(end 168.348529 88.348529)
+		(end 174.500002 82.197056)
 		(width 0.2)
 		(layer "B.Cu")
@@
 	)
 	(segment
-		(start 168.348529 88.348529)
-		(end 174.500002 82.197056)
-		(width 0.2)
-		(layer "B.Cu")
-		(net 58)
-	)
-	(segment
-		(start 167.313731 90.066551)
-		(end 167.3 90.080282)
-		(width 0.2)
-		(layer "B.Cu")
-		(net 58)
-	)
-	(segment
 		(start 150.044213 96.744213)
 		(end 150.488426 96.3)
@@
 	)
 	(segment
-		(start 160.7 74.5)
-		(end 160.7 81.300999)
-		(width 0.2)
-		(layer "B.Cu")
-		(net 62)
-	)
-	(segment
-		(start 160.7 81.300999)
-		(end 156.700999 85.3)
-		(width 0.2)
-		(layer "B.Cu")
-		(net 62)
-	)
-	(segment
 		(start 156.300999 85.7)
 		(end 152.2 85.7)
@@
 	(segment
 		(start 151.3 88.965686)
-		(end 151.834315 89.5)
+		(end 152.25 89.915685)
 		(width 0.2)
 		(layer "F.Cu")
@@
 	)
 	(segment
-		(start 151.834315 89.5)
-		(end 152.25 89.915685)
-		(width 0.2)
-		(layer "F.Cu")
-		(net 63)
-	)
-	(segment
 		(start 154.751001 79.751001)
 		(end 154 79)
@@
 	)
 	(segment
-		(start 146.56 161.04)
-		(end 146.2 161.04)
-		(width 0.2)
-		(layer "B.Cu")
-		(net 66)
-	)
-	(segment
