File: BPS-Leader.kicad_pcb (KiCad board)
At the start: 2 copper layers, 62.4 x 124 mm, 178 parts, among them J10 Fan2, J11 Fan3, J12 Fan4, J13 HV+ Connector, J14 HV- Connector, J15 Array Connector, J17 Fan5, J18 Strobe_Conn, J19 ADC SPI, J2 CarPowerConnector, J20 Fan I2C, J21 Segment1 Connector, J22 Segment2 Connector, J3 CANconn, J4 Fan I2C, J5 CANconn2, J6 I-CanConn, J8 E-STOP, J9 Fan1, Q1 IRLML0030, Q10 IRLML0030, Q11 IRLML0030, Q2 IRLML0030, Q3 IRLML0030, Q4 IRLML0030, Q5 IRLML0030, Q6 IRLML0030, Q7 IRLML0030, Q8 IRLML0030, Q9 IRLML0030, U10 EMC2305-1-AP-TR, U11 INA180A2, U2 TLA2518IRTER, U3 INA180A2, U4 INA180A2, U5 INA180A2, U6 INA180A2, U7 INA180A2, U8 INA180A2, U9 INA180A2

Commit message: traces cleaned up slightly (removed some accidental 90 degree bends
Routing:
- net GND: track 115.4 -> 104.7 mm, vias 44 -> 46
- net /SDO: track 70.9 -> 72.8 mm
- net /SCLK: track 75.1 -> 76.7 mm
- net /SDI: track 79.9 -> 80.7 mm
- net /Array SENSE: track 75.0 -> 74.4 mm

Commit message: everything should be finished now; tracks cleaned up, silkscreen issues fixed, new shunt/feedback/protection resistors chosen, BOM made, some other stuff i forgot probably
Parts:
- C10, C13, C16, C19, C22, C27, C4, C7: value 1.1uF -> 0.1uF
- C11, C14, C17, C20, C23, C28, C5, C8: value 0.16uF -> 0.15uF
- C12, C15, C18, C21, C24, C29, C6, C9: value 2.2uF -> 0.1uF
- D1, D10, D11, D12, D13, D14, D15, D16, D17, D18, D19, D2, D20, D21, D22, D23, D24, D27, D28, D29, D3, D30, D31, D32, D33, D34, D4, D5, D6, D7, D8, D9: footprint Diode_SMD:D_0805_2012Metric -> footprints:D_0805_2012Metric(adjsilk)
- R15, R22, R29, R36, R4, R43, R53, R68: value 3m -> 2.8m; footprint Resistor_SMD:R_0805_2012Metric -> Resistor_SMD:R_2512_6332Metric; moved to B.Cu
- R16, R17, R23, R24, R30, R31, R37, R38, R44, R45, R5, R54, R55, R6, R69, R70: value 5 -> 10
- R18, R25, R32, R39, R46, R56, R7, R71: value 0.9 -> 1
- U11, U3, U4, U5, U6, U7, U8, U9: footprint Package_TO_SOT_SMD:SOT-23-5 -> footprints:SOT-23-5(movedsilk)
- moved R4 2.02 mm to (129.9, 136.9)
- moved R22 2.02 mm to (168.7, 131.8)
- moved R36 2.01 mm to (130.0, 73.1)
- moved R15 2.01 mm to (168.7, 150.8)
- moved R29 2.01 mm to (168.7, 112.8)
- moved R68 2.00 mm to (129.9, 121.0)
- moved R53 2.00 mm to (129.9, 105.0)
- moved R43 1.97 mm to (129.9, 86.2)
- moved R46 0.17 mm to (136.8, 87.6)
- moved R39 0.16 mm to (136.8, 74.6)
- moved U8 0.15 mm to (137.8, 84.6)
- moved U7 0.11 mm to (137.8, 71.5)
- moved C21 0.07 mm to (139.5, 88.4)
- moved C16 0.07 mm to (141.6, 75.3)
- moved C18 0.07 mm to (139.5, 75.3)
Routing:
- net GND: track 104.7 -> 91.5 mm, vias 46 -> 49
- net +3.3V: track 330.2 -> 325.8 mm
- net /F2TACH: track 41.8 -> 38.1 mm
- net /F3TACH: track 56.5 -> 53.0 mm
- net /F5TACH: track 100.0 -> 97.1 mm
- net Net-(R4-Pad2): track 1.92 -> 4.49 mm, vias 0 -> 1
- net Net-(R22-Pad2): track 1.92 -> 4.47 mm, vias 0 -> 1
- net Net-(R68-Pad2): track 1.92 -> 4.47 mm, vias 0 -> 1
- net Net-(R36-Pad2): track 1.92 -> 4.46 mm, vias 0 -> 1
- net Net-(R15-Pad2): track 1.92 -> 4.46 mm, vias 0 -> 1
- net Net-(R29-Pad2): track 1.92 -> 4.45 mm, vias 0 -> 1
- net Net-(R53-Pad2): track 1.92 -> 4.32 mm, vias 0 -> 1
- net Net-(R43-Pad2): track 1.92 -> 4.29 mm, vias 0 -> 1
- net /F4TACH: track 76.5 -> 74.4 mm
- net /F1TACH: track 37.7 -> 35.8 mm
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Other:
- board size 62.4 x 124 mm -> 62.4 x 124.2 mm
- board text added: "1"
- board text added: "2"
- board text added: "3"
- board text added: "4"
- board text added: "5"
- board text added: "ADC"
- board text added: "Array"
- board text added: "CAN"
- board text added: "F4 F3 F2 F1"
- board text added: "FAN MCU"
- board text added: "FANERR ADDS SEL SCL SDA"
- board text added: "FANS"
- board text added: "FN5 ARY HV- HV+"
- board text added: "HV+"
- board text added: "HV-"
- board text added: "HV- STOP"
- board text added: "I-CAN"
- board text added: "PWR"
- board text added: "SDO SCLK SDI CS"
- board text added: "SEG_1"
- board text added: "SEG_2"
- board text added: "Strobe"
- board text added: "TEST PINS"
- board text added: "bypass_jmp"
- board text added: "gnd"
- board text added: "lsom :-)"

Commit message: I made small tweaks to various tracks throughout the week
Routing:
- net +3.3V: track 325.8 -> 326.9 mm
Changed lines of the file:
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@@
 	)
 	(segment
-		(start 174.3 69.6)
-		(end 174.3 72.7)
-		(width 0.3)
-		(layer "F.Cu")
-		(net 2)
-	)
-	(segment
 		(start 155 88.1125)
 		(end 157 88.1125)
@@
 		(start 176.8 67.1)
 		(end 176.8 65.359931)
-		(width 0.4)
+		(width 0.3)
 		(layer "F.Cu")
 		(net 2)
@@
 	)
 	(segment
+		(start 174.3 70.849939)
+		(end 174.3 69.6)
+		(width 0.3)
+		(layer "F.Cu")
+		(net 2)
+	)
+	(segment
 		(start 176.75 72.7)
 		(end 172.449939 72.7)
-		(width 0.4)
+		(width 0.3)
 		(layer "F.Cu")
 		(net 2)
@@
 		(start 174.3 69.6)
 		(end 176.8 67.1)
-		(width 0.4)
+		(width 0.3)
 		(layer "F.Cu")
 		(net 2)
@@
 		(start 172.449939 73.11391)
 		(end 172.449939 72.7)
-		(width 0.4)
+		(width 0.3)
 		(layer "F.Cu")
 		(net 2)
@@
 		(start 176.75 72.313971)
 		(end 176.749939 72.31391)
-		(width 0.4)
+		(width 0.3)
 		(layer "F.Cu")
 		(net 2)
@@
 	)
 	(segment
-		(start 172.449939 72.31397)
-		(end 172.449998 72.313911)
-		(width 0.4)
-		(layer "F.Cu")
-		(net 2)
-	)
-	(segment
 		(start 165 69.8)
 		(end 158.726001 76.073999)
@@
 		(start 176.75 73.11391)
 		(end 176.75 72.7)
-		(width 0.4)
+		(width 0.3)
 		(layer "F.Cu")
 		(net 2)
@@
 	)
 	(segment
+		(start 172.449939 72.7)
+		(end 174.3 70.849939)
+		(width 0.3)
+		(layer "F.Cu")
+		(net 2)
+	)
+	(segment
 		(start 138.596 136.3915)
 		(end 140.143 136.3915)
@@
 	)
 	(segment
-		(start 172.449939 72.7)
-		(end 172.449939 72.31397)
-		(width 0.4)
-		(layer "F.Cu")
-		(net 2)
-	)
-	(segment
 		(start 163.074999 93.972285)
 		(end 162.047283 95.000001)
@@
 		(start 176.75 72.7)
 		(end 176.75 72.313971)
-		(width 0.4)
+		(width 0.3)
 		(layer "F.Cu")
 		(net 2)
@@
 	)
 	(via
-		(at 174.3 72.7)
+		(at 172.449939 72.7)
 		(size 0.6)
 		(drill 0.3)
@@
 	)
 	(segment
-		(start 167.8375 95.8625)
-		(end 175.6 88.1)
-		(width 0.3)
-		(layer "B.Cu")
-		(net 2)
-	)
-	(segment
 		(start 165 69.8)
 		(end 165.9 68.9)
@@
 	)
 	(segment
-		(start 175.6 75.5)
-		(end 174.3 74.2)
+		(start 141.13975 86.44325)
+		(end 142.531844 86.44325)
 		(width 0.3)
 		(layer "B.Cu")
@@
 	)
 	(segment
-		(start 141.13975 86.44325)
-		(end 142.531844 86.44325)
+		(start 142.531844 86.44325)
+		(end 144.177724 88.08913)
 		(width 0.3)
 		(layer "B.Cu")
@@
 	)
 	(segment
-		(start 142.531844 86.44325)
-		(end 144.177724 88.08913)
+		(start 175.6 88.1)
+		(end 167.8375 95.8625)
 		(width 0.3)
 		(layer "B.Cu")
@@
 	)
 	(segment
-		(start 174.3 74.2)
-		(end 174.3 72.7)
+		(start 172.449939 72.719939)
+		(end 175.6 75.87)
 		(width 0.3)
 		(layer "B.Cu")
@@
 	)
 	(segment
-		(start 168.37825 120.21625)
-		(end 168.88175 120.71975)
+		(start 167.8375 95.8625)
+		(end 166.6375 95.8625)
 		(width 0.3)
 		(layer "B.Cu")
@@
 	)
 	(segment
-		(start 163.6 142.2)
-		(end 166.397 142.2)
+		(start 172.449939 72.7)
+		(end 172.449939 72.719939)
 		(width 0.3)
 		(layer "B.Cu")
@@
 	)
 	(segment
-		(start 166.6375 95.8625)
-		(end 167.8375 95.8625)
+		(start 168.37825 120.21625)
+		(end 168.88175 120.71975)
 		(width 0.3)
 		(layer "B.Cu")
@@
 	)
 	(segment
-		(start 143.8 75)
-		(end 142.06875 73.26875)
+		(start 163.6 142.2)
+		(end 166.397 142.2)
 		(width 0.3)
 		(layer "B.Cu")
@@
 	)
 	(segment
-		(start 165.9 68.9)
-		(end 170.8 68.9)
+		(start 143.8 75)
+		(end 142.06875 73.26875)
 		(width 0.3)
 		(layer "B.Cu")
@@
 	)
 	(segment
-		(start 175.6 88.1)
-		(end 175.6 75.5)
+		(start 165.9 68.9)
+		(end 170.8 68.9)
 		(width 0.3)
 		(layer "B.Cu")
@@
 	)
 	(segment
+		(start 175.6 75.87)
+		(end 175.6 88.1)
+		(width 0.3)
+		(layer "B.Cu")
+		(net 2)
+	)
+	(segment
 		(start 166.9155 103.7)
 		(end 168.88875 101.72675)
@@
 	)
 	(segment
+		(start 163.5 82.37)
+		(end 162.93 81.8)
+		(width 0.2)
+		(layer "F.Cu")
+		(net 82)
+	)
+	(segment
 		(start 162.798999 81.798998)
 		(end 157.675201 81.798998)
@@
 	)
 	(segment
-		(start 162.800001 81.8)
-		(end 162.798999 81.798998)
+		(start 147.3 90.55)
+		(end 146.777724 91.072276)
 		(width 0.2)
 		(layer "F.Cu")
@@
 	)
 	(segment
-		(start 163.5 82.1)
-		(end 163.2 81.8)
+		(start 134.466 141.178)
+		(end 133.328 140.04)
 		(width 0.2)
 		(layer "F.Cu")
@@
 	)
 	(segment
-		(start 147.3 90.55)
-		(end 146.777724 91.072276)
+		(start 146.777724 91.072276)
+		(end 146.777724 136.866276)
 		(width 0.2)
 		(layer "F.Cu")
@@
 	)
 	(segment
-		(start 163.2 81.8)
+		(start 162.93 81.8)
 		(end 162.800001 81.8)
 		(width 0.2)
@@
 	)
 	(segment
-		(start 134.466 141.178)
-		(end 133.328 140.04)
-		(width 0.2)
-		(layer "F.Cu")
-		(net 82)
-	)
-	(segment
-		(start 146.777724 91.072276)
-		(end 146.777724 136.866276)
+		(start 162.800001 81.8)
+		(end 162.798999 81.798998)
 		(width 0.2)
 		(layer "F.Cu")
@@
 	)
 	(via
-		(at 163.5 82.1)
+		(at 163.5 82.37)
 		(size 0.6)
 		(drill 0.3)
@@
 	)
 	(segment
-		(start 161.9 89.5)
-		(end 163.5 87.9)
+		(start 163.5 87.9)
+		(end 161.9 89.5)
 		(width 0.2)
 		(layer "B.Cu")
@@
 	(segment
 		(start 148.35 89.5)
-		(end 161.9 89.5)
+		(end 147.3 90.55)
 		(width 0.2)
 		(layer "B.Cu")
@@
 	)
 	(segment
-		(start 147.3 90.55)
+		(start 161.9 89.5)
 		(end 148.35 89.5)
 		(width 0.2)
@@
 	)
 	(segment
-		(start 163.5 87.9)
-		(end 163.5 82.1)
+		(start 163.5 82.37)
+		(end 163.5 87.9)
 		(width 0.2)
 		(layer "B.Cu")

Commit message: gerbers made, silkscreen adjusted to include pin labels
Parts:
- added G***: LOGO, Graphics:manface tiny, F.Cu at (143.0, 63.5)
- added G***: LOGO, UTSVT_Special:UTSVT_Logo_Symbol, F.Cu at (133.5, 129.0)
- added G***: LOGO, UTSVT_Special:Hallock_Image_Tiny, F.Cu at (150.0, 142.4)
- added G***: LOGO, LOGO, B.Cu at (159.0, 49.5)
Other:
- board text added: "+ -"
- board text added: "+ - T"
- board text added: "- +"
- board text added: "- ICH ICL +"
- board text added: "BPS Leader Clark Rucker Spring 2025"
- board text added: "L |CAN| H"
- board text added: "S1"
- board text added: "S2"
- board text added: "SG - S +"
- board text added: "SG S - +"
- board text added: "greetings and salutations"
- board text removed: "CAN"
- board text removed: "SEG_1"
- board text removed: "SEG_2"
- board text removed: "gnd"
