File: adc.kicad_sch (KiCad schematic)
At the start: 4 parts, among them U7 TLA2518IRTER

Commit message: Preliminary Schematic Finished
Parts:
- U3: renamed from U7; footprint WQFN16_RTE_TEX -> footprints:WQFN16_RTE_TEX
- renumbered C13 to C1, C14 to C2, C15 to C3
Connections:
- net +3.3V: no longer C1.2, U3.7 (AVDD)
- net GND: no longer C1.1
- new net AVDD: C1.1, U3.7 (AVDD)
- new net GNDA: C1.2
Other:
- moved on the sheet: C1
Changed lines of the file:
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@@
-		(color 0 0 0 0)
-	)
-	(junction
-		(at 105.41 71.12)
-		(diameter 0)
 		(color 0 0 0 0)
 	)
@@
 	(wire
 		(pts
-			(xy 96.52 71.12) (xy 105.41 71.12)
-		)
-		(stroke
-			(width 0)
-			(type default)
-		)
-	)
-	(wire
-		(pts
 			(xy 175.26 78.74) (xy 175.26 73.66)
 		)
@@
 	(wire
 		(pts
-			(xy 105.41 71.12) (xy 105.41 86.36)
-		)
-		(stroke
-			(width 0)
-			(type default)
-		)
-	)
-	(wire
-		(pts
-			(xy 133.35 86.36) (xy 172.72 86.36)
+			(xy 102.87 71.12) (xy 102.87 76.2)
 		)
 		(stroke
@@
 	(wire
 		(pts
+			(xy 102.87 71.12) (xy 106.68 71.12)
+		)
+		(stroke
+			(width 0)
+			(type default)
+		)
+	)
+	(wire
+		(pts
 			(xy 175.26 73.66) (xy 172.72 73.66)
 		)
@@
 	(wire
 		(pts
-			(xy 105.41 86.36) (xy 128.27 86.36)
-		)
-		(stroke
-			(width 0)
-			(type default)
-		)
-	)
-	(wire
-		(pts
 			(xy 184.15 73.66) (xy 175.26 73.66)
 		)
@@
 		)
 	)
-	(wire
-		(pts
-			(xy 106.68 71.12) (xy 105.41 71.12)
-		)
-		(stroke
-			(width 0)
-			(type default)
-		)
-	)
 	(hierarchical_label "CS"
 		(shape input)
@@
 			)
 			(justify left)
+		)
+	)
+	(hierarchical_label "AVDD"
+		(shape input)
+		(at 102.87 71.12 180)
+		(fields_autoplaced yes)
+		(effects
+			(font
+				(size 1.27 1.27)
+				(thickness 0.254)
+				(bold yes)
+			)
+			(justify right)
 		)
 	)
@@
 	(symbol
 		(lib_id "Device:C_Small")
-		(at 130.81 86.36 270)
+		(at 102.87 78.74 0)
 		(unit 1)
 		(exclude_from_sim no)
@@
 		(on_board yes)
 		(dnp no)
-		(property "Reference" "C13"
-			(at 130.81 77.47 90)
+		(property "Reference" "C1"
+			(at 99.06 77.978 0)
 			(effects
 				(font
@@
 		)
 		(property "Value" "1uF"
-			(at 130.81 80.01 90)
+			(at 99.06 80.518 0)
 			(effects
 				(font
@@
 		)
 		(property "Footprint" "Capacitor_SMD:C_0805_2012Metric"
-			(at 130.81 86.36 0)
+			(at 102.87 78.74 0)
 			(effects
 				(font
@@
 		)
 		(property "Datasheet" "~"
-			(at 130.81 86.36 0)
+			(at 102.87 78.74 0)
 			(effects
 				(font
@@
 		)
 		(property "Description" "Unpolarized capacitor, small symbol"
-			(at 130.81 86.36 0)
+			(at 102.87 78.74 0)
 			(effects
 				(font
@@
 			(project "BPS-Leader"
 				(path "/bca74250-80d8-4ae3-9726-634afabc9565/fe68b7ab-dadd-40ec-a34d-6c2925722947"
-					(reference "C13")
+					(reference "C1")
 					(unit 1)
 				)
@@
 		(on_board yes)
 		(dnp no)
-		(property "Reference" "C15"
+		(property "Reference" "C3"
 			(at 177.8 81.534 0)
 			(effects
@@
 			(project "BPS-Leader"
 				(path "/bca74250-80d8-4ae3-9726-634afabc9565/fe68b7ab-dadd-40ec-a34d-6c2925722947"
-					(reference "C15")
+					(reference "C3")
 					(unit 1)
 				)
@@
 		(dnp no)
 		(fields_autoplaced yes)
-		(property "Reference" "#PWR051"
+		(property "Reference" "#PWR013"
 			(at 172.72 93.98 0)
 			(effects
@@
 			(project ""
 				(path "/bca74250-80d8-4ae3-9726-634afabc9565/fe68b7ab-dadd-40ec-a34d-6c2925722947"
-					(reference "#PWR051")
+					(reference "#PWR013")
+					(unit 1)
+				)
+			)
+		)
+	)
+	(symbol
+		(lib_id "power:GNDA")
+		(at 102.87 81.28 0)
+		(unit 1)
+		(exclude_from_sim no)
+		(in_bom yes)
+		(on_board yes)
+		(dnp no)
+		(fields_autoplaced yes)
+		(property "Reference" "#PWR012"
+			(at 102.87 87.63 0)
+			(effects
+				(font
+					(size 1.27 1.27)
+				)
+				(hide yes)
+			)
+		)
+		(property "Value" "GNDA"
+			(at 102.87 86.36 0)
+			(effects
+				(font
+					(size 1.27 1.27)
+				)
+			)
+		)
+		(property "Footprint" ""
+			(at 102.87 81.28 0)
+			(effects
+				(font
+					(size 1.27 1.27)
+				)
+				(hide yes)
+			)
+		)
+		(property "Datasheet" ""
+			(at 102.87 81.28 0)
+			(effects
+				(font
+					(size 1.27 1.27)
+				)
+				(hide yes)
+			)
+		)
+		(property "Description" "Power symbol creates a global label with name \"GNDA\" , analog ground"
+			(at 102.87 81.28 0)
+			(effects
+				(font
+					(size 1.27 1.27)
+				)
+				(hide yes)
+			)
+		)
+		(pin "1"
+		)
+		(instances
+			(project "BPS-Leader"
+				(path "/bca74250-80d8-4ae3-9726-634afabc9565/fe68b7ab-dadd-40ec-a34d-6c2925722947"
+					(reference "#PWR012")
 					(unit 1)
 				)
@@
 		(dnp no)
 		(fields_autoplaced yes)
-		(property "Reference" "U7"
+		(property "Reference" "U3"
 			(at 139.7 45.72 0)
 			(effects
@@
 			)
 		)
-		(property "Footprint" "WQFN16_RTE_TEX"
+		(property "Footprint" "footprints:WQFN16_RTE_TEX"
 			(at 106.68 55.88 0)
 			(effects
@@
 			(project ""
 				(path "/bca74250-80d8-4ae3-9726-634afabc9565/fe68b7ab-dadd-40ec-a34d-6c2925722947"
-					(reference "U7")
-					(unit 1)
-				)
-			)
-		)
-	)
-	(symbol
-		(lib_id "power:+3.3V")
-		(at 96.52 71.12 0)
-		(unit 1)
-		(exclude_from_sim no)
-		(in_bom yes)
-		(on_board yes)
-		(dnp no)
-		(fields_autoplaced yes)
-		(property "Reference" "#PWR050"
-			(at 96.52 74.93 0)
-			(effects
-				(font
-					(size 1.27 1.27)
-				)
-				(hide yes)
-			)
-		)
-		(property "Value" "+3.3V"
-			(at 96.52 66.04 0)
-			(effects
-				(font
-					(size 1.27 1.27)
-				)
-			)
-		)
-		(property "Footprint" ""
-			(at 96.52 71.12 0)
-			(effects
-				(font
-					(size 1.27 1.27)
-				)
-				(hide yes)
-			)
-		)
-		(property "Datasheet" ""
-			(at 96.52 71.12 0)
-			(effects
-				(font
-					(size 1.27 1.27)
-				)
-				(hide yes)
-			)
-		)
-		(property "Description" "Power symbol creates a global label with name \"+3.3V\""
-			(at 96.52 71.12 0)
-			(effects
-				(font
-					(size 1.27 1.27)
-				)
-				(hide yes)
-			)
-		)
-		(pin "1"
-		)
-		(instances
-			(project "BPS-Leader"
-				(path "/bca74250-80d8-4ae3-9726-634afabc9565/fe68b7ab-dadd-40ec-a34d-6c2925722947"
-					(reference "#PWR050")
+					(reference "U3")
 					(unit 1)
 				)
@@
 		(dnp no)
 		(fields_autoplaced yes)
-		(property "Reference" "C14"
+		(property "Reference" "C2"
 			(at 139.6936 77.47 90)
 			(effects
@@
 			(project ""
 				(path "/bca74250-80d8-4ae3-9726-634afabc9565/fe68b7ab-dadd-40ec-a34d-6c2925722947"
-					(reference "C14")
+					(reference "C2")
 					(unit 1)
 				)
@@
 		(dnp no)
 		(fields_autoplaced yes)
-		(property "Reference" "#PWR049"
+		(property "Reference" "#PWR014"
 			(at 184.15 77.47 0)
 			(effects
@@
 			(project ""
 				(path "/bca74250-80d8-4ae3-9726-634afabc9565/fe68b7ab-dadd-40ec-a34d-6c2925722947"
-					(reference "#PWR049")
+					(reference "#PWR014")
 					(unit 1)
 				)
@@
 		(dnp no)
 		(fields_autoplaced yes)
-		(property "Reference" "#FLG04"
+		(property "Reference" "#FLG02"
 			(at 184.15 75.565 0)
 			(effects
@@
 			(project "BPS-Leader"
 				(path "/bca74250-80d8-4ae3-9726-634afabc9565/fe68b7ab-dadd-40ec-a34d-6c2925722947"
-					(reference "#FLG04")
+					(reference "#FLG02")
 					(unit 1)
 				)

Commit message: Preliminary Schematic
Parts:
- renumbered U3 to U2
Connections:
- net GND: now also U2.17 (GND)
- net Fan5: now reaches U2.6 (AIN7/GPIO7)
- no-connect marks 2 -> 0
Changed lines of the file:
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@@
 		(color 0 0 0 0)
 	)
-	(no_connect
-		(at 106.68 68.58)
-	)
-	(no_connect
-		(at 172.72 55.88)
-	)
 	(wire
 		(pts
@@
 	(wire
 		(pts
+			(xy 172.72 55.88) (xy 181.61 55.88)
+		)
+		(stroke
+			(width 0)
+			(type default)
+		)
+	)
+	(wire
+		(pts
 			(xy 106.68 73.66) (xy 106.68 83.82)
 		)
@@
 		(shape input)
 		(at 102.87 71.12 180)
+		(fields_autoplaced yes)
+		(effects
+			(font
+				(size 1.27 1.27)
+				(thickness 0.254)
+				(bold yes)
+			)
+			(justify right)
+		)
+	)
+	(hierarchical_label "Fan5"
+		(shape input)
+		(at 106.68 68.58 180)
 		(fields_autoplaced yes)
 		(effects
@@
 	(symbol
 		(lib_id "power:GND")
+		(at 181.61 55.88 0)
+		(unit 1)
+		(exclude_from_sim no)
+		(in_bom yes)
+		(on_board yes)
+		(dnp no)
+		(fields_autoplaced yes)
+		(property "Reference" "#PWR012"
+			(at 181.61 62.23 0)
+			(effects
+				(font
+					(size 1.27 1.27)
+				)
+				(hide yes)
+			)
+		)
+		(property "Value" "GND"
+			(at 181.61 60.96 0)
+			(effects
+				(font
+					(size 1.27 1.27)
+				)
+			)
+		)
+		(property "Footprint" ""
+			(at 181.61 55.88 0)
+			(effects
+				(font
+					(size 1.27 1.27)
+				)
+				(hide yes)
+			)
+		)
+		(property "Datasheet" ""
+			(at 181.61 55.88 0)
+			(effects
+				(font
+					(size 1.27 1.27)
+				)
+				(hide yes)
+			)
+		)
+		(property "Description" "Power symbol creates a global label with name \"GND\" , ground"
+			(at 181.61 55.88 0)
+			(effects
+				(font
+					(size 1.27 1.27)
+				)
+				(hide yes)
+			)
+		)
+		(pin "1"
+		)
+		(instances
+			(project "BPS-Leader"
+				(path "/bca74250-80d8-4ae3-9726-634afabc9565/fe68b7ab-dadd-40ec-a34d-6c2925722947"
+					(reference "#PWR012")
+					(unit 1)
+				)
+			)
+		)
+	)
+	(symbol
+		(lib_id "power:GND")
 		(at 172.72 87.63 0)
 		(unit 1)
@@
 		(dnp no)
 		(fields_autoplaced yes)
-		(property "Reference" "#PWR013"
+		(property "Reference" "#PWR011"
 			(at 172.72 93.98 0)
 			(effects
@@
 			(project ""
 				(path "/bca74250-80d8-4ae3-9726-634afabc9565/fe68b7ab-dadd-40ec-a34d-6c2925722947"
-					(reference "#PWR013")
+					(reference "#PWR011")
 					(unit 1)
 				)
@@
 		(dnp no)
 		(fields_autoplaced yes)
-		(property "Reference" "#PWR012"
+		(property "Reference" "#PWR010"
 			(at 102.87 87.63 0)
 			(effects
@@
 			(project "BPS-Leader"
 				(path "/bca74250-80d8-4ae3-9726-634afabc9565/fe68b7ab-dadd-40ec-a34d-6c2925722947"
-					(reference "#PWR012")
+					(reference "#PWR010")
 					(unit 1)
 				)
@@
 		(dnp no)
 		(fields_autoplaced yes)
-		(property "Reference" "U3"
+		(property "Reference" "U2"
 			(at 139.7 45.72 0)
 			(effects
@@
 			(project ""
 				(path "/bca74250-80d8-4ae3-9726-634afabc9565/fe68b7ab-dadd-40ec-a34d-6c2925722947"
-					(reference "U3")
+					(reference "U2")
 					(unit 1)
 				)
@@
 		(dnp no)
 		(fields_autoplaced yes)
-		(property "Reference" "#PWR014"
+		(property "Reference" "#PWR013"
 			(at 184.15 77.47 0)
 			(effects
@@
 			(project ""
 				(path "/bca74250-80d8-4ae3-9726-634afabc9565/fe68b7ab-dadd-40ec-a34d-6c2925722947"
-					(reference "#PWR014")
+					(reference "#PWR013")
 					(unit 1)
 				)

Commit message: adjusted shunt, added bypass caps to fan, high net removed, opamp output test pins added
Connections:
- net AVDD is gone; now on net +3.3V: C1.1, U2.7 (AVDD)
- net GNDA is gone; now on net GND: C1.2
Changed lines of the file:
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@@
+	)
+	(junction
+		(at 102.87 71.12)
+		(diameter 0)
+		(color 0 0 0 0)
 	)
 	(junction
@@
 	(wire
 		(pts
+			(xy 96.52 71.12) (xy 102.87 71.12)
+		)
+		(stroke
+			(width 0)
+			(type default)
+		)
+	)
+	(wire
+		(pts
 			(xy 102.87 71.12) (xy 106.68 71.12)
 		)
@@
 			)
 			(justify left)
-		)
-	)
-	(hierarchical_label "AVDD"
-		(shape input)
-		(at 102.87 71.12 180)
-		(fields_autoplaced yes)
-		(effects
-			(font
-				(size 1.27 1.27)
-				(thickness 0.254)
-				(bold yes)
-			)
-			(justify right)
 		)
 	)
@@
 	)
 	(symbol
-		(lib_id "power:GNDA")
-		(at 102.87 81.28 0)
-		(unit 1)
-		(exclude_from_sim no)
-		(in_bom yes)
-		(on_board yes)
-		(dnp no)
-		(fields_autoplaced yes)
-		(property "Reference" "#PWR010"
-			(at 102.87 87.63 0)
-			(effects
-				(font
-					(size 1.27 1.27)
-				)
-				(hide yes)
-			)
-		)
-		(property "Value" "GNDA"
-			(at 102.87 86.36 0)
-			(effects
-				(font
-					(size 1.27 1.27)
-				)
-			)
-		)
-		(property "Footprint" ""
-			(at 102.87 81.28 0)
-			(effects
-				(font
-					(size 1.27 1.27)
-				)
-				(hide yes)
-			)
-		)
-		(property "Datasheet" ""
-			(at 102.87 81.28 0)
-			(effects
-				(font
-					(size 1.27 1.27)
-				)
-				(hide yes)
-			)
-		)
-		(property "Description" "Power symbol creates a global label with name \"GNDA\" , analog ground"
-			(at 102.87 81.28 0)
-			(effects
-				(font
-					(size 1.27 1.27)
-				)
-				(hide yes)
-			)
-		)
-		(pin "1"
-		)
-		(instances
-			(project "BPS-Leader"
-				(path "/bca74250-80d8-4ae3-9726-634afabc9565/fe68b7ab-dadd-40ec-a34d-6c2925722947"
-					(reference "#PWR010")
-					(unit 1)
-				)
-			)
-		)
-	)
-	(symbol
 		(lib_id "2024-10-26_20-27-39:TLA2518IRTER")
 		(at 106.68 55.88 0)
@@
 					(unit 1)
 				)
+			)
+		)
+	)
+	(symbol
+		(lib_id "power:+3.3V")
+		(at 96.52 71.12 0)
+		(unit 1)
+		(exclude_from_sim no)
+		(in_bom yes)
+		(on_board yes)
+		(dnp no)
+		(fields_autoplaced yes)
+		(property "Reference" "#PWR0101"
+			(at 96.52 74.93 0)
+			(effects
+				(font
+					(size 1.27 1.27)
+				)
+				(hide yes)
+			)
+		)
+		(property "Value" "+3.3V"
+			(at 96.52 66.04 0)
+			(effects
+				(font
+					(size 1.27 1.27)
+				)
+			)
+		)
+		(property "Footprint" ""
+			(at 96.52 71.12 0)
+			(effects
+				(font
+					(size 1.27 1.27)
+				)
+				(hide yes)
+			)
+		)
+		(property "Datasheet" ""
+			(at 96.52 71.12 0)
+			(effects
+				(font
+					(size 1.27 1.27)
+				)
+				(hide yes)
+			)
+		)
+		(property "Description" "Power symbol creates a global label with name \"+3.3V\""
+			(at 96.52 71.12 0)
+			(effects
+				(font
+					(size 1.27 1.27)
+				)
+				(hide yes)
+			)
+		)
+		(pin "1"
+		)
+		(instances
+			(project "BPS-Leader"
+				(path "/bca74250-80d8-4ae3-9726-634afabc9565/fe68b7ab-dadd-40ec-a34d-6c2925722947"
+					(reference "#PWR0101")
+					(unit 1)
+				)
+			)
+		)
+	)
+	(symbol
+		(lib_id "power:GND")
+		(at 102.87 81.28 0)
+		(unit 1)
+		(exclude_from_sim no)
+		(in_bom yes)
+		(on_board yes)
+		(dnp no)
+		(fields_autoplaced yes)
+		(property "Reference" "#PWR010"
+			(at 102.87 87.63 0)
+			(effects
+				(font
+					(size 1.27 1.27)
+				)
+				(hide yes)
+			)
+		)
+		(property "Value" "GND"
+			(at 102.87 86.36 0)
+			(effects
+				(font
+					(size 1.27 1.27)
+				)
+			)
+		)
+		(property "Footprint" ""
+			(at 102.87 81.28 0)
+			(effects
+				(font
+					(size 1.27 1.27)
+				)
+				(hide yes)
+			)
+		)
+		(property "Datasheet" ""
+			(at 102.87 81.28 0)
+			(effects
+				(font
+					(size 1.27 1.27)
+				)
+				(hide yes)
+			)
+		)
+		(property "Description" "Power symbol creates a global label with name \"GND\" , ground"
+			(at 102.87 81.28 0)
+			(effects
+				(font
+					(size 1.27 1.27)
+				)
+				(hide yes)
+			)
+		)
+		(pin "1"
+		)
+		(instances
+			(project "BPS-Leader"
+				(path "/bca74250-80d8-4ae3-9726-634afabc9565/fe68b7ab-dadd-40ec-a34d-6c2925722947"
+					(reference "#PWR010")
+					(unit 1)
+				)

Commit message: everything should be finished now; tracks cleaned up, silkscreen issues fixed, new shunt/feedback/protection resistors chosen, BOM made, some other stuff i forgot probably
Parts:
- C1, C2, C3: P/N (none) -> C0805C105K5PACTU
- U2: P/N (none) -> TLA2518IRTER
Changed lines of the file:
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@@
 			)
 		)
-		(property "Datasheet" "~"
+		(property "Datasheet" "https://www.mouser.com/datasheet/2/447/KEM_C1006_X5R_SMD-3316465.pdf"
 			(at 102.87 78.74 0)
 			(effects
@@
 			)
 		)
+		(property "P/N" "C0805C105K5PACTU"
+			(at 102.87 78.74 0)
+			(effects
+				(font
+					(size 1.27 1.27)
+				)
+				(hide yes)
+			)
+		)
 		(pin "2"
 		)
@@
 			)
 		)
-		(property "Datasheet" "~"
+		(property "Datasheet" "https://www.mouser.com/datasheet/2/447/KEM_C1006_X5R_SMD-3316465.pdf"
 			(at 175.26 81.28 0)
 			(effects
@@
 		)
 		(property "Description" "Unpolarized capacitor, small symbol"
+			(at 175.26 81.28 0)
+			(effects
+				(font
+					(size 1.27 1.27)
+				)
+				(hide yes)
+			)
+		)
+		(property "P/N" "C0805C105K5PACTU"
 			(at 175.26 81.28 0)
 			(effects
@@
 			)
 		)
-		(property "Datasheet" "TLA2518IRTER"
+		(property "Datasheet" "https://www.ti.com/lit/ds/symlink/tla2518.pdf?ts=1737821011794&ref_url=https%253A%252F%252Fwww.mouser.com%252F"
 			(at 106.68 55.88 0)
 			(effects
@@
 		)
 		(property "Description" ""
+			(at 106.68 55.88 0)
+			(effects
+				(font
+					(size 1.27 1.27)
+				)
+				(hide yes)
+			)
+		)
+		(property "P/N" "TLA2518IRTER"
 			(at 106.68 55.88 0)
 			(effects
@@
 			)
 		)
-		(property "Datasheet" "~"
+		(property "Datasheet" "https://www.mouser.com/datasheet/2/447/KEM_C1006_X5R_SMD-3316465.pdf"
 			(at 139.7 83.82 0)
 			(effects
@@
 			(at 139.7 83.82 0)
 			(effects
+				(font
+					(size 1.27 1.27)
+				)
+				(hide yes)
+			)
+		)
+		(property "P/N" "C0805C105K5PACTU"
+			(at 139.7 83.82 0)
+			(effects
