File: currentsense.kicad_sch (KiCad schematic)
At the start: 15 parts, among them Q6 IRLML0030, U4 INA180B1

Commit message: Preliminary Schematic Finished
Parts:
- D7: renamed from D10; footprint (none) -> Diode_SMD:D_0805_2012Metric
- D8: renamed from D11; footprint (none) -> Diode_SMD:D_0805_2012Metric
- renumbered C7 to C10, C8 to C11, Q6 to Q4, R34 to R28, R35 to R29, R36 to R30, R37 to R31, R38 to R32, R39 to R33, R40 to R34, R41 to R35, R42 to R36, U4 to U7

Commit message: Preliminary Schematic
Parts:
- removed R34, R36: R, Resistor_SMD:R_0805_2012Metric, symbol Device:R
- removed U7: INA180B1, Package_TO_SOT_SMD:SOT-23-5, symbol Amplifier_Current:INA180B1
- added C20: 0.16uF, Capacitor_SMD:C_0805_2012Metric, symbol Device:C_Small
- added U3: INA180A2, Package_TO_SOT_SMD:SOT-23-5, symbol Amplifier_Current:INA180A2
- R40: renamed from R31; value R -> 1.8m
- R41: renamed from R32; value R -> 5
- R42: renamed from R33; value R -> 5
- R44: renamed from R35; value R -> 0.9
- renumbered C10 to C12, C11 to C13, D8 to D10, D7 to D9, Q4 to Q5, R28 to R37, R29 to R38, R30 to R39
Connections:
- net +3.3V: now also U3.5 (V+)
- net GND: now also U3.2 (GND)
- net OAO: now also R44.2, U3.1
- net at R42.2, R44.1: now also C20.2, U3.4 (-)
- net at R41.2: now also C20.1, U3.3 (+)

Commit message: adjusted shunt, added bypass caps to fan, high net removed, opamp output test pins added
Parts:
- added D19, D27: 1N448W, Diode_SMD:D_0805_2012Metric, symbol Device:D
- R40: value 1.8m -> 3m
- renumbered C20 to C24, U3 to U7
Connections:
- net +3.3V: now also D27.1 (K)
- net GND: now also D19.2 (A)
- net OAO: now also D19.1 (K), D27.2 (A)
- net High: no longer names the net of R40.2, R42.1
Other:
- moved on the sheet: C12, C13

Commit message: preliminary schematic completed
Parts:
- renumbered C12 to C16, C24 to C17, C13 to C18, D9 to D17, D10 to D18, D27 to D19, D19 to D20, Q5 to Q7, R37 to R33, R38 to R34, R39 to R35, R40 to R36, R41 to R37, R42 to R38, R44 to R39, U7 to U3

Commit message: Very rough layout of the board - maybe too long?
Parts:
- renumbered U3 to U7
Changed lines of the file:
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@@
 		(on_board yes)
 		(dnp no)
-		(property "Reference" "U3"
+		(property "Reference" "U7"
 			(at 105.918 42.926 0)
 			(effects

Commit message: everything should be finished now; tracks cleaned up, silkscreen issues fixed, new shunt/feedback/protection resistors chosen, BOM made, some other stuff i forgot probably
Parts:
- C16: value 1.1uF -> 0.1uF; P/N (none) -> C0805C104M5RACTU
- C17: value 0.16uF -> 0.15uF; P/N (none) -> 08051C154KAT2A
- C18: value 2.2uF -> 0.1uF; P/N (none) -> C0805C104M5RACTU
- D17: footprint Diode_SMD:D_0805_2012Metric -> footprints:D_0805_2012Metric(adjsilk); P/N (none) -> HSMQ-C170-T0000
- D18, D19, D20: footprint Diode_SMD:D_0805_2012Metric -> footprints:D_0805_2012Metric(adjsilk); P/N (none) -> 1N4448W-G3-18
- Q7: P/N (none) -> IRLML0030
- R33: P/N (none) -> CRCW0805100KFKEAC
- R34: P/N (none) -> CRCW080510K0FKEAC
- R35: P/N (none) -> CRCW08051K00FKEAC
- R36: value 3m -> 2.8m; footprint Resistor_SMD:R_0805_2012Metric -> Resistor_SMD:R_2512_6332Metric; P/N (none) -> WSLP25122L800FEA
- R37, R38: value 5 -> 10; P/N (none) -> CRGP0805F10R
- R39: value 0.9 -> 1; P/N (none) -> CRM0805-FW-1R00ELF
- U7: footprint Package_TO_SOT_SMD:SOT-23-5 -> footprints:SOT-23-5(movedsilk); P/N (none) -> INA180A2
