File: drivernosense.kicad_sch (KiCad schematic)
At the start: 6 parts, among them Q2 IRLML0030, Q3 IRLML0030

Commit message: everything should be finished now; tracks cleaned up, silkscreen issues fixed, new shunt/feedback/protection resistors chosen, BOM made, some other stuff i forgot probably
Parts:
- Q2, Q3: P/N (none) -> IRLML0030
- R10, R8: P/N (none) -> CRCW0805100KFKEAC
- R11, R9: P/N (none) -> CRCW08051K00FKEAC
Changed lines of the file:
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@@
+			)
+		)
+		(property "P/N" "IRLML0030"
+			(at 35.56 43.18 0)
+			(effects
+				(font
+					(size 1.27 1.27)
+				)
+				(hide yes)
 			)
 		)
@@
 			)
 		)
-		(property "Datasheet" "~"
+		(property "Datasheet" "https://www.mouser.com/ProductDetail/Vishay-Dale/CRCW0805100KFKEAC?qs=sGAEpiMZZMvdGkrng054t0DrEhLhGh8gZRT9GjFuHWDV3jEqj5sSqw%3D%3D"
 			(at 58.42 49.53 0)
 			(effects
@@
 			)
 		)
+		(property "P/N" "CRCW0805100KFKEAC"
+			(at 58.42 49.53 0)
+			(effects
+				(font
+					(size 1.27 1.27)
+				)
+				(hide yes)
+			)
+		)
 		(pin "1"
 		)
@@
 			)
 		)
-		(property "Datasheet" "~"
+		(property "Datasheet" "https://www.mouser.com/ProductDetail/71-CRCW08051K00FKEAC"
 			(at 63.5 43.18 0)
 			(effects
@@
 			)
 		)
+		(property "P/N" "CRCW08051K00FKEAC"
+			(at 63.5 43.18 0)
+			(effects
+				(font
+					(size 1.27 1.27)
+				)
+				(hide yes)
+			)
+		)
 		(pin "1"
 		)
@@
 			)
 		)
-		(property "Datasheet" "~"
+		(property "Datasheet" "https://www.mouser.com/ProductDetail/71-CRCW08051K00FKEAC"
 			(at 25.4 43.18 0)
 			(effects
@@
 			)
 		)
+		(property "P/N" "CRCW08051K00FKEAC"
+			(at 25.4 43.18 0)
+			(effects
+				(font
+					(size 1.27 1.27)
+				)
+				(hide yes)
+			)
+		)
 		(pin "1"
 		)
@@
 			)
 		)
+		(property "P/N" "IRLML0030"
+			(at 73.66 43.18 0)
+			(effects
+				(font
+					(size 1.27 1.27)
+				)
+				(hide yes)
+			)
+		)
 		(pin "2"
 		)
@@
 			)
 		)
-		(property "Datasheet" "~"
+		(property "Datasheet" "https://www.mouser.com/ProductDetail/Vishay-Dale/CRCW0805100KFKEAC?qs=sGAEpiMZZMvdGkrng054t0DrEhLhGh8gZRT9GjFuHWDV3jEqj5sSqw%3D%3D"
 			(at 20.32 49.53 0)
 			(effects
@@
 			(at 20.32 49.53 0)
 			(effects
+				(font
+					(size 1.27 1.27)
+				)
+				(hide yes)
+			)
+		)
+		(property "P/N" "CRCW0805100KFKEAC"
+			(at 20.32 49.53 0)
+			(effects
