File: fancntrlr.kicad_sch (KiCad schematic)
At the start: 13 parts, among them U1 EMC2305-1-AP-TR

Commit message: Preliminary Schematic
Parts:
- removed R68, R69, R72, R76, R77: 100k, Resistor_SMD:R_0805_2012Metric, symbol Device:R
- added R74: 15k, Resistor_SMD:R_0805_2012Metric, symbol Device:R
- R72: renamed from R67; value 100k -> 33k
- renumbered R70 to R67, R73 to R68, R74 to R69, R75 to R70, R78 to R73, U1 to U10
Connections:
- net +3.3V: now also R74.1
- net PWM3: no longer R71.2
- net at U10.11 (CLK): now also R74.2
- net PWM5: now reaches U10.15 (PWM5)
- net TACH5: now reaches U10.16 (TACH5)
- net TACH5: now also R71.2
- no-connect marks 3 -> 0
Other:
- note added: "Default Fan Speed"
- moved on the sheet: R67, R68, R69, R70, R72, R73

Commit message: adjusted shunt, added bypass caps to fan, high net removed, opamp output test pins added
Parts:
- added C28, C29: 1uF, Capacitor_SMD:C_0805_2012Metric, symbol Device:C_Small
Connections:
- net +3.3V: now also C28.1, C29.1
- net GND: now also C28.2, C29.2
Other:
- note added: "I2C1_SCL I2C1_SDA"
- moved on the sheet: R74, U10

Commit message: preliminary schematic completed
Parts:
- renumbered C28 to C25, C29 to C26, R67 to R57, R68 to R58, R69 to R59, R70 to R60, R71 to R61, R72 to R62, R73 to R63, R74 to R64
Changed lines of the file:
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@@
 		(on_board yes)
 		(dnp no)
-		(property "Reference" "#PWR080"
+		(property "Reference" "#PWR0102"
 			(at 25.4 66.04 0)
 			(effects
@@
 			(project "BPS-Leader"
 				(path "/bca74250-80d8-4ae3-9726-634afabc9565/9150f836-09cb-45bb-b39a-93624518a94e"
-					(reference "#PWR080")
+					(reference "#PWR0102")
 					(unit 1)
 				)
@@
 		(on_board yes)
 		(dnp no)
-		(property "Reference" "R73"
+		(property "Reference" "R63"
 			(at 48.768 80.772 90)
 			(effects
@@
 			(project "BPS-Leader"
 				(path "/bca74250-80d8-4ae3-9726-634afabc9565/9150f836-09cb-45bb-b39a-93624518a94e"
-					(reference "R73")
+					(reference "R63")
 					(unit 1)
 				)
@@
 		(on_board yes)
 		(dnp no)
-		(property "Reference" "#PWR099"
+		(property "Reference" "#PWR0109"
 			(at 46.99 41.91 0)
 			(effects
@@
 			(project "BPS-Leader"
 				(path "/bca74250-80d8-4ae3-9726-634afabc9565/9150f836-09cb-45bb-b39a-93624518a94e"
-					(reference "#PWR099")
+					(reference "#PWR0109")
 					(unit 1)
 				)
@@
 		(on_board yes)
 		(dnp no)
-		(property "Reference" "R68"
+		(property "Reference" "R58"
 			(at 23.368 81.026 90)
 			(effects
@@
 			(project "BPS-Leader"
 				(path "/bca74250-80d8-4ae3-9726-634afabc9565/9150f836-09cb-45bb-b39a-93624518a94e"
-					(reference "R68")
+					(reference "R58")
 					(unit 1)
 				)
@@
 		(on_board yes)
 		(dnp no)
-		(property "Reference" "C28"
+		(property "Reference" "C25"
 			(at 35.56 32.258 0)
 			(effects
@@
 			(project "BPS-Leader"
 				(path "/bca74250-80d8-4ae3-9726-634afabc9565/9150f836-09cb-45bb-b39a-93624518a94e"
-					(reference "C28")
+					(reference "C25")
 					(unit 1)
 				)
@@
 		(on_board yes)
 		(dnp no)
-		(property "Reference" "#PWR084"
+		(property "Reference" "#PWR0106"
 			(at 25.4 118.11 0)
 			(effects
@@
 			(project "BPS-Leader"
 				(path "/bca74250-80d8-4ae3-9726-634afabc9565/9150f836-09cb-45bb-b39a-93624518a94e"
-					(reference "#PWR084")
+					(reference "#PWR0106")
 					(unit 1)
 				)
@@
 		(on_board yes)
 		(dnp no)
-		(property "Reference" "R70"
+		(property "Reference" "R60"
 			(at 23.368 106.426 90)
 			(effects
@@
 			(project "BPS-Leader"
 				(path "/bca74250-80d8-4ae3-9726-634afabc9565/9150f836-09cb-45bb-b39a-93624518a94e"
-					(reference "R70")
+					(reference "R60")
 					(unit 1)
 				)
@@
 		(on_board yes)
 		(dnp no)
-		(property "Reference" "#PWR0100"
+		(property "Reference" "#PWR0108"
 			(at 39.37 41.91 0)
 			(effects
@@
 			(project "BPS-Leader"
 				(path "/bca74250-80d8-4ae3-9726-634afabc9565/9150f836-09cb-45bb-b39a-93624518a94e"
-					(reference "#PWR0100")
+					(reference "#PWR0108")
 					(unit 1)
 				)
@@
 		(on_board yes)
 		(dnp no)
-		(property "Reference" "#PWR082"
+		(property "Reference" "#PWR0104"
 			(at 25.4 91.44 0)
 			(effects
@@
 			(project "BPS-Leader"
 				(path "/bca74250-80d8-4ae3-9726-634afabc9565/9150f836-09cb-45bb-b39a-93624518a94e"
-					(reference "#PWR082")
+					(reference "#PWR0104")
 					(unit 1)
 				)
@@
 		(on_board yes)
 		(dnp no)
-		(property "Reference" "#PWR079"
+		(property "Reference" "#PWR0107"
 			(at 39.37 34.29 0)
 			(effects
@@
 			(project ""
 				(path "/bca74250-80d8-4ae3-9726-634afabc9565/9150f836-09cb-45bb-b39a-93624518a94e"
-					(reference "#PWR079")
+					(reference "#PWR0107")
 					(unit 1)
 				)
@@
 		(on_board yes)
 		(dnp no)
-		(property "Reference" "R67"
+		(property "Reference" "R57"
 			(at 23.368 68.072 90)
 			(effects
@@
 			(project "BPS-Leader"
 				(path "/bca74250-80d8-4ae3-9726-634afabc9565/9150f836-09cb-45bb-b39a-93624518a94e"
-					(reference "R67")
+					(reference "R57")
 					(unit 1)
 				)
@@
 		(on_board yes)
 		(dnp no)
-		(property "Reference" "#PWR086"
+		(property "Reference" "#PWR0111"
 			(at 50.8 78.74 0)
 			(effects
@@
 			(project "BPS-Leader"
 				(path "/bca74250-80d8-4ae3-9726-634afabc9565/9150f836-09cb-45bb-b39a-93624518a94e"
-					(reference "#PWR086")
+					(reference "#PWR0111")
 					(unit 1)
 				)
@@
 		(on_board yes)
 		(dnp no)
-		(property "Reference" "R69"
+		(property "Reference" "R59"
 			(at 23.114 93.472 90)
 			(effects
@@
 			(project "BPS-Leader"
 				(path "/bca74250-80d8-4ae3-9726-634afabc9565/9150f836-09cb-45bb-b39a-93624518a94e"
-					(reference "R69")
+					(reference "R59")
 					(unit 1)
 				)
@@
 		(on_board yes)
 		(dnp no)
-		(property "Reference" "#PWR087"
+		(property "Reference" "#PWR0112"
 			(at 123.19 31.75 0)
 			(effects
@@
 			(project ""
 				(path "/bca74250-80d8-4ae3-9726-634afabc9565/9150f836-09cb-45bb-b39a-93624518a94e"
-					(reference "#PWR087")
+					(reference "#PWR0112")
 					(unit 1)
 				)
@@
 		(on_board yes)
 		(dnp no)
-		(property "Reference" "#PWR081"
+		(property "Reference" "#PWR0103"
 			(at 25.4 78.74 0)
 			(effects
@@
 			(project "BPS-Leader"
 				(path "/bca74250-80d8-4ae3-9726-634afabc9565/9150f836-09cb-45bb-b39a-93624518a94e"
-					(reference "#PWR081")
+					(reference "#PWR0103")
 					(unit 1)
 				)
@@
 		(on_board yes)
 		(dnp no)
-		(property "Reference" "#PWR083"
+		(property "Reference" "#PWR0105"
 			(at 25.4 104.14 0)
 			(effects
@@
 			(project "BPS-Leader"
 				(path "/bca74250-80d8-4ae3-9726-634afabc9565/9150f836-09cb-45bb-b39a-93624518a94e"
-					(reference "#PWR083")
+					(reference "#PWR0105")
 					(unit 1)
 				)
@@
 		(on_board yes)
 		(dnp no)
-		(property "Reference" "#PWR085"
+		(property "Reference" "#PWR0110"
 			(at 50.8 66.04 0)
 			(effects
@@
 			(project "BPS-Leader"
 				(path "/bca74250-80d8-4ae3-9726-634afabc9565/9150f836-09cb-45bb-b39a-93624518a94e"
-					(reference "#PWR085")
+					(reference "#PWR0110")
 					(unit 1)
 				)
@@
 		(on_board yes)
 		(dnp no)
-		(property "Reference" "R74"
+		(property "Reference" "R64"
 			(at 123.698 38.608 90)
 			(effects
@@
 			(project "BPS-Leader"
 				(path "/bca74250-80d8-4ae3-9726-634afabc9565/9150f836-09cb-45bb-b39a-93624518a94e"
-					(reference "R74")
+					(reference "R64")
 					(unit 1)
 				)
@@
 		(on_board yes)
 		(dnp no)
-		(property "Reference" "R72"
+		(property "Reference" "R62"
 			(at 48.768 68.072 90)
 			(effects
@@
 			(project "BPS-Leader"
 				(path "/bca74250-80d8-4ae3-9726-634afabc9565/9150f836-09cb-45bb-b39a-93624518a94e"
-					(reference "R72")
+					(reference "R62")
 					(unit 1)
 				)
@@
 		(on_board yes)
 		(dnp no)
-		(property "Reference" "C29"
+		(property "Reference" "C26"
 			(at 43.18 32.258 0)
 			(effects
@@
 			(project "BPS-Leader"
 				(path "/bca74250-80d8-4ae3-9726-634afabc9565/9150f836-09cb-45bb-b39a-93624518a94e"
-					(reference "C29")
+					(reference "C26")
 					(unit 1)
 				)
@@
 		(on_board yes)
 		(dnp no)
-		(property "Reference" "R71"
+		(property "Reference" "R61"
 			(at 23.368 120.396 90)
 			(effects
@@
 			(project "BPS-Leader"
 				(path "/bca74250-80d8-4ae3-9726-634afabc9565/9150f836-09cb-45bb-b39a-93624518a94e"
-					(reference "R71")
+					(reference "R61")
 					(unit 1)
 				)
@@
 		(on_board yes)
 		(dnp no)
-		(property "Reference" "#PWR088"
+		(property "Reference" "#PWR0113"
 			(at 125.73 36.83 0)
 			(effects
@@
 			(project "BPS-Leader"
 				(path "/bca74250-80d8-4ae3-9726-634afabc9565/9150f836-09cb-45bb-b39a-93624518a94e"
-					(reference "#PWR088")
-					(unit 1)
-				)
+					(reference "#PWR0113")
+					(unit 1)
+				)

Commit message: everything should be finished now; tracks cleaned up, silkscreen issues fixed, new shunt/feedback/protection resistors chosen, BOM made, some other stuff i forgot probably
Parts:
- C25, C26: P/N (none) -> C0805C105K5PACTU
- R57, R58, R59, R60, R61, R63: P/N (none) -> CRCW0805100KFKEAC
- R62: P/N (none) -> ERA-6ARB333V
- R64: P/N (none) -> ERA-6VEB1502V
- U10: P/N (none) -> EMC2305-1-AP-TR
Changed lines of the file:
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@@
 			)
 		)
-		(property "Datasheet" "~"
+		(property "Datasheet" "https://www.mouser.com/ProductDetail/Vishay-Dale/CRCW0805100KFKEAC?qs=sGAEpiMZZMvdGkrng054t0DrEhLhGh8gZRT9GjFuHWDV3jEqj5sSqw%3D%3D"
 			(at 50.8 78.74 0)
 			(effects
@@
 			)
 		)
+		(property "P/N" "CRCW0805100KFKEAC"
+			(at 50.8 78.74 0)
+			(effects
+				(font
+					(size 1.27 1.27)
+				)
+				(hide yes)
+			)
+		)
 		(pin "1"
 		)
@@
 			)
 		)
-		(property "Datasheet" "~"
+		(property "Datasheet" "https://www.mouser.com/ProductDetail/Vishay-Dale/CRCW0805100KFKEAC?qs=sGAEpiMZZMvdGkrng054t0DrEhLhGh8gZRT9GjFuHWDV3jEqj5sSqw%3D%3D"
 			(at 25.4 78.74 0)
 			(effects
@@
 			)
 		)
+		(property "P/N" "CRCW0805100KFKEAC"
+			(at 25.4 78.74 0)
+			(effects
+				(font
+					(size 1.27 1.27)
+				)
+				(hide yes)
+			)
+		)
 		(pin "1"
 		)
@@
 			)
 		)
-		(property "Datasheet" "~"
+		(property "Datasheet" "https://www.mouser.com/datasheet/2/447/KEM_C1006_X5R_SMD-3316465.pdf"
 			(at 39.37 33.02 0)
 			(effects
@@
 			)
 		)
+		(property "P/N" "C0805C105K5PACTU"
+			(at 39.37 33.02 0)
+			(effects
+				(font
+					(size 1.27 1.27)
+				)
+				(hide yes)
+			)
+		)
 		(pin "2"
 		)
@@
 			)
 		)
-		(property "Datasheet" "~"
+		(property "Datasheet" "https://www.mouser.com/ProductDetail/Vishay-Dale/CRCW0805100KFKEAC?qs=sGAEpiMZZMvdGkrng054t0DrEhLhGh8gZRT9GjFuHWDV3jEqj5sSqw%3D%3D"
 			(at 25.4 104.14 0)
 			(effects
@@
 			)
 		)
+		(property "P/N" "CRCW0805100KFKEAC"
+			(at 25.4 104.14 0)
+			(effects
+				(font
+					(size 1.27 1.27)
+				)
+				(hide yes)
+			)
+		)
 		(pin "1"
 		)
@@
 			)
 		)
-		(property "Datasheet" "~"
+		(property "Datasheet" "https://www.mouser.com/ProductDetail/Vishay-Dale/CRCW0805100KFKEAC?qs=sGAEpiMZZMvdGkrng054t0DrEhLhGh8gZRT9GjFuHWDV3jEqj5sSqw%3D%3D"
 			(at 25.4 66.04 0)
 			(effects
@@
 			)
 		)
+		(property "P/N" "CRCW0805100KFKEAC"
+			(at 25.4 66.04 0)
+			(effects
+				(font
+					(size 1.27 1.27)
+				)
+				(hide yes)
+			)
+		)
 		(pin "1"
 		)
@@
 			)
 		)
-		(property "Datasheet" "~"
+		(property "Datasheet" "https://www.mouser.com/ProductDetail/Vishay-Dale/CRCW0805100KFKEAC?qs=sGAEpiMZZMvdGkrng054t0DrEhLhGh8gZRT9GjFuHWDV3jEqj5sSqw%3D%3D"
 			(at 25.4 91.44 0)
 			(effects
@@
 		)
 		(property "Description" "Resistor"
+			(at 25.4 91.44 0)
+			(effects
+				(font
+					(size 1.27 1.27)
+				)
+				(hide yes)
+			)
+		)
+		(property "P/N" "CRCW0805100KFKEAC"
 			(at 25.4 91.44 0)
 			(effects
@@
 			)
 		)
-		(property "Datasheet" "EMC2305-1-AP-TR"
+		(property "Datasheet" "https://ww1.microchip.com/downloads/aemDocuments/documents/MSLD/ProductDocuments/DataSheets/EMC2301-2-3-5-Data-Sheet-DS20006532A.pdf"
 			(at 60.96 25.4 0)
 			(effects
@@
 			)
 		)
+		(property "P/N" "EMC2305-1-AP-TR"
+			(at 60.96 25.4 0)
+			(effects
+				(font
+					(size 1.27 1.27)
+				)
+				(hide yes)
+			)
+		)
 		(pin "8"
 		)
@@
 			)
 		)
-		(property "Datasheet" "~"
+		(property "Datasheet" "https://www.mouser.com/catalog/specsheets/Panasonic_ERA.pdf"
 			(at 125.73 36.83 0)
 			(effects
@@
 			)
 		)
+		(property "P/N" "ERA-6VEB1502V"
+			(at 125.73 36.83 0)
+			(effects
+				(font
+					(size 1.27 1.27)
+				)
+				(hide yes)
+			)
+		)
 		(pin "1"
 		)
@@
 			)
 		)
-		(property "Datasheet" "~"
+		(property "Datasheet" "https://industrial.panasonic.com/cdbs/www-data/pdf/RDM0000/AOA0000C307.pdf"
 			(at 50.8 66.04 0)
 			(effects
@@
 			)
 		)
+		(property "P/N" "ERA-6ARB333V"
+			(at 50.8 66.04 0)
+			(effects
+				(font
+					(size 1.27 1.27)
+				)
+				(hide yes)
+			)
+		)
 		(pin "1"
 		)
@@
 			)
 		)
-		(property "Datasheet" "~"
+		(property "Datasheet" "https://www.mouser.com/datasheet/2/447/KEM_C1006_X5R_SMD-3316465.pdf"
 			(at 46.99 33.02 0)
 			(effects
@@
 			)
 		)
+		(property "P/N" "C0805C105K5PACTU"
+			(at 46.99 33.02 0)
+			(effects
+				(font
+					(size 1.27 1.27)
+				)
+				(hide yes)
+			)
+		)
 		(pin "2"
 		)
@@
 			)
 		)
-		(property "Datasheet" "~"
+		(property "Datasheet" "https://www.mouser.com/ProductDetail/Vishay-Dale/CRCW0805100KFKEAC?qs=sGAEpiMZZMvdGkrng054t0DrEhLhGh8gZRT9GjFuHWDV3jEqj5sSqw%3D%3D"
 			(at 25.4 118.11 0)
 			(effects
@@
 			(at 25.4 118.11 0)
 			(effects
+				(font
+					(size 1.27 1.27)
+				)
+				(hide yes)
+			)
+		)
+		(property "P/N" "CRCW0805100KFKEAC"
+			(at 25.4 118.11 0)
+			(effects
