File: strobe.kicad_sch (KiCad schematic)
At the start: 6 parts, among them Q8 IRLML0030

Commit message: Added pull-up resistors to the fan control chip
Other:
- moved on the sheet: D15, D16, Q8, R64, R65, R66

Commit message: Preliminary Schematic
Parts:
- renumbered D15 to D13, D16 to D14, Q8 to Q7, R64 to R55, R65 to R56, R66 to R57
Changed lines of the file:
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@@
 		(on_board yes)
 		(dnp no)
-		(property "Reference" "D16"
+		(property "Reference" "D14"
 			(at 33.274 43.688 90)
 			(effects
@@
 			(project "BPS-Leader"
 				(path "/bca74250-80d8-4ae3-9726-634afabc9565/52b3a4d4-955c-43e8-a21b-33fe1a04884d"
-					(reference "D16")
+					(reference "D14")
 					(unit 1)
 				)
@@
 		(on_board yes)
 		(dnp no)
-		(property "Reference" "R65"
+		(property "Reference" "R56"
 			(at 21.082 34.544 0)
 			(effects
@@
 			(project "BPS-Leader"
 				(path "/bca74250-80d8-4ae3-9726-634afabc9565/52b3a4d4-955c-43e8-a21b-33fe1a04884d"
-					(reference "R65")
+					(reference "R56")
 					(unit 1)
 				)
@@
 		(dnp no)
 		(fields_autoplaced yes)
-		(property "Reference" "#PWR078"
+		(property "Reference" "#PWR068"
 			(at 39.37 29.21 0)
 			(effects
@@
 			(project "BPS-Leader"
 				(path "/bca74250-80d8-4ae3-9726-634afabc9565/52b3a4d4-955c-43e8-a21b-33fe1a04884d"
-					(reference "#PWR078")
+					(reference "#PWR068")
 					(unit 1)
 				)
@@
 		(on_board yes)
 		(dnp no)
-		(property "Reference" "D15"
+		(property "Reference" "D13"
 			(at 20.828 42.164 90)
 			(effects
@@
 			(project "BPS-Leader"
 				(path "/bca74250-80d8-4ae3-9726-634afabc9565/52b3a4d4-955c-43e8-a21b-33fe1a04884d"
-					(reference "D15")
+					(reference "D13")
 					(unit 1)
 				)
@@
 		(dnp no)
 		(fields_autoplaced yes)
-		(property "Reference" "#PWR079"
+		(property "Reference" "#PWR069"
 			(at 39.37 73.66 0)
 			(effects
@@
 			(project "BPS-Leader"
 				(path "/bca74250-80d8-4ae3-9726-634afabc9565/52b3a4d4-955c-43e8-a21b-33fe1a04884d"
-					(reference "#PWR079")
+					(reference "#PWR069")
 					(unit 1)
 				)
@@
 		(on_board yes)
 		(dnp no)
-		(property "Reference" "R64"
+		(property "Reference" "R55"
 			(at 19.558 64.77 90)
 			(effects
@@
 			(project "BPS-Leader"
 				(path "/bca74250-80d8-4ae3-9726-634afabc9565/52b3a4d4-955c-43e8-a21b-33fe1a04884d"
-					(reference "R64")
+					(reference "R55")
 					(unit 1)
 				)
@@
 		(dnp no)
 		(fields_autoplaced yes)
-		(property "Reference" "Q8"
+		(property "Reference" "Q7"
 			(at 43.18 55.8799 0)
 			(effects
@@
 			(project "BPS-Leader"
 				(path "/bca74250-80d8-4ae3-9726-634afabc9565/52b3a4d4-955c-43e8-a21b-33fe1a04884d"
-					(reference "Q8")
+					(reference "Q7")
 					(unit 1)
 				)
@@
 		(on_board yes)
 		(dnp no)
-		(property "Reference" "R66"
+		(property "Reference" "R57"
 			(at 26.67 55.118 90)
 			(effects
@@
 			(project "BPS-Leader"
 				(path "/bca74250-80d8-4ae3-9726-634afabc9565/52b3a4d4-955c-43e8-a21b-33fe1a04884d"
-					(reference "R66")
-					(unit 1)
-				)
+					(reference "R57")
+					(unit 1)
+				)

Commit message: adjusted shunt, added bypass caps to fan, high net removed, opamp output test pins added
Changed lines of the file:
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@@
 	(paper "A4")
-	(junction
-		(at 39.37 26.67)
-		(diameter 0)
-		(color 0 0 0 0)
-	)
 	(junction
 		(at 33.02 26.67)
@@
 	(wire
 		(pts
-			(xy 39.37 26.67) (xy 39.37 36.83)
-		)
-		(stroke
-			(width 0)
-			(type default)
-		)
-	)
-	(wire
-		(pts
 			(xy 26.67 50.8) (xy 26.67 46.99)
 		)
@@
 		)
 	)
-	(hierarchical_label "High"
-		(shape input)
-		(at 39.37 36.83 0)
-		(fields_autoplaced yes)
-		(effects
-			(font
-				(size 1.27 1.27)
-				(thickness 0.254)
-				(bold yes)
-			)
-			(justify left)
-		)
-	)

Commit message: preliminary schematic completed
Parts:
- renumbered D13 to D25, D14 to D26, Q7 to Q9, R55 to R47, R56 to R48, R57 to R49
Changed lines of the file:
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@@
 		(on_board yes)
 		(dnp no)
-		(property "Reference" "D14"
+		(property "Reference" "D26"
 			(at 33.274 43.688 90)
 			(effects
@@
 			(project "BPS-Leader"
 				(path "/bca74250-80d8-4ae3-9726-634afabc9565/52b3a4d4-955c-43e8-a21b-33fe1a04884d"
-					(reference "D14")
+					(reference "D26")
 					(unit 1)
 				)
@@
 		(on_board yes)
 		(dnp no)
-		(property "Reference" "R56"
+		(property "Reference" "R48"
 			(at 21.082 34.544 0)
 			(effects
@@
 			(project "BPS-Leader"
 				(path "/bca74250-80d8-4ae3-9726-634afabc9565/52b3a4d4-955c-43e8-a21b-33fe1a04884d"
-					(reference "R56")
+					(reference "R48")
 					(unit 1)
 				)
@@
 		(dnp no)
 		(fields_autoplaced yes)
-		(property "Reference" "#PWR068"
+		(property "Reference" "#PWR090"
 			(at 39.37 29.21 0)
 			(effects
@@
 			(project "BPS-Leader"
 				(path "/bca74250-80d8-4ae3-9726-634afabc9565/52b3a4d4-955c-43e8-a21b-33fe1a04884d"
-					(reference "#PWR068")
+					(reference "#PWR090")
 					(unit 1)
 				)
@@
 		(on_board yes)
 		(dnp no)
-		(property "Reference" "D13"
+		(property "Reference" "D25"
 			(at 20.828 42.164 90)
 			(effects
@@
 			(project "BPS-Leader"
 				(path "/bca74250-80d8-4ae3-9726-634afabc9565/52b3a4d4-955c-43e8-a21b-33fe1a04884d"
-					(reference "D13")
+					(reference "D25")
 					(unit 1)
 				)
@@
 		(dnp no)
 		(fields_autoplaced yes)
-		(property "Reference" "#PWR069"
+		(property "Reference" "#PWR091"
 			(at 39.37 73.66 0)
 			(effects
@@
 			(project "BPS-Leader"
 				(path "/bca74250-80d8-4ae3-9726-634afabc9565/52b3a4d4-955c-43e8-a21b-33fe1a04884d"
-					(reference "#PWR069")
+					(reference "#PWR091")
 					(unit 1)
 				)
@@
 		(on_board yes)
 		(dnp no)
-		(property "Reference" "R55"
+		(property "Reference" "R47"
 			(at 19.558 64.77 90)
 			(effects
@@
 			(project "BPS-Leader"
 				(path "/bca74250-80d8-4ae3-9726-634afabc9565/52b3a4d4-955c-43e8-a21b-33fe1a04884d"
-					(reference "R55")
+					(reference "R47")
 					(unit 1)
 				)
@@
 		(dnp no)
 		(fields_autoplaced yes)
-		(property "Reference" "Q7"
+		(property "Reference" "Q9"
 			(at 43.18 55.8799 0)
 			(effects
@@
 			(project "BPS-Leader"
 				(path "/bca74250-80d8-4ae3-9726-634afabc9565/52b3a4d4-955c-43e8-a21b-33fe1a04884d"
-					(reference "Q7")
+					(reference "Q9")
 					(unit 1)
 				)
@@
 		(on_board yes)
 		(dnp no)
-		(property "Reference" "R57"
+		(property "Reference" "R49"
 			(at 26.67 55.118 90)
 			(effects
@@
 			(project "BPS-Leader"
 				(path "/bca74250-80d8-4ae3-9726-634afabc9565/52b3a4d4-955c-43e8-a21b-33fe1a04884d"
-					(reference "R57")
-					(unit 1)
-				)
+					(reference "R49")
+					(unit 1)
+				)

Commit message: Very rough layout of the board - maybe too long?
Parts:
- removed D26: 1N448W, Diode_SMD:D_0805_2012Metric, symbol Device:D
Other:
- moved on the sheet: D25, R48
Changed lines of the file:
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@@
 	(paper "A4")
-	(junction
-		(at 33.02 26.67)
-		(diameter 0)
-		(color 0 0 0 0)
-	)
 	(junction
 		(at 39.37 67.31)
@@
 	)
 	(junction
-		(at 33.02 50.8)
-		(diameter 0)
-		(color 0 0 0 0)
-	)
-	(junction
 		(at 21.59 57.15)
 		(diameter 0)
@@
 	(wire
 		(pts
-			(xy 33.02 26.67) (xy 26.67 26.67)
+			(xy 34.29 26.67) (xy 39.37 26.67)
 		)
 		(stroke
@@
 	(wire
 		(pts
-			(xy 33.02 50.8) (xy 26.67 50.8)
-		)
-		(stroke
-			(width 0)
-			(type default)
-		)
-	)
-	(wire
-		(pts
 			(xy 39.37 62.23) (xy 39.37 67.31)
 		)
@@
 	(wire
 		(pts
-			(xy 39.37 50.8) (xy 33.02 50.8)
+			(xy 34.29 50.8) (xy 39.37 50.8)
 		)
 		(stroke
@@
 	(wire
 		(pts
-			(xy 33.02 26.67) (xy 33.02 34.29)
-		)
-		(stroke
-			(width 0)
-			(type default)
-		)
-	)
-	(wire
-		(pts
-			(xy 39.37 26.67) (xy 33.02 26.67)
-		)
-		(stroke
-			(width 0)
-			(type default)
-		)
-	)
-	(wire
-		(pts
 			(xy 21.59 67.31) (xy 39.37 67.31)
 		)
@@
 	(wire
 		(pts
-			(xy 33.02 41.91) (xy 33.02 50.8)
-		)
-		(stroke
-			(width 0)
-			(type default)
-		)
-	)
-	(wire
-		(pts
 			(xy 21.59 57.15) (xy 21.59 59.69)
 		)
@@
 	(wire
 		(pts
-			(xy 26.67 26.67) (xy 26.67 30.48)
-		)
-		(stroke
-			(width 0)
-			(type default)
-		)
-	)
-	(wire
-		(pts
-			(xy 26.67 50.8) (xy 26.67 46.99)
-		)
-		(stroke
-			(width 0)
-			(type default)
-		)
-	)
-	(wire
-		(pts
-			(xy 26.67 38.1) (xy 26.67 39.37)
+			(xy 34.29 26.67) (xy 34.29 30.48)
+		)
+		(stroke
+			(width 0)
+			(type default)
+		)
+	)
+	(wire
+		(pts
+			(xy 34.29 50.8) (xy 34.29 46.99)
+		)
+		(stroke
+			(width 0)
+			(type default)
+		)
+	)
+	(wire
+		(pts
+			(xy 34.29 38.1) (xy 34.29 39.37)
 		)
 		(stroke
@@
 	)
 	(symbol
-		(lib_id "Device:D")
-		(at 33.02 38.1 270)
-		(unit 1)
-		(exclude_from_sim no)
-		(in_bom yes)
-		(on_board yes)
-		(dnp no)
-		(property "Reference" "D26"
-			(at 33.274 43.688 90)
-			(effects
-				(font
-					(size 1.27 1.27)
-				)
-				(justify left)
-			)
-		)
-		(property "Value" "1N448W"
-			(at 35.814 34.29 0)
-			(effects
-				(font
-					(size 1.27 1.27)
-				)
-				(justify left)
-			)
-		)
-		(property "Footprint" "Diode_SMD:D_0805_2012Metric"
-			(at 33.02 38.1 0)
-			(effects
-				(font
-					(size 1.27 1.27)
-				)
-				(hide yes)
-			)
-		)
-		(property "Datasheet" "~"
-			(at 33.02 38.1 0)
-			(effects
-				(font
-					(size 1.27 1.27)
-				)
-				(hide yes)
-			)
-		)
-		(property "Description" "Diode"
-			(at 33.02 38.1 0)
-			(effects
-				(font
-					(size 1.27 1.27)
-				)
-				(hide yes)
-			)
-		)
-		(property "Sim.Device" "D"
-			(at 33.02 38.1 0)
-			(effects
-				(font
-					(size 1.27 1.27)
-				)
-				(hide yes)
-			)
-		)
-		(property "Sim.Pins" "1=K 2=A"
-			(at 33.02 38.1 0)
-			(effects
-				(font
-					(size 1.27 1.27)
-				)
-				(hide yes)
-			)
-		)
-		(pin "1"
-		)
-		(pin "2"
-		)
-		(instances
-			(project "BPS-Leader"
-				(path "/bca74250-80d8-4ae3-9726-634afabc9565/52b3a4d4-955c-43e8-a21b-33fe1a04884d"
-					(reference "D26")
-					(unit 1)
-				)
-			)
-		)
-	)
-	(symbol
 		(lib_id "Device:R")
-		(at 26.67 34.29 0)
+		(at 34.29 34.29 0)
 		(mirror y)
 		(unit 1)
@@
 		(dnp no)
 		(property "Reference" "R48"
-			(at 21.082 34.544 0)
+			(at 28.702 34.544 0)
 			(effects
 				(font
@@
 		)
 		(property "Value" "10k"
-			(at 26.67 32.512 90)
+			(at 34.29 32.512 90)
 			(effects
 				(font
@@
 		)
 		(property "Footprint" "Resistor_SMD:R_0805_2012Metric"
-			(at 28.448 34.29 90)
+			(at 36.068 34.29 90)
 			(effects
 				(font
@@
 		)
 		(property "Datasheet" "~"
-			(at 26.67 34.29 0)
+			(at 34.29 34.29 0)
 			(effects
 				(font
@@
 		)
 		(property "Description" "Resistor"
-			(at 26.67 34.29 0)
+			(at 34.29 34.29 0)
 			(effects
 				(font
@@
 	(symbol
 		(lib_id "Device:LED")
-		(at 26.67 43.18 90)
+		(at 34.29 43.18 90)
 		(unit 1)
 		(exclude_from_sim no)
@@
 		(dnp no)
 		(property "Reference" "D25"
-			(at 20.828 42.164 90)
+			(at 28.448 42.164 90)
 			(effects
 				(font
@@
 		)
 		(property "Value" "Green"
-			(at 19.558 43.942 90)
+			(at 27.178 43.942 90)
 			(effects
 				(font
@@
 		)
 		(property "Footprint" "Diode_SMD:D_0805_2012Metric"
-			(at 26.67 43.18 0)
+			(at 34.29 43.18 0)
 			(effects
 				(font
@@
 		)
 		(property "Datasheet" "~"
-			(at 26.67 43.18 0)
+			(at 34.29 43.18 0)
 			(effects
 				(font
@@
 		)
 		(property "Description" "Light emitting diode"
-			(at 26.67 43.18 0)
-			(effects
-				(font
+			(at 34.29 43.18 0)
+			(effects
+				(font

Commit message: everything should be finished now; tracks cleaned up, silkscreen issues fixed, new shunt/feedback/protection resistors chosen, BOM made, some other stuff i forgot probably
Parts:
- D25: P/N (none) -> HSMQ-C170-T0000
- Q9: P/N (none) -> IRLML0030
- R47: P/N (none) -> CRCW0805100KFKEAC
- R48: P/N (none) -> CRCW080510K0FKEAC
- R49: P/N (none) -> CRCW08051K00FKEAC
Changed lines of the file:
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@@
 			)
 		)
-		(property "Datasheet" "~"
+		(property "Datasheet" "https://www.mouser.com/ProductDetail/71-CRCW080510K0FKEAC"
 			(at 34.29 34.29 0)
 			(effects
@@
 		)
 		(property "Description" "Resistor"
+			(at 34.29 34.29 0)
+			(effects
+				(font
+					(size 1.27 1.27)
+				)
+				(hide yes)
+			)
+		)
+		(property "P/N" "CRCW080510K0FKEAC"
 			(at 34.29 34.29 0)
 			(effects
@@
 			)
 		)
-		(property "Datasheet" "~"
+		(property "Datasheet" "https://www.mouser.com/datasheet/2/678/hsmq_c170_t0000_ds100-2498198.pdf"
 			(at 34.29 43.18 0)
 			(effects
@@
 		)
 		(property "Description" "Light emitting diode"
+			(at 34.29 43.18 0)
+			(effects
+				(font
+					(size 1.27 1.27)
+				)
+				(hide yes)
+			)
+		)
+		(property "P/N" "HSMQ-C170-T0000"
 			(at 34.29 43.18 0)
 			(effects
@@
 			)
 		)
-		(property "Datasheet" "~"
+		(property "Datasheet" "https://www.mouser.com/ProductDetail/Vishay-Dale/CRCW0805100KFKEAC?qs=sGAEpiMZZMvdGkrng054t0DrEhLhGh8gZRT9GjFuHWDV3jEqj5sSqw%3D%3D"
 			(at 21.59 63.5 0)
 			(effects
@@
 		)
 		(property "Description" "Resistor"
+			(at 21.59 63.5 0)
+			(effects
+				(font
+					(size 1.27 1.27)
+				)
+				(hide yes)
+			)
+		)
+		(property "P/N" "CRCW0805100KFKEAC"
 			(at 21.59 63.5 0)
 			(effects
@@
 			)
 		)
+		(property "P/N" "IRLML0030"
+			(at 36.83 57.15 0)
+			(effects
+				(font
+					(size 1.27 1.27)
+				)
+				(hide yes)
+			)
+		)
 		(pin "2"
 		)
@@
 			)
 		)
-		(property "Datasheet" "~"
+		(property "Datasheet" "https://www.mouser.com/ProductDetail/71-CRCW08051K00FKEAC"
 			(at 26.67 57.15 0)
 			(effects
@@
 			(at 26.67 57.15 0)
 			(effects
+				(font
+					(size 1.27 1.27)
+				)
+				(hide yes)
+			)
+		)
+		(property "P/N" "CRCW08051K00FKEAC"
+			(at 26.67 57.15 0)
+			(effects

Commit message: math for shunt added, BOM excel file added
Parts:
- D25: footprint Diode_SMD:D_0805_2012Metric -> footprints:D_0805_2012Metric(adjsilk)
Changed lines of the file:
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@@
 			)
 		)
-		(property "Footprint" "Diode_SMD:D_0805_2012Metric"
+		(property "Footprint" "footprints:D_0805_2012Metric(adjsilk)"
 			(at 34.29 43.18 0)
 			(effects
